Commit message: set parameters

File: urdf/rs_bpearl_lidar.urdf.xacro (robot description, xacro)
@@ -36,4 +36,5 @@
       <parent link="${prefix}_base_link"/>
       <child link="${prefix}_link" />
+      <origin xyz="0 0 0.06" rpy="0 0 0"/>
     </joint>
     <link name="${prefix}_link"/>
@@ -53,5 +54,5 @@
         <sensor type="${ray_type}" name="${prefix}_sensor">
           <pose>0 0 0 0 0 0.0</pose>
-          <visualize>false</visualize>
+          <visualize>true</visualize>
           <update_rate>${fps}</update_rate>
           <ray>
@@ -65,6 +66,6 @@
               <vertical>
                 <samples>${vfov/vres}</samples>
-                <min_angle>-${vfov/2.0*M_PI/180.0}</min_angle>
-                <max_angle>${vfov/2.0*M_PI/180.0}</max_angle>
+                <min_angle>0</min_angle>
+                <max_angle>90</max_angle>
               </vertical>
             </scan>

Commit message: Updated parameters

File: urdf/rs_bpearl_lidar.urdf.xacro (robot description, xacro)
@@ -2,5 +2,5 @@
 <robot name="sensor_rs_bpearl_lidar" xmlns:xacro="http://wiki.ros.org/xacro">
   <xacro:property name="M_PI" value="3.1415926535897931" />
-  <xacro:macro name="sensor_rs_bpearl_lidar" params="prefix parent prefix_topic *origin range_min range_max hfov hres vfov vres fps gpu:=^|true">
+  <xacro:macro name="sensor_rs_bpearl_lidar" params="prefix parent prefix_topic *origin range_min range_max hfov samples vfov lasers fps gpu:=^|true">
     <material name="black_alu">
       <color rgba="0.9 0.9 0.9 1"/>
@@ -36,10 +36,10 @@
       <parent link="${prefix}_base_link"/>
       <child link="${prefix}_link" />
-      <origin xyz="0 0 0.06" rpy="0 0 0"/>
+      <origin xyz="0 0 0.06" rpy="0 ${5*M_PI/180.0} 0"/>
     </joint>
     <link name="${prefix}_link"/>
-  <sensor_rs_bpearl_lidar_gazebo range_min="${range_min}" range_max="${range_max}" hfov="${hfov}" hres="${hres}" vfov="${vfov}" vres="${vres}" fps="${fps}" gpu="${gpu}"/>
+  <sensor_rs_bpearl_lidar_gazebo range_min="${range_min}" range_max="${range_max}" hfov="${hfov}" samples="${samples}" vfov="${vfov}" lasers="${lasers}" fps="${fps}" gpu="${gpu}"/>
   </xacro:macro>
-  <xacro:macro name="sensor_rs_bpearl_lidar_gazebo" params="range_min range_max hfov hres vfov vres fps gpu">
+  <xacro:macro name="sensor_rs_bpearl_lidar_gazebo" params="range_min range_max hfov samples vfov lasers fps gpu">
     <gazebo reference="${prefix}_link">
       <xacro:if value="${gpu}">
@@ -60,12 +60,12 @@
               <horizontal>
 				<!-- for a high quality simulation -->
-                <samples>${hfov/hres}</samples>
-                <min_angle>-${hfov/2.0*M_PI/180.0}</min_angle>
-                <max_angle>${hfov/2.0*M_PI/180.0}</max_angle>
+                <samples>${samples}</samples>
+                <min_angle>-${hfov/2*M_PI/180.0}</min_angle>
+                <max_angle>${hfov/2*M_PI/180.0}</max_angle>
               </horizontal>
               <vertical>
-                <samples>${vfov/vres}</samples>
-                <min_angle>0</min_angle>
-                <max_angle>90</max_angle>
+                <samples>${lasers}</samples>
+                <min_angle>-${5*M_PI/180.0}</min_angle>  <!-- bpearl has 90 degrees of vertival field of view-->
+                <max_angle> ${(vfov-5)*M_PI/180.0}</max_angle>
               </vertical>
             </scan>
