Commit message: Update ueye_cp_gige inertia

File: urdf/ueye_cp_gige.urdf.xacro (robot description, xacro)
@@ -7,9 +7,9 @@
       <child link="${prefix}_base_link"/>
     </joint>
-    <link name="${prefix}_base_link"> <!-- TODO: review masses, inertial -->
+    <link name="${prefix}_base_link">
       <inertial>
-        <origin xyz="0.0 0.0 0." rpy="0 0 0"/>
-        <mass value="0.1"/>
-        <origin xyz="0 0 0" rpy="0 0 0"/>
+        <mass value="0.0088"/>
+        <origin xyz="0.007 0 0.0145" rpy="0 0 0"/>
+        <xacro:solid_cuboid_inertia m="0.0088" w="0.0604" h="0.029" d="0.029" />
         <inertia ixx="0.1" ixy="0" ixz="0" iyy="0.1" iyz="0" izz="0.1"/>
       </inertial>
@@ -37,11 +37,9 @@
     </joint>
     <link name="${prefix}_rgb_frame_link">
-    <inertial>
-      <mass value="0.001" />
-      <origin xyz="0 0 0" />
-      <inertia ixx="0.0001" ixy="0.0" ixz="0.0"
-               iyy="0.0001" iyz="0.0"
-               izz="0.0001" />
-    </inertial>
+      <inertial>
+        <mass value="0.0001" />
+        <origin xyz="0 0 0" />
+        <xacro:solid_cuboid_inertia m="0.0001" w="0.0604" h="0.029" d="0.029" />
+      </inertial>
     </link>
     <joint name="${prefix}_rgb_optical_joint" type="fixed">
@@ -52,9 +50,7 @@
     <link name="${prefix}_rgb_optical_frame_link">
     <inertial>
-      <mass value="0.001" />
-      <origin xyz="0 0 0" />
-      <inertia ixx="0.0001" ixy="0.0" ixz="0.0"
-               iyy="0.0001" iyz="0.0"
-               izz="0.0001" />
+      <mass value="0.0001" />
+        <origin xyz="0 0 0" />
+        <xacro:solid_cuboid_inertia m="0.0001" w="0.0604" h="0.029" d="0.029" />
     </inertial>
     </link>
