Commit message: Update teraranger
- Update inertias
- Add gazebo plugins

File: urdf/teraranger_tr_duo.urdf.xacro (robot description, xacro)
@@ -1,5 +1,5 @@
 <?xml version="1.0"?>
 <robot name="sensor_teraranger_duo" xmlns:xacro="http://wiki.ros.org/xacro">
-  <xacro:macro name="sensor_teraranger_duo" params="prefix parent prefix_topic:='teraranger_duo' *origin">
+  <xacro:macro name="sensor_teraranger_duo" params="prefix parent prefix_topic:='teraranger_duo' *origin min_angle:=-0.02618 max_angle:=0.02618">
     <joint name="${prefix}_base_joint" type="fixed">
       <xacro:insert_block name="origin" />
@@ -21,7 +21,7 @@
 		</visual>
 		<inertial>
-			<mass value="1e-5" />
-			<origin xyz="0 0 0" rpy="0 0 0"/>
-			<inertia ixx="1e-6" ixy="0" ixz="0" iyy="1e-6" iyz="0" izz="1e-6" />
+			<mass value="0.016" />
+			<origin xyz="0.01 0 0" rpy="0 0 0"/>
+	        <xacro:solid_cuboid_inertia m="0.016" w="0.02" h="0.03" d="0.053" />
 		</inertial>
 	</link>
@@ -41,4 +41,76 @@
     </link>
 	<!-- TODO add Gazebo stuff for simulation-->
+	<gazebo reference="${prefix}_sonar_link">
+		<material>Gazebo/Yellow</material>
+      	<sensor type="ray" name="${prefix}_sensor">
+			<visualize>false</visualize>
+			<update_rate>100</update_rate>
+			<ray>
+				<scan>
+					<horizontal>
+						<samples>10</samples>
+						<resolution>1</resolution>
+						<min_angle>-0.02618</min_angle>
+						<max_angle>0.02618</max_angle>
+					</horizontal>
+					<vertical>
+						<samples>10</samples>
+						<resolution>1</resolution>
+						<min_angle>-0.02618</min_angle>
+						<max_angle>0.02618</max_angle>
+					</vertical>
+				</scan>
+				<range>
+					<min>0.02</min>
+					<max>14</max>
+					<resolution>0.05</resolution>
+				</range>
+			</ray>
+			<plugin name="${prefix}_sonar_controller" filename="libgazebo_ros_range.so">
+				<topicName>${prefix_topic}/sonar</topicName>
+				<frameName>${prefix}_laser_link</frameName>
+				<gaussianNoise>0</gaussianNoise>
+				<updateRate>20</updateRate>
+				<radiation>ultrasound</radiation>
+				<fov>0.05</fov>
+			</plugin>
+		</sensor>
+	</gazebo>
+	<gazebo reference="${prefix}_laser_link">
+		<material>Gazebo/Yellow</material>
+      	<sensor type="ray" name="${prefix}_sensor">
+			<visualize>false</visualize>
+			<update_rate>100</update_rate>
+			<ray>
+				<scan>
+					<horizontal>
+						<samples>10</samples>
+						<resolution>1</resolution>
+						<min_angle>-0.02618</min_angle>
+						<max_angle>0.02618</max_angle>
+					</horizontal>
+					<vertical>
+						<samples>10</samples>
+						<resolution>1</resolution>
+						<min_angle>-0.02618</min_angle>
+						<max_angle>0.02618</max_angle>
+					</vertical>
+				</scan>
+				<range>
+					<min>0.02</min>
+					<max>14</max>
+					<resolution>0.05</resolution>
+				</range>
+			</ray>
+			<plugin name="${prefix}_range_controller" filename="libgazebo_ros_range.so">
+				<topicName>${prefix_topic}/scan</topicName>
+				<frameName>${prefix}_laser_link</frameName>
+				<gaussianNoise>0</gaussianNoise>
+				<updateRate>20</updateRate>
+				<radiation>infrared</radiation>
+				<fov>0.05</fov>
+			</plugin>
+		</sensor>
+	</gazebo>
   </xacro:macro>
 </robot>
