Commit message: Fix sick tim551 inertia

File: urdf/sick_tim551.urdf.xacro (robot description, xacro)
@@ -21,7 +21,7 @@
       </visual>
       <inertial>
-        <mass value="1e-5" />
-        <origin xyz="0 0 0" rpy="0 0 0"/>
-        <inertia ixx="1e-6" ixy="0" ixz="0" iyy="1e-6" iyz="0" izz="1e-6" />
+        <mass value="0.25" />
+        <origin xyz="-0.0017 0 0.042875" rpy="0 0 0"/>
+        <xacro:solid_cuboid_inertia m="0.25" w="0.061" h="0.06" d="0.08575" />
       </inertial>
     </link>
