Commit message: Update sick_s3000
- Fix inertia
- Update ray link

File: urdf/sick_s3000.urdf.xacro (robot description, xacro)
@@ -2,5 +2,5 @@
 <robot name="sensor_sick_s3000" xmlns:xacro="http://wiki.ros.org/xacro">
   <xacro:macro name="sensor_sick_s3000" params="prefix parent ns='' prefix_topic:='front_laser' *origin gpu:=^|true">
-    <joint name="${prefix}_joint" type="fixed">
+    <joint name="${prefix}_base_joint" type="fixed">
       <xacro:insert_block name="origin" />
       <parent link="${parent}"/>
@@ -9,5 +9,6 @@
 	<link name="${prefix}_base_link">
 		<collision>
-			<origin xyz="-0.093 0 -0.0625" rpy="0 0 0"/>
+			<!--origin xyz="-0.093 0 -0.0625" rpy="0 0 0"/-->
+			<origin xyz="0.0 0.0 0.0" rpy="0 0 0"/>
 			<geometry>
 	     		<mesh filename="package://robotnik_sensors/meshes/sick_s3000.dae"/>
@@ -15,5 +16,6 @@
 		</collision>
 		<visual>
-			<origin xyz="-0.093 0 -0.0625" rpy="0 0 0"/>
+			<origin xyz="0.0 0.0 0.0" rpy="0 0 0"/>
+			<!--origin xyz="-0.093 0 -0.0625" rpy="0 0 0"/-->
 			<geometry>
 	     		<mesh filename="package://robotnik_sensors/meshes/sick_s3000.dae"/>
@@ -21,14 +23,20 @@
 		</visual>
 		<inertial>
-			<mass value="1e-5" />
-			<origin xyz="0 0 0" rpy="0 0 0"/>
-			<inertia ixx="1e-6" ixy="0" ixz="0" iyy="1e-6" iyz="0" izz="1e-6" />
+			<mass value="3.3" />
+            <origin xyz="0.08 0 0.0925" rpy="0 0 0"/>
+            <xacro:solid_cuboid_inertia m="3.3" w="0.16" h="0.160" d="0.185" />
 		</inertial>
 	</link>
+    <joint name="${prefix}_joint" type="fixed">
+      <parent link="${prefix}_base_link"/>
+      <child link="${prefix}_link"/>
+      <origin xyz="0.093 0 0.0625" rpy="0 0 0"/>
+	</joint>
+	<link name="${prefix}_link" />
 	<!-- Sick sensor sensor for simulation -->
 	<sensor_sick_s3000_gazebo/>
   </xacro:macro>
   <xacro:macro name="sensor_sick_s3000_gazebo">
-    <gazebo reference="${prefix}_base_link">
+    <gazebo reference="${prefix}_link">
 		<xacro:if value="${gpu}">
 			<xacro:property name="ray_type" value="gpu_ray" />
@@ -65,5 +73,5 @@
 			<plugin name="${prefix}_controller" filename="${plugin_lib}">
 				<topicName>${ns}${prefix_topic}/scan</topicName>
-				<frameName>/${prefix}_base_link</frameName>
+				<frameName>/${prefix}_link</frameName>
 			</plugin>
 		</sensor>
