Commit message: adding prefix_scan to rplidars

File: urdf/rplidar.urdf.xacro (robot description, xacro)
@@ -1,5 +1,5 @@
 <?xml version="1.0"?>
 <robot xmlns:xacro="http://www.ros.org/wiki/xacro">
-  <xacro:macro name="sensor_rplidar" params="prefix parent *origin min_angle:=3.14159 max_angle:=-3.14159">
+  <xacro:macro name="sensor_rplidar" params="prefix parent prefix_scan *origin min_angle:=3.14159 max_angle:=-3.14159">
     <joint name="${prefix}_laser_base_joint" type="fixed">
       <xacro:insert_block name="origin" />
@@ -62,5 +62,5 @@
 				</ray>
 				<plugin name="gazebo_ros_rplidar_controller" filename="libgazebo_ros_laser.so">
-					<topicName>scan</topicName>
+					<topicName>${prefix_scan}/scan</topicName>
 					<frameName>${prefix}_laser_link</frameName>
 					<ignoreTfPrefix>1</ignoreTfPrefix>

File: urdf/rplidar_a2.urdf.xacro (robot description, xacro)
@@ -1,5 +1,5 @@
 <?xml version="1.0"?>
 <robot xmlns:xacro="http://www.ros.org/wiki/xacro">
-  <xacro:macro name="sensor_rplidar_a2" params="prefix parent *origin min_angle:=-3.14159 max_angle:=3.14159">
+  <xacro:macro name="sensor_rplidar_a2" params="prefix parent prefix_scan *origin min_angle:=-3.14159 max_angle:=3.14159">
     <joint name="${prefix}_base_joint" type="fixed">
       <xacro:insert_block name="origin" />
@@ -62,5 +62,5 @@
 				</ray>
 				<plugin name="${prefix}gazebo_ros_rplidar_a2_controller" filename="libgazebo_ros_laser.so">
-					<topicName>scan</topicName>
+					<topicName>${prefix_scan}/scan</topicName>
 					<frameName>${prefix}_link</frameName>
 					<ignoreTfPrefix>1</ignoreTfPrefix>

Commit message: Fix rplidar inertia

File: urdf/rplidar.urdf.xacro (robot description, xacro)
@@ -1,5 +1,5 @@
 <?xml version="1.0"?>
 <robot xmlns:xacro="http://wiki.ros.org/xacro">
-  <xacro:macro name="sensor_rplidar" params="prefix parent prefix_topic:='front_laser' *origin min_angle:=3.14159 max_angle:=-3.14159 gpu:=^|true">
+  <xacro:macro name="sensor_rplidar" params="prefix parent prefix_topic:='front_laser' *origin min_angle:=3.14159 max_angle:=-3.14159 gpu:=^|false">
     <joint name="${prefix}_laser_base_joint" type="fixed">
       <xacro:insert_block name="origin" />
@@ -21,7 +21,7 @@
       </visual>
       <inertial>
-        <mass value="1e-5" />
-        <origin xyz="0 0 0" rpy="0 0 0"/>
-        <inertia ixx="1e-6" ixy="0" ixz="0" iyy="1e-6" iyz="0" izz="1e-6" />
+        <mass value="0.190" />
+        <origin xyz="0.01 0 0.028" rpy="0 0 0"/>
+        <xacro:solid_cuboid_inertia m="0.190" w="0.09674" h="0.056" d="0.056" />
       </inertial>
     </link>
