Commit message: Fix rplidar_a2 inertia

File: urdf/rplidar_a2.urdf.xacro (robot description, xacro)
@@ -21,7 +21,7 @@
       </visual>
       <inertial>
-        <mass value="1e-5" />
-        <origin xyz="0 0 0" rpy="0 0 0"/>
-        <inertia ixx="1e-6" ixy="0" ixz="0" iyy="1e-6" iyz="0" izz="1e-6" />
+        <mass value="0.190" />
+        <origin xyz="0 0 0.02040" rpy="0 0 0"/>
+        <xacro:solid_cuboid_inertia m="0.190" w="0.07570" h="0.07570" d="0.04080" />
       </inertial>
     </link>
