Commit message: Fix roboteq mgs inertia

File: urdf/roboteq_mgs.urdf.xacro (robot description, xacro)
@@ -9,7 +9,7 @@
     <link name="${prefix}_base_link">
       <inertial>
-        <mass value="0.5" />
+        <mass value="0.255" />
         <origin xyz="0 0 0" />
-        <inertia ixx="0.1" ixy="0" ixz="0" iyy="0.1" iyz="0" izz="0.1"/>
+        <xacro:solid_cuboid_inertia m="0.255" w="0.025" h="0.165" d="0.025" />
       </inertial>
     </link>
