Commit message: removed dependancy from rbcar, modified sensor links and samples

File: urdf/hokuyo3d.urdf.xacro (robot description, xacro)
@@ -2,10 +2,10 @@
 <robot name="sensor_hokuyo3d" xmlns:xacro="http://ros.org/wiki/xacro">
   <xacro:macro name="sensor_hokuyo3d" params="name parent *origin">
-    <joint name="${name}_laser_joint" type="fixed">
+    <joint name="${name}_laser_fix_joint" type="fixed">
       <insert_block name="origin" />
       <parent link="${parent}"/>
-      <child link="${name}_laser_link"/>
+      <child link="${name}_laser_fix_link"/>
 	</joint>
-	<link name="${name}_laser_link">
+	<link name="${name}_laser_fix_link">
 		<collision>
 			<origin xyz="0 0 0" rpy="0 0 0"/>
@@ -17,5 +17,5 @@
 			<origin xyz="0 0 0" rpy="0 0 0"/>
 			<geometry>
-	     		<mesh filename="package://rbcar_description/meshes/sensors/hokuyo3d.dae"/>
+	     		<mesh filename="package://robotnik_sensors/meshes/hokuyo3d.stl"/>
 			</geometry>
 		</visual>
@@ -26,4 +26,11 @@
 		</inertial>
 	</link>
+	<link name="${name}_laser_link">
+	</link>
+    <joint name="${name}_laser_joint" type="fixed">
+      <parent link="${name}_laser_fix_link"/>
+      <child link="${name}_laser_link"/>
+      <origin xyz="0.08 0 0.08" rpy="0 0 0"/>
+	</joint>
 	<!-- Hokuyo sensor for simulation -->
 	<sensor_hokuyo3d_gazebo/>
@@ -34,9 +41,9 @@
 				<pose>0 0 0 0 0 0</pose>
 				<visualize>false</visualize>
-				<update_rate>20</update_rate>
+				<update_rate>5</update_rate>
 				<ray>
 					<scan>
                         <horizontal>
-                            <samples>16</samples>
+                            <samples>144</samples>
                             <resolution>1.0</resolution>
                             <min_angle>-1.83591184</min_angle>
@@ -44,8 +51,8 @@
                         </horizontal>
                         <vertical>
-                            <samples>162</samples>
+                            <samples>74</samples>
                             <resolution>1.0</resolution>
-                            <min_angle>-0.0872664626</min_angle>
-                            <max_angle>0.610865238</max_angle>
+                            <min_angle>-0.610865238</min_angle>
+                            <max_angle>0.0872664626</max_angle>
                         </vertical>
 					</scan>

Commit message: Setting hokuyo3d.dae path correctly

File: urdf/hokuyo3d.urdf.xacro (robot description, xacro)
@@ -17,5 +17,5 @@
 			<origin xyz="0 0 0" rpy="0 0 0"/>
 			<geometry>
-	     		<mesh filename="package://rbcar_description/meshes/sensors/hokuyo3d.dae"/>
+	     		<mesh filename="package://robotnik_sensors/meshes/hokuyo3d.dae"/>
 			</geometry>
 		</visual>

Commit message: minor change in collision box

File: urdf/hokuyo3d.urdf.xacro (robot description, xacro)
@@ -11,5 +11,5 @@
 			<origin xyz="0 0 0" rpy="0 0 0"/>
 			<geometry>
-				<box size="0.1 0.1 0.08"/>
+				<box size="0.05 0.05 0.08"/>
 			</geometry>
 		</collision>

Commit message: Fix hokuyo 3d inertia

File: urdf/hokuyo3d.urdf.xacro (robot description, xacro)
@@ -21,7 +21,7 @@
         </visual>
         <inertial>
-            <mass value="1e-5" />
-            <origin xyz="0 0 0" rpy="0 0 0"/>
-            <inertia ixx="1e-6" ixy="0" ixz="0" iyy="1e-6" iyz="0" izz="1e-6" />
+            <mass value="0.65" />
+            <origin xyz="0.0475 0.0 0.053" rpy="0 0 0"/>
+            <xacro:solid_cuboid_inertia m="0.65" w="0.095" h="0.07" d="0.106" />
         </inertial>
     </link>
