Commit message: Axis_p5514 name standarization: urdf, stl and dae

File: urdf/axis_p5514.urdf.xacro (robot description, xacro)
@@ -27,5 +27,5 @@
         </material>
         <geometry>
-          <mesh filename="package://robotnik_sensors/meshes/camera_axis_p5514.stl" scale="1.0 1.0 1.0"/>
+          <mesh filename="package://robotnik_sensors/meshes/axis_p5514.stl" scale="1.0 1.0 1.0"/>
         </geometry>
       </visual>
@@ -34,5 +34,5 @@
         <!-- because the origin of the mesh file is not at the "center" of the model-->
         <geometry>
-          <mesh filename="package://robotnik_sensors/meshes/camera_axis_p5514.stl" scale="1.0 1.0 1.0"/>
+          <mesh filename="package://robotnik_sensors/meshes/axis_p5514.stl" scale="1.0 1.0 1.0"/>
         </geometry>
       </collision>
