Commit message: axis_m5525: Add prefix_topic argument

File: urdf/axis_m5525.urdf.xacro (robot description, xacro)
@@ -7,5 +7,5 @@
   <xacro:property name="ptz_mechanical_reduction" value="1.0"/>
   <xacro:property name="PI" value="3.14159265359"/>
-  <xacro:macro name="sensor_axis_m5525" params="prefix parent *origin far:=^|8.0 near:=^|0.05">
+  <xacro:macro name="sensor_axis_m5525" params="prefix parent *origin far:=^|8.0 near:=^|0.05 prefix_topic:=^ptz_camera">
     <joint name="${prefix}_joint" type="fixed">
       <axis xyz="0 1 0"/>
@@ -127,5 +127,5 @@
 			<sensor type="camera" name="${prefix}_sensor">
 				<update_rate>30.0</update_rate>
-				<camera name="${prefix}">
+				<camera name="${prefix_topic}">
 					<horizontal_fov>${60.0*M_PI/180.0}</horizontal_fov>
 					<image>
@@ -140,8 +140,7 @@
 				</camera>
 				<plugin name="${prefix}_controller" filename="libgazebo_ros_camera.so">
-				    <cameraName>${prefix}</cameraName>
 					<alwaysOn>true</alwaysOn>
 					<updateRate>0.0</updateRate>
-					<cameraName>${prefix}</cameraName>
+					<cameraName>${prefix_topic}</cameraName>
 					<imageTopicName>image_raw</imageTopicName>
 					<cameraInfoTopicName>camera_info</cameraInfoTopicName>

Commit message: axis_m5525: Fix inertias

File: urdf/axis_m5525.urdf.xacro (robot description, xacro)
@@ -1,6 +1,6 @@
 <?xml version="1.0"?>
 <robot xmlns:xacro="http://wiki.ros.org/xacro" name="sensor_axis_m5525">
-  <xacro:property name="ptz_joint_effort_limit" value="100.0"/>
-  <xacro:property name="ptz_joint_velocity_limit" value="100.0"/>
+  <xacro:property name="ptz_joint_effort_limit" value="1.0"/>
+  <xacro:property name="ptz_joint_velocity_limit" value="1.0"/>
   <xacro:property name="ptz_joint_friction" value="0.1"/>
   <xacro:property name="ptz_joint_damping" value="0.1"/>
@@ -21,6 +21,6 @@
         <origin xyz="0 0 0" rpy="0 0 0"/>
         <mass value="0.1"/>
-        <origin xyz="0 0 0" rpy="0 0 0"/>
-        <inertia ixx="0.1" ixy="0" ixz="0" iyy="0.1" iyz="0" izz="0.1"/>
+        <xacro:solid_cuboid_inertia m="0.1" x="0.165" y="0.165" z="0.165" />
+        <!--inertia ixx="0.001" ixy="0" ixz="0" iyy="0.001" iyz="0" izz="0.001"/-->
       </inertial>
       <visual>
@@ -43,5 +43,5 @@
     <joint name="${prefix}_pan_joint" type="revolute">
       <axis xyz="1 0 0"/>
-      <origin xyz="0.0 0.0 0.087" rpy="0 0 0"/>
+      <origin xyz="0.087 0.0 0.0" rpy="0 0 0"/>
       <!-- check the displacement -->
       <parent link="${prefix}_base_link"/>
@@ -52,7 +52,8 @@
     <link name="${prefix}_pan_link">
       <inertial>
-        <mass value="0.1"/>
+        <mass value="0.01"/>
         <origin xyz="0 0 0" rpy="0 0 0"/>
-        <inertia ixx="0.1" ixy="0" ixz="0" iyy="0.1" iyz="0" izz="0.1"/>
+        <xacro:solid_cuboid_inertia m="0.01" x="0.0165" y="0.0165" z="0.0165" />
+        <!--inertia ixx="0.001" ixy="0" ixz="0" iyy="0.001" iyz="0" izz="0.001"/-->
       </inertial>
     </link>
@@ -77,7 +78,8 @@
     <link name="${prefix}_tilt_link">
       <inertial>
-        <mass value="0.1"/>
+        <mass value="0.01"/>
         <origin xyz="0 0 0" rpy="0 0 0"/>
-        <inertia ixx="0.1" ixy="0" ixz="0" iyy="0.1" iyz="0" izz="0.1"/>
+        <xacro:solid_cuboid_inertia m="0.01" x="0.0165" y="0.0165" z="0.0165" />
+        <!--inertia ixx="0.001" ixy="0" ixz="0" iyy="0.001" iyz="0" izz="0.001"/-->
       </inertial>
     </link>
@@ -99,7 +101,8 @@
     <link name="${prefix}_frame_link">
       <inertial>
-        <mass value="0.001"/>
+        <mass value="0.00001"/>
         <origin xyz="0 0 0"/>
-        <inertia ixx="0.0001" ixy="0.0" ixz="0.0" iyy="0.0001" iyz="0.0" izz="0.0001"/>
+        <xacro:solid_cuboid_inertia m="0.00001" x="0.165" y="0.165" z="0.165" />
+        <!--inertia ixx="0.0001" ixy="0.0" ixz="0.0" iyy="0.0001" iyz="0.0" izz="0.0001"/-->
       </inertial>
     </link>
@@ -112,7 +115,8 @@
     <link name="${prefix}_optical_frame_link">
       <inertial>
-        <mass value="0.001"/>
+        <mass value="0.00001"/>
         <origin xyz="0 0 0"/>
-        <inertia ixx="0.0001" ixy="0.0" ixz="0.0" iyy="0.0001" iyz="0.0" izz="0.0001"/>
+        <xacro:solid_cuboid_inertia m="0.00001" x="0.165" y="0.165" z="0.165" />
+        <!--inertia ixx="0.0001" ixy="0.0" ixz="0.0" iyy="0.0001" iyz="0.0" izz="0.0001"/-->
       </inertial>
     </link>

Commit message: Fix solid_cuboid_inertia with old params

File: urdf/axis_m5525.urdf.xacro (robot description, xacro)
@@ -21,5 +21,5 @@
         <origin xyz="0 0 0" rpy="0 0 0"/>
         <mass value="0.1"/>
-        <xacro:solid_cuboid_inertia m="0.1" x="0.165" y="0.165" z="0.165" />
+        <xacro:solid_cuboid_inertia m="0.1" w="0.165" h="0.165" d="0.165" />
         <!--inertia ixx="0.001" ixy="0" ixz="0" iyy="0.001" iyz="0" izz="0.001"/-->
       </inertial>
@@ -54,5 +54,5 @@
         <mass value="0.01"/>
         <origin xyz="0 0 0" rpy="0 0 0"/>
-        <xacro:solid_cuboid_inertia m="0.01" x="0.0165" y="0.0165" z="0.0165" />
+        <xacro:solid_cuboid_inertia m="0.01" w="0.0165" h="0.0165" d="0.0165" />
         <!--inertia ixx="0.001" ixy="0" ixz="0" iyy="0.001" iyz="0" izz="0.001"/-->
       </inertial>
@@ -80,5 +80,5 @@
         <mass value="0.01"/>
         <origin xyz="0 0 0" rpy="0 0 0"/>
-        <xacro:solid_cuboid_inertia m="0.01" x="0.0165" y="0.0165" z="0.0165" />
+        <xacro:solid_cuboid_inertia m="0.01" w="0.0165" h="0.0165" d="0.0165" />
         <!--inertia ixx="0.001" ixy="0" ixz="0" iyy="0.001" iyz="0" izz="0.001"/-->
       </inertial>
@@ -103,5 +103,5 @@
         <mass value="0.00001"/>
         <origin xyz="0 0 0"/>
-        <xacro:solid_cuboid_inertia m="0.00001" x="0.165" y="0.165" z="0.165" />
+        <xacro:solid_cuboid_inertia m="0.00001" w="0.165" h="0.165" d="0.165" />
         <!--inertia ixx="0.0001" ixy="0.0" ixz="0.0" iyy="0.0001" iyz="0.0" izz="0.0001"/-->
       </inertial>
@@ -117,5 +117,5 @@
         <mass value="0.00001"/>
         <origin xyz="0 0 0"/>
-        <xacro:solid_cuboid_inertia m="0.00001" x="0.165" y="0.165" z="0.165" />
+        <xacro:solid_cuboid_inertia m="0.00001" w="0.165" h="0.165" d="0.165" />
         <!--inertia ixx="0.0001" ixy="0.0" ixz="0.0" iyy="0.0001" iyz="0.0" izz="0.0001"/-->
       </inertial>

File: urdf/utils/inertia.urdf.xacro (robot description, xacro)
@@ -33,8 +33,8 @@
   <!-- w relates to X axis, d to Z axis, and h to Y axis -->
   <!-- Keep this comment -->
-  <xacro:macro name="solid_cuboid_inertia" params="m x y z">
-    <inertia  ixx="${(m*(y*y+z*z))/12}" ixy = "0" ixz = "0"
-              iyy="${(m*(x*x+z*z))/12}" iyz = "0"
-              izz="${(m*(x*x+y*y))/12}"
+  <xacro:macro name="solid_cuboid_inertia" params="m w h d">
+    <inertia  ixx="${(m*(h*h+d*d))/12}" ixy = "0" ixz = "0"
+              iyy="${(m*(w*w+d*d))/12}" iyz = "0"
+              izz="${(m*(w*w+h*h))/12}"
      />
   </xacro:macro>

Commit message: urdf: updated axis_m5525 inertia

File: urdf/axis_m5525.urdf.xacro (robot description, xacro)
@@ -19,8 +19,7 @@
     <link name="${prefix}_base_link">
       <inertial>
-        <origin xyz="0 0 0" rpy="0 0 0"/>
-        <mass value="0.1"/>
-        <xacro:solid_cuboid_inertia m="0.1" w="0.165" h="0.165" d="0.165" />
-        <!--inertia ixx="0.001" ixy="0" ixz="0" iyy="0.001" iyz="0" izz="0.001"/-->
+        <origin xyz="0.066 0 0" rpy="0 ${M_PI/2} 0"/>
+        <mass value="0.8"/>
+        <xacro:solid_cuboid_inertia m="0.8" w="0.165" h="0.165" d="0.132" />
       </inertial>
       <visual>
@@ -52,8 +51,7 @@
     <link name="${prefix}_pan_link">
       <inertial>
-        <mass value="0.01"/>
+        <mass value="0.1"/>
         <origin xyz="0 0 0" rpy="0 0 0"/>
-        <xacro:solid_cuboid_inertia m="0.01" w="0.0165" h="0.0165" d="0.0165" />
-        <!--inertia ixx="0.001" ixy="0" ixz="0" iyy="0.001" iyz="0" izz="0.001"/-->
+        <xacro:solid_cuboid_inertia m="0.1" w="0.1" h="0.11" d="0.11" />
       </inertial>
     </link>
@@ -78,8 +76,7 @@
     <link name="${prefix}_tilt_link">
       <inertial>
-        <mass value="0.01"/>
+        <mass value="0.1"/>
         <origin xyz="0 0 0" rpy="0 0 0"/>
-        <xacro:solid_cuboid_inertia m="0.01" w="0.0165" h="0.0165" d="0.0165" />
-        <!--inertia ixx="0.001" ixy="0" ixz="0" iyy="0.001" iyz="0" izz="0.001"/-->
+        <xacro:solid_cuboid_inertia m="0.1" w="0.11" h="0.11" d="0.1" />
       </inertial>
     </link>
@@ -101,8 +98,7 @@
     <link name="${prefix}_frame_link">
       <inertial>
-        <mass value="0.00001"/>
+        <mass value="0.1"/>
         <origin xyz="0 0 0"/>
-        <xacro:solid_cuboid_inertia m="0.00001" w="0.165" h="0.165" d="0.165" />
-        <!--inertia ixx="0.0001" ixy="0.0" ixz="0.0" iyy="0.0001" iyz="0.0" izz="0.0001"/-->
+        <xacro:solid_cuboid_inertia m="0.1" w="0.11" h="0.11" d="0.1" />
       </inertial>
     </link>
@@ -115,12 +111,11 @@
     <link name="${prefix}_optical_frame_link">
       <inertial>
-        <mass value="0.00001"/>
+        <mass value="0.1"/>
         <origin xyz="0 0 0"/>
-        <xacro:solid_cuboid_inertia m="0.00001" w="0.165" h="0.165" d="0.165" />
-        <!--inertia ixx="0.0001" ixy="0.0" ixz="0.0" iyy="0.0001" iyz="0.0" izz="0.0001"/-->
+        <xacro:solid_cuboid_inertia m="0.1" w="0.11" h="0.11" d="0.1" />
       </inertial>
     </link>
     <gazebo reference="${prefix}_base_link">
-      <material>Gazebo/FlatBlack</material>
+      <material>Gazebo/DarkGrey</material>
     </gazebo>
     <!-- Axis sensor for simulation -->

Commit message: Fix issue on axis m5525 simulation

File: urdf/axis_m5525.urdf.xacro (robot description, xacro)
@@ -104,4 +104,16 @@
       </inertial>
     </link>
+    <joint name="${prefix}_frame_simulation_joint" type="fixed">
+      <origin xyz="0 0 0" rpy="${M_PI} 0 0"/>
+      <parent link="${prefix}_tilt_link"/>
+      <child link="${prefix}_frame_simulation_link"/>
+    </joint>
+    <link name="${prefix}_frame_simulation_link">
+      <inertial>
+        <mass value="0.1"/>
+        <origin xyz="0 0 0"/>
+        <xacro:solid_cuboid_inertia m="0.1" w="0.11" h="0.11" d="0.1" />
+      </inertial>
+    </link>
     <!-- Optical frame -->
     <joint name="${prefix}_optical_joint" type="fixed">
@@ -117,6 +129,19 @@
       </inertial>
     </link>
-    <gazebo reference="${prefix}_base_link">
-      <material>Gazebo/FlatBlack</material>
+    <!-- For simulation, the link has to be inverted -->
+    <joint name="${prefix}_optical_simulation_joint" type="fixed">
+      <origin xyz="0 0 0" rpy="${-M_PI/2} 0 ${-M_PI/2}"/>
+      <parent link="${prefix}_frame_simulation_link"/>
+      <child link="${prefix}_optical_frame_simulation_link"/>
+    </joint>
+    <link name="${prefix}_optical_frame_simulation_link">
+      <inertial>
+        <mass value="0.1"/>
+        <origin xyz="0 0 0"/>
+        <xacro:solid_cuboid_inertia m="0.1" w="0.11" h="0.11" d="0.1" />
+      </inertial>
+    </link>
+    <gazebo reference="${prefix}_base_simulation_link">
+      <material>Gazebo/DarkGrey</material>
     </gazebo>
     <!-- Axis sensor for simulation -->
@@ -124,5 +149,5 @@
   </xacro:macro>
 	<xacro:macro name="sensor_axis_m5525_gazebo">
-		<gazebo reference="${prefix}_frame_link"> <!-- the image will be generated from this (${name}_frame) point of view, with the front being the X axis -->
+		<gazebo reference="${prefix}_frame_simulation_link"> <!-- the image will be generated from this (${name}_frame) point of view, with the front being the X axis -->
 			<sensor type="camera" name="${prefix}_sensor">
 				<update_rate>30.0</update_rate>
@@ -146,5 +171,5 @@
 					<imageTopicName>image_raw</imageTopicName>
 					<cameraInfoTopicName>camera_info</cameraInfoTopicName>
-					<frameName>${prefix}_optical_frame_link</frameName>
+					<frameName>${prefix}_optical_frame_simulation_link</frameName>
 					<!-- this is just which name the Image msg will have, it does not affect the simulation.
 					     However must be set to the optical_frame,  -->

Commit message: Fix axis m5525 TF

File: urdf/axis_m5525.urdf.xacro (robot description, xacro)
@@ -69,5 +69,5 @@
     <joint name="${prefix}_tilt_joint" type="revolute">
       <axis xyz="0 -1 0"/>
-      <origin xyz="0.0 0.0 0.0" rpy="0 ${-PI/2} 0"/>
+      <origin xyz="0.0 0.0 0.0" rpy="0 ${PI/2} 0"/>
       <parent link="${prefix}_pan_link"/>
       <child link="${prefix}_tilt_link"/>
@@ -104,16 +104,4 @@
       </inertial>
     </link>
-    <joint name="${prefix}_frame_simulation_joint" type="fixed">
-      <origin xyz="0 0 0" rpy="${M_PI} 0 0"/>
-      <parent link="${prefix}_tilt_link"/>
-      <child link="${prefix}_frame_simulation_link"/>
-    </joint>
-    <link name="${prefix}_frame_simulation_link">
-      <inertial>
-        <mass value="0.1"/>
-        <origin xyz="0 0 0"/>
-        <xacro:solid_cuboid_inertia m="0.1" w="0.11" h="0.11" d="0.1" />
-      </inertial>
-    </link>
     <!-- Optical frame -->
     <joint name="${prefix}_optical_joint" type="fixed">
@@ -129,18 +117,5 @@
       </inertial>
     </link>
-    <!-- For simulation, the link has to be inverted -->
-    <joint name="${prefix}_optical_simulation_joint" type="fixed">
-      <origin xyz="0 0 0" rpy="${-M_PI/2} 0 ${-M_PI/2}"/>
-      <parent link="${prefix}_frame_simulation_link"/>
-      <child link="${prefix}_optical_frame_simulation_link"/>
-    </joint>
-    <link name="${prefix}_optical_frame_simulation_link">
-      <inertial>
-        <mass value="0.1"/>
-        <origin xyz="0 0 0"/>
-        <xacro:solid_cuboid_inertia m="0.1" w="0.11" h="0.11" d="0.1" />
-      </inertial>
-    </link>
-    <gazebo reference="${prefix}_base_simulation_link">
+    <gazebo reference="${prefix}_base_link">
       <material>Gazebo/DarkGrey</material>
     </gazebo>
@@ -149,5 +124,5 @@
   </xacro:macro>
 	<xacro:macro name="sensor_axis_m5525_gazebo">
-		<gazebo reference="${prefix}_frame_simulation_link"> <!-- the image will be generated from this (${name}_frame) point of view, with the front being the X axis -->
+		<gazebo reference="${prefix}_frame_link"> <!-- the image will be generated from this (${name}_frame) point of view, with the front being the X axis -->
 			<sensor type="camera" name="${prefix}_sensor">
 				<update_rate>30.0</update_rate>
@@ -171,5 +146,5 @@
 					<imageTopicName>image_raw</imageTopicName>
 					<cameraInfoTopicName>camera_info</cameraInfoTopicName>
-					<frameName>${prefix}_optical_frame_simulation_link</frameName>
+					<frameName>${prefix}_optical_frame_link</frameName>
 					<!-- this is just which name the Image msg will have, it does not affect the simulation.
 					     However must be set to the optical_frame,  -->
