Commit message: rslidar has optional gpu

File: urdf/rslidar.urdf.xacro (robot description, xacro)
@@ -2,5 +2,5 @@
 <robot name="sensor_rslidar" xmlns:xacro="http://wiki.ros.org/xacro">
   <xacro:property name="M_PI" value="3.1415926535897931" />
-  <xacro:macro name="sensor_rslidar" params="prefix parent prefix_topic *origin range_min range_max hfov hres vfov vres fps gpu">
+  <xacro:macro name="sensor_rslidar" params="prefix parent prefix_topic *origin range_min range_max hfov hres vfov vres fps gpu:=^|true">
     <material name="black_alu">
       <color rgba="0.9 0.9 0.9 1"/>

Commit message: Fix rslidar inertia

File: urdf/rslidar.urdf.xacro (robot description, xacro)
@@ -27,8 +27,7 @@
       </collision>
       <inertial>
-        <!-- The following are not reliable values, and should not be used for modeling -->
-        <mass value="0.564" />
-        <origin xyz="0 0 0" />
-        <inertia ixx="0.003881243" ixy="0.0" ixz="0.0" iyy="0.000498940" iyz="0.0" izz="0.003879257" />
+        <mass value="0.840" />
+        <origin xyz="0 0 0.04135" />
+				<xacro:solid_cuboid_inertia m="0.840" w="0.109" h="0.109" d="0.0827" />
       </inertial>
     </link>

Commit message: Add z offset to rslidar link

File: urdf/rslidar.urdf.xacro (robot description, xacro)
@@ -36,4 +36,5 @@
       <parent link="${prefix}_base_link"/>
       <child link="${prefix}_link" />
+      <origin xyz="0.0 0 0.038" rpy="0 0 0"/>
     </joint>
     <link name="${prefix}_link"/>
