Commit message: Add range_min and range_max parameters to velodyne_vlp16

File: urdf/velodyne_vlp16.urdf.xacro (robot description, xacro)
@@ -1,5 +1,5 @@
 <?xml version="1.0"?>
 <robot name="sensor_velodyne_vlp16" xmlns:xacro="http://wiki.ros.org/xacro">
-  <xacro:macro name="sensor_velodyne_vlp16" params="prefix parent prefix_topic:='velodyne' *origin gpu:=^|true">
+  <xacro:macro name="sensor_velodyne_vlp16" params="prefix parent prefix_topic:='velodyne' *origin range_min range_max gpu:=^|true">
     <joint name="${prefix}_base_joint" type="fixed">
       <xacro:insert_block name="origin" />
@@ -34,7 +34,7 @@
     </link>
     <!-- Velodyne sensor for simulation -->
-    <sensor_velodyne_vlp16_gazebo gpu="${gpu}" />
+    <sensor_velodyne_vlp16_gazebo range_min="${range_min}" range_max="${range_max}" gpu="${gpu}" />
   </xacro:macro>
-  <xacro:macro name="sensor_velodyne_vlp16_gazebo" params="gpu">
+  <xacro:macro name="sensor_velodyne_vlp16_gazebo" params="range_min range_max gpu">
     <gazebo reference="${prefix}_link">
       <xacro:if value="${gpu}">
@@ -67,6 +67,6 @@
               </scan>
               <range>
-                  <min>0.10</min>
-                  <max>30.0</max>
+              <min>${range_min}</min>
+              <max>${range_max}</max>
                   <resolution>0.01</resolution>
               </range>

Commit message: Fix velodyne inertia

File: urdf/velodyne_vlp16.urdf.xacro (robot description, xacro)
@@ -21,7 +21,7 @@
         </visual>
         <inertial>
-            <mass value="1e-5" />
-            <origin xyz="0 0 0" rpy="0 0 0"/>
-            <inertia ixx="1e-6" ixy="0" ixz="0" iyy="1e-6" iyz="0" izz="1e-6" />
+            <mass value="0.830" />
+            <origin xyz="0 0 0.03555" rpy="0 0 0"/>
+            <xacro:solid_cuboid_inertia m="0.830" w="0.1033" h="0.1033" d="0.0711" />
         </inertial>
     </link>

Commit message: Updated parameters for a correct vlp16 configuration

File: urdf/velodyne_vlp16.urdf.xacro (robot description, xacro)
@@ -1,5 +1,6 @@
 <?xml version="1.0"?>
 <robot name="sensor_velodyne_vlp16" xmlns:xacro="http://wiki.ros.org/xacro">
-  <xacro:macro name="sensor_velodyne_vlp16" params="prefix parent prefix_topic:='velodyne' *origin range_min range_max gpu:=^|true">
+  <xacro:property name="M_PI" value="3.1415926535897931" />
+  <xacro:macro name="sensor_velodyne_vlp16" params="prefix parent prefix_topic:='velodyne' *origin range_min range_max fps:=15 hsamples:=300 vsamples:=100 hfov:=360.0 vfov:=30.0 gpu:=^|true">
     <joint name="${prefix}_base_joint" type="fixed">
       <xacro:insert_block name="origin" />
@@ -50,18 +51,18 @@
           <pose>0 0 0 0 0 0</pose>
           <visualize>false</visualize>
-          <update_rate>15</update_rate>
+          <update_rate>${fps}</update_rate>
           <ray>
               <scan>
                   <horizontal>
-                      <samples>300</samples>
+                      <samples>${hsamples}</samples>
                       <resolution>1.0</resolution>
-                      <min_angle>-1.83591184</min_angle>
-                      <max_angle>1.83591184</max_angle>
+                      <min_angle>-${hfov/2.0*M_PI/180.0}</min_angle>
+                      <max_angle>${hfov/2.0*M_PI/180.0}</max_angle>
                   </horizontal>
                   <vertical>
-                      <samples>100</samples>
+                      <samples>${vsamples}</samples>
                       <resolution>1.0</resolution>
-                      <min_angle>-0.610865238</min_angle>
-                      <max_angle>1.83591184</max_angle>
+                      <min_angle>-${vfov/2.0*M_PI/180.0}</min_angle>
+                      <max_angle>${vfov/2.0*M_PI/180.0}</max_angle>
                   </vertical>
               </scan>
