Commit message: fotonic_e format

File: urdf/fotonic_e.urdf.xacro (robot description, xacro)
@@ -3,113 +3,113 @@
   <xacro:macro name="sensor_fotonic" params="prefix parent *origin">
     <joint name="${prefix}_joint" type="fixed">
-			<xacro:insert_block name="origin"/>
+      <xacro:insert_block name="origin"/>
       <parent link="${parent}"/>
       <child link="${prefix}_base_link"/>
-	  </joint>
-	  <link name="${prefix}_base_link">
-	    <inertial>
-			<origin xyz="0.0 0 0.0" rpy="0 0 0" />
-	      <mass value="0.0001" />
-	      <origin xyz="0 0 0" />
-	      <inertia ixx="0.0001" ixy="0.0" ixz="0.0"
-	               iyy="0.0001" iyz="0.0"
-	               izz="0.0001" />
-	    </inertial>
-	    <visual>
-	      <origin xyz="0.0 0.0 -0.04" rpy="0 0 0" /> <!-- to center the .dae model -->
-	      <material name="fotonic_color">
-           <color rgba="0.5 0.5 0.5 1"/>
+    </joint>
+    <link name="${prefix}_base_link">
+      <inertial>
+        <origin xyz="0.0 0 0.0" rpy="0 0 0" />
+        <mass value="0.0001" />
+        <origin xyz="0 0 0" />
+        <inertia ixx="0.0001" ixy="0.0" ixz="0.0"
+                  iyy="0.0001" iyz="0.0"
+                  izz="0.0001" />
+      </inertial>
+      <visual>
+        <origin xyz="0.0 0.0 -0.04" rpy="0 0 0" /> <!-- to center the .dae model -->
+        <material name="fotonic_color">
+          <color rgba="0.5 0.5 0.5 1"/>
         </material>
-	      <geometry>
-					<mesh filename= "package://robotnik_sensors/meshes/fotonic_e.stl" scale="1.0 1.0 1.0"/>
-	      </geometry>
-	    </visual>
-	    <collision>
-	      <origin xyz="0.0 0 -0.04" rpy="0 0 0" />
-	      <geometry>
-					<mesh filename= "package://robotnik_sensors/meshes/fotonic_e.stl" scale="1.0 1.0 1.0"/>
-	      </geometry>
-	    </collision>
-	  </link>
-	  <joint name="${prefix}_depth_joint" type="fixed">
-			<origin xyz="0.0375 0 0" rpy="0 0 0" />
-	    <parent link="${prefix}_base_link" />
-	    <child link="${prefix}_depth_frame_link" />
-	  </joint>
-	  <link name="${prefix}_depth_frame_link">
-	    <inertial>
-	      <mass value="0.0001" />
-	      <origin xyz="0 0 0" />
-	      <inertia ixx="0.0001" ixy="0.0" ixz="0.0"
-	               iyy="0.0001" iyz="0.0"
-	               izz="0.0001" />
-	    </inertial>
-	  </link>
-	  <joint name="${prefix}_depth_optical_joint" type="fixed">
-	    <origin xyz="0 0 0" rpy="-1.5708 0 -1.5708" />
-	    <parent link="${prefix}_depth_frame_link" />
-	    <child link="${prefix}_depth_optical_frame_link" />
-	  </joint>
-	  <link name="${prefix}_depth_optical_frame_link">
-	    <inertial>
-	      <mass value="0.0001" />
-	      <origin xyz="0 0 0" />
-	      <inertia ixx="0.0001" ixy="0.0" ixz="0.0"
-	               iyy="0.0001" iyz="0.0"
-	               izz="0.0001" />
-	    </inertial>
-	  </link>
-		<!-- Fotonic sensor for simulation -->
-		<sensor_fotonic_gazebo/>
+        <geometry>
+          <mesh filename= "package://robotnik_sensors/meshes/fotonic_e.stl" scale="1.0 1.0 1.0"/>
+        </geometry>
+      </visual>
+      <collision>
+        <origin xyz="0.0 0 -0.04" rpy="0 0 0" />
+        <geometry>
+          <mesh filename= "package://robotnik_sensors/meshes/fotonic_e.stl" scale="1.0 1.0 1.0"/>
+        </geometry>
+      </collision>
+    </link>
+    <joint name="${prefix}_depth_joint" type="fixed">
+      <origin xyz="0.0375 0 0" rpy="0 0 0" />
+      <parent link="${prefix}_base_link" />
+      <child link="${prefix}_depth_frame_link" />
+    </joint>
+    <link name="${prefix}_depth_frame_link">
+      <inertial>
+        <mass value="0.0001" />
+        <origin xyz="0 0 0" />
+        <inertia ixx="0.0001" ixy="0.0" ixz="0.0"
+                  iyy="0.0001" iyz="0.0"
+                  izz="0.0001" />
+      </inertial>
+    </link>
+    <joint name="${prefix}_depth_optical_joint" type="fixed">
+      <origin xyz="0 0 0" rpy="-1.5708 0 -1.5708" />
+      <parent link="${prefix}_depth_frame_link" />
+      <child link="${prefix}_depth_optical_frame_link" />
+    </joint>
+    <link name="${prefix}_depth_optical_frame_link">
+      <inertial>
+        <mass value="0.0001" />
+        <origin xyz="0 0 0" />
+        <inertia ixx="0.0001" ixy="0.0" ixz="0.0"
+                  iyy="0.0001" iyz="0.0"
+                  izz="0.0001" />
+      </inertial>
+    </link>
+    <!-- Fotonic sensor for simulation -->
+    <sensor_fotonic_gazebo/>
   </xacro:macro>
   <xacro:macro name="sensor_fotonic_gazebo">
-		<gazebo reference="${prefix}_base_link">
+    <gazebo reference="${prefix}_base_link">
       <material>Gazebo/Grey</material>
     </gazebo>
     <gazebo reference="${prefix}_depth_frame_link">
-	    <sensor type="depth" name="${prefix}_sensor">
-	      <update_rate>30.0</update_rate>
-	      <camera name="fotonic">
-	        <horizontal_fov>1.221730476</horizontal_fov>  <!-- 70 deg -->
-	        <image>
-	          <width>160</width>  <!-- 160 -->
-	          <height>120</height> <!-- 120 -->
-	          <format>L8</format> <!-- gray -->
-	        </image>
-	        <clip>
-	          <near>0.05</near>
-	          <far>7.0</far>         <!-- outdoor down to 3m depending on luminosity -->
-	        </clip>
-	        <noise>
-	          <type>gaussian</type>
-	          <mean>0.0</mean>
-	          <stddev>0.007</stddev>
-	        </noise>
-	      </camera>
-		    <plugin name="${prefix}_controller" filename="libgazebo_ros_openni_kinect.so">
-					<alwaysOn>true</alwaysOn>
-					<updateRate>10.0</updateRate>
-					<cameraName>${prefix}</cameraName>
-					<imageTopicName>ir/image_raw</imageTopicName>
-					<cameraInfoTopicName>ir/camera_info</cameraInfoTopicName>
-					<depthImageTopicName>depth/image_raw</depthImageTopicName>
-					<depthImageCameraInfoTopicName>depth/camera_info</depthImageCameraInfoTopicName>
-					<pointCloudTopicName>points</pointCloudTopicName>
-					<frameName>${prefix}_depth_optical_frame_link</frameName>
-					<pointCloudCutoff>0.5</pointCloudCutoff>
-					<distortionK1>0</distortionK1>
-					<distortionK2>0</distortionK2>
-					<distortionK3>0</distortionK3>
-					<distortionT1>0</distortionT1>
-					<distortionT2>0</distortionT2>
-					<CxPrime>0</CxPrime>
-					<Cx>0</Cx>
-					<Cy>0</Cy>
-					<focalLength>0</focalLength>
-					<hackBaseline>0</hackBaseline>
-					<ignoreTfPrefix>1</ignoreTfPrefix>
-			  </plugin>
-	    </sensor>
-	  </gazebo>
+      <sensor type="depth" name="${prefix}_sensor">
+        <update_rate>30.0</update_rate>
+        <camera name="fotonic">
+          <horizontal_fov>1.221730476</horizontal_fov>  <!-- 70 deg -->
+          <image>
+            <width>160</width>  <!-- 160 -->
+            <height>120</height> <!-- 120 -->
+            <format>L8</format> <!-- gray -->
+          </image>
+          <clip>
+            <near>0.05</near>
+            <far>7.0</far>         <!-- outdoor down to 3m depending on luminosity -->
+          </clip>
+          <noise>
+            <type>gaussian</type>
+            <mean>0.0</mean>
+            <stddev>0.007</stddev>
+          </noise>
+        </camera>
+        <plugin name="${prefix}_controller" filename="libgazebo_ros_openni_kinect.so">
+          <alwaysOn>true</alwaysOn>
+          <updateRate>10.0</updateRate>
+          <cameraName>${prefix}</cameraName>
+          <imageTopicName>ir/image_raw</imageTopicName>
+          <cameraInfoTopicName>ir/camera_info</cameraInfoTopicName>
+          <depthImageTopicName>depth/image_raw</depthImageTopicName>
+          <depthImageCameraInfoTopicName>depth/camera_info</depthImageCameraInfoTopicName>
+          <pointCloudTopicName>points</pointCloudTopicName>
+          <frameName>${prefix}_depth_optical_frame_link</frameName>
+          <pointCloudCutoff>0.5</pointCloudCutoff>
+          <distortionK1>0</distortionK1>
+          <distortionK2>0</distortionK2>
+          <distortionK3>0</distortionK3>
+          <distortionT1>0</distortionT1>
+          <distortionT2>0</distortionT2>
+          <CxPrime>0</CxPrime>
+          <Cx>0</Cx>
+          <Cy>0</Cy>
+          <focalLength>0</focalLength>
+          <hackBaseline>0</hackBaseline>
+          <ignoreTfPrefix>1</ignoreTfPrefix>
+        </plugin>
+      </sensor>
+    </gazebo>
   </xacro:macro>
 </robot>

Commit message: Update fotonic_e inertia

File: urdf/fotonic_e.urdf.xacro (robot description, xacro)
@@ -10,9 +10,6 @@
       <inertial>
         <origin xyz="0.0 0 0.0" rpy="0 0 0" />
-        <mass value="0.0001" />
-        <origin xyz="0 0 0" />
-        <inertia ixx="0.0001" ixy="0.0" ixz="0.0"
-                  iyy="0.0001" iyz="0.0"
-                  izz="0.0001" />
+        <mass value="0.79" />
+        <xacro:solid_cuboid_inertia m="0.79" w="0.08" h="0.0863" d="0.08" />
       </inertial>
       <visual>
@@ -39,9 +36,7 @@
     <link name="${prefix}_depth_frame_link">
       <inertial>
-        <mass value="0.0001" />
-        <origin xyz="0 0 0" />
-        <inertia ixx="0.0001" ixy="0.0" ixz="0.0"
-                  iyy="0.0001" iyz="0.0"
-                  izz="0.0001" />
+        <origin xyz="-0.0375 0 0.0" rpy="0 0 0" />
+        <mass value="0.01" />
+        <xacro:solid_cuboid_inertia m="0.01" w="0.08" h="0.0863" d="0.08" />
       </inertial>
     </link>
@@ -52,11 +47,9 @@
     </joint>
     <link name="${prefix}_depth_optical_frame_link">
-      <inertial>
-        <mass value="0.0001" />
-        <origin xyz="0 0 0" />
-        <inertia ixx="0.0001" ixy="0.0" ixz="0.0"
-                  iyy="0.0001" iyz="0.0"
-                  izz="0.0001" />
-      </inertial>
+      <!--inertial>
+        <origin xyz="-0.0375 0 0.0" rpy="0 0 0" />
+        <mass value="0.01" />
+        <xacro:solid_cuboid_inertia m="0.01" w="0.08" h="0.0863" d="0.08" />
+      </inertial-->
     </link>
     <!-- Fotonic sensor for simulation -->
