Commit message: robotnik_sensors: adding min and max angle params to hokuyo sensors

File: urdf/hokuyo_urg04lx.urdf.xacro (robot description, xacro)
@@ -1,5 +1,5 @@
 <?xml version="1.0"?>
 <robot name="sensor_hokuyo_urg04lx" xmlns:xacro="http://ros.org/wiki/xacro">
-  <xacro:macro name="sensor_hokuyo_urg04lx" params="name parent *origin">
+  <xacro:macro name="sensor_hokuyo_urg04lx" params="name parent *origin min_angle:=2.0943 max_angle:=-2.0943">
     <joint name="${name}_laser_joint" type="fixed">
       <!-- FRONT MOUNT  -->
@@ -10,28 +10,28 @@
       <parent link="${parent}"/>
       <child link="${name}_laser_link"/>
-	</joint>
-	<link name="${name}_laser_link">
-		<collision>
-			<origin xyz="0 0 -0.05" rpy="0 0 0"/>
-			<geometry>
-				<box size="0.1 0.1 0.08"/>
-			</geometry>
-		</collision>
-		<visual>
-			<origin xyz="0 0 -0.05" rpy="0 0 0"/>
-			<geometry>
-	     		<mesh filename="package://robotnik_sensors/meshes/hokuyo_urg_04lx.dae"/>
-			</geometry>
-		</visual>
-		<inertial>
-			<mass value="1e-5" />
-			<origin xyz="0 0 0" rpy="0 0 0"/>
-			<inertia ixx="1e-6" ixy="0" ixz="0" iyy="1e-6" iyz="0" izz="1e-6" />
-		</inertial>
-	</link>
-	<!-- Hokuyo sensor for simulation -->
-	<sensor_hokuyo_gazebo/>
+    </joint>
+    <link name="${name}_laser_link">
+      <collision>
+        <origin xyz="0 0 -0.05" rpy="0 0 0"/>
+        <geometry>
+          <box size="0.1 0.1 0.08"/>
+        </geometry>
+      </collision>
+      <visual>
+        <origin xyz="0 0 -0.05" rpy="0 0 0"/>
+        <geometry>
+            <mesh filename="package://robotnik_sensors/meshes/hokuyo_urg_04lx.dae"/>
+        </geometry>
+      </visual>
+      <inertial>
+        <mass value="1e-5" />
+        <origin xyz="0 0 0" rpy="0 0 0"/>
+        <inertia ixx="1e-6" ixy="0" ixz="0" iyy="1e-6" iyz="0" izz="1e-6" />
+      </inertial>
+    </link>
+    <!-- Hokuyo sensor for simulation -->
+    <sensor_hokuyo_urg_gazebo/>
   </xacro:macro>
-  <xacro:macro name="sensor_hokuyo_gazebo">
+  <xacro:macro name="sensor_hokuyo_urg_gazebo">
     <gazebo reference="${name}_laser_link">
 			<sensor type="ray" name="${name}_sensor">
@@ -44,6 +44,6 @@
 							<samples>640</samples>
 							<resolution>1</resolution>
-							<min_angle>2.0943951</min_angle>
-							<max_angle>-2.0943951</max_angle>
+							<min_angle>${min_angle}</min_angle>
+							<max_angle>${max_angle}</max_angle>
 						</horizontal>
 					</scan>

File: urdf/hokuyo_ust10lx.urdf.xacro (robot description, xacro)
@@ -1,33 +1,33 @@
 <?xml version="1.0"?>
 <robot name="sensor_hokuyo_ust10lx" xmlns:xacro="http://ros.org/wiki/xacro">
-  <xacro:macro name="sensor_hokuyo_ust10lx" params="name parent *origin">
+  <xacro:macro name="sensor_hokuyo_ust10lx" params="name parent *origin min_angle:=2.35 max_angle:=-2.35">
     <joint name="${name}_laser_joint" type="fixed">
       <insert_block name="origin" />
       <parent link="${parent}"/>
       <child link="${name}_laser_link"/>
-	</joint>
-	<link name="${name}_laser_link">
-		<collision>
-			<origin xyz="0 0 -0.05" rpy="0 0 0"/>
-			<geometry>
-				<box size="0.1 0.1 0.08"/>
-			</geometry>
-		</collision>
-		<visual>
-			<origin xyz="0 0 -0.05" rpy="0 0 0"/>
-			<geometry>
-	     		<mesh filename="package://robotnik_sensors/meshes/hokuyo_ust_10lx.dae"/>
-			</geometry>
-		</visual>
-		<inertial>
-			<mass value="1e-5" />
-			<origin xyz="0 0 0" rpy="0 0 0"/>
-			<inertia ixx="1e-6" ixy="0" ixz="0" iyy="1e-6" iyz="0" izz="1e-6" />
-		</inertial>
-	</link>
-	<!-- Hokuyo sensor for simulation -->
-	<sensor_hokuyo_gazebo/>
+    </joint>
+    <link name="${name}_laser_link">
+      <collision>
+        <origin xyz="0 0 -0.05" rpy="0 0 0"/>
+        <geometry>
+          <box size="0.1 0.1 0.08"/>
+        </geometry>
+      </collision>
+      <visual>
+        <origin xyz="0 0 -0.05" rpy="0 0 0"/>
+        <geometry>
+            <mesh filename="package://robotnik_sensors/meshes/hokuyo_ust_10lx.dae"/>
+        </geometry>
+      </visual>
+      <inertial>
+        <mass value="1e-5" />
+        <origin xyz="0 0 0" rpy="0 0 0"/>
+        <inertia ixx="1e-6" ixy="0" ixz="0" iyy="1e-6" iyz="0" izz="1e-6" />
+      </inertial>
+    </link>
+    <!-- Hokuyo sensor for simulation -->
+    <sensor_hokuyo_ust_gazebo/>
   </xacro:macro>
-  <xacro:macro name="sensor_hokuyo_gazebo">
+  <xacro:macro name="sensor_hokuyo_ust_gazebo">
     <gazebo reference="${name}_laser_link">
 			<sensor type="ray" name="${name}_sensor">
@@ -40,6 +40,6 @@
 							<samples>1081</samples>
 							<resolution>1</resolution>
-							<min_angle>2.35619449</min_angle>
-							<max_angle>-2.35619449</max_angle>
+							<min_angle>${min_angle}</min_angle>
+							<max_angle>${max_angle}</max_angle>
 						</horizontal>
 					</scan>

File: urdf/hokuyo_utm30lx.urdf.xacro (robot description, xacro)
@@ -1,5 +1,5 @@
 <?xml version="1.0"?>
 <robot name="sensor_hokuyo_utm30lx" xmlns:xacro="http://ros.org/wiki/xacro">
-  <xacro:macro name="sensor_hokuyo_utm30lx" params="name parent *origin">
+  <xacro:macro name="sensor_hokuyo_utm30lx" params="name parent *origin min_angle:=2.35 max_angle:=-2.35">
     <joint name="${name}_laser_joint" type="fixed">
       <!-- FRONT MOUNT  -->
@@ -10,22 +10,22 @@
       <parent link="${parent}"/>
       <child link="${name}_laser_link"/>
-	</joint>
-	<link name="${name}_laser_link">
-		<visual>
-			<origin xyz="0 0 0" rpy="0 0 0"/>
-			<geometry>
-	     		<mesh filename="package://robotnik_sensors/meshes/hokuyo_utm_30lx.dae"/>
-			</geometry>
-		</visual>
-		<inertial>
-			<mass value="1e-5" />
-			<origin xyz="0 0 0" rpy="0 0 0"/>
-			<inertia ixx="1e-6" ixy="0" ixz="0" iyy="1e-6" iyz="0" izz="1e-6" />
-		</inertial>
-	</link>
-	<!-- Hokuyo sensor for simulation -->
-	<sensor_hokuyo_gazebo/>
+    </joint>
+    <link name="${name}_laser_link">
+      <visual>
+        <origin xyz="0 0 0" rpy="0 0 0"/>
+        <geometry>
+            <mesh filename="package://robotnik_sensors/meshes/hokuyo_utm_30lx.dae"/>
+        </geometry>
+      </visual>
+      <inertial>
+        <mass value="1e-5" />
+        <origin xyz="0 0 0" rpy="0 0 0"/>
+        <inertia ixx="1e-6" ixy="0" ixz="0" iyy="1e-6" iyz="0" izz="1e-6" />
+      </inertial>
+    </link>
+    <!-- Hokuyo sensor for simulation -->
+    <sensor_hokuyo_utm_gazebo/>
   </xacro:macro>
-  <xacro:macro name="sensor_hokuyo_gazebo">
+  <xacro:macro name="sensor_hokuyo_utm_gazebo">
     <gazebo reference="${name}_laser_link">
 			<sensor type="ray" name="${name}_sensor">
@@ -38,6 +38,6 @@
 							<samples>1081</samples>
 							<resolution>1</resolution>
-							<min_angle>2.35619449</min_angle>  <!-- +/-135 deg -->
-							<max_angle>-2.35619449</max_angle>
+							<min_angle>${min_angle}</min_angle>
+							<max_angle>${max_angle}</max_angle>
 						</horizontal>
 					</scan>

Commit message: added link position to hokuyo lasers

File: urdf/hokuyo_urg04lx.urdf.xacro (robot description, xacro)
@@ -30,9 +30,16 @@
       </inertial>
     </link>
+    <link name="${prefix}_link">
+	</link>
+    <joint name="${prefix}_joint" type="fixed">
+      <parent link="${prefix}_base_link"/>
+      <child link="${prefix}_link"/>
+      <origin xyz="0.00 0 0.05" rpy="0 0 0"/>
+	</joint>
     <!-- Hokuyo sensor for simulation -->
     <sensor_hokuyo_urg_gazebo/>
   </xacro:macro>
   <xacro:macro name="sensor_hokuyo_urg_gazebo">
-    <gazebo reference="${prefix}_base_link">
+    <gazebo reference="${prefix}_link">
 			<sensor type="ray" name="${prefix}_sensor">
 				<pose>0 0 0 0 0 0</pose>
@@ -61,5 +68,5 @@
 				<plugin name="${name}_controller" filename="libgazebo_ros_laser.so">
 					<topicName>scan</topicName>
-					<frameName>${prefix}_base_link</frameName>
+					<frameName>${prefix}_link</frameName>
 					<ignoreTfPrefix>1</ignoreTfPrefix>
 				</plugin>

File: urdf/hokuyo_ust10lx.urdf.xacro (robot description, xacro)
@@ -27,9 +27,16 @@
       </inertial>
     </link>
+    <link name="${prefix}_link">
+	</link>
+    <joint name="${prefix}_joint" type="fixed">
+      <parent link="${prefix}_base_link"/>
+      <child link="${prefix}_link"/>
+      <origin xyz="0.00 0 0.0474" rpy="0 0 0"/>
+	</joint>
     <!-- Hokuyo sensor for simulation -->
     <xacro:sensor_hokuyo_ust_gazebo/>
   </xacro:macro>
   <xacro:macro name="sensor_hokuyo_ust_gazebo">
-    <gazebo reference="${prefix}_base_link">
+    <gazebo reference="${prefix}_link">
 			<sensor type="ray" name="${prefix}_sensor">
 				<pose>0 0 0 0 0 0</pose>
@@ -60,5 +67,5 @@
 				<plugin name="${prefix}_controller" filename="libgazebo_ros_laser.so">
 					<topicName>scan</topicName>
-					<frameName>${prefix}_base_link</frameName>
+					<frameName>${prefix}_link</frameName>
 					<ignoreTfPrefix>1</ignoreTfPrefix>
 				</plugin>

File: urdf/hokuyo_utm30lx.urdf.xacro (robot description, xacro)
@@ -24,9 +24,16 @@
       </inertial>
     </link>
+	<link name="${prefix}_link">
+	</link>
+    <joint name="${prefix}_joint" type="fixed">
+      <parent link="${prefix}_base_link"/>
+      <child link="${prefix}_link"/>
+      <origin xyz="0.00 0 0.055" rpy="0 0 0"/>
+	</joint>
     <!-- Hokuyo sensor for simulation -->
     <sensor_hokuyo_utm_gazebo/>
   </xacro:macro>
   <xacro:macro name="sensor_hokuyo_utm_gazebo">
-    <gazebo reference="${prefix}_base_link">
+    <gazebo reference="${prefix}_link">
 			<sensor type="ray" name="${prefix}_sensor">
 				<pose>0 0 0 0 0 0</pose>
@@ -55,5 +62,5 @@
 				<plugin name="${prefix}_controller" filename="libgazebo_ros_laser.so">
 					<topicName>scan</topicName>
-					<frameName>${prefix}_base_link</frameName>
+					<frameName>${prefix}_link</frameName>
 					<ignoreTfPrefix>1</ignoreTfPrefix>
 				</plugin>

Commit message: hokuyo_urg04 model updated

File: urdf/hokuyo_urg04lx.urdf.xacro (robot description, xacro)
@@ -4,5 +4,5 @@
     <joint name="${prefix}_base_joint" type="fixed">
       <!-- FRONT MOUNT  -->
-      <!-- origin xyz="0.29 0 0.1" -->
+      <!--origin xyz="0.29 0 0.1" -->
       <!-- TOP MOUNT -->
       <!-- origin xyz="0.0 0.0 0.325"-->
@@ -12,14 +12,8 @@
     </joint>
     <link name="${prefix}_base_link">
-      <collision>
-        <origin xyz="0 0 -0.05" rpy="0 0 0"/>
-        <geometry>
-          <box size="0.1 0.1 0.08"/>
-        </geometry>
-      </collision>
       <visual>
         <origin xyz="0 0 -0.05" rpy="0 0 0"/>
         <geometry>
-            <mesh filename="package://robotnik_sensors/meshes/hokuyo_urg_04lx.dae"/>
+            <mesh filename="package://robotnik_sensors/meshes/hokuyo_urg_04lx2.dae"/>
         </geometry>
       </visual>
@@ -66,5 +60,5 @@
 					</noise>
 				</ray>
-				<plugin name="${name}_controller" filename="libgazebo_ros_laser.so">
+				<plugin name="${prefix}_controller" filename="libgazebo_ros_laser.so">
 					<topicName>scan</topicName>
 					<frameName>${prefix}_link</frameName>

Commit message: laser hokuyo_urg04lx updated

File: urdf/hokuyo_urg04lx.urdf.xacro (robot description, xacro)
@@ -15,5 +15,5 @@
         <origin xyz="0 0 -0.05" rpy="0 0 0"/>
         <geometry>
-            <mesh filename="package://robotnik_sensors/meshes/hokuyo_urg_04lx2.dae"/>
+            <mesh filename="package://robotnik_sensors/meshes/hokuyo_urg_04lx.dae"/>
         </geometry>
       </visual>

Commit message: adding prefix_scan to all 2d lasers

File: urdf/hokuyo_urg04lx.urdf.xacro (robot description, xacro)
@@ -1,5 +1,5 @@
 <?xml version="1.0"?>
 <robot name="sensor_hokuyo_urg04lx" xmlns:xacro="http://www.ros.org/wiki/xacro">
-  <xacro:macro name="sensor_hokuyo_urg04lx" params="prefix parent *origin min_angle:=-2.0943 max_angle:=2.0943">
+  <xacro:macro name="sensor_hokuyo_urg04lx" params="prefix parent prefix_scan *origin min_angle:=-2.0943 max_angle:=2.0943">
     <joint name="${prefix}_base_joint" type="fixed">
       <!-- FRONT MOUNT  -->
@@ -32,7 +32,7 @@
 	</joint>
     <!-- Hokuyo sensor for simulation -->
-    <sensor_hokuyo_urg_gazebo/>
+    <sensor_hokuyo_urg04lx_gazebo/>
   </xacro:macro>
-  <xacro:macro name="sensor_hokuyo_urg_gazebo">
+  <xacro:macro name="sensor_hokuyo_urg04lx_gazebo">
     <gazebo reference="${prefix}_link">
 			<sensor type="ray" name="${prefix}_sensor">
@@ -61,5 +61,5 @@
 				</ray>
 				<plugin name="${prefix}_controller" filename="libgazebo_ros_laser.so">
-					<topicName>scan</topicName>
+					<topicName>${prefix_scan}/scan</topicName>
 					<frameName>${prefix}_link</frameName>
 					<ignoreTfPrefix>1</ignoreTfPrefix>

File: urdf/hokuyo_ust10lx.urdf.xacro (robot description, xacro)
@@ -1,5 +1,5 @@
 <?xml version="1.0"?>
 <robot name="sensor_hokuyo_ust10lx" xmlns:xacro="http://www.ros.org/wiki/xacro">
-  <xacro:macro name="sensor_hokuyo_ust10lx" params="prefix parent *origin min_angle:=-2.3562 max_angle:=2.3562">
+  <xacro:macro name="sensor_hokuyo_ust10lx" params="prefix parent prefix_scan *origin min_angle:=-2.3562 max_angle:=2.3562">
 			<!--arg name="namespace" value="$(arg namespace)"/-->
     <joint name="${prefix}_base_joint" type="fixed">
@@ -35,7 +35,7 @@
 	</joint>
     <!-- Hokuyo sensor for simulation -->
-    <xacro:sensor_hokuyo_ust_gazebo/>
+    <xacro:sensor_hokuyo_ust10_gazebo/>
   </xacro:macro>
-  <xacro:macro name="sensor_hokuyo_ust_gazebo">
+  <xacro:macro name="sensor_hokuyo_ust10_gazebo">
     <gazebo reference="${prefix}_link">
 			<sensor type="ray" name="${prefix}_sensor">
@@ -66,5 +66,5 @@
 				</ray>
 				<plugin name="${prefix}_controller" filename="libgazebo_ros_laser.so">
-					<topicName>scan</topicName>
+					<topicName>${prefix_scan}/scan</topicName>
 					<frameName>${prefix}_link</frameName>
 					<ignoreTfPrefix>1</ignoreTfPrefix>

File: urdf/hokuyo_ust20lx.urdf.xacro (robot description, xacro)
@@ -1,5 +1,5 @@
 <?xml version="1.0"?>
 <robot name="sensor_hokuyo_ust20lx" xmlns:xacro="http://www.ros.org/wiki/xacro">
-  <xacro:macro name="sensor_hokuyo_ust20lx" params="prefix parent *origin min_angle:=-2.3562 max_angle:=2.3562">
+  <xacro:macro name="sensor_hokuyo_ust20lx" params="prefix parent prefix_scan *origin min_angle:=-2.3562 max_angle:=2.3562">
 			<!--arg name="namespace" value="$(arg namespace)"/-->
     <joint name="${prefix}_base_joint" type="fixed">
@@ -35,7 +35,7 @@
 	</joint>
     <!-- Hokuyo sensor for simulation -->
-    <xacro:sensor_hokuyo_ust_gazebo/>
+    <xacro:sensor_hokuyo_ust20_gazebo/>
   </xacro:macro>
-  <xacro:macro name="sensor_hokuyo_ust_gazebo">
+  <xacro:macro name="sensor_hokuyo_ust20_gazebo">
     <gazebo reference="${prefix}_link">
 			<sensor type="ray" name="${prefix}_sensor">
@@ -54,5 +54,5 @@
 					<range>
 						<min>0.06</min>
-						<max>10.0</max>
+						<max>20.0</max>
 						<!-- resolution>0.004363323</resolution -->
 						<resolution>0.004359297</resolution>
@@ -66,5 +66,5 @@
 				</ray>
 				<plugin name="${prefix}_controller" filename="libgazebo_ros_laser.so">
-					<topicName>scan</topicName>
+					<topicName>${prefix_scan}/scan</topicName>
 					<frameName>${prefix}_link</frameName>
 					<ignoreTfPrefix>1</ignoreTfPrefix>

File: urdf/hokuyo_utm30lx.urdf.xacro (robot description, xacro)
@@ -1,5 +1,5 @@
 <?xml version="1.0"?>
 <robot name="sensor_hokuyo_utm30lx" xmlns:xacro="http://www.ros.org/wiki/xacro">
-  <xacro:macro name="sensor_hokuyo_utm30lx" params="prefix parent *origin min_angle:=-2.35 max_angle:=2.35">
+  <xacro:macro name="sensor_hokuyo_utm30lx" params="prefix parent prefix_scan *origin min_angle:=-2.35 max_angle:=2.35">
     <joint name="${prefix}_base_joint" type="fixed">
       <!-- FRONT MOUNT  -->
@@ -61,5 +61,5 @@
 				</ray>
 				<plugin name="${prefix}_controller" filename="libgazebo_ros_laser.so">
-					<topicName>scan</topicName>
+					<topicName>${prefix_scan}/scan</topicName>
 					<frameName>${prefix}_link</frameName>
 					<ignoreTfPrefix>1</ignoreTfPrefix>

File: urdf/sick_s300.urdf.xacro (robot description, xacro)
@@ -1,5 +1,5 @@
 <?xml version="1.0"?>
 <robot name="sensor_sick_s300" xmlns:xacro="http://www.ros.org/wiki/xacro">
-  <xacro:macro name="sensor_sick_s300" params="prefix parent *origin">
+  <xacro:macro name="sensor_sick_s300" params="prefix parent prefix_scan *origin">
     <joint name="${prefix}_base_joint" type="fixed">
       <xacro:insert_block name="origin" />
@@ -64,5 +64,5 @@
 				</ray>
 				<plugin name="${prefix}_controller" filename="libgazebo_ros_laser.so">
-					<topicName>scan</topicName>
+					<topicName>${prefix_scan}/scan</topicName>
 					<frameName>${prefix}_link</frameName><!-- if not global (leading /) sets the current namespace as a prefix (/ns/name_laser_link) -->
 					<ignoreTfPrefix>1</ignoreTfPrefix>

File: urdf/sick_s3000.urdf.xacro (robot description, xacro)
@@ -1,5 +1,5 @@
 <?xml version="1.0"?>
 <robot name="sensor_sick_s3000" xmlns:xacro="http://www.ros.org/wiki/xacro">
-  <xacro:macro name="sensor_sick_s3000" params="prefix parent *origin">
+  <xacro:macro name="sensor_sick_s3000" params="prefix parent prefix_scan *origin">
     <joint name="${prefix}_joint" type="fixed">
       <xacro:insert_block name="origin" />
@@ -56,5 +56,5 @@
 				</ray>
 				<plugin name="${prefix}_controller" filename="libgazebo_ros_laser.so">
-					<topicName>scan</topicName>
+					<topicName>${prefix_scan}/scan</topicName>
 					<frameName>${prefix}_base_link</frameName>
 					<ignoreTfPrefix>1</ignoreTfPrefix>

File: urdf/sick_tim551.urdf.xacro (robot description, xacro)
@@ -1,5 +1,5 @@
 <?xml version="1.0"?>
 <robot xmlns:xacro="http://www.ros.org/wiki/xacro">
-  <xacro:macro name="sensor_sick_tim551" params="prefix parent *origin min_angle:=-2.36 max_angle:=2.36">
+  <xacro:macro name="sensor_sick_tim551" params="prefix parent prefix_scan *origin min_angle:=-2.36 max_angle:=2.36">
     <joint name="${prefix}_base_joint" type="fixed">
       <xacro:insert_block name="origin" />
@@ -62,5 +62,5 @@
 				</ray>
 				<plugin name="${prefix}_controller" filename="libgazebo_ros_laser.so">
-					<topicName>scan</topicName>
+					<topicName>${prefix_scan}/scan</topicName>
 					<frameName>${prefix}_link</frameName> <!-- leading / avoids that current namespace is added as prefix in the frame name (/ns/prefix_link) -->
 					<ignoreTfPrefix>1</ignoreTfPrefix>

File: urdf/sick_tim571.urdf.xacro (robot description, xacro)
@@ -1,5 +1,5 @@
 <?xml version="1.0"?>
 <robot xmlns:xacro="http://www.ros.org/wiki/xacro">
-  <xacro:macro name="sensor_sick_tim571" params="prefix parent *origin min_angle:=-2.36 max_angle:=2.36">
+  <xacro:macro name="sensor_sick_tim571" params="prefix parent prefix_scan *origin min_angle:=-2.36 max_angle:=2.36">
     <joint name="${prefix}_base_joint" type="fixed">
       <xacro:insert_block name="origin" />
@@ -62,5 +62,5 @@
 				</ray>
 				<plugin name="${prefix}_controller" filename="libgazebo_ros_laser.so">
-					<topicName>scan</topicName>
+					<topicName>${prefix_scan}/scan</topicName>
 					<frameName>${prefix}_link</frameName>
 					<ignoreTfPrefix>1</ignoreTfPrefix>
