Commit message: renamig prefix_scan with prefix_topic for all the 2d lasers

File: urdf/hokuyo_urg04lx.urdf.xacro (robot description, xacro)
@@ -1,5 +1,5 @@
 <?xml version="1.0"?>
 <robot name="sensor_hokuyo_urg04lx" xmlns:xacro="http://www.ros.org/wiki/xacro">
-  <xacro:macro name="sensor_hokuyo_urg04lx" params="prefix parent prefix_scan *origin min_angle:=-2.0943 max_angle:=2.0943">
+  <xacro:macro name="sensor_hokuyo_urg04lx" params="prefix parent prefix_topic *origin min_angle:=-2.0943 max_angle:=2.0943">
     <joint name="${prefix}_base_joint" type="fixed">
       <!-- FRONT MOUNT  -->
@@ -61,5 +61,5 @@
 				</ray>
 				<plugin name="${prefix}_controller" filename="libgazebo_ros_laser.so">
-					<topicName>${prefix_scan}/scan</topicName>
+					<topicName>${prefix_topic}/scan</topicName>
 					<frameName>${prefix}_link</frameName>
 					<ignoreTfPrefix>1</ignoreTfPrefix>

File: urdf/hokuyo_ust10lx.urdf.xacro (robot description, xacro)
@@ -1,5 +1,5 @@
 <?xml version="1.0"?>
 <robot name="sensor_hokuyo_ust10lx" xmlns:xacro="http://www.ros.org/wiki/xacro">
-  <xacro:macro name="sensor_hokuyo_ust10lx" params="prefix parent prefix_scan *origin min_angle:=-2.3562 max_angle:=2.3562">
+  <xacro:macro name="sensor_hokuyo_ust10lx" params="prefix parent prefix_topic *origin min_angle:=-2.3562 max_angle:=2.3562">
 			<!--arg name="namespace" value="$(arg namespace)"/-->
     <joint name="${prefix}_base_joint" type="fixed">
@@ -66,5 +66,5 @@
 				</ray>
 				<plugin name="${prefix}_controller" filename="libgazebo_ros_laser.so">
-					<topicName>${prefix_scan}/scan</topicName>
+					<topicName>${prefix_topic}/scan</topicName>
 					<frameName>${prefix}_link</frameName>
 					<ignoreTfPrefix>1</ignoreTfPrefix>

File: urdf/hokuyo_ust20lx.urdf.xacro (robot description, xacro)
@@ -1,5 +1,5 @@
 <?xml version="1.0"?>
 <robot name="sensor_hokuyo_ust20lx" xmlns:xacro="http://www.ros.org/wiki/xacro">
-  <xacro:macro name="sensor_hokuyo_ust20lx" params="prefix parent prefix_scan *origin min_angle:=-2.3562 max_angle:=2.3562">
+  <xacro:macro name="sensor_hokuyo_ust20lx" params="prefix parent prefix_topic *origin min_angle:=-2.3562 max_angle:=2.3562">
 			<!--arg name="namespace" value="$(arg namespace)"/-->
     <joint name="${prefix}_base_joint" type="fixed">
@@ -66,5 +66,5 @@
 				</ray>
 				<plugin name="${prefix}_controller" filename="libgazebo_ros_laser.so">
-					<topicName>${prefix_scan}/scan</topicName>
+					<topicName>${prefix_topic}/scan</topicName>
 					<frameName>${prefix}_link</frameName>
 					<ignoreTfPrefix>1</ignoreTfPrefix>

File: urdf/hokuyo_utm30lx.urdf.xacro (robot description, xacro)
@@ -1,5 +1,5 @@
 <?xml version="1.0"?>
 <robot name="sensor_hokuyo_utm30lx" xmlns:xacro="http://www.ros.org/wiki/xacro">
-  <xacro:macro name="sensor_hokuyo_utm30lx" params="prefix parent prefix_scan *origin min_angle:=-2.35 max_angle:=2.35">
+  <xacro:macro name="sensor_hokuyo_utm30lx" params="prefix parent prefix_topic *origin min_angle:=-2.35 max_angle:=2.35">
     <joint name="${prefix}_base_joint" type="fixed">
       <!-- FRONT MOUNT  -->
@@ -61,5 +61,5 @@
 				</ray>
 				<plugin name="${prefix}_controller" filename="libgazebo_ros_laser.so">
-					<topicName>${prefix_scan}/scan</topicName>
+					<topicName>${prefix_topic}/scan</topicName>
 					<frameName>${prefix}_link</frameName>
 					<ignoreTfPrefix>1</ignoreTfPrefix>

File: urdf/rplidar.urdf.xacro (robot description, xacro)
@@ -1,5 +1,5 @@
 <?xml version="1.0"?>
 <robot xmlns:xacro="http://www.ros.org/wiki/xacro">
-  <xacro:macro name="sensor_rplidar" params="prefix parent prefix_scan *origin min_angle:=3.14159 max_angle:=-3.14159">
+  <xacro:macro name="sensor_rplidar" params="prefix parent prefix_topic *origin min_angle:=3.14159 max_angle:=-3.14159">
     <joint name="${prefix}_laser_base_joint" type="fixed">
       <xacro:insert_block name="origin" />
@@ -62,5 +62,5 @@
 				</ray>
 				<plugin name="gazebo_ros_rplidar_controller" filename="libgazebo_ros_laser.so">
-					<topicName>${prefix_scan}/scan</topicName>
+					<topicName>${prefix_topic}/scan</topicName>
 					<frameName>${prefix}_laser_link</frameName>
 					<ignoreTfPrefix>1</ignoreTfPrefix>

File: urdf/rplidar_a2.urdf.xacro (robot description, xacro)
@@ -1,5 +1,5 @@
 <?xml version="1.0"?>
 <robot xmlns:xacro="http://www.ros.org/wiki/xacro">
-  <xacro:macro name="sensor_rplidar_a2" params="prefix parent prefix_scan *origin min_angle:=-3.14159 max_angle:=3.14159">
+  <xacro:macro name="sensor_rplidar_a2" params="prefix parent prefix_topic *origin min_angle:=-3.14159 max_angle:=3.14159">
     <joint name="${prefix}_base_joint" type="fixed">
       <xacro:insert_block name="origin" />
@@ -62,5 +62,5 @@
 				</ray>
 				<plugin name="${prefix}gazebo_ros_rplidar_a2_controller" filename="libgazebo_ros_laser.so">
-					<topicName>${prefix_scan}/scan</topicName>
+					<topicName>${prefix_topic}/scan</topicName>
 					<frameName>${prefix}_link</frameName>
 					<ignoreTfPrefix>1</ignoreTfPrefix>

File: urdf/sick_s3000.urdf.xacro (robot description, xacro)
@@ -1,5 +1,5 @@
 <?xml version="1.0"?>
 <robot name="sensor_sick_s3000" xmlns:xacro="http://www.ros.org/wiki/xacro">
-  <xacro:macro name="sensor_sick_s3000" params="prefix parent prefix_scan *origin">
+  <xacro:macro name="sensor_sick_s3000" params="prefix parent prefix_topic *origin">
     <joint name="${prefix}_joint" type="fixed">
       <xacro:insert_block name="origin" />
@@ -56,5 +56,5 @@
 				</ray>
 				<plugin name="${prefix}_controller" filename="libgazebo_ros_laser.so">
-					<topicName>${prefix_scan}/scan</topicName>
+					<topicName>${prefix_topic}/scan</topicName>
 					<frameName>${prefix}_base_link</frameName>
 					<ignoreTfPrefix>1</ignoreTfPrefix>

File: urdf/sick_tim551.urdf.xacro (robot description, xacro)
@@ -1,5 +1,5 @@
 <?xml version="1.0"?>
 <robot xmlns:xacro="http://www.ros.org/wiki/xacro">
-  <xacro:macro name="sensor_sick_tim551" params="prefix parent prefix_scan *origin min_angle:=-2.36 max_angle:=2.36">
+  <xacro:macro name="sensor_sick_tim551" params="prefix parent prefix_topic *origin min_angle:=-2.36 max_angle:=2.36">
     <joint name="${prefix}_base_joint" type="fixed">
       <xacro:insert_block name="origin" />
@@ -62,5 +62,5 @@
 				</ray>
 				<plugin name="${prefix}_controller" filename="libgazebo_ros_laser.so">
-					<topicName>${prefix_scan}/scan</topicName>
+					<topicName>${prefix_topic}/scan</topicName>
 					<frameName>${prefix}_link</frameName> <!-- leading / avoids that current namespace is added as prefix in the frame name (/ns/prefix_link) -->
 					<ignoreTfPrefix>1</ignoreTfPrefix>

File: urdf/sick_tim571.urdf.xacro (robot description, xacro)
@@ -1,5 +1,5 @@
 <?xml version="1.0"?>
 <robot xmlns:xacro="http://www.ros.org/wiki/xacro">
-  <xacro:macro name="sensor_sick_tim571" params="prefix parent prefix_scan *origin min_angle:=-2.36 max_angle:=2.36">
+  <xacro:macro name="sensor_sick_tim571" params="prefix parent prefix_topic *origin min_angle:=-2.36 max_angle:=2.36">
     <joint name="${prefix}_base_joint" type="fixed">
       <xacro:insert_block name="origin" />
@@ -62,5 +62,5 @@
 				</ray>
 				<plugin name="${prefix}_controller" filename="libgazebo_ros_laser.so">
-					<topicName>${prefix_scan}/scan</topicName>
+					<topicName>${prefix_topic}/scan</topicName>
 					<frameName>${prefix}_link</frameName>
 					<ignoreTfPrefix>1</ignoreTfPrefix>

Commit message: setting hokuyos laser_link z to 0.0 from the base_link

File: urdf/hokuyo_urg04lx.urdf.xacro (robot description, xacro)
@@ -29,5 +29,5 @@
       <parent link="${prefix}_base_link"/>
       <child link="${prefix}_link"/>
-      <origin xyz="0.00 0 0.05" rpy="0 0 0"/>
+      <origin xyz="0.00 0 0.00" rpy="0 0 0"/>
 	</joint>
     <!-- Hokuyo sensor for simulation -->

File: urdf/hokuyo_ust10lx.urdf.xacro (robot description, xacro)
@@ -32,5 +32,6 @@
       <parent link="${prefix}_base_link"/>
       <child link="${prefix}_link"/>
-      <origin xyz="0.00 0 0.0474" rpy="0 0 0"/>
+      <origin xyz="0.00 0 0.0" rpy="0 0 0"/>
+      <!--origin xyz="0.00 0 0.0474" rpy="0 0 0"/-->
 	</joint>
     <!-- Hokuyo sensor for simulation -->

File: urdf/hokuyo_ust20lx.urdf.xacro (robot description, xacro)
@@ -32,5 +32,5 @@
       <parent link="${prefix}_base_link"/>
       <child link="${prefix}_link"/>
-      <origin xyz="0.00 0 0.0474" rpy="0 0 0"/>
+      <origin xyz="0.00 0 0.0" rpy="0 0 0"/>
 	</joint>
     <!-- Hokuyo sensor for simulation -->

Commit message: prefix_topic param set to default values

File: urdf/hokuyo_urg04lx.urdf.xacro (robot description, xacro)
@@ -1,5 +1,5 @@
 <?xml version="1.0"?>
 <robot name="sensor_hokuyo_urg04lx" xmlns:xacro="http://www.ros.org/wiki/xacro">
-  <xacro:macro name="sensor_hokuyo_urg04lx" params="prefix parent prefix_topic *origin min_angle:=-2.0943 max_angle:=2.0943">
+  <xacro:macro name="sensor_hokuyo_urg04lx" params="prefix parent prefix_topic:='front_laser' *origin min_angle:=-2.0943 max_angle:=2.0943">
     <joint name="${prefix}_base_joint" type="fixed">
       <!-- FRONT MOUNT  -->

File: urdf/hokuyo_ust10lx.urdf.xacro (robot description, xacro)
@@ -1,5 +1,5 @@
 <?xml version="1.0"?>
 <robot name="sensor_hokuyo_ust10lx" xmlns:xacro="http://www.ros.org/wiki/xacro">
-  <xacro:macro name="sensor_hokuyo_ust10lx" params="prefix parent prefix_topic *origin min_angle:=-2.3562 max_angle:=2.3562">
+  <xacro:macro name="sensor_hokuyo_ust10lx" params="prefix parent prefix_topic:='front_laser' *origin min_angle:=-2.3562 max_angle:=2.3562">
 			<!--arg name="namespace" value="$(arg namespace)"/-->
     <joint name="${prefix}_base_joint" type="fixed">

File: urdf/hokuyo_ust20lx.urdf.xacro (robot description, xacro)
@@ -1,5 +1,5 @@
 <?xml version="1.0"?>
 <robot name="sensor_hokuyo_ust20lx" xmlns:xacro="http://www.ros.org/wiki/xacro">
-  <xacro:macro name="sensor_hokuyo_ust20lx" params="prefix parent prefix_topic *origin min_angle:=-2.3562 max_angle:=2.3562">
+  <xacro:macro name="sensor_hokuyo_ust20lx" params="prefix parent prefix_topic:='front_laser' *origin min_angle:=-2.3562 max_angle:=2.3562">
 			<!--arg name="namespace" value="$(arg namespace)"/-->
     <joint name="${prefix}_base_joint" type="fixed">

File: urdf/hokuyo_utm30lx.urdf.xacro (robot description, xacro)
@@ -1,5 +1,5 @@
 <?xml version="1.0"?>
 <robot name="sensor_hokuyo_utm30lx" xmlns:xacro="http://www.ros.org/wiki/xacro">
-  <xacro:macro name="sensor_hokuyo_utm30lx" params="prefix parent prefix_topic *origin min_angle:=-2.35 max_angle:=2.35">
+  <xacro:macro name="sensor_hokuyo_utm30lx" params="prefix parent prefix_topic:='front_laser *origin min_angle:=-2.35 max_angle:=2.35">
     <joint name="${prefix}_base_joint" type="fixed">
       <!-- FRONT MOUNT  -->

File: urdf/orbbec_astra.urdf.xacro (robot description, xacro)
@@ -13,5 +13,5 @@
   <xacro:property name="orbbec_astra_depth_rel_rgb_pz" value="0.0" />
   <xacro:property name="M_PI" value="3.1415926535897931" />
-  <xacro:macro name="sensor_orbbec_astra" params="prefix parent prefix_topic *origin">
+  <xacro:macro name="sensor_orbbec_astra" params="prefix parent prefix_topic:='front_rgbd_camera' *origin">
     <joint name="${prefix}_rgb_joint" type="fixed">
 	  <xacro:insert_block name="origin" />

File: urdf/rplidar.urdf.xacro (robot description, xacro)
@@ -1,5 +1,5 @@
 <?xml version="1.0"?>
 <robot xmlns:xacro="http://www.ros.org/wiki/xacro">
-  <xacro:macro name="sensor_rplidar" params="prefix parent prefix_topic *origin min_angle:=3.14159 max_angle:=-3.14159">
+  <xacro:macro name="sensor_rplidar" params="prefix parent prefix_topic:='front_laser' *origin min_angle:=3.14159 max_angle:=-3.14159">
     <joint name="${prefix}_laser_base_joint" type="fixed">
       <xacro:insert_block name="origin" />

File: urdf/rplidar_a2.urdf.xacro (robot description, xacro)
@@ -1,5 +1,5 @@
 <?xml version="1.0"?>
 <robot xmlns:xacro="http://www.ros.org/wiki/xacro">
-  <xacro:macro name="sensor_rplidar_a2" params="prefix parent prefix_topic *origin min_angle:=-3.14159 max_angle:=3.14159">
+  <xacro:macro name="sensor_rplidar_a2" params="prefix parent prefix_topic:='front_laser' *origin min_angle:=-3.14159 max_angle:=3.14159">
     <joint name="${prefix}_base_joint" type="fixed">
       <xacro:insert_block name="origin" />

File: urdf/sick_s300.urdf.xacro (robot description, xacro)
@@ -1,5 +1,5 @@
 <?xml version="1.0"?>
 <robot name="sensor_sick_s300" xmlns:xacro="http://www.ros.org/wiki/xacro">
-  <xacro:macro name="sensor_sick_s300" params="prefix parent prefix_scan *origin">
+  <xacro:macro name="sensor_sick_s300" params="prefix parent prefix_topic:='front_laser' *origin">
     <joint name="${prefix}_base_joint" type="fixed">
       <xacro:insert_block name="origin" />
@@ -64,5 +64,5 @@
 				</ray>
 				<plugin name="${prefix}_controller" filename="libgazebo_ros_laser.so">
-					<topicName>${prefix_scan}/scan</topicName>
+					<topicName>${prefix_laser}/scan</topicName>
 					<frameName>${prefix}_link</frameName><!-- if not global (leading /) sets the current namespace as a prefix (/ns/name_laser_link) -->
 					<ignoreTfPrefix>1</ignoreTfPrefix>

File: urdf/sick_s3000.urdf.xacro (robot description, xacro)
@@ -1,5 +1,5 @@
 <?xml version="1.0"?>
 <robot name="sensor_sick_s3000" xmlns:xacro="http://www.ros.org/wiki/xacro">
-  <xacro:macro name="sensor_sick_s3000" params="prefix parent prefix_topic *origin">
+  <xacro:macro name="sensor_sick_s3000" params="prefix parent prefix_topic:='front_laser' *origin">
     <joint name="${prefix}_joint" type="fixed">
       <xacro:insert_block name="origin" />

File: urdf/sick_tim551.urdf.xacro (robot description, xacro)
@@ -1,5 +1,5 @@
 <?xml version="1.0"?>
 <robot xmlns:xacro="http://www.ros.org/wiki/xacro">
-  <xacro:macro name="sensor_sick_tim551" params="prefix parent prefix_topic *origin min_angle:=-2.36 max_angle:=2.36">
+  <xacro:macro name="sensor_sick_tim551" params="prefix parent prefix_topic:='front_laser' *origin min_angle:=-2.36 max_angle:=2.36">
     <joint name="${prefix}_base_joint" type="fixed">
       <xacro:insert_block name="origin" />

File: urdf/sick_tim571.urdf.xacro (robot description, xacro)
@@ -1,5 +1,5 @@
 <?xml version="1.0"?>
 <robot xmlns:xacro="http://www.ros.org/wiki/xacro">
-  <xacro:macro name="sensor_sick_tim571" params="prefix parent prefix_topic *origin min_angle:=-2.36 max_angle:=2.36">
+  <xacro:macro name="sensor_sick_tim571" params="prefix parent prefix_topic:='front_laser' *origin min_angle:=-2.36 max_angle:=2.36">
     <joint name="${prefix}_base_joint" type="fixed">
       <xacro:insert_block name="origin" />

Commit message: Update hokuyo_urg04lx
- Fixes inertia
- Updates gazebo plugin min range
- Sets links correctly based on datasheet

File: urdf/hokuyo_urg04lx.urdf.xacro (robot description, xacro)
@@ -13,5 +13,5 @@
     <link name="${prefix}_base_link">
       <visual>
-        <origin xyz="0 0 -0.05" rpy="0 0 0"/>
+        <origin xyz="0.0 0.0 0.0" rpy="0 0 0"/>
         <geometry>
             <mesh filename="package://robotnik_sensors/meshes/hokuyo_urg_04lx.dae"/>
@@ -19,16 +19,16 @@
       </visual>
       <inertial>
-        <mass value="1e-5" />
-        <origin xyz="0 0 0" rpy="0 0 0"/>
-        <inertia ixx="1e-6" ixy="0" ixz="0" iyy="1e-6" iyz="0" izz="1e-6" />
+        <origin xyz="0.0 0 0.035" rpy="0 0 0" />
+        <mass value="0.160" />
+        <xacro:solid_cuboid_inertia m="0.160" w="0.05" h="0.05" d="0.07" />
       </inertial>
     </link>
     <link name="${prefix}_link">
-	</link>
+  </link>
     <joint name="${prefix}_joint" type="fixed">
       <parent link="${prefix}_base_link"/>
       <child link="${prefix}_link"/>
-      <origin xyz="0.00 0 0.00" rpy="0 0 0"/>
-	</joint>
+      <origin xyz="0.00 0 0.05315" rpy="0 0 0"/>
+  </joint>
     <!-- Hokuyo sensor for simulation -->
     <sensor_hokuyo_urg04lx_gazebo/>
@@ -44,35 +44,35 @@
         <xacro:property name="plugin_lib" value="libgazebo_ros_laser.so" />
       </xacro:unless>
-			<sensor type="${ray_type}" name="${prefix}_sensor">
-				<pose>0 0 0 0 0 0</pose>
-				<visualize>false</visualize>
-				<update_rate>10</update_rate>
-				<ray>
-					<scan>
-						<horizontal>
-							<samples>640</samples>
-							<resolution>1</resolution>
-							<min_angle>${min_angle}</min_angle>
-							<max_angle>${max_angle}</max_angle>
-						</horizontal>
-					</scan>
-					<range>
-						<min>0.02</min>
-						<max>4.0</max>
-						<resolution>0.00628318531</resolution>
-					</range>
-					<noise>
-						<type>gaussian</type>
-						<mean>0.0</mean>
-						<stddev>0.01</stddev>
-					</noise>
-				</ray>
-				<plugin name="${prefix}_controller" filename="${plugin_lib}">
-					<topicName>${prefix_topic}/scan</topicName>
-					<frameName>${prefix}_link</frameName>
-					<ignoreTfPrefix>1</ignoreTfPrefix>
-				</plugin>
-			</sensor>
-	</gazebo>
+      <sensor type="${ray_type}" name="${prefix}_sensor">
+        <pose>0 0 0 0 0 0</pose>
+        <visualize>false</visualize>
+        <update_rate>10</update_rate>
+        <ray>
+          <scan>
+            <horizontal>
+              <samples>640</samples>
+              <resolution>1</resolution>
+              <min_angle>${min_angle}</min_angle>
+              <max_angle>${max_angle}</max_angle>
+            </horizontal>
+          </scan>
+          <range>
+            <min>0.06</min>
+            <max>4.0</max>
+            <resolution>0.00628318531</resolution>
+          </range>
+          <noise>
+            <type>gaussian</type>
+            <mean>0.0</mean>
+            <stddev>0.01</stddev>
+          </noise>
+        </ray>
+        <plugin name="${prefix}_controller" filename="${plugin_lib}">
+          <topicName>${prefix_topic}/scan</topicName>
+          <frameName>${prefix}_link</frameName>
+          <ignoreTfPrefix>1</ignoreTfPrefix>
+        </plugin>
+      </sensor>
+  </gazebo>
   </xacro:macro>
 </robot>
