Commit message: changed collision box of ust10

File: urdf/hokuyo_ust10lx.urdf.xacro (robot description, xacro)
@@ -1,5 +1,5 @@
 <?xml version="1.0"?>
 <robot name="sensor_hokuyo_ust10lx" xmlns:xacro="http://ros.org/wiki/xacro">
-  <xacro:macro name="sensor_hokuyo_ust10lx" params="name parent *origin min_angle:=2.35 max_angle:=-2.35">
+  <xacro:macro name="sensor_hokuyo_ust10lx" params="name parent *origin min_angle:=2.3562 max_angle:=-2.3562">
     <joint name="${name}_laser_joint" type="fixed">
       <insert_block name="origin" />
@@ -11,5 +11,5 @@
         <origin xyz="0 0 -0.05" rpy="0 0 0"/>
         <geometry>
-          <box size="0.1 0.1 0.08"/>
+          <box size="0.010 0.010 0.010"/>
         </geometry>
       </collision>
@@ -45,7 +45,9 @@
 					</scan>
 					<range>
-						<min>0.02</min>
+						<min>0.06</min>
 						<max>20.0</max>
-						<resolution>0.004363323</resolution>
+						<!-- resolution>0.004363323</resolution -->
+						<resolution>0.004359297</resolution>
+						<!-- resolution>0.001</resolution -->
 					</range>
 					<noise>

Commit message: adding prefix_frame and prefix_topic

File: urdf/hokuyo_ust10lx.urdf.xacro (robot description, xacro)
@@ -1,11 +1,12 @@
 <?xml version="1.0"?>
 <robot name="sensor_hokuyo_ust10lx" xmlns:xacro="http://www.ros.org/wiki/xacro">
-  <xacro:macro name="sensor_hokuyo_ust10lx" params="name parent *origin min_angle:=-2.3562 max_angle:=2.3562">
-    <joint name="${name}_joint" type="fixed">
+  <xacro:macro name="sensor_hokuyo_ust10lx" params="prefix_frame prefix_topic parent *origin min_angle:=-2.3562 max_angle:=2.3562">
+			<!--arg name="namespace" value="$(arg namespace)"/-->
+    <joint name="${prefix_frame}_joint" type="fixed">
       <xacro:insert_block name="origin" />
       <parent link="${parent}"/>
-      <child link="${name}_link"/>
+      <child link="${prefix_frame}_link"/>
     </joint>
-    <link name="${name}_link">
+    <link name="${prefix_frame}_link">
       <collision>
         <origin xyz="0 0 -0.05" rpy="0 0 0"/>
@@ -30,6 +31,6 @@
   </xacro:macro>
   <xacro:macro name="sensor_hokuyo_ust_gazebo">
-    <gazebo reference="${name}_link">
-			<sensor type="ray" name="${name}_sensor">
+    <gazebo reference="${prefix_frame}_link">
+			<sensor type="ray" name="${prefix_frame}_sensor">
 				<pose>0 0 0 0 0 0</pose>
 				<visualize>false</visualize>
@@ -57,7 +58,7 @@
 					</noise>
 				</ray>
-				<plugin name="${name}_controller" filename="libgazebo_ros_laser.so">
-					<topicName>${name}/scan</topicName>
-					<frameName>${name}_link</frameName>
+				<plugin name="${prefix_frame}_controller" filename="libgazebo_ros_laser.so">
+					<topicName>${prefix_topic}hokuyo_base/scan</topicName>
+					<frameName>${prefix_frame}_link</frameName>
 					<ignoreTfPrefix>1</ignoreTfPrefix>
 				</plugin>

Commit message: hokuyo ust10lx. changing links relation

File: urdf/hokuyo_ust10lx.urdf.xacro (robot description, xacro)
@@ -2,13 +2,19 @@
 <robot name="sensor_hokuyo_ust10lx" xmlns:xacro="http://www.ros.org/wiki/xacro">
   <xacro:macro name="sensor_hokuyo_ust10lx" params="prefix parent prefix_topic *origin min_angle:=-2.3562 max_angle:=2.3562">
-			<!--arg name="namespace" value="$(arg namespace)"/-->
+    <link name="${prefix}_link">
+	</link>
+    <joint name="${prefix}_joint" type="fixed">
+      <parent link="${parent}"/>
+      <child link="${prefix}_link"/>
+      <xacro:insert_block name="origin" />
+	</joint>
     <joint name="${prefix}_base_joint" type="fixed">
-      <xacro:insert_block name="origin" />
-      <parent link="${parent}"/>
+      <origin xyz="0.00 0 -0.05" rpy="0 0 0"/>
+      <parent link="${prefix}_link"/>
       <child link="${prefix}_base_link"/>
     </joint>
     <link name="${prefix}_base_link">
       <collision>
-        <origin xyz="0 0 -0.05" rpy="0 0 0"/>
+        <origin xyz="0 0 0.0" rpy="0 0 0"/>
         <geometry>
           <box size="0.010 0.010 0.010"/>
@@ -16,5 +22,6 @@
       </collision>
       <visual>
-        <origin xyz="0 0 -0.05" rpy="0 0 0"/>
+        <!--origin xyz="0 0 -0.05" rpy="0 0 0"/-->
+        <origin xyz="0 0 0.0" rpy="0 0 0"/>
         <geometry>
             <mesh filename="package://robotnik_sensors/meshes/hokuyo_ust_10lx.dae"/>
@@ -27,12 +34,4 @@
       </inertial>
     </link>
-    <link name="${prefix}_link">
-	</link>
-    <joint name="${prefix}_joint" type="fixed">
-      <parent link="${prefix}_base_link"/>
-      <child link="${prefix}_link"/>
-      <origin xyz="0.00 0 0.0" rpy="0 0 0"/>
-      <!--origin xyz="0.00 0 0.0474" rpy="0 0 0"/-->
-	</joint>
     <!-- Hokuyo sensor for simulation -->
     <xacro:sensor_hokuyo_ust10_gazebo/>

Commit message: Update hokuyo_ust10lx
- Fixes inertias
- Sets links correctly based on datasheet

File: urdf/hokuyo_ust10lx.urdf.xacro (robot description, xacro)
@@ -2,14 +2,7 @@
 <robot name="sensor_hokuyo_ust10lx" xmlns:xacro="http://wiki.ros.org/xacro">
   <xacro:macro name="sensor_hokuyo_ust10lx" params="prefix parent prefix_topic:='front_laser' *origin min_angle:=-2.3562 max_angle:=2.3562 gpu:=^|true">
-    <link name="${prefix}_link">
-	</link>
-    <joint name="${prefix}_joint" type="fixed">
+    <joint name="${prefix}_base_joint" type="fixed">
+      <xacro:insert_block name="origin" />
       <parent link="${parent}"/>
-      <child link="${prefix}_link"/>
-      <xacro:insert_block name="origin" />
-	</joint>
-    <joint name="${prefix}_base_joint" type="fixed">
-      <origin xyz="0.00 0 -0.05" rpy="0 0 0"/>
-      <parent link="${prefix}_link"/>
       <child link="${prefix}_base_link"/>
     </joint>
@@ -28,8 +21,15 @@
       </visual>
       <inertial>
-        <mass value="1e-5" />
-        <origin xyz="0 0 0" rpy="0 0 0"/>
-        <inertia ixx="1e-6" ixy="0" ixz="0" iyy="1e-6" iyz="0" izz="1e-6" />
+        <origin xyz="0.0 0 0.035" rpy="0 0 0" />
+        <mass value="0.130" />
+        <xacro:solid_cuboid_inertia m="0.130" w="0.05" h="0.05" d="0.07" />
       </inertial>
+    </link>
+    <joint name="${prefix}_joint" type="fixed">
+      <origin xyz="0 0 0.0474" rpy="0 0 0"/>
+      <parent link="${prefix}_base_link"/>
+      <child link="${prefix}_link"/>
+    </joint>
+    <link name="${prefix}_link">
     </link>
     <!-- Hokuyo sensor for simulation -->
