Commit message: Update r430 inertia

File: urdf/intel_r430.urdf.xacro (robot description, xacro)
@@ -45,8 +45,7 @@
       </collision>
       <inertial>
-        <!-- The following are not reliable values, and should not be used for modeling -->
-        <mass value="0.564" />
-        <origin xyz="0 0 0" />
-        <inertia ixx="0.003881243" ixy="0.0" ixz="0.0" iyy="0.000498940" iyz="0.0" izz="0.003879257" />
+        <origin xyz="-0.0125 0.0 0.0" rpy="0 0 0" />
+        <mass value="0.1" />
+        <xacro:solid_cuboid_inertia m="0.1" w="0.025" h="0.09" d="0.025" />
       </inertial>
     </link>
