Commit message: corrected mesh file link

File: urdf/kinect.urdf.xacro (robot description, xacro)
@@ -46,5 +46,5 @@
      <origin xyz="0 0 0" rpy="0 0 ${M_PI/2}"/>
       <geometry>
-       <mesh filename="package://robotnik_sensors/meshes/sensors/kinect.dae"/>
+       <mesh filename="package://robotnik_sensors/meshes/kinect.dae"/>
       </geometry>
     </visual>

Commit message: Update kinect inertia

File: urdf/kinect.urdf.xacro (robot description, xacro)
@@ -15,11 +15,4 @@
     </joint>
     <link name="${prefix}_rgb_base_link">
-      <inertial>
-        <mass value="0.001" />
-        <origin xyz="0 0 0" />
-        <inertia ixx="0.0001" ixy="0.0" ixz="0.0"
-                 iyy="0.0001" iyz="0.0"
-                 izz="0.0001" />
-      </inertial>
     </link>
     <joint name="${prefix}_rgb_optical_joint" type="fixed">
@@ -29,11 +22,4 @@
     </joint>
     <link name="${prefix}_rgb_optical_frame">
-      <inertial>
-        <mass value="0.001" />
-        <origin xyz="0 0 0" />
-        <inertia ixx="0.0001" ixy="0.0" ixz="0.0"
-                 iyy="0.0001" iyz="0.0"
-                 izz="0.0001" />
-      </inertial>
     </link>
   <joint name="${prefix}_joint" type="fixed">
@@ -56,9 +42,7 @@
 	  </collision>
     <inertial>
-      <mass value="0.001" />
-      <origin xyz="0 0 0" />
-      <inertia ixx="0.0001" ixy="0.0" ixz="0.0"
-               iyy="0.0001" iyz="0.0"
-               izz="0.0001" />
+      <origin xyz="-0.0 0.0 0.015" rpy="0 0 0" />
+      <mass value="0.2" />
+      <xacro:solid_cuboid_inertia m="0.2" w="0.06" h="0.24" d="0.04" />
     </inertial>
   </link>
@@ -72,11 +56,4 @@
 	</joint>
 	<link name="${prefix}_depth_link">
-    <inertial>
-      <mass value="0.001" />
-      <origin xyz="0 0 0" />
-      <inertia ixx="0.0001" ixy="0.0" ixz="0.0"
-               iyy="0.0001" iyz="0.0"
-               izz="0.0001" />
-    </inertial>
 	</link>
 	<joint name="${prefix}_depth_optical_joint" type="fixed">
@@ -86,11 +63,4 @@
 	</joint>
 	<link name="${prefix}_depth_optical_frame">
-    <inertial>
-      <mass value="0.001" />
-      <origin xyz="0 0 0" />
-      <inertia ixx="0.0001" ixy="0.0" ixz="0.0"
-               iyy="0.0001" iyz="0.0"
-               izz="0.0001" />
-    </inertial>
 	</link>
 		<!-- Kinect sensor for simulation -->
