Commit message: added kinectv2

File: urdf/kinectv2.urdf.xacro (robot description, xacro)
@@ -46,5 +46,5 @@
      <origin xyz="0 0 0" rpy="0 0 ${M_PI/2}"/>
       <geometry>
-       <mesh filename="package://robotnik_sensors/meshes/sensors/kinect.dae"/>
+       <mesh filename="package://robotnik_sensors/meshes/sensors/kinectv2.dae"/>
       </geometry>
     </visual>

Commit message: Make far and pointCloudCutoffMax parameters configurable

File: urdf/kinectv2.urdf.xacro (robot description, xacro)
@@ -8,5 +8,5 @@
     <xacro:property name="cam_op" value="0" />
     <xacro:property name="cam_oy" value="0" />
-  <xacro:macro name="sensor_kinectv2" params="prefix parent base:=true *origin">
+  <xacro:macro name="sensor_kinectv2" params="prefix parent base:=true *origin cloudCutoffMax:=5.0 far:=8.0">
     <joint name="${prefix}_rgb_joint" type="fixed">
       <xacro:insert_block name="origin" />
@@ -115,7 +115,7 @@
     </link>
         <!-- Kinect sensor for simulation -->
-      <sensor_kinectv2_gazebo/>
+      <sensor_kinectv2_gazebo cloudCutoffMax="${cloudCutoffMax}" far="${far}"/>
   </xacro:macro>
-  <xacro:macro name="sensor_kinectv2_gazebo">
+  <xacro:macro name="sensor_kinectv2_gazebo" params="cloudCutoffMax:=5.0 far:=8.0">
     <gazebo reference="${prefix}_link">
       <sensor type="depth" name="${prefix}_sensor">
@@ -131,5 +131,5 @@
           <clip>
             <near>0.05</near>
-            <far>8.0</far>
+            <far>${far}</far>
           </clip>
         </camera>
@@ -151,5 +151,5 @@
           <distortion_t2>0.0</distortion_t2>
           <pointCloudCutoff>0.4</pointCloudCutoff>
-          <pointCloudCutoffMax>5.0</pointCloudCutoffMax>
+          <pointCloudCutoffMax>${cloudCutoffMax}</pointCloudCutoffMax>
         </plugin>
       </sensor>

Commit message: Update kinectv2 inertia

File: urdf/kinectv2.urdf.xacro (robot description, xacro)
@@ -15,11 +15,4 @@
     </joint>
     <link name="${prefix}_rgb_base_link">
-      <inertial>
-        <mass value="0.001" />
-        <origin xyz="0 0 0" />
-        <inertia ixx="0.0001" ixy="0.0" ixz="0.0"
-                 iyy="0.0001" iyz="0.0"
-                 izz="0.0001" />
-      </inertial>
     </link>
     <joint name="${prefix}_rgb_optical_joint" type="fixed">
@@ -29,11 +22,4 @@
     </joint>
     <link name="${prefix}_rgb_optical_frame">
-      <inertial>
-        <mass value="0.001" />
-        <origin xyz="0 0 0" />
-        <inertia ixx="0.0001" ixy="0.0" ixz="0.0"
-                 iyy="0.0001" iyz="0.0"
-                 izz="0.0001" />
-      </inertial>
     </link>
   <joint name="${prefix}_joint" type="fixed">
@@ -76,9 +62,7 @@
     </collision>
     <inertial>
-      <mass value="0.001" />
-      <origin xyz="0 0 0" />
-      <inertia ixx="0.0001" ixy="0.0" ixz="0.0"
-               iyy="0.0001" iyz="0.0"
-               izz="0.0001" />
+      <origin xyz="-0.0 0.0 0.025" rpy="0 0 0" />
+      <mass value="0.2" />
+      <xacro:solid_cuboid_inertia m="0.2" w="0.06" h="0.24" d="0.04" />
     </inertial>
   </link>
@@ -92,11 +76,4 @@
     </joint>
     <link name="${prefix}_depth_link">
-    <inertial>
-      <mass value="0.001" />
-      <origin xyz="0 0 0" />
-      <inertia ixx="0.0001" ixy="0.0" ixz="0.0"
-               iyy="0.0001" iyz="0.0"
-               izz="0.0001" />
-    </inertial>
     </link>
     <joint name="${prefix}_depth_optical_joint" type="fixed">
@@ -106,11 +83,4 @@
     </joint>
     <link name="${prefix}_depth_optical_frame">
-    <inertial>
-      <mass value="0.001" />
-      <origin xyz="0 0 0" />
-      <inertia ixx="0.0001" ixy="0.0" ixz="0.0"
-               iyy="0.0001" iyz="0.0"
-               izz="0.0001" />
-    </inertial>
     </link>
         <!-- Kinect sensor for simulation -->
