Commit message: Update bumblebee2 inertia

File: urdf/pointgrey_bumblebee2.urdf.xacro (robot description, xacro)
@@ -76,19 +76,10 @@
       </collision>
       <inertial>
-        <mass value="0.342" />
-        <inertia
-          ixx="${1/12*0.342*(0.036*0.036 + 0.0474*0.0474)}" ixy="0" ixz="0"
-          iyy="${1/12*0.342*(0.157*0.157 + 0.0474*0.0474)}" iyz="0"
-          izz="${1/12*0.342*(0.157*0.157 + 0.036*0.036)}" />
+        <origin xyz="-0.0 0.0 0.0" rpy="0 0 0" />
+        <mass value="2.0" />
+        <xacro:solid_cuboid_inertia m="2.0" w="0.0474" h="0.157" d="0.036" />
       </inertial>
     </link>
     <link name="${prefix}_optical_frame">
-      <inertial>
-        <mass value="1E-5" />
-        <inertia
-          ixx="1E-10" ixy="0" ixz="0"
-          iyy="1E-10" iyz="0"
-          izz="1E-10" />
-      </inertial>
     </link>
     <joint name="${frame}_optical_joint" type="fixed">
