Commit message: robotnik_sensors: removed collision model of the utm30lx sensor (it was colliding with itself)

File: urdf/hokuyo_utm30lx.urdf.xacro (robot description, xacro)
@@ -12,10 +12,4 @@
 	</joint>
 	<link name="${name}_laser_link">
-		<collision>
-			<origin xyz="0 0 0" rpy="0 0 0"/>
-			<geometry>
-				<box size="0.1 0.1 0.08"/>
-			</geometry>
-		</collision>
 		<visual>
 			<origin xyz="0 0 0" rpy="0 0 0"/>

Commit message: Missing apostrophe after front_laser added.

File: urdf/hokuyo_utm30lx.urdf.xacro (robot description, xacro)
@@ -1,5 +1,5 @@
 <?xml version="1.0"?>
 <robot name="sensor_hokuyo_utm30lx" xmlns:xacro="http://www.ros.org/wiki/xacro">
-  <xacro:macro name="sensor_hokuyo_utm30lx" params="prefix parent prefix_topic:='front_laser *origin min_angle:=-2.35 max_angle:=2.35">
+  <xacro:macro name="sensor_hokuyo_utm30lx" params="prefix parent prefix_topic:='front_laser' *origin min_angle:=-2.35 max_angle:=2.35">
     <joint name="${prefix}_base_joint" type="fixed">
       <!-- FRONT MOUNT  -->

Commit message: Update hokuyo_utm30lx inertia

File: urdf/hokuyo_utm30lx.urdf.xacro (robot description, xacro)
@@ -13,5 +13,5 @@
     <link name="${prefix}_base_link">
       <visual>
-        <origin xyz="0 0 0" rpy="0 0 0"/>
+        <origin xyz="0 0 0.055" rpy="0 0 0"/>
         <geometry>
             <mesh filename="package://robotnik_sensors/meshes/hokuyo_utm_30lx.dae"/>
@@ -19,7 +19,7 @@
       </visual>
       <inertial>
-        <mass value="1e-5" />
-        <origin xyz="0 0 0" rpy="0 0 0"/>
-        <inertia ixx="1e-6" ixy="0" ixz="0" iyy="1e-6" iyz="0" izz="1e-6" />
+        <origin xyz="0.0 0 0.0435" rpy="0 0 0" />
+        <mass value="0.370" />
+        <xacro:solid_cuboid_inertia m="0.370" w="0.06" h="0.06" d="0.087" />
       </inertial>
     </link>

Commit message: Update the utm30lx's visual position

File: urdf/hokuyo_utm30lx.urdf.xacro (robot description, xacro)
@@ -13,5 +13,5 @@
     <link name="${prefix}_base_link">
       <visual>
-        <origin xyz="0 0 0" rpy="0 0 0"/>
+        <origin xyz="0 0 0.055" rpy="0 0 0"/>
         <geometry>
             <mesh filename="package://robotnik_sensors/meshes/hokuyo_utm_30lx.dae"/>
