Commit message: corrected embedded s near clip and plugin frame

File: urdf/embedded_s.urdf.xacro (robot description, xacro)
@@ -14,4 +14,7 @@
           <!--box size="0.0148 0.0686 0.02235"/-->
         </geometry>
+        <material name="dark_grey">
+          <color rgba="0.4 0.4 0.4 1.0"/>
+        </material>
       </visual>
       <collision>
@@ -59,5 +62,5 @@
   </xacro:macro>
    <xacro:macro name="sensor_astra_embedded_s_gazebo">
-    <gazebo reference="${prefix}_rgb_optical_frame">
+    <gazebo reference="${prefix}_link">
       <sensor type="depth" name="${prefix}_depth_sensor">
         <always_on>true</always_on>
@@ -71,5 +74,5 @@
           </image>
           <clip>
-            <near>0.05</near>
+            <near>0.1</near>
             <far>3.5</far>
           </clip>
