Commit message: flir_ptu_5: Fix inertias

File: urdf/flir_ptu_5.urdf.xacro (robot description, xacro)
@@ -13,5 +13,5 @@
                 <mass value="0.05" />
                 <origin xyz="0 0 0" />
-                <inertia  ixx="1.0" ixy="0.0"  ixz="0.0"  iyy="1.0"  iyz="0.0"  izz="1.0" />
+                <inertia  ixx="0.001043333" ixy="0.0"  ixz="0.0"  iyy="0.001052083"  iyz="0.0"  izz="0.000177083" />
             </inertial>
             <visual>
@@ -38,6 +38,6 @@
         <!-- BODY -->
         <joint name="${prefix}_pan_joint" type="revolute">
-            <limit lower="-2.93197861" upper="2.93215" effort="1.0" velocity="1.4"/>
-            <axis xyz="0 -1 0"/>
+            <limit lower="-2.93197861" upper="2.93215" effort="10.0" velocity="1.4"/>
+            <axis xyz="0 0 -1"/>
             <origin xyz="0 0 0.0232" rpy="0.0 0.0 0.0" />
             <parent link="${prefix}_base_link"/>
@@ -47,8 +47,8 @@
             <type>transmission_interface/SimpleTransmission</type>
             <joint name="${prefix}_pan_joint">
-                <hardwareInterface>hardware_interface/PositionJointInterface</hardwareInterface>
+                <hardwareInterface>hardware_interface/VelocityJointInterface</hardwareInterface>
             </joint>
             <actuator name="${prefix}_pan_motor">
-                <hardwareInterface>hardware_interface/PositionJointInterface</hardwareInterface>
+                <hardwareInterface>hardware_interface/VelocityJointInterface</hardwareInterface>
                 <mechanicalReduction>1.0</mechanicalReduction>
             </actuator>
@@ -58,5 +58,5 @@
                 <mass value="0.25" />
                 <origin xyz="0 0 0" />
-                <inertia  ixx="1.0" ixy="0.0"  ixz="0.0"  iyy="1.0"  iyz="0.0"  izz="1.0" />
+                <inertia  ixx="0.000677083" ixy="0.0"  ixz="0.0"  iyy="0.000570833"  iyz="0.0"  izz="0.000310417" />
             </inertial>
             <visual>
@@ -82,5 +82,5 @@
         <!-- STAND -->
         <joint name="${prefix}_tilt_joint" type="revolute">
-            <limit lower="-1.5706218" upper="0.523599" effort="1.0" velocity="1.2"/>
+            <limit lower="-1.5706218" upper="0.523599" effort="10.0" velocity="1.2"/>
             <axis xyz="0 -1 0"/>
             <origin xyz="0.005 0 0.0753" rpy="0.0 0.0 0.0" />
@@ -91,8 +91,8 @@
             <type>transmission_interface/SimpleTransmission</type>
             <joint name="${prefix}_tilt_joint">
-                <hardwareInterface>hardware_interface/PositionJointInterface</hardwareInterface>
+                <hardwareInterface>hardware_interface/VelocityJointInterface</hardwareInterface>
             </joint>
             <actuator name="${prefix}_tilt_motor">
-                <hardwareInterface>hardware_interface/PositionJointInterface</hardwareInterface>
+                <hardwareInterface>hardware_interface/VelocityJointInterface</hardwareInterface>
                 <mechanicalReduction>1.0</mechanicalReduction>
             </actuator>
@@ -102,5 +102,5 @@
                 <mass value="0.05" />
                 <origin xyz="0 0 0" />
-                <inertia  ixx="1.0" ixy="0.0"  ixz="0.0"  iyy="1.0"  iyz="0.0"  izz="1.0" />
+                <inertia  ixx="0.001043333" ixy="0.0"  ixz="0.0"  iyy="0.001052083"  iyz="0.0"  izz="0.000177083" />
             </inertial>
             <visual>

Commit message: flir_ptu_5: Update urdf

File: urdf/flir_ptu_5.urdf.xacro (robot description, xacro)
@@ -40,5 +40,5 @@
             <limit lower="-2.93197861" upper="2.93215" effort="10.0" velocity="1.4"/>
             <axis xyz="0 0 -1"/>
-            <origin xyz="0 0 0.0232" rpy="0.0 0.0 0.0" />
+            <origin xyz="0 0 0.0251" rpy="0.0 0.0 0.0" />
             <parent link="${prefix}_base_link"/>
             <child link="${prefix}_body_link" />
@@ -84,5 +84,5 @@
             <limit lower="-1.5706218" upper="0.523599" effort="10.0" velocity="1.2"/>
             <axis xyz="0 -1 0"/>
-            <origin xyz="0.005 0 0.0753" rpy="0.0 0.0 0.0" />
+            <origin xyz="0.00725 0 0.0725" rpy="0.0 0.0 0.0" />
             <parent link="${prefix}_body_link"/>
             <child link="${prefix}_stand_link" />
@@ -105,5 +105,5 @@
             </inertial>
             <visual>
-                <origin xyz="0.0 -0.0625 0.0" rpy="0 0 ${M_PI}" />
+                <origin xyz="0.0 -0.0555 0.0" rpy="0 0 ${M_PI}" />
                 <geometry>
                     <mesh filename="package://robotnik_sensors/meshes/flir_ptu_5_stand.stl" scale="1 1 1"/>
@@ -114,5 +114,5 @@
             </visual>
             <collision>
-                <origin xyz="0.0 -0.0625 0" rpy="0 0 ${M_PI}" />
+                <origin xyz="0.0 -0.0555 0" rpy="0 0 ${M_PI}" />
                 <geometry>
                     <mesh filename="package://robotnik_sensors/meshes/flir_ptu_5_stand.stl" scale="1 1 1"/>
@@ -120,5 +120,5 @@
             </collision>
             <visual>
-                <origin xyz="0.0 0.0625 0.0" rpy="0 0 0" />
+                <origin xyz="0.0 0.0555 0.0" rpy="0 0 0" />
                 <geometry>
                     <mesh filename="package://robotnik_sensors/meshes/flir_ptu_5_stand.stl" scale="1 1 1"/>
@@ -129,5 +129,5 @@
             </visual>
             <collision>
-                <origin xyz="0.0 0.0625 0" rpy="0 0 0" />
+                <origin xyz="0.0 0.0555 0" rpy="0 0 0" />
                 <geometry>
                     <mesh filename="package://robotnik_sensors/meshes/flir_ptu_5_stand.stl" scale="1 1 1"/>
