Commit message: added gpu plugin to benewake (needs velodyne plugin)

File: urdf/benewake_ce30.urdf.xacro (robot description, xacro)
@@ -8,5 +8,5 @@
   <xacro:property name="ce30d_depth_py" value="-0.0115"/>
   <xacro:property name="ce30d_depth_pz" value="0.0"/>
-  <xacro:macro name="sensor_benewake_ce30" params="prefix parent *origin range_min range_max hfov vfov fps">
+  <xacro:macro name="sensor_benewake_ce30" params="prefix parent *origin range_min range_max hfov vfov fps gpu">
     <material name="black_alu">
       <color rgba="0.9 0.9 0.9 1"/>
@@ -47,10 +47,18 @@
     </joint>
     <link name="${prefix}_link"/>
-  <!-- Ray sensor for simulation, same as Hokuyo3d -->
-  <sensor_benewake_ce30_gazebo range_min="${range_min}" range_max="${range_max}" hfov="${hfov}" vfov="${vfov}" fps="${fps}"/>
+  <sensor_benewake_ce30_gazebo range_min="${range_min}" range_max="${range_max}" hfov="${hfov}" vfov="${vfov}" fps="${fps}" gpu="${gpu}"/>
   </xacro:macro>
-  <xacro:macro name="sensor_benewake_ce30_gazebo" params="range_min range_max hfov vfov fps">
+  <xacro:macro name="sensor_benewake_ce30_gazebo" params="range_min range_max hfov vfov fps gpu">
     <gazebo reference="${prefix}_link">
-      <sensor type="ray" name="${prefix}_sensor">
+      <xacro:if value="${gpu}">
+        <!-- Using GPU needs: https://github.com/RobotnikAutomation/velodyne_simulator -->
+        <xacro:property name="ray_type" value="gpu_ray" />
+        <xacro:property name="plugin_lib" value="libgazebo_ros_velodyne_gpu_laser.so" />
+      </xacro:if>
+      <xacro:unless value="${gpu}">
+        <xacro:property name="ray_type" value="ray" />
+        <xacro:property name="plugin_lib" value="libgazebo_ros_block_laser.so" />
+      </xacro:unless>
+        <sensor type="${ray_type}" name="${prefix}_sensor">
           <pose>0 0 0 0 0 0.0</pose>
           <visualize>false</visualize>
@@ -76,10 +84,8 @@
             </range>
             <noise>
-              <type>gaussian</type>
-              <mean>0.1</mean>
-              <stddev>0.1</stddev>
+              <type>none</type>
             </noise>
           </ray>
-          <plugin name="gazebo_ros_laser_controller" filename="libgazebo_ros_block_laser.so">
+          <plugin name="gazebo_ros_laser_controller" filename="${plugin_lib}">
             <topicName>${prefix}/points</topicName>
             <frameName>${prefix}_link</frameName>
@@ -89,16 +95,16 @@
     </gazebo>
   </xacro:macro>
-  <xacro:macro name="sensor_benewake_ce30a" params="prefix parent *origin">
-    <sensor_benewake_ce30 prefix="${prefix}" parent="${parent}" range_min="0.1" range_max="4.0" hfov="132.0" vfov="9.0" fps="20.0" >
+  <xacro:macro name="sensor_benewake_ce30a" params="prefix parent *origin gpu:=false">
+    <sensor_benewake_ce30 prefix="${prefix}" parent="${parent}" range_min="0.1" range_max="4.0" hfov="132.0" vfov="9.0" fps="20.0" gpu="${gpu}" >
       <xacro:insert_block name="origin" />
     </sensor_benewake_ce30>
   </xacro:macro>
-  <xacro:macro name="sensor_benewake_ce30c" params="prefix parent *origin">
-    <sensor_benewake_ce30 prefix="${prefix}" parent="${parent}" range_min="0.1" range_max="4.0" hfov="132.0" vfov="9.0" fps="20.0" >
+  <xacro:macro name="sensor_benewake_ce30c" params="prefix parent *origin gpu:=false">
+    <sensor_benewake_ce30 prefix="${prefix}" parent="${parent}" range_min="0.1" range_max="4.0" hfov="132.0" vfov="9.0" fps="20.0" gpu="${gpu}" >
       <xacro:insert_block name="origin" />
     </sensor_benewake_ce30>
   </xacro:macro>
-  <xacro:macro name="sensor_benewake_ce30d" params="prefix parent *origin">
-    <sensor_benewake_ce30 prefix="${prefix}" parent="${parent}" range_min="0.4" range_max="28.0" hfov="60.0" vfov="20.0" fps="30.0" >
+  <xacro:macro name="sensor_benewake_ce30d" params="prefix parent *origin gpu:=false">
+    <sensor_benewake_ce30 prefix="${prefix}" parent="${parent}" range_min="0.4" range_max="28.0" hfov="60.0" vfov="20.0" fps="30.0" gpu="${gpu}" >
       <xacro:insert_block name="origin" />
     </sensor_benewake_ce30>

Commit message: switched laser sensors to use gpu
improves realtime simulation

File: urdf/benewake_ce30.urdf.xacro (robot description, xacro)
@@ -87,5 +87,5 @@
             </noise>
           </ray>
-          <plugin name="gazebo_ros_laser_controller" filename="${plugin_lib}">
+          <plugin name="${prefix}_controller" filename="${plugin_lib}">
             <topicName>${prefix}/points</topicName>
             <frameName>${prefix}_link</frameName>

File: urdf/hokuyo3d.urdf.xacro (robot description, xacro)
@@ -1,78 +1,87 @@
 <?xml version="1.0"?>
 <robot name="sensor_hokuyo3d" xmlns:xacro="http://www.ros.org/wiki/xacro">
-  <xacro:macro name="sensor_hokuyo3d" params="prefix parent *origin">
+  <xacro:macro name="sensor_hokuyo3d" params="prefix parent *origin gpu:=false">
     <joint name="${prefix}_fix_joint" type="fixed">
       <xacro:insert_block name="origin" />
       <parent link="${parent}"/>
       <child link="${prefix}_base_link"/>
-	</joint>
-	<link name="${prefix}_base_link">
-		<collision>
-			<origin xyz="0 0 0" rpy="0 0 0"/>
-			<geometry>
-				<box size="0.05 0.05 0.08"/>
-			</geometry>
-		</collision>
-		<visual>
-			<origin xyz="0 0 0" rpy="0 0 0"/>
-			<geometry>
-	     		<mesh filename="package://robotnik_sensors/meshes/hokuyo3d.stl"/>
-			</geometry>
-		</visual>
-		<inertial>
-			<mass value="1e-5" />
-			<origin xyz="0 0 0" rpy="0 0 0"/>
-			<inertia ixx="1e-6" ixy="0" ixz="0" iyy="1e-6" iyz="0" izz="1e-6" />
-		</inertial>
-	</link>
-	<link name="${prefix}_link">
-	</link>
+    </joint>
+    <link name="${prefix}_base_link">
+        <collision>
+            <origin xyz="0 0 0" rpy="0 0 0"/>
+            <geometry>
+                <box size="0.05 0.05 0.08"/>
+            </geometry>
+        </collision>
+        <visual>
+            <origin xyz="0 0 0" rpy="0 0 0"/>
+            <geometry>
+                <mesh filename="package://robotnik_sensors/meshes/hokuyo3d.stl"/>
+            </geometry>
+        </visual>
+        <inertial>
+            <mass value="1e-5" />
+            <origin xyz="0 0 0" rpy="0 0 0"/>
+            <inertia ixx="1e-6" ixy="0" ixz="0" iyy="1e-6" iyz="0" izz="1e-6" />
+        </inertial>
+    </link>
+    <link name="${prefix}_link">
+    </link>
     <joint name="${prefix}_joint" type="fixed">
       <parent link="${prefix}_base_link"/>
       <child link="${prefix}_link"/>
       <origin xyz="0.08 0 0.08" rpy="0 0 0"/>
-	</joint>
-	<!-- Hokuyo sensor for simulation -->
-	<sensor_hokuyo3d_gazebo/>
+    </joint>
+    <!-- Hokuyo sensor for simulation -->
+    <sensor_hokuyo3d_gazebo gpu="${gpu}"/>
   </xacro:macro>
-  <xacro:macro name="sensor_hokuyo3d_gazebo">
+  <xacro:macro name="sensor_hokuyo3d_gazebo" params="gpu">
     <gazebo reference="${prefix}_link">
-			<sensor type="ray" name="${prefix}_sensor">
-				<pose>0 0 0 0 0 0</pose>
-				<visualize>false</visualize>
-				<update_rate>5</update_rate>
-				<ray>
-					<scan>
-                        <horizontal>
-                            <samples>144</samples>
-                            <resolution>1.0</resolution>
-                            <min_angle>-1.83591184</min_angle>
-                            <max_angle>1.83591184</max_angle>
-                        </horizontal>
-                        <vertical>
-                            <samples>74</samples>
-                            <resolution>1.0</resolution>
-                            <min_angle>-0.610865238</min_angle>
-                            <max_angle>0.0872664626</max_angle>
-                        </vertical>
-					</scan>
-					<range>
-						<min>0.10</min>
-						<max>20.0</max>
-						<resolution>0.01</resolution>
-					</range>
-					<noise>
-						<type>gaussian</type>
-						<mean>0.0</mean>
-						<stddev>0.01</stddev>
-					</noise>
-				</ray>
-				<plugin name="${prefix}_controller" filename="libgazebo_ros_block_laser.so">
-					<topicName>points</topicName>
-					<frameName>${prefix}_link</frameName>
-					        <ignoreTfPrefix>1</ignoreTfPrefix>
-				</plugin>
-			</sensor>
-		</gazebo>
+      <xacro:if value="${gpu}">
+        <!-- Using GPU needs: https://github.com/RobotnikAutomation/velodyne_simulator -->
+        <xacro:property name="ray_type" value="gpu_ray" />
+        <xacro:property name="plugin_lib" value="libgazebo_ros_velodyne_gpu_laser.so" />
+      </xacro:if>
+      <xacro:unless value="${gpu}">
+        <xacro:property name="ray_type" value="ray" />
+        <xacro:property name="plugin_lib" value="libgazebo_ros_block_laser.so" />
+      </xacro:unless>
+      <sensor type="${ray_type}" name="${prefix}_sensor">
+          <pose>0 0 0 0 0 0</pose>
+          <visualize>false</visualize>
+          <update_rate>5</update_rate>
+          <ray>
+              <scan>
+                  <horizontal>
+                      <samples>144</samples>
+                      <resolution>1.0</resolution>
+                      <min_angle>-1.83591184</min_angle>
+                      <max_angle>1.83591184</max_angle>
+                  </horizontal>
+                  <vertical>
+                      <samples>74</samples>
+                      <resolution>1.0</resolution>
+                      <min_angle>-0.610865238</min_angle>
+                      <max_angle>0.0872664626</max_angle>
+                  </vertical>
+              </scan>
+              <range>
+                  <min>0.10</min>
+                  <max>20.0</max>
+                  <resolution>0.01</resolution>
+              </range>
+              <noise>
+                  <type>gaussian</type>
+                  <mean>0.0</mean>
+                  <stddev>0.01</stddev>
+              </noise>
+          </ray>
+          <plugin name="${prefix}_controller" filename="${plugin_lib}">
+                    <topicName>points</topicName>
+                    <frameName>${prefix}_link</frameName>
+                            <ignoreTfPrefix>1</ignoreTfPrefix>
+                </plugin>
+            </sensor>
+        </gazebo>
   </xacro:macro>
 </robot>

File: urdf/hokuyo_urg04lx.urdf.xacro (robot description, xacro)
@@ -36,5 +36,5 @@
   <xacro:macro name="sensor_hokuyo_urg04lx_gazebo">
     <gazebo reference="${prefix}_link">
-			<sensor type="ray" name="${prefix}_sensor">
+			<sensor type="gpu_ray" name="${prefix}_sensor">
 				<pose>0 0 0 0 0 0</pose>
 				<visualize>false</visualize>
@@ -60,5 +60,5 @@
 					</noise>
 				</ray>
-				<plugin name="${prefix}_controller" filename="libgazebo_ros_laser.so">
+				<plugin name="${prefix}_controller" filename="libgazebo_ros_gpu_laser.so">
 					<topicName>${prefix_topic}/scan</topicName>
 					<frameName>${prefix}_link</frameName>

File: urdf/hokuyo_ust10lx.urdf.xacro (robot description, xacro)
@@ -38,5 +38,5 @@
   <xacro:macro name="sensor_hokuyo_ust10_gazebo">
     <gazebo reference="${prefix}_link">
-			<sensor type="ray" name="${prefix}_sensor">
+			<sensor type="gpu_ray" name="${prefix}_sensor">
 				<pose>0 0 0 0 0 0</pose>
 				<visualize>false</visualize>
@@ -64,5 +64,5 @@
 					</noise>
 				</ray>
-				<plugin name="${prefix}_controller" filename="libgazebo_ros_laser.so">
+				<plugin name="${prefix}_controller" filename="libgazebo_ros_gpu_laser.so">
 					<topicName>${prefix_topic}/scan</topicName>
 					<frameName>/${prefix}_link</frameName>

File: urdf/hokuyo_ust20lx.urdf.xacro (robot description, xacro)
@@ -39,5 +39,5 @@
   <xacro:macro name="sensor_hokuyo_ust20_gazebo">
     <gazebo reference="${prefix}_link">
-			<sensor type="ray" name="${prefix}_sensor">
+			<sensor type="gpu_ray" name="${prefix}_sensor">
 				<pose>0 0 0 0 0 0</pose>
 				<visualize>false</visualize>
@@ -65,5 +65,5 @@
 					</noise>
 				</ray>
-				<plugin name="${prefix}_controller" filename="libgazebo_ros_laser.so">
+				<plugin name="${prefix}_controller" filename="libgazebo_ros_gpu_laser.so">
 					<topicName>${prefix_topic}/scan</topicName>
 					<frameName>/${prefix}_link</frameName>

File: urdf/hokuyo_utm30lx.urdf.xacro (robot description, xacro)
@@ -36,5 +36,5 @@
   <xacro:macro name="sensor_hokuyo_utm_gazebo">
     <gazebo reference="${prefix}_link">
-			<sensor type="ray" name="${prefix}_sensor">
+			<sensor type="gpu_ray" name="${prefix}_sensor">
 				<pose>0 0 0 0 0 0</pose>
 				<visualize>false</visualize>
@@ -60,5 +60,5 @@
 					</noise>
 				</ray>
-				<plugin name="${prefix}_controller" filename="libgazebo_ros_laser.so">
+				<plugin name="${prefix}_controller" filename="libgazebo_ros_gpu_laser.so">
 					<topicName>${prefix_topic}/scan</topicName>
 					<frameName>/${prefix}_link</frameName>

File: urdf/rplidar.urdf.xacro (robot description, xacro)
@@ -37,5 +37,5 @@
   <xacro:macro name="${prefix}_sensor_rplidar_gazebo">
     <gazebo reference="${prefix}_laser_link">
-			<sensor type="ray" name="${prefix}_rplidar_sensor">
+			<sensor type="gpu_ray" name="${prefix}_rplidar_sensor">
 				<pose>0 0 0 0 0 0</pose>
 				<visualize>false</visualize>
@@ -61,5 +61,5 @@
 					</noise>
 				</ray>
-				<plugin name="gazebo_ros_rplidar_controller" filename="libgazebo_ros_laser.so">
+				<plugin name="${prefix}_controller" filename="libgazebo_ros_gpu_laser.so">
 					<topicName>${prefix_topic}/scan</topicName>
 					<frameName>/${prefix}_laser_link</frameName>

File: urdf/rplidar_a2.urdf.xacro (robot description, xacro)
@@ -37,5 +37,5 @@
   <xacro:macro name="sensor_rplidar_a2_gazebo">
     <gazebo reference="${prefix}_link">
-			<sensor type="ray" name="${prefix}_rplidar_a2_sensor">
+			<sensor type="gpu_ray" name="${prefix}_rplidar_a2_sensor">
 				<pose>0 0 0 0 0 0</pose>
 				<visualize>false</visualize>
@@ -61,5 +61,5 @@
 					</noise>
 				</ray>
-				<plugin name="${prefix}gazebo_ros_rplidar_a2_controller" filename="libgazebo_ros_laser.so">
+				<plugin name="${prefix}_controller" filename="libgazebo_ros_gpu_laser.so">
 					<topicName>${prefix_topic}/scan</topicName>
 					<frameName>/${prefix}_link</frameName>

File: urdf/sick_s300.urdf.xacro (robot description, xacro)
@@ -39,5 +39,5 @@
   <xacro:macro name="sensor_sick_s300_gazebo">
     <gazebo reference="${prefix}_link">
-			<sensor type="ray" name="${prefix}_sensor">
+			<sensor type="gpu_ray" name="${prefix}_sensor">
 				<pose>0 0 0 0 0 0</pose>
 				<visualize>false</visualize>
@@ -63,5 +63,5 @@
 					</noise>
 				</ray>
-				<plugin name="${prefix}_controller" filename="libgazebo_ros_laser.so">
+				<plugin name="${prefix}_controller" filename="libgazebo_ros_gpu_laser.so">
 					<topicName>${prefix_topic}/scan</topicName>
 					<frameName>/${prefix}_link</frameName><!-- if not global (leading /) sets the current namespace as a prefix (/ns/name_laser_link) -->

File: urdf/sick_s3000.urdf.xacro (robot description, xacro)
@@ -31,5 +31,5 @@
   <xacro:macro name="sensor_sick_s3000_gazebo">
     <gazebo reference="${prefix}_base_link">
-			<sensor type="ray" name="${prefix}_sensor">
+			<sensor type="gpu_ray" name="${prefix}_sensor">
 				<pose>0 0 0 0 0 0</pose>
 				<visualize>false</visualize>
@@ -55,5 +55,5 @@
 					</noise>
 				</ray>
-				<plugin name="${prefix}_controller" filename="libgazebo_ros_laser.so">
+				<plugin name="${prefix}_controller" filename="libgazebo_ros_gpu_laser.so">
 					<topicName>${ns}${prefix_topic}/scan</topicName>
 					<frameName>/${prefix}_base_link</frameName>

File: urdf/sick_tim551.urdf.xacro (robot description, xacro)
@@ -37,5 +37,5 @@
   <xacro:macro name="sensor_sick_tim551_gazebo">
     <gazebo reference="${prefix}_link">
-			<sensor type="ray" name="${prefix}_sensor">
+			<sensor type="gpu_ray" name="${prefix}_sensor">
 				<pose>0 0 0 0 0 0</pose>
 				<visualize>false</visualize>
@@ -61,5 +61,5 @@
 					</noise>
 				</ray>
-				<plugin name="${prefix}_controller" filename="libgazebo_ros_laser.so">
+				<plugin name="${prefix}_controller" filename="libgazebo_ros_gpu_laser.so">
 					<topicName>${prefix_topic}/scan</topicName>
 					<frameName>/${prefix}_link</frameName> <!-- leading / avoids that current namespace is added as prefix in the frame name (/ns/prefix_link) -->

File: urdf/sick_tim571.urdf.xacro (robot description, xacro)
@@ -37,5 +37,5 @@
   <xacro:macro name="sensor_sick_tim571_gazebo">
 	<gazebo reference="${prefix}_link">
-			<sensor type="ray" name="${prefix}_sensor">
+			<sensor type="gpu_ray" name="${prefix}_sensor">
 				<pose>0 0 0 0 0 0</pose>
 				<visualize>false</visualize>
@@ -61,5 +61,5 @@
 					</noise>
 				</ray>
-				<plugin name="${prefix}_controller" filename="libgazebo_ros_laser.so">
+				<plugin name="${prefix}_controller" filename="libgazebo_ros_gpu_laser.so">
 					<topicName>${prefix_topic}/scan</topicName>
 					<frameName>/${prefix}_link</frameName>

File: urdf/velodyne_vlp16.urdf.xacro (robot description, xacro)
@@ -1,78 +1,87 @@
 <?xml version="1.0"?>
 <robot name="sensor_velodyne_vlp16" xmlns:xacro="http://www.ros.org/wiki/xacro">
-  <xacro:macro name="sensor_velodyne_vlp16" params="prefix parent prefix_topic:='velodyne' *origin">
+  <xacro:macro name="sensor_velodyne_vlp16" params="prefix parent prefix_topic:='velodyne' *origin gpu:=false">
     <joint name="${prefix}_base_joint" type="fixed">
       <xacro:insert_block name="origin" />
       <parent link="${parent}"/>
       <child link="${prefix}_base_link"/>
-	</joint>
-	<link name="${prefix}_base_link">
-		<collision>
-			<origin xyz="0 0 0" rpy="0 0 0"/>
-			<geometry>
-	     		<mesh filename="package://robotnik_sensors/meshes/velodyne_vlp16.dae"/>
-			</geometry>
-		</collision>
-		<visual>
-			<origin xyz="0 0 0" rpy="0 0 0"/>
-			<geometry>
-	     		<mesh filename="package://robotnik_sensors/meshes/velodyne_vlp16.dae"/>
-			</geometry>
-		</visual>
-		<inertial>
-			<mass value="1e-5" />
-			<origin xyz="0 0 0" rpy="0 0 0"/>
-			<inertia ixx="1e-6" ixy="0" ixz="0" iyy="1e-6" iyz="0" izz="1e-6" />
-		</inertial>
-	</link>
+    </joint>
+    <link name="${prefix}_base_link">
+        <collision>
+            <origin xyz="0 0 0" rpy="0 0 0"/>
+            <geometry>
+                <mesh filename="package://robotnik_sensors/meshes/velodyne_vlp16.dae"/>
+            </geometry>
+        </collision>
+        <visual>
+            <origin xyz="0 0 0" rpy="0 0 0"/>
+            <geometry>
+                <mesh filename="package://robotnik_sensors/meshes/velodyne_vlp16.dae"/>
+            </geometry>
+        </visual>
+        <inertial>
+            <mass value="1e-5" />
+            <origin xyz="0 0 0" rpy="0 0 0"/>
+            <inertia ixx="1e-6" ixy="0" ixz="0" iyy="1e-6" iyz="0" izz="1e-6" />
+        </inertial>
+    </link>
     <joint name="${prefix}_joint" type="fixed">
       <parent link="${prefix}_base_link"/>
       <child link="${prefix}_link"/>
       <origin xyz="0.0 0 0.035" rpy="0 0 0"/>
-	</joint>
-	<link name="${prefix}_link">
+    </joint>
+    <link name="${prefix}_link">
     </link>
-	<!-- Velodyne sensor for simulation -->
-	<sensor_velodyne_vlp16_gazebo />
+    <!-- Velodyne sensor for simulation -->
+    <sensor_velodyne_vlp16_gazebo gpu="${gpu}" />
   </xacro:macro>
-  <xacro:macro name="sensor_velodyne_vlp16_gazebo">
+  <xacro:macro name="sensor_velodyne_vlp16_gazebo" params="gpu">
     <gazebo reference="${prefix}_link">
-			<sensor type="ray" name="${prefix}_sensor">
-				<pose>0 0 0 0 0 0</pose>
-                <visualize>false</visualize>
-				<update_rate>15</update_rate>
-				<ray>
-					<scan>
-						<horizontal>
-							<samples>300</samples>
-							<resolution>1.0</resolution>
-							<min_angle>-1.83591184</min_angle>
-							<max_angle>1.83591184</max_angle>
-						</horizontal>
-                        <vertical>
-							<samples>100</samples>
-							<resolution>1.0</resolution>
-							<min_angle>-0.610865238</min_angle>
-							<max_angle>1.83591184</max_angle>
-						</vertical>
-					</scan>
-					<range>
-						<min>0.10</min>
-						<max>30.0</max>
-						<resolution>0.01</resolution>
-					</range>
-					<noise>
-						<type>gaussian</type>
-						<mean>0.0</mean>
-						<stddev>0.01</stddev>
-					</noise>
-				</ray>
-				<plugin name="${prefix}_controller" filename="libgazebo_ros_block_laser.so">
-					<topicName>${prefix_topic}/point_cloud</topicName>
-					<frameName>/${prefix}_link</frameName>
-    				<ignoreTfPrefix>1</ignoreTfPrefix>
-				</plugin>
-			</sensor>
-		</gazebo>
+      <xacro:if value="${gpu}">
+        <!-- Using GPU needs: https://github.com/RobotnikAutomation/velodyne_simulator -->
+        <xacro:property name="ray_type" value="gpu_ray" />
+        <xacro:property name="plugin_lib" value="libgazebo_ros_velodyne_gpu_laser.so" />
+      </xacro:if>
+      <xacro:unless value="${gpu}">
+        <xacro:property name="ray_type" value="ray" />
+        <xacro:property name="plugin_lib" value="libgazebo_ros_block_laser.so" />
+      </xacro:unless>
+      <sensor type="${ray_type}" name="${prefix}_sensor">
+          <pose>0 0 0 0 0 0</pose>
+          <visualize>false</visualize>
+          <update_rate>15</update_rate>
+          <ray>
+              <scan>
+                  <horizontal>
+                      <samples>300</samples>
+                      <resolution>1.0</resolution>
+                      <min_angle>-1.83591184</min_angle>
+                      <max_angle>1.83591184</max_angle>
+                  </horizontal>
+                  <vertical>
+                      <samples>100</samples>
+                      <resolution>1.0</resolution>
+                      <min_angle>-0.610865238</min_angle>
+                      <max_angle>1.83591184</max_angle>
+                  </vertical>
+              </scan>
+              <range>
+                  <min>0.10</min>
+                  <max>30.0</max>
+                  <resolution>0.01</resolution>
+              </range>
+              <noise>
+                  <type>gaussian</type>
+                  <mean>0.0</mean>
+                  <stddev>0.01</stddev>
+              </noise>
+          </ray>
+          <plugin name="${prefix}_controller" filename="${plugin_lib}">
+              <topicName>${prefix_topic}/point_cloud</topicName>
+              <frameName>/${prefix}_link</frameName>
+              <ignoreTfPrefix>1</ignoreTfPrefix>
+          </plugin>
+      </sensor>
+    </gazebo>
   </xacro:macro>
 </robot>
