Commit message: Add model param to benewake sensor

File: urdf/benewake_ce30.urdf.xacro (robot description, xacro)
@@ -8,5 +8,5 @@
   <xacro:property name="ce30d_depth_py" value="-0.0115"/>
   <xacro:property name="ce30d_depth_pz" value="0.0"/>
-  <xacro:macro name="sensor_benewake_ce30" params="prefix parent *origin range_min range_max hfov vfov fps gpu">
+  <xacro:macro name="sensor_benewake_ce30" params="model prefix parent *origin range_min range_max hfov vfov fps gpu">
     <material name="black_alu">
       <color rgba="0.9 0.9 0.9 1"/>
@@ -22,14 +22,13 @@
       <origin xyz="0 0 0" rpy="0 0 0"/>
         <geometry>
-          <!-- box size="${ce30d_width} ${ce30d_length} ${ce30d_height}"/ -->
-          <!-- mesh filename="package://robotnik_sensors/meshes/benewake_ce30d.dae" / -->
-          <box size="${ce30d_length} ${ce30d_width} ${ce30d_height}"/>
+          <mesh filename="package://robotnik_sensors/meshes/benewake_ce30${model}.stl" />
+          <!--box size="${ce30d_length} ${ce30d_width} ${ce30d_height}"/-->
         </geometry>
         <material name="black_alu"/>
       </visual>
       <collision>
-        <origin xyz="${-ce30d_length/2} ${-ce30d_width/2} 0.0" rpy="0 0 0"/>
+        <origin xyz="0 0 0" rpy="0 0 0"/>
         <geometry>
-        <box size="${ce30d_length} ${ce30d_width} ${ce30d_height}"/>
+          <mesh filename="package://robotnik_sensors/meshes/benewake_ce30${model}.stl" />
         </geometry>
       </collision>
@@ -96,15 +95,15 @@
   </xacro:macro>
   <xacro:macro name="sensor_benewake_ce30a" params="prefix parent *origin gpu:=false">
-    <sensor_benewake_ce30 prefix="${prefix}" parent="${parent}" range_min="0.1" range_max="4.0" hfov="132.0" vfov="9.0" fps="20.0" gpu="${gpu}" >
+    <sensor_benewake_ce30 model="a" prefix="${prefix}" parent="${parent}" range_min="0.1" range_max="4.0" hfov="132.0" vfov="9.0" fps="20.0" gpu="${gpu}" >
       <xacro:insert_block name="origin" />
     </sensor_benewake_ce30>
   </xacro:macro>
   <xacro:macro name="sensor_benewake_ce30c" params="prefix parent *origin gpu:=false">
-    <sensor_benewake_ce30 prefix="${prefix}" parent="${parent}" range_min="0.1" range_max="4.0" hfov="132.0" vfov="9.0" fps="20.0" gpu="${gpu}" >
+    <sensor_benewake_ce30 model="c" prefix="${prefix}" parent="${parent}" range_min="0.1" range_max="4.0" hfov="132.0" vfov="9.0" fps="20.0" gpu="${gpu}" >
       <xacro:insert_block name="origin" />
     </sensor_benewake_ce30>
   </xacro:macro>
   <xacro:macro name="sensor_benewake_ce30d" params="prefix parent *origin gpu:=false">
-    <sensor_benewake_ce30 prefix="${prefix}" parent="${parent}" range_min="0.4" range_max="28.0" hfov="60.0" vfov="20.0" fps="30.0" gpu="${gpu}" >
+    <sensor_benewake_ce30 model="d" prefix="${prefix}" parent="${parent}" range_min="0.4" range_max="28.0" hfov="60.0" vfov="20.0" fps="30.0" gpu="${gpu}" >
       <xacro:insert_block name="origin" />
     </sensor_benewake_ce30>

Commit message: Correction on benewake origin

File: urdf/benewake_ce30.urdf.xacro (robot description, xacro)
@@ -20,5 +20,5 @@
       <visual>
       <!-- origin xyz="0 0 0" rpy="0 0 1.5708"/ -->
-      <origin xyz="0 0 0" rpy="0 0 0"/>
+      <origin xyz="0.02 0 -0.025" rpy="0 0 0"/>
         <geometry>
           <mesh filename="package://robotnik_sensors/meshes/benewake_ce30${model}.stl" />
@@ -28,5 +28,5 @@
       </visual>
       <collision>
-        <origin xyz="0 0 0" rpy="0 0 0"/>
+        <origin xyz="0.02 0 -0.025" rpy="0 0 0"/>
         <geometry>
           <mesh filename="package://robotnik_sensors/meshes/benewake_ce30${model}.stl" />

Commit message: Correction on benewake origin position

File: urdf/benewake_ce30.urdf.xacro (robot description, xacro)
@@ -20,5 +20,5 @@
       <visual>
       <!-- origin xyz="0 0 0" rpy="0 0 1.5708"/ -->
-      <origin xyz="0.02 0 -0.025" rpy="0 0 0"/>
+      <origin xyz="0 0 0" rpy="0 0 0"/>
         <geometry>
           <mesh filename="package://robotnik_sensors/meshes/benewake_ce30${model}.stl" />
@@ -28,5 +28,5 @@
       </visual>
       <collision>
-        <origin xyz="0.02 0 -0.025" rpy="0 0 0"/>
+        <origin xyz="0 0 0" rpy="0 0 0"/>
         <geometry>
           <mesh filename="package://robotnik_sensors/meshes/benewake_ce30${model}.stl" />

Commit message: removing benewake model until we have actual meshes

File: urdf/benewake_ce30.urdf.xacro (robot description, xacro)
@@ -8,5 +8,5 @@
   <xacro:property name="ce30d_depth_py" value="-0.0115"/>
   <xacro:property name="ce30d_depth_pz" value="0.0"/>
-  <xacro:macro name="sensor_benewake_ce30" params="model prefix parent *origin range_min range_max hfov vfov fps gpu">
+  <xacro:macro name="sensor_benewake_ce30" params="prefix parent *origin range_min range_max hfov vfov fps gpu">
     <material name="black_alu">
       <color rgba="0.9 0.9 0.9 1"/>
@@ -22,5 +22,5 @@
       <origin xyz="0 0 0" rpy="0 0 0"/>
         <geometry>
-          <mesh filename="package://robotnik_sensors/meshes/benewake_ce30${model}.stl" />
+          <mesh filename="package://robotnik_sensors/meshes/benewake_ce30.stl" />
           <!--box size="${ce30d_length} ${ce30d_width} ${ce30d_height}"/-->
         </geometry>
@@ -30,5 +30,5 @@
         <origin xyz="0 0 0" rpy="0 0 0"/>
         <geometry>
-          <mesh filename="package://robotnik_sensors/meshes/benewake_ce30${model}.stl" />
+          <mesh filename="package://robotnik_sensors/meshes/benewake_ce30.stl" />
         </geometry>
       </collision>
@@ -95,15 +95,15 @@
   </xacro:macro>
   <xacro:macro name="sensor_benewake_ce30a" params="prefix parent *origin gpu:=false">
-    <sensor_benewake_ce30 model="a" prefix="${prefix}" parent="${parent}" range_min="0.1" range_max="4.0" hfov="132.0" vfov="9.0" fps="20.0" gpu="${gpu}" >
+    <sensor_benewake_ce30 prefix="${prefix}" parent="${parent}" range_min="0.1" range_max="4.0" hfov="132.0" vfov="9.0" fps="20.0" gpu="${gpu}" >
       <xacro:insert_block name="origin" />
     </sensor_benewake_ce30>
   </xacro:macro>
   <xacro:macro name="sensor_benewake_ce30c" params="prefix parent *origin gpu:=false">
-    <sensor_benewake_ce30 model="c" prefix="${prefix}" parent="${parent}" range_min="0.1" range_max="4.0" hfov="132.0" vfov="9.0" fps="20.0" gpu="${gpu}" >
+    <sensor_benewake_ce30 prefix="${prefix}" parent="${parent}" range_min="0.1" range_max="4.0" hfov="132.0" vfov="9.0" fps="20.0" gpu="${gpu}" >
       <xacro:insert_block name="origin" />
     </sensor_benewake_ce30>
   </xacro:macro>
   <xacro:macro name="sensor_benewake_ce30d" params="prefix parent *origin gpu:=false">
-    <sensor_benewake_ce30 model="d" prefix="${prefix}" parent="${parent}" range_min="0.4" range_max="28.0" hfov="60.0" vfov="20.0" fps="30.0" gpu="${gpu}" >
+    <sensor_benewake_ce30 prefix="${prefix}" parent="${parent}" range_min="0.4" range_max="28.0" hfov="60.0" vfov="20.0" fps="30.0" gpu="${gpu}" >
       <xacro:insert_block name="origin" />
     </sensor_benewake_ce30>

Commit message: added prefix_topic to benewake

File: urdf/benewake_ce30.urdf.xacro (robot description, xacro)
@@ -8,5 +8,5 @@
   <xacro:property name="ce30d_depth_py" value="-0.0115"/>
   <xacro:property name="ce30d_depth_pz" value="0.0"/>
-  <xacro:macro name="sensor_benewake_ce30" params="prefix parent *origin range_min range_max hfov vfov fps gpu">
+  <xacro:macro name="sensor_benewake_ce30" params="prefix parent prefix_topic *origin range_min range_max hfov vfov fps gpu">
     <material name="black_alu">
       <color rgba="0.9 0.9 0.9 1"/>
@@ -78,5 +78,5 @@
             </scan>
             <range>
-              <min>0.4</min>
+              <min>${range_min}</min>
               <max>${range_max}</max>
               <resolution>0.01</resolution>
@@ -87,6 +87,6 @@
           </ray>
           <plugin name="${prefix}_controller" filename="${plugin_lib}">
-            <topicName>${prefix}/points</topicName>
-            <frameName>${prefix}_link</frameName>
+            <topicName>${prefix_topic}/points</topicName>
+            <frameName>/${prefix}_link</frameName>
             <gaussianNoise>0.008</gaussianNoise>
           </plugin>
@@ -94,16 +94,16 @@
     </gazebo>
   </xacro:macro>
-  <xacro:macro name="sensor_benewake_ce30a" params="prefix parent *origin gpu:=false">
-    <sensor_benewake_ce30 prefix="${prefix}" parent="${parent}" range_min="0.1" range_max="4.0" hfov="132.0" vfov="9.0" fps="20.0" gpu="${gpu}" >
+  <xacro:macro name="sensor_benewake_ce30a" params="prefix parent prefix_topic:='lidar_3d' *origin gpu:=false">
+    <sensor_benewake_ce30 prefix="${prefix}" parent="${parent}" prefix_topic="${prefix_topic}" range_min="0.1" range_max="4.0" hfov="132.0" vfov="9.0" fps="20.0" gpu="${gpu}" >
       <xacro:insert_block name="origin" />
     </sensor_benewake_ce30>
   </xacro:macro>
-  <xacro:macro name="sensor_benewake_ce30c" params="prefix parent *origin gpu:=false">
-    <sensor_benewake_ce30 prefix="${prefix}" parent="${parent}" range_min="0.1" range_max="4.0" hfov="132.0" vfov="9.0" fps="20.0" gpu="${gpu}" >
+  <xacro:macro name="sensor_benewake_ce30c" params="prefix parent prefix_topic:='lidar_3d' *origin gpu:=false">
+    <sensor_benewake_ce30 prefix="${prefix}" parent="${parent}" prefix_topic="${prefix_topic}" range_min="0.1" range_max="4.0" hfov="132.0" vfov="9.0" fps="20.0" gpu="${gpu}" >
       <xacro:insert_block name="origin" />
     </sensor_benewake_ce30>
   </xacro:macro>
-  <xacro:macro name="sensor_benewake_ce30d" params="prefix parent *origin gpu:=false">
-    <sensor_benewake_ce30 prefix="${prefix}" parent="${parent}" range_min="0.4" range_max="28.0" hfov="60.0" vfov="20.0" fps="30.0" gpu="${gpu}" >
+  <xacro:macro name="sensor_benewake_ce30d" params="prefix parent prefix_topic:='lidar_3d' *origin gpu:=false">
+    <sensor_benewake_ce30 prefix="${prefix}" parent="${parent}" prefix_topic="${prefix_topic}" range_min="0.4" range_max="28.0" hfov="60.0" vfov="20.0" fps="30.0" gpu="${gpu}" >
       <xacro:insert_block name="origin" />
     </sensor_benewake_ce30>
