Commit message: Add setting the use of GPU for lasers from launch file

File: urdf/benewake_ce30.urdf.xacro (robot description, xacro)
@@ -8,5 +8,5 @@
   <xacro:property name="ce30d_depth_py" value="-0.0115"/>
   <xacro:property name="ce30d_depth_pz" value="0.0"/>
-  <xacro:macro name="sensor_benewake_ce30" params="prefix parent prefix_topic *origin range_min range_max hfov vfov fps gpu">
+  <xacro:macro name="sensor_benewake_ce30" params="prefix parent prefix_topic *origin range_min range_max hfov vfov fps gpu:=^|true">
     <material name="black_alu">
       <color rgba="0.9 0.9 0.9 1"/>

File: urdf/hokuyo3d.urdf.xacro (robot description, xacro)
@@ -1,5 +1,5 @@
 <?xml version="1.0"?>
 <robot name="sensor_hokuyo3d" xmlns:xacro="http://wiki.ros.org/xacro">
-  <xacro:macro name="sensor_hokuyo3d" params="prefix parent *origin gpu:=false">
+  <xacro:macro name="sensor_hokuyo3d" params="prefix parent *origin gpu:=^|true">
     <joint name="${prefix}_fix_joint" type="fixed">
       <xacro:insert_block name="origin" />

File: urdf/hokuyo_urg04lx.urdf.xacro (robot description, xacro)
@@ -1,5 +1,5 @@
 <?xml version="1.0"?>
 <robot name="sensor_hokuyo_urg04lx" xmlns:xacro="http://wiki.ros.org/xacro">
-  <xacro:macro name="sensor_hokuyo_urg04lx" params="prefix parent prefix_topic:='front_laser' *origin min_angle:=-2.0943 max_angle:=2.0943">
+  <xacro:macro name="sensor_hokuyo_urg04lx" params="prefix parent prefix_topic:='front_laser' *origin min_angle:=-2.0943 max_angle:=2.0943  gpu:=^|true">
     <joint name="${prefix}_base_joint" type="fixed">
       <!-- FRONT MOUNT  -->
@@ -36,5 +36,13 @@
   <xacro:macro name="sensor_hokuyo_urg04lx_gazebo">
     <gazebo reference="${prefix}_link">
-			<sensor type="gpu_ray" name="${prefix}_sensor">
+      <xacro:if value="${gpu}">
+        <xacro:property name="ray_type" value="gpu_ray" />
+        <xacro:property name="plugin_lib" value="libgazebo_ros_gpu_laser.so" />
+      </xacro:if>
+      <xacro:unless value="${gpu}">
+        <xacro:property name="ray_type" value="ray" />
+        <xacro:property name="plugin_lib" value="libgazebo_ros_laser.so" />
+      </xacro:unless>
+			<sensor type="${ray_type}" name="${prefix}_sensor">
 				<pose>0 0 0 0 0 0</pose>
 				<visualize>false</visualize>
@@ -60,5 +68,5 @@
 					</noise>
 				</ray>
-				<plugin name="${prefix}_controller" filename="libgazebo_ros_gpu_laser.so">
+				<plugin name="${prefix}_controller" filename="${plugin_lib}">
 					<topicName>${prefix_topic}/scan</topicName>
 					<frameName>${prefix}_link</frameName>

File: urdf/hokuyo_ust10lx.urdf.xacro (robot description, xacro)
@@ -1,5 +1,5 @@
 <?xml version="1.0"?>
 <robot name="sensor_hokuyo_ust10lx" xmlns:xacro="http://wiki.ros.org/xacro">
-  <xacro:macro name="sensor_hokuyo_ust10lx" params="prefix parent prefix_topic:='front_laser' *origin min_angle:=-2.3562 max_angle:=2.3562">
+  <xacro:macro name="sensor_hokuyo_ust10lx" params="prefix parent prefix_topic:='front_laser' *origin min_angle:=-2.3562 max_angle:=2.3562 gpu:=^|true">
     <link name="${prefix}_link">
 	</link>
@@ -38,5 +38,13 @@
   <xacro:macro name="sensor_hokuyo_ust10_gazebo">
     <gazebo reference="${prefix}_link">
-			<sensor type="gpu_ray" name="${prefix}_sensor">
+			<xacro:if value="${gpu}">
+        <xacro:property name="ray_type" value="gpu_ray" />
+        <xacro:property name="plugin_lib" value="libgazebo_ros_gpu_laser.so" />
+      </xacro:if>
+      <xacro:unless value="${gpu}">
+        <xacro:property name="ray_type" value="ray" />
+        <xacro:property name="plugin_lib" value="libgazebo_ros_laser.so" />
+      </xacro:unless>
+			<sensor type="${ray_type}" name="${prefix}_sensor">
 				<pose>0 0 0 0 0 0</pose>
 				<visualize>false</visualize>
@@ -64,5 +72,5 @@
 					</noise>
 				</ray>
-				<plugin name="${prefix}_controller" filename="libgazebo_ros_gpu_laser.so">
+				<plugin name="${prefix}_controller" filename="${plugin_lib}">
 					<topicName>${prefix_topic}/scan</topicName>
 					<frameName>/${prefix}_link</frameName>

File: urdf/hokuyo_ust20lx.urdf.xacro (robot description, xacro)
@@ -1,5 +1,5 @@
 <?xml version="1.0"?>
 <robot name="sensor_hokuyo_ust20lx" xmlns:xacro="http://wiki.ros.org/xacro">
-  <xacro:macro name="sensor_hokuyo_ust20lx" params="prefix parent prefix_topic:='front_laser' *origin min_angle:=-2.3562 max_angle:=2.3562">
+  <xacro:macro name="sensor_hokuyo_ust20lx" params="prefix parent prefix_topic:='front_laser' *origin min_angle:=-2.3562 max_angle:=2.3562 gpu:=^|true">
 			<!--arg name="namespace" value="$(arg namespace)"/-->
     <joint name="${prefix}_base_joint" type="fixed">
@@ -39,5 +39,13 @@
   <xacro:macro name="sensor_hokuyo_ust20_gazebo">
     <gazebo reference="${prefix}_link">
-			<sensor type="gpu_ray" name="${prefix}_sensor">
+			<xacro:if value="${gpu}">
+        <xacro:property name="ray_type" value="gpu_ray" />
+        <xacro:property name="plugin_lib" value="libgazebo_ros_gpu_laser.so" />
+      </xacro:if>
+      <xacro:unless value="${gpu}">
+        <xacro:property name="ray_type" value="ray" />
+        <xacro:property name="plugin_lib" value="libgazebo_ros_laser.so" />
+      </xacro:unless>
+			<sensor type="${ray_type}" name="${prefix}_sensor">
 				<pose>0 0 0 0 0 0</pose>
 				<visualize>false</visualize>
@@ -65,5 +73,5 @@
 					</noise>
 				</ray>
-				<plugin name="${prefix}_controller" filename="libgazebo_ros_gpu_laser.so">
+				<plugin name="${prefix}_controller" filename="${plugin_lib}">
 					<topicName>${prefix_topic}/scan</topicName>
 					<frameName>/${prefix}_link</frameName>

File: urdf/hokuyo_utm30lx.urdf.xacro (robot description, xacro)
@@ -1,5 +1,5 @@
 <?xml version="1.0"?>
 <robot name="sensor_hokuyo_utm30lx" xmlns:xacro="http://wiki.ros.org/xacro">
-  <xacro:macro name="sensor_hokuyo_utm30lx" params="prefix parent prefix_topic:='front_laser' *origin min_angle:=-2.35 max_angle:=2.35">
+  <xacro:macro name="sensor_hokuyo_utm30lx" params="prefix parent prefix_topic:='front_laser' *origin min_angle:=-2.35 max_angle:=2.35 gpu:=^|true">
     <joint name="${prefix}_base_joint" type="fixed">
       <!-- FRONT MOUNT  -->
@@ -36,5 +36,13 @@
   <xacro:macro name="sensor_hokuyo_utm_gazebo">
     <gazebo reference="${prefix}_link">
-			<sensor type="gpu_ray" name="${prefix}_sensor">
+			<xacro:if value="${gpu}">
+        <xacro:property name="ray_type" value="gpu_ray" />
+        <xacro:property name="plugin_lib" value="libgazebo_ros_gpu_laser.so" />
+      </xacro:if>
+      <xacro:unless value="${gpu}">
+        <xacro:property name="ray_type" value="ray" />
+        <xacro:property name="plugin_lib" value="libgazebo_ros_laser.so" />
+      </xacro:unless>
+			<sensor type="${ray_type}" name="${prefix}_sensor">
 				<pose>0 0 0 0 0 0</pose>
 				<visualize>false</visualize>
@@ -60,5 +68,5 @@
 					</noise>
 				</ray>
-				<plugin name="${prefix}_controller" filename="libgazebo_ros_gpu_laser.so">
+				<plugin name="${prefix}_controller" filename="${plugin_lib}">
 					<topicName>${prefix_topic}/scan</topicName>
 					<frameName>/${prefix}_link</frameName>

File: urdf/rplidar.urdf.xacro (robot description, xacro)
@@ -1,5 +1,5 @@
 <?xml version="1.0"?>
 <robot xmlns:xacro="http://wiki.ros.org/xacro">
-  <xacro:macro name="sensor_rplidar" params="prefix parent prefix_topic:='front_laser' *origin min_angle:=3.14159 max_angle:=-3.14159">
+  <xacro:macro name="sensor_rplidar" params="prefix parent prefix_topic:='front_laser' *origin min_angle:=3.14159 max_angle:=-3.14159 gpu:=^|true">
     <joint name="${prefix}_laser_base_joint" type="fixed">
       <xacro:insert_block name="origin" />
@@ -37,5 +37,13 @@
   <xacro:macro name="${prefix}_sensor_rplidar_gazebo">
     <gazebo reference="${prefix}_laser_link">
-			<sensor type="gpu_ray" name="${prefix}_rplidar_sensor">
+			<xacro:if value="${gpu}">
+        <xacro:property name="ray_type" value="gpu_ray" />
+        <xacro:property name="plugin_lib" value="libgazebo_ros_gpu_laser.so" />
+      </xacro:if>
+      <xacro:unless value="${gpu}">
+        <xacro:property name="ray_type" value="ray" />
+        <xacro:property name="plugin_lib" value="libgazebo_ros_laser.so" />
+      </xacro:unless>
+			<sensor type="${ray_type}" name="${prefix}_rplidar_sensor">
 				<pose>0 0 0 0 0 0</pose>
 				<visualize>false</visualize>
@@ -61,5 +69,5 @@
 					</noise>
 				</ray>
-				<plugin name="${prefix}_controller" filename="libgazebo_ros_gpu_laser.so">
+				<plugin name="${prefix}_controller" filename="${plugin_lib}">
 					<topicName>${prefix_topic}/scan</topicName>
 					<frameName>/${prefix}_laser_link</frameName>

File: urdf/rplidar_a2.urdf.xacro (robot description, xacro)
@@ -1,5 +1,5 @@
 <?xml version="1.0"?>
 <robot xmlns:xacro="http://wiki.ros.org/xacro">
-  <xacro:macro name="sensor_rplidar_a2" params="prefix parent prefix_topic:='front_laser' *origin min_angle:=-3.14159 max_angle:=3.14159">
+  <xacro:macro name="sensor_rplidar_a2" params="prefix parent prefix_topic:='front_laser' *origin min_angle:=-3.14159 max_angle:=3.14159 gpu:=^|true">
     <joint name="${prefix}_base_joint" type="fixed">
       <xacro:insert_block name="origin" />
@@ -37,5 +37,13 @@
   <xacro:macro name="sensor_rplidar_a2_gazebo">
     <gazebo reference="${prefix}_link">
-			<sensor type="gpu_ray" name="${prefix}_rplidar_a2_sensor">
+			<xacro:if value="${gpu}">
+        <xacro:property name="ray_type" value="gpu_ray" />
+        <xacro:property name="plugin_lib" value="libgazebo_ros_gpu_laser.so" />
+      </xacro:if>
+      <xacro:unless value="${gpu}">
+        <xacro:property name="ray_type" value="ray" />
+        <xacro:property name="plugin_lib" value="libgazebo_ros_laser.so" />
+      </xacro:unless>
+			<sensor type="${ray_type}" name="${prefix}_rplidar_a2_sensor">
 				<pose>0 0 0 0 0 0</pose>
 				<visualize>false</visualize>
@@ -61,5 +69,5 @@
 					</noise>
 				</ray>
-				<plugin name="${prefix}_controller" filename="libgazebo_ros_gpu_laser.so">
+				<plugin name="${prefix}_controller" filename="${plugin_lib}">
 					<topicName>${prefix_topic}/scan</topicName>
 					<frameName>/${prefix}_link</frameName>

File: urdf/sick_s300.urdf.xacro (robot description, xacro)
@@ -1,5 +1,5 @@
 <?xml version="1.0"?>
 <robot name="sensor_sick_s300" xmlns:xacro="http://wiki.ros.org/xacro">
-  <xacro:macro name="sensor_sick_s300" params="prefix parent prefix_topic:='front_laser' *origin min_angle:=-2.3562 max_angle:=2.3562">
+  <xacro:macro name="sensor_sick_s300" params="prefix parent prefix_topic:='front_laser' *origin min_angle:=-2.3562 max_angle:=2.3562 gpu:=^|true">
     <joint name="${prefix}_base_joint" type="fixed">
       <xacro:insert_block name="origin" />
@@ -39,34 +39,42 @@
   <xacro:macro name="sensor_sick_s300_gazebo">
     <gazebo reference="${prefix}_link">
-			<sensor type="gpu_ray" name="${prefix}_sensor">
-				<pose>0 0 0 0 0 0</pose>
-				<visualize>false</visualize>
-				<update_rate>12.5</update_rate>
-				<ray>
-					<scan>
-						<horizontal>
-							<samples>541</samples>
-							<resolution>1</resolution>
-							<min_angle>${min_angle}</min_angle>
-							<max_angle>${max_angle}</max_angle>
-						</horizontal>
-					</scan>
-					<range>
-						<min>0.10</min>
-						<max>30.0</max>
-						<resolution>0.03</resolution>
-					</range>
-					<noise>
-						<type>gaussian</type>
-						<mean>0.0</mean>
-						<stddev>0.03</stddev>
-					</noise>
-				</ray>
-				<plugin name="${prefix}_controller" filename="libgazebo_ros_gpu_laser.so">
-					<topicName>${prefix_topic}/scan</topicName>
-					<frameName>/${prefix}_link</frameName><!-- if not global (leading /) sets the current namespace as a prefix (/ns/name_laser_link) -->
-				</plugin>
-			</sensor>
-		</gazebo>
+		<xacro:if value="${gpu}">
+			<xacro:property name="ray_type" value="gpu_ray" />
+			<xacro:property name="plugin_lib" value="libgazebo_ros_gpu_laser.so" />
+		</xacro:if>
+		<xacro:unless value="${gpu}">
+			<xacro:property name="ray_type" value="ray" />
+			<xacro:property name="plugin_lib" value="libgazebo_ros_laser.so" />
+		</xacro:unless>
+		<sensor type="${ray_type}" name="${prefix}_sensor">
+			<pose>0 0 0 0 0 0</pose>
+			<visualize>false</visualize>
+			<update_rate>12.5</update_rate>
+			<ray>
+				<scan>
+					<horizontal>
+						<samples>541</samples>
+						<resolution>1</resolution>
+						<min_angle>${min_angle}</min_angle>
+						<max_angle>${max_angle}</max_angle>
+					</horizontal>
+				</scan>
+				<range>
+					<min>0.10</min>
+					<max>30.0</max>
+					<resolution>0.03</resolution>
+				</range>
+				<noise>
+					<type>gaussian</type>
+					<mean>0.0</mean>
+					<stddev>0.03</stddev>
+				</noise>
+			</ray>
+			<plugin name="${prefix}_controller" filename="${plugin_lib}">
+				<topicName>${prefix_topic}/scan</topicName>
+				<frameName>/${prefix}_link</frameName><!-- if not global (leading /) sets the current namespace as a prefix (/ns/name_laser_link) -->
+			</plugin>
+		</sensor>
+	</gazebo>
   </xacro:macro>
 </robot>

File: urdf/sick_s3000.urdf.xacro (robot description, xacro)
@@ -1,5 +1,5 @@
 <?xml version="1.0"?>
 <robot name="sensor_sick_s3000" xmlns:xacro="http://wiki.ros.org/xacro">
-  <xacro:macro name="sensor_sick_s3000" params="prefix parent ns='' prefix_topic:='front_laser' *origin">
+  <xacro:macro name="sensor_sick_s3000" params="prefix parent ns='' prefix_topic:='front_laser' *origin gpu:=^|true">
     <joint name="${prefix}_joint" type="fixed">
       <xacro:insert_block name="origin" />
@@ -31,34 +31,42 @@
   <xacro:macro name="sensor_sick_s3000_gazebo">
     <gazebo reference="${prefix}_base_link">
-			<sensor type="gpu_ray" name="${prefix}_sensor">
-				<pose>0 0 0 0 0 0</pose>
-				<visualize>false</visualize>
-				<update_rate>16.6</update_rate>
-				<ray>
-					<scan>
-						<horizontal>
-							<samples>761</samples>
-							<resolution>1</resolution>
-							<min_angle>-1.6580</min_angle>
-							<max_angle>1.6580</max_angle>
-						</horizontal>
-					</scan>
-					<range>
-						<min>0.10</min>
-						<max>49.0</max>
-						<resolution>0.01</resolution>
-					</range>
-					<noise>
-						<type>gaussian</type>
-						<mean>0.0</mean>
-						<stddev>0.01</stddev>
-					</noise>
-				</ray>
-				<plugin name="${prefix}_controller" filename="libgazebo_ros_gpu_laser.so">
-					<topicName>${ns}${prefix_topic}/scan</topicName>
-					<frameName>/${prefix}_base_link</frameName>
-				</plugin>
-			</sensor>
-		</gazebo>
+		<xacro:if value="${gpu}">
+			<xacro:property name="ray_type" value="gpu_ray" />
+			<xacro:property name="plugin_lib" value="libgazebo_ros_gpu_laser.so" />
+		</xacro:if>
+		<xacro:unless value="${gpu}">
+			<xacro:property name="ray_type" value="ray" />
+			<xacro:property name="plugin_lib" value="libgazebo_ros_laser.so" />
+		</xacro:unless>
+		<sensor type="${ray_type}" name="${prefix}_sensor">
+			<pose>0 0 0 0 0 0</pose>
+			<visualize>false</visualize>
+			<update_rate>16.6</update_rate>
+			<ray>
+				<scan>
+					<horizontal>
+						<samples>761</samples>
+						<resolution>1</resolution>
+						<min_angle>-1.6580</min_angle>
+						<max_angle>1.6580</max_angle>
+					</horizontal>
+				</scan>
+				<range>
+					<min>0.10</min>
+					<max>49.0</max>
+					<resolution>0.01</resolution>
+				</range>
+				<noise>
+					<type>gaussian</type>
+					<mean>0.0</mean>
+					<stddev>0.01</stddev>
+				</noise>
+			</ray>
+			<plugin name="${prefix}_controller" filename="${plugin_lib}">
+				<topicName>${ns}${prefix_topic}/scan</topicName>
+				<frameName>/${prefix}_base_link</frameName>
+			</plugin>
+		</sensor>
+	</gazebo>
   </xacro:macro>
 </robot>

File: urdf/sick_tim551.urdf.xacro (robot description, xacro)
@@ -1,5 +1,5 @@
 <?xml version="1.0"?>
 <robot xmlns:xacro="http://wiki.ros.org/xacro">
-  <xacro:macro name="sensor_sick_tim551" params="prefix parent prefix_topic:='front_laser' *origin min_angle:=-2.36 max_angle:=2.36">
+  <xacro:macro name="sensor_sick_tim551" params="prefix parent prefix_topic:='front_laser' *origin min_angle:=-2.36 max_angle:=2.36 gpu:=^|true">
     <joint name="${prefix}_base_joint" type="fixed">
       <xacro:insert_block name="origin" />
@@ -37,5 +37,13 @@
   <xacro:macro name="sensor_sick_tim551_gazebo">
     <gazebo reference="${prefix}_link">
-			<sensor type="gpu_ray" name="${prefix}_sensor">
+			<xacro:if value="${gpu}">
+        <xacro:property name="ray_type" value="gpu_ray" />
+        <xacro:property name="plugin_lib" value="libgazebo_ros_gpu_laser.so" />
+      </xacro:if>
+      <xacro:unless value="${gpu}">
+        <xacro:property name="ray_type" value="ray" />
+        <xacro:property name="plugin_lib" value="libgazebo_ros_laser.so" />
+      </xacro:unless>
+			<sensor type="${ray_type}" name="${prefix}_sensor">
 				<pose>0 0 0 0 0 0</pose>
 				<visualize>false</visualize>
@@ -61,5 +69,5 @@
 					</noise>
 				</ray>
-				<plugin name="${prefix}_controller" filename="libgazebo_ros_gpu_laser.so">
+				<plugin name="${prefix}_controller" filename="${plugin_lib}">
 					<topicName>${prefix_topic}/scan</topicName>
 					<frameName>/${prefix}_link</frameName> <!-- leading / avoids that current namespace is added as prefix in the frame name (/ns/prefix_link) -->

File: urdf/sick_tim571.urdf.xacro (robot description, xacro)
@@ -1,5 +1,5 @@
 <?xml version="1.0"?>
 <robot xmlns:xacro="http://wiki.ros.org/xacro">
-  <xacro:macro name="sensor_sick_tim571" params="prefix parent prefix_topic:='front_laser' *origin min_angle:=-2.36 max_angle:=2.36">
+  <xacro:macro name="sensor_sick_tim571" params="prefix parent prefix_topic:='front_laser' *origin min_angle:=-2.36 max_angle:=2.36 gpu:=^|true">
     <joint name="${prefix}_base_joint" type="fixed">
       <xacro:insert_block name="origin" />
@@ -36,6 +36,14 @@
   </xacro:macro>
   <xacro:macro name="sensor_sick_tim571_gazebo">
-	<gazebo reference="${prefix}_link">
-			<sensor type="gpu_ray" name="${prefix}_sensor">
+	  <gazebo reference="${prefix}_link">
+			<xacro:if value="${gpu}">
+        <xacro:property name="ray_type" value="gpu_ray" />
+        <xacro:property name="plugin_lib" value="libgazebo_ros_gpu_laser.so" />
+      </xacro:if>
+      <xacro:unless value="${gpu}">
+        <xacro:property name="ray_type" value="ray" />
+        <xacro:property name="plugin_lib" value="libgazebo_ros_laser.so" />
+      </xacro:unless>
+			<sensor type="${ray_type}" name="${prefix}_sensor">
 				<pose>0 0 0 0 0 0</pose>
 				<visualize>false</visualize>
@@ -61,10 +69,10 @@
 					</noise>
 				</ray>
-				<plugin name="${prefix}_controller" filename="libgazebo_ros_gpu_laser.so">
+				<plugin name="${prefix}_controller" filename="${plugin_lib}">
 					<topicName>${prefix_topic}/scan</topicName>
 					<frameName>/${prefix}_link</frameName>
 				</plugin>
 			</sensor>
-	</gazebo>
+	  </gazebo>
   </xacro:macro>
 </robot>

File: urdf/velodyne_vlp16.urdf.xacro (robot description, xacro)
@@ -1,5 +1,5 @@
 <?xml version="1.0"?>
 <robot name="sensor_velodyne_vlp16" xmlns:xacro="http://wiki.ros.org/xacro">
-  <xacro:macro name="sensor_velodyne_vlp16" params="prefix parent prefix_topic:='velodyne' *origin gpu:=false">
+  <xacro:macro name="sensor_velodyne_vlp16" params="prefix parent prefix_topic:='velodyne' *origin gpu:=^|true">
     <joint name="${prefix}_base_joint" type="fixed">
       <xacro:insert_block name="origin" />

Commit message: Fix Benewake_ce30 inertia

File: urdf/benewake_ce30.urdf.xacro (robot description, xacro)
@@ -35,7 +35,7 @@
       <inertial>
         <!-- The following are not reliable values, and should not be used for modeling -->
-        <mass value="0.564" />
-        <origin xyz="0 0 0" />
-        <inertia ixx="0.003881243" ixy="0.0" ixz="0.0" iyy="0.000498940" iyz="0.0" izz="0.003879257" />
+        <mass value="0.219" />
+        <origin xyz="0 0 0.025" />
+        <xacro:solid_cuboid_inertia m="0.219" w="0.047" h="0.079" d="0.05" />
       </inertial>
     </link>
