Commit message: Deleted benewake_ce30d from benewake_ce30 urdf + Deleted unused properties

File: urdf/benewake_ce30.urdf.xacro (robot description, xacro)
@@ -2,10 +2,4 @@
 <robot name="sensor_benewake_ce30" xmlns:xacro="http://wiki.ros.org/xacro">
   <xacro:property name="M_PI" value="3.1415926535897931" />
-  <xacro:property name="ce30d_width" value="0.079"/>
-  <xacro:property name="ce30d_length" value="0.050"/>
-  <xacro:property name="ce30d_height" value="0.047"/>
-  <xacro:property name="ce30d_depth_px" value="0.00"/>
-  <xacro:property name="ce30d_depth_py" value="-0.0115"/>
-  <xacro:property name="ce30d_depth_pz" value="0.0"/>
   <xacro:macro name="sensor_benewake_ce30" params="prefix parent prefix_topic *origin range_min range_max hfov vfov fps gpu:=^|true">
     <material name="black_alu">
@@ -23,5 +17,4 @@
         <geometry>
           <mesh filename="package://robotnik_sensors/meshes/benewake_ce30.stl" />
-          <!--box size="${ce30d_length} ${ce30d_width} ${ce30d_height}"/-->
         </geometry>
         <material name="black_alu"/>
@@ -104,8 +97,3 @@
     </sensor_benewake_ce30>
   </xacro:macro>
-  <xacro:macro name="sensor_benewake_ce30d" params="prefix parent prefix_topic:='lidar_3d' *origin gpu:=false">
-    <sensor_benewake_ce30 prefix="${prefix}" parent="${parent}" prefix_topic="${prefix_topic}" range_min="0.4" range_max="28.0" hfov="60.0" vfov="20.0" fps="30.0" gpu="${gpu}" >
-      <xacro:insert_block name="origin" />
-    </sensor_benewake_ce30>
-  </xacro:macro>
 </robot>

File: urdf/benewake_ce30d.urdf.xacro (robot description, xacro)
@@ -1,12 +1,6 @@
 <?xml version="1.0"?>
-<robot name="sensor_benewake_ce30" xmlns:xacro="http://wiki.ros.org/xacro">
+<robot name="sensor_benewake_ce30d" xmlns:xacro="http://wiki.ros.org/xacro">
   <xacro:property name="M_PI" value="3.1415926535897931" />
-  <xacro:property name="ce30d_width" value="0.079"/>
-  <xacro:property name="ce30d_length" value="0.050"/>
-  <xacro:property name="ce30d_height" value="0.047"/>
-  <xacro:property name="ce30d_depth_px" value="0.00"/>
-  <xacro:property name="ce30d_depth_py" value="-0.0115"/>
-  <xacro:property name="ce30d_depth_pz" value="0.0"/>
-  <xacro:macro name="sensor_benewake_ce30" params="prefix parent prefix_topic *origin range_min range_max hfov vfov fps gpu:=^|true">
+  <xacro:macro name="sensor_benewake_ce30d" params="prefix parent prefix_topic *origin range_min range_max hfov vfov fps gpu:=^|true">
     <material name="black_alu">
       <color rgba="0.9 0.9 0.9 1"/>
@@ -46,7 +40,7 @@
     </joint>
     <link name="${prefix}_link"/>
-  <sensor_benewake_ce30_gazebo range_min="${range_min}" range_max="${range_max}" hfov="${hfov}" vfov="${vfov}" fps="${fps}" gpu="${gpu}"/>
+  <sensor_benewake_ce30d_gazebo range_min="${range_min}" range_max="${range_max}" hfov="${hfov}" vfov="${vfov}" fps="${fps}" gpu="${gpu}"/>
   </xacro:macro>
-  <xacro:macro name="sensor_benewake_ce30_gazebo" params="range_min range_max hfov vfov fps gpu">
+  <xacro:macro name="sensor_benewake_ce30d_gazebo" params="range_min range_max hfov vfov fps gpu">
     <gazebo reference="${prefix}_link">
       <xacro:if value="${gpu}">
@@ -94,18 +88,3 @@
     </gazebo>
   </xacro:macro>
-  <xacro:macro name="sensor_benewake_ce30a" params="prefix parent prefix_topic:='lidar_3d' *origin gpu:=false">
-    <sensor_benewake_ce30 prefix="${prefix}" parent="${parent}" prefix_topic="${prefix_topic}" range_min="0.1" range_max="4.0" hfov="132.0" vfov="9.0" fps="20.0" gpu="${gpu}" >
-      <xacro:insert_block name="origin" />
-    </sensor_benewake_ce30>
-  </xacro:macro>
-  <xacro:macro name="sensor_benewake_ce30c" params="prefix parent prefix_topic:='lidar_3d' *origin gpu:=false">
-    <sensor_benewake_ce30 prefix="${prefix}" parent="${parent}" prefix_topic="${prefix_topic}" range_min="0.1" range_max="4.0" hfov="132.0" vfov="9.0" fps="20.0" gpu="${gpu}" >
-      <xacro:insert_block name="origin" />
-    </sensor_benewake_ce30>
-  </xacro:macro>
-  <xacro:macro name="sensor_benewake_ce30d" params="prefix parent prefix_topic:='lidar_3d' *origin gpu:=false">
-    <sensor_benewake_ce30 prefix="${prefix}" parent="${parent}" prefix_topic="${prefix_topic}" range_min="0.4" range_max="28.0" hfov="60.0" vfov="20.0" fps="30.0" gpu="${gpu}" >
-      <xacro:insert_block name="origin" />
-    </sensor_benewake_ce30>
-  </xacro:macro>
 </robot>

Commit message: 3d laser in use velodyne cpu plugin instead of block

File: urdf/benewake_ce30.urdf.xacro (robot description, xacro)
@@ -57,5 +57,5 @@
       <xacro:unless value="${gpu}">
         <xacro:property name="ray_type" value="ray" />
-        <xacro:property name="plugin_lib" value="libgazebo_ros_block_laser.so" />
+        <xacro:property name="plugin_lib" value="libgazebo_ros_velodyne_laser.so" />
       </xacro:unless>
         <sensor type="${ray_type}" name="${prefix}_sensor">

File: urdf/hokuyo3d.urdf.xacro (robot description, xacro)
@@ -45,5 +45,5 @@
       <xacro:unless value="${gpu}">
         <xacro:property name="ray_type" value="ray" />
-        <xacro:property name="plugin_lib" value="libgazebo_ros_block_laser.so" />
+        <xacro:property name="plugin_lib" value="libgazebo_ros_velodyne_laser.so" />
       </xacro:unless>
       <sensor type="${ray_type}" name="${prefix}_sensor">

File: urdf/ouster1.urdf.xacro (robot description, xacro)
@@ -49,5 +49,5 @@
       <xacro:unless value="${gpu}">
         <xacro:property name="ray_type" value="ray" />
-        <xacro:property name="plugin_lib" value="libgazebo_ros_block_laser.so" />
+        <xacro:property name="plugin_lib" value="libgazebo_ros_velodyne_laser.so" />
       </xacro:unless>
       <sensor type="${ray_type}" name="${prefix}_sensor">

File: urdf/rs_bpearl.urdf.xacro (robot description, xacro)
@@ -50,5 +50,5 @@
       <xacro:unless value="${gpu}">
         <xacro:property name="ray_type" value="ray" />
-        <xacro:property name="plugin_lib" value="libgazebo_ros_block_laser.so" />
+        <xacro:property name="plugin_lib" value="libgazebo_ros_velodyne_laser.so" />
       </xacro:unless>
         <sensor type="${ray_type}" name="${prefix}_sensor">

File: urdf/rslidar.urdf.xacro (robot description, xacro)
@@ -49,5 +49,5 @@
       <xacro:unless value="${gpu}">
         <xacro:property name="ray_type" value="ray" />
-        <xacro:property name="plugin_lib" value="libgazebo_ros_block_laser.so" />
+        <xacro:property name="plugin_lib" value="libgazebo_ros_velodyne_laser.so" />
       </xacro:unless>
         <sensor type="${ray_type}" name="${prefix}_sensor">

File: urdf/rslidar_mems.urdf.xacro (robot description, xacro)
@@ -45,5 +45,5 @@
       <xacro:unless value="${gpu}">
         <xacro:property name="ray_type" value="ray" />
-        <xacro:property name="plugin_lib" value="libgazebo_ros_block_laser.so" />
+        <xacro:property name="plugin_lib" value="libgazebo_ros_velodyne_laser.so" />
       </xacro:unless>
       <sensor type="${ray_type}" name="${prefix}_sensor">

File: urdf/velodyne_vlp16.urdf.xacro (robot description, xacro)
@@ -45,5 +45,5 @@
       <xacro:unless value="${gpu}">
         <xacro:property name="ray_type" value="ray" />
-        <xacro:property name="plugin_lib" value="libgazebo_ros_block_laser.so" />
+        <xacro:property name="plugin_lib" value="libgazebo_ros_velodyne_laser.so" />
       </xacro:unless>
       <sensor type="${ray_type}" name="${prefix}_sensor">

Commit message: cherry-pick from kinetic-devel to change gazebo plugin for using cpu

File: urdf/benewake_ce30.urdf.xacro (robot description, xacro)
@@ -50,5 +50,5 @@
       <xacro:unless value="${gpu}">
         <xacro:property name="ray_type" value="ray" />
-        <xacro:property name="plugin_lib" value="libgazebo_ros_block_laser.so" />
+        <xacro:property name="plugin_lib" value="libgazebo_ros_velodyne_laser.so" />
       </xacro:unless>
         <sensor type="${ray_type}" name="${prefix}_sensor">

File: urdf/hokuyo3d.urdf.xacro (robot description, xacro)
@@ -45,5 +45,5 @@
       <xacro:unless value="${gpu}">
         <xacro:property name="ray_type" value="ray" />
-        <xacro:property name="plugin_lib" value="libgazebo_ros_block_laser.so" />
+        <xacro:property name="plugin_lib" value="libgazebo_ros_velodyne_laser.so" />
       </xacro:unless>
       <sensor type="${ray_type}" name="${prefix}_sensor">

File: urdf/ouster1.urdf.xacro (robot description, xacro)
@@ -48,5 +48,5 @@
       <xacro:unless value="${gpu}">
         <xacro:property name="ray_type" value="ray" />
-        <xacro:property name="plugin_lib" value="libgazebo_ros_block_laser.so" />
+        <xacro:property name="plugin_lib" value="libgazebo_ros_velodyne_laser.so" />
       </xacro:unless>
       <sensor type="${ray_type}" name="${prefix}_sensor">

File: urdf/rs_bpearl.urdf.xacro (robot description, xacro)
@@ -67,5 +67,5 @@
       <xacro:unless value="${gpu}">
         <xacro:property name="ray_type" value="ray" />
-        <xacro:property name="plugin_lib" value="libgazebo_ros_block_laser.so" />
+        <xacro:property name="plugin_lib" value="libgazebo_ros_velodyne_laser.so" />
       </xacro:unless>
         <sensor type="${ray_type}" name="${prefix}_sensor">

File: urdf/rslidar.urdf.xacro (robot description, xacro)
@@ -49,5 +49,5 @@
       <xacro:unless value="${gpu}">
         <xacro:property name="ray_type" value="ray" />
-        <xacro:property name="plugin_lib" value="libgazebo_ros_block_laser.so" />
+        <xacro:property name="plugin_lib" value="libgazebo_ros_velodyne_laser.so" />
       </xacro:unless>
         <sensor type="${ray_type}" name="${prefix}_sensor">

File: urdf/rslidar_mems.urdf.xacro (robot description, xacro)
@@ -38,4 +38,55 @@
     </joint>
     <link name="${prefix}_link"/>
+    <!-- sensor for simulation -->
+    <sensor_rslidar_mems_gazebo range_min="1" range_max="180" gpu="false" />
+  </xacro:macro>
+  <xacro:macro name="sensor_rslidar_mems_gazebo" params="range_min range_max gpu">
+    <gazebo reference="${prefix}_link">
+      <xacro:if value="${gpu}">
+        <!-- Using GPU needs: https://github.com/RobotnikAutomation/velodyne_simulator -->
+        <xacro:property name="ray_type" value="gpu_ray" />
+        <xacro:property name="plugin_lib" value="libgazebo_ros_velodyne_gpu_laser.so" />
+      </xacro:if>
+      <xacro:unless value="${gpu}">
+        <xacro:property name="ray_type" value="ray" />
+        <xacro:property name="plugin_lib" value="libgazebo_ros_velodyne_laser.so" />
+      </xacro:unless>
+      <sensor type="${ray_type}" name="${prefix}_sensor">
+          <pose>0 0 0 0 0 0</pose>
+          <visualize>false</visualize>
+          <update_rate>15</update_rate>
+          <ray>
+              <scan>
+                  <horizontal>
+                      <samples>100</samples>
+                      <resolution>1.0</resolution>
+                      <min_angle>-1.0472</min_angle>
+                      <max_angle>1.0472</max_angle>
+                  </horizontal>
+                  <vertical>
+                      <samples>100</samples>
+                      <resolution>1.0</resolution>
+                      <min_angle>-0.610865238</min_angle>
+                      <max_angle>1.83591184</max_angle>
+                  </vertical>
+              </scan>
+              <range>
+              <min>${range_min}</min>
+              <max>${range_max}</max>
+                  <resolution>0.0035</resolution>
+              </range>
+              <noise>
+                  <type>gaussian</type>
+                  <mean>0.0</mean>
+                  <stddev>0.01</stddev>
+              </noise>
+          </ray>
+          <plugin name="${prefix}_controller" filename="${plugin_lib}">
+              <topicName>/robot/front_3d_laser/point_cloud</topicName>
+              <frameName>/${prefix}_link</frameName>
+              <ignoreTfPrefix>1</ignoreTfPrefix>
+          </plugin>
+      </sensor>
+    </gazebo>
   </xacro:macro>
 </robot>

File: urdf/velodyne_vlp16.urdf.xacro (robot description, xacro)
@@ -45,5 +45,5 @@
       <xacro:unless value="${gpu}">
         <xacro:property name="ray_type" value="ray" />
-        <xacro:property name="plugin_lib" value="libgazebo_ros_block_laser.so" />
+        <xacro:property name="plugin_lib" value="libgazebo_ros_velodyne_laser.so" />
       </xacro:unless>
       <sensor type="${ray_type}" name="${prefix}_sensor">

Commit message: Fix: benewake_ce30d duplicated and urdf/benewake_ce30d.urdf.xacro without default parameter values

File: urdf/benewake_ce30.urdf.xacro (robot description, xacro)
@@ -97,8 +97,3 @@
     </sensor_benewake_ce30>
   </xacro:macro>
-  <xacro:macro name="sensor_benewake_ce30d" params="prefix parent prefix_topic:='lidar_3d' *origin gpu:=false">
-    <sensor_benewake_ce30 prefix="${prefix}" parent="${parent}" prefix_topic="${prefix_topic}" range_min="0.4" range_max="28.0" hfov="60.0" vfov="4.0" fps="30.0" gpu="${gpu}" >
-      <xacro:insert_block name="origin" />
-    </sensor_benewake_ce30>
-  </xacro:macro>
 </robot>

File: urdf/benewake_ce30d.urdf.xacro (robot description, xacro)
@@ -2,5 +2,5 @@
 <robot name="sensor_benewake_ce30d" xmlns:xacro="http://wiki.ros.org/xacro">
   <xacro:property name="M_PI" value="3.1415926535897931" />
-  <xacro:macro name="sensor_benewake_ce30d" params="prefix parent prefix_topic *origin range_min range_max hfov vfov fps gpu:=^|true">
+  <xacro:macro name="sensor_benewake_ce30d" params="prefix parent prefix_topic:='lidar_3d' *origin range_min:=0.4 range_max:=28.0 hfov:=60.0 vfov:=4.0 fps:=30.0 gpu:=^|true">
     <material name="black_alu">
       <color rgba="0.9 0.9 0.9 1"/>

Commit message: material bug fixed

File: urdf/benewake_ce30.urdf.xacro (robot description, xacro)
@@ -3,7 +3,4 @@
   <xacro:property name="M_PI" value="3.1415926535897931" />
   <xacro:macro name="sensor_benewake_ce30" params="prefix parent prefix_topic *origin range_min range_max hfov vfov fps gpu:=^|true">
-    <material name="black_alu">
-      <color rgba="0.9 0.9 0.9 1"/>
-    </material>
     <joint name="${prefix}_base_joint" type="fixed">
       <xacro:insert_block name="origin" />
@@ -18,5 +15,7 @@
           <mesh filename="package://robotnik_sensors/meshes/benewake_ce30.stl" />
         </geometry>
-        <material name="black_alu"/>
+        <material name="black_alu">
+          <color rgba="0.9 0.9 0.9 1"/>
+        </material>
       </visual>
       <collision>

File: urdf/rslidar.urdf.xacro (robot description, xacro)
@@ -3,7 +3,4 @@
   <xacro:property name="M_PI" value="3.1415926535897931" />
   <xacro:macro name="sensor_rslidar" params="prefix parent prefix_topic *origin range_min range_max hfov hres vfov vres fps gpu:=^|true">
-    <material name="black_alu">
-      <color rgba="0.9 0.9 0.9 1"/>
-    </material>
     <joint name="${prefix}_base_joint" type="fixed">
       <xacro:insert_block name="origin" />
@@ -18,5 +15,7 @@
           <mesh filename="package://robotnik_sensors/meshes/rslidar.stl" />
         </geometry>
-        <material name="black_alu"/>
+        <material name="black_alu">
+          <color rgba="0.9 0.9 0.9 1"/>
+        </material>
       </visual>
       <collision>
