Commit message: Updates benewake visual

File: urdf/benewake_ce30d.urdf.xacro (robot description, xacro)
@@ -14,5 +14,5 @@
       <visual>
       <!-- origin xyz="0 0 0" rpy="0 0 1.5708"/ -->
-      <origin xyz="0 0 0" rpy="0 0 0"/>
+      <origin xyz="0 0 0" rpy="1.5708 0 1.5708"/>
         <geometry>
           <mesh filename="package://robotnik_sensors/meshes/benewake_ce30d.stl" />
