Commit message: corrected viper model

File: urdf/rubedos_viper.urdf.xacro (robot description, xacro)
@@ -74,5 +74,5 @@
         <origin xyz="0 0 0" rpy="0 0 0"/>
         <geometry>
-          <box size="${rubedos_viper_width} ${rubedos_viper_height} ${rubedos_viper_depth}"/>
+          <box size="${rubedos_viper_depth} ${rubedos_viper_height} ${rubedos_viper_width}"/>
           <!--<mesh filename="package://pointgrey_camera_description/meshes/rubedos_viper.dae"/>-->
         </geometry>
@@ -81,5 +81,5 @@
         <origin xyz="0 0 0" rpy="0 0 0"/>
         <geometry>
-          <box size="${rubedos_viper_width} ${rubedos_viper_height} ${rubedos_viper_depth}"/>
+          <box size="${rubedos_viper_depth} ${rubedos_viper_height} ${rubedos_viper_width}"/>
         </geometry>
       </collision>

Commit message: new 3D viper model added

File: urdf/rubedos_viper.urdf.xacro (robot description, xacro)
@@ -74,6 +74,6 @@
         <origin xyz="0 0 0" rpy="0 0 0"/>
         <geometry>
-          <box size="${rubedos_viper_depth} ${rubedos_viper_height} ${rubedos_viper_width}"/>
-          <!--<mesh filename="package://pointgrey_camera_description/meshes/rubedos_viper.dae"/>-->
+          <!--box size="${rubedos_viper_depth} ${rubedos_viper_width} ${rubedos_viper_height}"/-->
+          <mesh filename="package://robotnik_sensors/meshes/viper.dae"/>
         </geometry>
       </visual>
@@ -81,5 +81,5 @@
         <origin xyz="0 0 0" rpy="0 0 0"/>
         <geometry>
-          <box size="${rubedos_viper_depth} ${rubedos_viper_height} ${rubedos_viper_width}"/>
+          <box size="${rubedos_viper_depth} ${rubedos_viper_width} ${rubedos_viper_height}"/>
         </geometry>
       </collision>
@@ -93,6 +93,6 @@
     </link>
     <joint name="${prefix}_optical_joint" type="fixed">
-      <origin xyz="0 0 0" rpy="-1.570796 0 -1.570796" />
-      <!--<origin xyz="0 0 0" rpy="0 0 0" />-->
+      <!--origin xyz="0 0 0" rpy="-1.570796 0 -1.570796" /-->
+      <origin xyz="0 0 0" rpy="0 0 0" />
       <parent link="${prefix}_base_link" />
       <child link="${prefix}_optical_frame" />

Commit message: Update rubedos_viper inertia

File: urdf/rubedos_viper.urdf.xacro (robot description, xacro)
@@ -85,9 +85,7 @@
       </collision>
       <inertial>
+        <origin xyz="-0.0 0.0 0.0" rpy="0 0 0" />
         <mass value="0.8" />
-        <inertia
-          ixx="${1/12*0.8*(0.036*0.036 + 0.0474*0.0474)}" ixy="0" ixz="0"
-          iyy="${1/12*0.8*(0.157*0.157 + 0.0474*0.0474)}" iyz="0"
-          izz="${1/12*0.8*(0.157*0.157 + 0.036*0.036)}" />
+        <xacro:solid_cuboid_inertia m="0.8" w="0.0574" h="0.187" d="0.036" />
       </inertial>
     </link>
@@ -99,5 +97,5 @@
     </joint>
     <link name="${prefix}_optical_frame">
-      <inertial>
+      <!--inertial>
         <mass value="1E-5" />
         <inertia
@@ -105,5 +103,5 @@
           iyy="1E-10" iyz="0"
           izz="1E-10" />
-      </inertial>
+      </inertial-->
     </link>
       <xacro:stereo_camera

Commit message: Fix viper and zed frames to properly run

File: urdf/rubedos_viper.urdf.xacro (robot description, xacro)
@@ -50,5 +50,5 @@
           <imageTopicName>image_raw</imageTopicName>
           <cameraInfoTopicName>camera_info</cameraInfoTopicName>
-          <frameName>${prefix}_optical_frame</frameName>
+          <frameName>/${prefix}_optical_frame</frameName>
           <hackBaseline>${baseline}</hackBaseline>
           <!-- NOTE: Distortion is currently unused -->
@@ -91,5 +91,5 @@
     </link>
     <joint name="${prefix}_optical_joint" type="fixed">
-      <!--origin xyz="0 0 0" rpy="-1.570796 0 -1.570796" /-->
+      <origin xyz="0 0 0" rpy="-1.570796 0 -1.570796" />
       <origin xyz="0 0 0" rpy="0 0 0" />
       <parent link="${prefix}_base_link" />
@@ -109,7 +109,7 @@
         hfov="1.2217"
         baseline="0.20"
-        fps="40"
-        width="640"
-        height="480"
+        fps="60"
+        width="2304"
+        height="1535"
         format="${format}"
         near="${near}"
