Commit message: Update axis_q8641 inertia

File: urdf/axis_q8641.urdf.xacro (robot description, xacro)
@@ -2,5 +2,5 @@
 <robot xmlns:xacro="http://wiki.ros.org/xacro" name="sensor_axis_q8641">
   <xacro:property name="ptz_joint_effort_limit" value="100.0"/>
-  <xacro:property name="ptz_joint_velocity_limit" value="100.0"/>
+  <xacro:property name="ptz_joint_velocity_limit" value="1.0"/>
   <xacro:property name="ptz_joint_friction" value="0.1"/>
   <xacro:property name="ptz_joint_damping" value="0.1"/>
@@ -15,8 +15,7 @@
     <link name="${prefix}_base_link">
       <inertial>
-        <origin xyz="0.0 0.0 0.0" rpy="0 0 0"/>
-        <mass value="0.1"/>
-        <origin xyz="0 0 0" rpy="0 0 0"/>
-        <inertia ixx="0.1" ixy="0" ixz="0" iyy="0.1" iyz="0" izz="0.1"/>
+        <mass value="2"/>
+        <origin xyz="0 0 0.06" rpy="0 0 0"/>
+        <xacro:solid_cuboid_inertia m="2" w="0.175" h="0.175" d="0.12" />
       </inertial>
       <visual>
@@ -49,7 +48,7 @@
     <link name="${prefix}_pan_link">
       <inertial>
-        <mass value="0.1"/>
-        <origin xyz="0 0 0" rpy="0 0 0"/>
-        <inertia ixx="0.1" ixy="0" ixz="0" iyy="0.1" iyz="0" izz="0.1"/>
+        <mass value="5.0"/>
+        <origin xyz="0 0 0.12" rpy="0 0 0"/>
+        <xacro:solid_cuboid_inertia m="5.0" w="0.175" h="0.175" d="0.24" />
       </inertial>
       <visual>
@@ -91,7 +90,7 @@
     <link name="${prefix}_tilt_link">
       <inertial>
-        <mass value="0.1"/>
-        <origin xyz="0 0 0" rpy="0 0 0"/>
-        <inertia ixx="0.1" ixy="0" ixz="0" iyy="0.1" iyz="0" izz="0.1"/>
+        <mass value="5.0"/>
+        <origin xyz="0.04875 0 0.11" rpy="0 0 0"/>
+        <xacro:solid_cuboid_inertia m="5.0" w="0.24" h="0.09" d="0.09" />
       </inertial>
       <visual>
@@ -129,9 +128,9 @@
     </joint>
     <link name="${prefix}_frame_link">
-      <inertial>
+      <!--inertial>
         <mass value="0.001"/>
         <origin xyz="0 0 0"/>
         <inertia ixx="0.0001" ixy="0.0" ixz="0.0" iyy="0.0001" iyz="0.0" izz="0.0001"/>
-      </inertial>
+      </inertial-->
     </link>
     <!-- Optical frame -->
@@ -142,9 +141,9 @@
     </joint>
     <link name="${prefix}_optical_frame_link">
-      <inertial>
+      <!--inertial>
         <mass value="0.001"/>
         <origin xyz="0 0 0"/>
         <inertia ixx="0.0001" ixy="0.0" ixz="0.0" iyy="0.0001" iyz="0.0" izz="0.0001"/>
-      </inertial>
+      </inertial-->
     </link>
     <gazebo reference="${prefix}_base_link">

Commit message: axis_q8641:default inertia values set to 0.001

File: urdf/axis_q8641.urdf.xacro (robot description, xacro)
@@ -14,8 +14,12 @@
     </joint>
     <link name="${prefix}_base_link">
-      <inertial>
+      <!--inertial>
         <mass value="2"/>
         <origin xyz="0 0 0.06" rpy="0 0 0"/>
         <xacro:solid_cuboid_inertia m="2" w="0.175" h="0.175" d="0.12" />
+      </inertial-->
+      <inertial>
+        <mass value="0.001"/>
+        <inertia ixx="0.001" ixy="0" ixz="0" iyy="0.001" iyz="0" izz="0.001"/>
       </inertial>
       <visual>
@@ -47,8 +51,12 @@
     </joint>
     <link name="${prefix}_pan_link">
-      <inertial>
+      <!--inertial>
         <mass value="5.0"/>
         <origin xyz="0 0 0.12" rpy="0 0 0"/>
         <xacro:solid_cuboid_inertia m="5.0" w="0.175" h="0.175" d="0.24" />
+      </inertial-->
+      <inertial>
+        <mass value="0.001"/>
+        <inertia ixx="0.001" ixy="0" ixz="0" iyy="0.001" iyz="0" izz="0.001"/>
       </inertial>
       <visual>
@@ -89,8 +97,12 @@
     </joint>
     <link name="${prefix}_tilt_link">
-      <inertial>
+      <!--inertial>
         <mass value="5.0"/>
         <origin xyz="0.04875 0 0.11" rpy="0 0 0"/>
         <xacro:solid_cuboid_inertia m="5.0" w="0.24" h="0.09" d="0.09" />
+      </inertial-->
+      <inertial>
+        <mass value="0.001"/>
+        <inertia ixx="0.001" ixy="0" ixz="0" iyy="0.001" iyz="0" izz="0.001"/>
       </inertial>
       <visual>
