Commit message: Update zed2.urdf.xacro: Add prefix_topic in zed2 camera simulation

File: urdf/zed2.urdf.xacro (robot description, xacro)
@@ -2,5 +2,5 @@
 <robot xmlns:xacro="http://wiki.ros.org/xacro">
   <xacro:macro name="depth_camera"
-    params="prefix fps baseline hfov width height format near far">
+    params="prefix fps baseline hfov width height format near far  prefix_topic:='zed_node'">
     <gazebo reference="${prefix}_base_link">
       <visual>
@@ -37,10 +37,10 @@
             will control the frame rate. -->
           <updateRate>0.0</updateRate>
-          <cameraName>${prefix}</cameraName>
-          <imageTopicName>zed_node/rgb/image_raw</imageTopicName>
-          <cameraInfoTopicName>zed_node/rgb/camera_info</cameraInfoTopicName>
-          <depthImageTopicName>zed_node/depth/image_raw</depthImageTopicName>
-          <depthImageCameraInfoTopicName>zed_node/depth/camera_info</depthImageCameraInfoTopicName>
-          <pointCloudTopicName>zed_node/depth/points</pointCloudTopicName>
+          <cameraName>${prefix_topic}</cameraName>
+          <imageTopicName> rgb/image_raw</imageTopicName>
+          <cameraInfoTopicName>rgb/camera_info</cameraInfoTopicName>
+          <depthImageTopicName>depth/image_raw</depthImageTopicName>
+          <depthImageCameraInfoTopicName>depth/camera_info</depthImageCameraInfoTopicName>
+          <pointCloudTopicName>depth/points</pointCloudTopicName>
           <frameName>/${prefix}_depth_optical_frame</frameName>
           <pointCloudCutoff>${near}</pointCloudCutoff>
@@ -61,5 +61,5 @@
   </xacro:macro>
   <xacro:macro name="stereolabs_zed2"
-    params="prefix:=zed parent *origin model:=zed format:=R8G8B8 near:=0.5 far:=30">
+    params="prefix:=zed parent *origin model:=zed format:=R8G8B8 near:=0.5 far:=30  prefix_topic:=zed_node">
     <xacro:if value="${model == 'zed'}">
         <xacro:property name="baseline" value="0.12" />
@@ -146,8 +146,10 @@
         format="${format}"
         near="${near}"
-        far="${far}"/>
+        far="${far}"
+        prefix_topic="${prefix_topic}"
+        />
   </xacro:macro>
-  <xacro:macro name="sensor_zed2" params="prefix:=zed2 parent *origin model:=zed2" >
-    <stereolabs_zed2 prefix="${prefix}" parent="${parent}" model="${model}">
+  <xacro:macro name="sensor_zed2" params="prefix:=zed2 parent *origin model:=zed2  prefix_topic:=zed_node" >
+    <stereolabs_zed2 prefix="${prefix}" parent="${parent}" model="${model}" prefix_topic="${prefix_topic}">
       <xacro:insert_block name="origin" />
     </stereolabs_zed2>

Commit message: zed2: change rgb_ to camera_

File: urdf/zed2.urdf.xacro (robot description, xacro)
@@ -99,29 +99,29 @@
     </link>
    <!-- Left camera -->
-    <joint name="${prefix}_rgb_left_joint" type="fixed">
+    <joint name="${prefix}_camera_left_joint" type="fixed">
       <origin xyz="0.0 0.06 0.0" rpy="0.0 0.0 0.0" />
       <parent link="${prefix}_base_link" />
-      <child link="${prefix}_left_rgb_frame" />
+      <child link="${prefix}_left_camera_frame" />
     </joint>
-    <link name="${prefix}_left_rgb_frame"/>
-    <joint name="${prefix}_rgb_left_optical_joint" type="fixed">
+    <link name="${prefix}_left_camera_frame"/>
+    <joint name="${prefix}_camera_left_optical_joint" type="fixed">
       <origin xyz="0.0 0.0 0.0" rpy="${-M_PI/2} 0.0 ${-M_PI/2}" />
-      <parent link="${prefix}_left_rgb_frame" />
-      <child link="${prefix}_left_rgb_optical_frame" />
+      <parent link="${prefix}_left_camera_frame" />
+      <child link="${prefix}_left_camera_optical_frame" />
     </joint>
-    <link name="${prefix}_left_rgb_optical_frame"/>
+    <link name="${prefix}_left_camera_optical_frame"/>
     <!-- Right camera-->
-    <joint name="${prefix}_rgb_right_joint" type="fixed">
+    <joint name="${prefix}_camera_right_joint" type="fixed">
       <origin xyz="0.0 -0.06 0.0" rpy="0.0 0.0 0.0" />
       <parent link="${prefix}_base_link" />
-      <child link="${prefix}_right_rgb_frame" />
+      <child link="${prefix}_right_camera_frame" />
     </joint>
-    <link name="${prefix}_right_rgb_frame"/>
-    <joint name="${prefix}_rgb_right_optical_joint" type="fixed">
+    <link name="${prefix}_right_camera_frame"/>
+    <joint name="${prefix}_camera_right_optical_joint" type="fixed">
       <origin xyz="0.0 0 0.0" rpy="${-M_PI/2} 0.0 ${-M_PI/2}" />
-      <parent link="${prefix}_right_rgb_frame" />
-      <child link="${prefix}_right_rgb_optical_frame" />
+      <parent link="${prefix}_right_camera_frame" />
+      <child link="${prefix}_right_camera_optical_frame" />
     </joint>
-    <link name="${prefix}_right_rgb_optical_frame"/>
+    <link name="${prefix}_right_camera_optical_frame"/>
     <!-- Depth image-->
     <joint name="${prefix}_depth_joint" type="fixed">
