Commit message: Update gps_with_mast inertia

File: urdf/gps_with_mast.urdf.xacro (robot description, xacro)
@@ -13,9 +13,9 @@
 	  </joint>
 	  <link name="${prefix}_mast_base_link">
-	    <inertial>
-	      <mass value="0.001"/>
-	      <origin rpy="0 0 0" xyz="0 0 0"/>
-	      <inertia ixx="0.0001" ixy="0" ixz="0" iyy="0.000001" iyz="0" izz="0.0001"/>
-	    </inertial>
+		<inertial>
+			<origin xyz="0.0 0 0.0" rpy="0 0 0" />
+			<mass value="1.0" />
+			<xacro:solid_cuboid_inertia m="1.0" w="${mast_radius}" h="${mast_radius}" d="${mast_height}" />
+		</inertial>
 	    <visual>
 	      <origin rpy="0 0 0" xyz="0 0 0"/>
@@ -47,8 +47,8 @@
 	  <link name="${prefix}_link">
 	    <inertial>
-	      <mass value="0.001"/>
-	      <origin rpy="0 0 0" xyz="0 0 0"/>
-	      <inertia ixx="0.0001" ixy="0" ixz="0" iyy="0.000001" iyz="0" izz="0.0001"/>
-	    </inertial>
+			<origin xyz="0.0 0 0.015" rpy="0 0 0" />
+			<mass value="0.2" />
+			<xacro:solid_cuboid_inertia m="0.2" w="0.081" h="0.081" d="0.03" />
+      	</inertial>
 	    <visual>
 	      <origin rpy="0 0 0" xyz="0 0 0"/>

Commit message: Fix gps_with_mast model

File: urdf/gps_with_mast.urdf.xacro (robot description, xacro)
@@ -4,5 +4,5 @@
   <xacro:property name="mast_radius" value="0.010" />
   <!-- if no latitude/longitud is specified, then use Fuente del Jarro as default -->
-  <xacro:macro name="sensor_gps_with_mast" params="prefix parent *origin gps_latitude:=^|39.5080331 gps_longitude:=^|-0.4619816">
+  <xacro:macro name="sensor_gps_with_mast" params="prefix parent *origin gps_latitude:=^|39.5080331 gps_longitude:=^|-0.4619816 update_rate:=^|5">
 	  <!-- MAST OF THE ANTENNA GPS -->
 	  <joint name="${prefix}_joint" type="fixed">
@@ -37,5 +37,5 @@
 	    <axis xyz="0 1 0"/>
 	    <parent link="${prefix}_mast_base_link"/>
-	    <child link="${prefix}_link"/>
+	    <child link="${prefix}_base_link"/>
 	    <origin xyz="0 0 ${mast_height/2.0}" rpy="0 0 0" />
 	  </joint>
@@ -45,5 +45,5 @@
 	  </gazebo>
       <!-- ANTENNA GPS -->
-	  <link name="${prefix}_link">
+	  <link name="${prefix}_base_link">
 	    <inertial>
 			<origin xyz="0.0 0 0.015" rpy="0 0 0" />
@@ -67,5 +67,5 @@
 	    </collision>
 	  </link>
-	  <gazebo reference="${prefix}_link">
+	  <gazebo reference="${prefix}_base_link">
 	    <material>Gazebo/White</material>
 	    <gravity>true</gravity>
@@ -74,8 +74,8 @@
       <plugin name="${prefix}_controller" filename="libhector_gazebo_ros_gps.so">
         <alwaysOn>1</alwaysOn>
-        <updateRate>5</updateRate>
-        <bodyName>${prefix}_link</bodyName> <!-- must be the link of the gps device, not the base_link or base_footprint -->
-        <frameId>${prefix}_link</frameId>   <!-- which frame_id would be on the published message -->
-        <topicName>fix</topicName>
+        <updateRate>${update_rate}</updateRate>
+        <bodyName>${prefix}_base_link</bodyName> <!-- must be the link of the gps device, not the base_link or base_footprint -->
+        <frameId>${prefix}_base_link</frameId>   <!-- which frame_id would be on the published message -->
+        <topicName>gps/fix</topicName>
         <!-- GPS coordinates -->
         <referenceLatitude>${gps_latitude}</referenceLatitude>
@@ -83,14 +83,13 @@
         <!-- To set heading in ENU orientation (degrees) -->
         <referenceHeading>90</referenceHeading>
-        <velocityTopicName>fix_velocity</velocityTopicName>
+        <velocityTopicName>gps/fix_velocity</velocityTopicName>
         <drift>0.0 0.0 0.0</drift>
         <!--<drift>0.0001 0.0001 0.0001</drift>-->
         <!--<drift>0.3 0.3 0.3</drift>-->
-        <gaussianNoise>0.1 0.1 0.1</gaussianNoise>
+        <gaussianNoise>0.00001 0.00001 0.00001</gaussianNoise>
         <!--<gaussianNoise>0.00001 0.00001 0.00001</gaussianNoise>-->
         <velocityDrift>0.00001 0.00001 0.00001</velocityDrift>
         <!--<velocityGaussianNoise>0.1 0.1 0.1</velocityGaussianNoise>-->
         <velocityGaussianNoise>0.00001 0.00001 0.00001</velocityGaussianNoise>
-        <ignoreTfPrefix>1</ignoreTfPrefix>
       </plugin>
 	</gazebo>
