Commit message: adding prefix_frame and prefix_topic

File: urdf/imu.urdf.xacro (robot description, xacro)
@@ -1,5 +1,5 @@
 <?xml version="1.0"?>
 <robot name="sensor_imu" xmlns:xacro="http://www.ros.org/wiki/xacro">
-  <xacro:macro name="sensor_imu" params="name parent *origin">
+  <xacro:macro name="sensor_imu" params="name prefix_frame prefix_topic parent *origin">
 	  <joint name="${name}_joint" type="fixed">
 	      <axis xyz="1 0 0"/>
@@ -7,5 +7,5 @@
 	      <xacro:insert_block name="origin"/>
 	      <parent link="${parent}"/>
-	      <child link="${name}_link"/>
+	      <child link="${prefix_frame}_link"/>
 	  </joint>
 	  <link name="${name}_link">
@@ -30,7 +30,7 @@
 	  <gazebo>
 	    <plugin name="${name}_controller" filename="libgazebo_ros_imu.so">
-	       <topicName>${name}/data</topicName>
-		   <serviceName>${name}/service</serviceName>
-		   <bodyName>${name}_link</bodyName>
+	       <topicName>${prefix_topic}/data</topicName>
+		   <serviceName>${prefix_topic}/service</serviceName>
+		   <bodyName>${prefix_frame}_link</bodyName>
 	       <gaussianNoise>0.005</gaussianNoise>
 	    </plugin>

Commit message: updating imu_plugin: topic and link names

File: urdf/imu.urdf.xacro (robot description, xacro)
@@ -2,12 +2,12 @@
 <robot name="sensor_imu" xmlns:xacro="http://www.ros.org/wiki/xacro">
   <xacro:macro name="sensor_imu" params="prefix parent *origin">
-	  <joint name="${prefix}_base_joint" type="fixed">
+	  <joint name="${prefix}_joint" type="fixed">
 	      <axis xyz="1 0 0"/>
 	      <!--origin xyz="0 0 0.2825"/-->
 	      <xacro:insert_block name="origin"/>
 	      <parent link="${parent}"/>
-	      <child link="${prefix}_base_link"/>
+	      <child link="${prefix}_link"/>
 	  </joint>
-	  <link name="${prefix}_base_link">
+	  <link name="${prefix}_link">
 	      <inertial>
 	        <mass value="0.001"/>
@@ -30,7 +30,8 @@
 	  <gazebo>
 	    <plugin name="${prefix}_controller" filename="libgazebo_ros_imu.so">
-	       <topicName>data</topicName>
-		   <serviceName>${prefix}service</serviceName>
-		   <bodyName>/${prefix}_base_link</bodyName>
+	       <topicName>imu/data</topicName>
+	       <serviceName>imu/service</serviceName>
+		   <bodyName>${prefix}_link</bodyName>
+		   <updateRateHZ>50.0</updateRateHZ>
 	       <gaussianNoise>0.005</gaussianNoise>
 	    </plugin>

Commit message: Added left zero of floar numbers

File: urdf/imu.urdf.xacro (robot description, xacro)
@@ -24,5 +24,5 @@
 	        <origin rpy="0 0 0" xyz="0 0 0"/>
 	        <geometry>
-	          <box size=".001 .001 .001"/>
+	          <box size="0.001 0.001 0.001"/>
 	        </geometry>
 	      </collision>

Commit message: Change imu sensors default topic - from data to data_raw

File: urdf/imu.urdf.xacro (robot description, xacro)
@@ -1,59 +1,44 @@
 <?xml version="1.0"?>
 <robot name="sensor_imu" xmlns:xacro="http://wiki.ros.org/xacro">
-  <xacro:macro name="sensor_imu" params="prefix ns:='' parent *origin">
+  <xacro:macro name="sensor_imu" params="prefix ns:='' parent *origin prefix_topic:='imu'">
 	  <joint name="${prefix}_joint" type="fixed">
-	      <axis xyz="1 0 0"/>
-	      <!--origin xyz="0 0 0.2825"/-->
-	      <xacro:insert_block name="origin"/>
-	      <parent link="${parent}"/>
-	      <child link="${prefix}_link"/>
+      <axis xyz="1 0 0"/>
+      <!--origin xyz="0 0 0.2825"/-->
+      <xacro:insert_block name="origin"/>
+      <parent link="${parent}"/>
+      <child link="${prefix}_link"/>
 	  </joint>
-	  <link name="${prefix}_link">
-	      <inertial>
-	        <mass value="0.001"/>
-	        <origin rpy="0 0 0" xyz="0 0 0"/>
-	        <inertia ixx="0.00000000167" ixy="0" ixz="0" iyy="0.00000000167" iyz="0" izz="0.00000000167"/>
-	      </inertial>
-	      <visual>
-	        <origin rpy="0 0 0" xyz="0 0 0"/>
-	        <geometry>
-	          <box size="0.001 0.001 0.001"/>
-	        </geometry>
-	      </visual>
-	      <!--collision>
-	        <origin rpy="0 0 0" xyz="0 0 0"/>
-	        <geometry>
-	          <box size=".001 .001 .001"/>
-	        </geometry>
-	      </collision-->
-	  </link>
-	  <!--<gazebo>-->
-		<!--<plugin name="${prefix}_controller" filename="libgazebo_ros_imu.so">-->
-		   <!--<topicName>${ns}imu/data</topicName>-->
-		   <!--<serviceName>imu/service</serviceName>-->
-		   <!--<bodyName>${prefix}_link</bodyName>-->
-		   <!--<updateRateHZ>50.0</updateRateHZ>-->
-		   <!--<gaussianNoise>0.0</gaussianNoise>-->
-		<!--</plugin>-->
-	  <!--</gazebo>-->
- <gazebo reference="${prefix}_link">
-    <gravity>true</gravity>
-    <sensor name="${prefix}_imu_sensor" type="imu">
-      <always_on>true</always_on>
-      <update_rate>100</update_rate>
-      <visualize>true</visualize>
-      <topic>__default_topic__</topic>
-      <plugin filename="libgazebo_ros_imu_sensor.so" name="${prefix}_imu_plugin">
-        <topicName>imu/data</topicName>
-		<bodyName>${prefix}_link</bodyName>
-        <updateRateHZ>100.0</updateRateHZ>
-        <gaussianNoise>0.0</gaussianNoise>
-        <xyzOffset>0 0 0</xyzOffset>
-        <rpyOffset>0 0 0</rpyOffset>
-		<frameName>${prefix}_link</frameName>
-      </plugin>
-      <pose>0 0 0 0 0 0</pose>
-    </sensor>
-  </gazebo>
+    <link name="${prefix}_link">
+      <inertial>
+        <mass value="0.001"/>
+        <origin rpy="0 0 0" xyz="0 0 0"/>
+        <inertia ixx="0.00000000167" ixy="0" ixz="0" iyy="0.00000000167" iyz="0" izz="0.00000000167"/>
+      </inertial>
+      <visual>
+        <origin rpy="0 0 0" xyz="0 0 0"/>
+        <geometry>
+          <box size="0.001 0.001 0.001"/>
+        </geometry>
+      </visual>
+    </link>
+    <gazebo reference="${prefix}_link">
+      <gravity>true</gravity>
+      <sensor name="${prefix}_imu_sensor" type="imu">
+        <always_on>true</always_on>
+        <update_rate>100</update_rate>
+        <visualize>true</visualize>
+        <topic>__default_topic__</topic>
+        <plugin filename="libgazebo_ros_imu_sensor.so" name="${prefix}_imu_plugin">
+          <topicName>${prefix_topic}/data_raw</topicName>
+  		    <bodyName>${prefix}_link</bodyName>
+          <updateRateHZ>100.0</updateRateHZ>
+          <gaussianNoise>0.0</gaussianNoise>
+          <xyzOffset>0 0 0</xyzOffset>
+          <rpyOffset>0 0 0</rpyOffset>
+  		    <frameName>${prefix}_link</frameName>
+        </plugin>
+        <pose>0 0 0 0 0 0</pose>
+      </sensor>
+    </gazebo>
   </xacro:macro>
 </robot>

File: urdf/imu_hector_plugin.urdf.xacro (robot description, xacro)
@@ -1,51 +1,51 @@
 <?xml version="1.0"?>
 <robot name="sensor_imu" xmlns:xacro="http://wiki.ros.org/xacro">
-  <xacro:macro name="sensor_imu_hector" params="prefix parent *origin">
+  <xacro:macro name="sensor_imu_hector" params="prefix parent *origin prefix_topic:='imu'">
 	  <joint name="${prefix}_joint" type="fixed">
-	      <axis xyz="1 0 0"/>
-	      <!--origin xyz="0 0 0.2825"/-->
-	      <xacro:insert_block name="origin"/>
-	      <parent link="${parent}"/>
-	      <child link="${prefix}_link"/>
+      <axis xyz="1 0 0"/>
+      <!--origin xyz="0 0 0.2825"/-->
+      <xacro:insert_block name="origin"/>
+      <parent link="${parent}"/>
+      <child link="${prefix}_link"/>
 	  </joint>
 	  <link name="${prefix}_link">
-	      <inertial>
-	        <mass value="0.001"/>
-	        <origin rpy="0 0 0" xyz="0 0 0"/>
-	        <inertia ixx="0.0001" ixy="0" ixz="0" iyy="0.000001" iyz="0" izz="0.0001"/>
-	      </inertial>
-	      <visual>
-	        <origin rpy="0 0 0" xyz="0 0 0"/>
-	        <geometry>
-	          <box size="0.001 0.001 0.001"/>
-	        </geometry>
-	      </visual>
-	      <collision>
-	        <origin rpy="0 0 0" xyz="0 0 0"/>
-	        <geometry>
-	          <box size=".001 .001 .001"/>
-	        </geometry>
-	      </collision>
+      <inertial>
+        <mass value="0.001"/>
+        <origin rpy="0 0 0" xyz="0 0 0"/>
+        <inertia ixx="0.0001" ixy="0" ixz="0" iyy="0.000001" iyz="0" izz="0.0001"/>
+      </inertial>
+      <visual>
+        <origin rpy="0 0 0" xyz="0 0 0"/>
+        <geometry>
+          <box size="0.001 0.001 0.001"/>
+        </geometry>
+      </visual>
+      <collision>
+        <origin rpy="0 0 0" xyz="0 0 0"/>
+        <geometry>
+          <box size=".001 .001 .001"/>
+        </geometry>
+      </collision>
 	  </link>
 	  <gazebo>
 	    <plugin name="${prefix}_controller" filename="libhector_gazebo_ros_imu.so">
-	       <alwaysOn>true</alwaysOn>
-	       <topicName>imu/data</topicName>
-		   <serviceName>${prefix}imu/service</serviceName>
-		   <bodyName>${prefix}_link</bodyName>
-		   <frameId>${prefix}_link</frameId>
-	       <updateRate>50.0</updateRate>
-	       <gaussianNoise>0.00</gaussianNoise>
-           <yawOffset>0.0</yawOffset>
-           <yawDrift>0.0</yawDrift>
-           <yawGaussianNoise>0.0</yawGaussianNoise>
-           <!-- angular velocities parameters -->
-           <rateOffset>0.0 0.0 0.0</rateOffset>
-           <rateDrift>0.0 0.0 0.0</rateDrift>
-           <rateGaussianNoise>0.0 0.0 0.0</rateGaussianNoise>
-           <!-- linear accelerations parameters -->
-           <accelOffset>0.0 0.0 0.0</accelOffset>
-           <accelDrift>0.0 0.0 0.0</accelDrift>
-           <accelGaussianNoise>0.0 0.0 0.0</accelGaussianNoise>
+       <alwaysOn>true</alwaysOn>
+       <topicName>${prefix_topic}/data_raw</topicName>
+  	   <serviceName>${prefix}imu/service</serviceName>
+  	   <bodyName>${prefix}_link</bodyName>
+  	   <frameId>${prefix}_link</frameId>
+       <updateRate>50.0</updateRate>
+       <gaussianNoise>0.00</gaussianNoise>
+       <yawOffset>0.0</yawOffset>
+       <yawDrift>0.0</yawDrift>
+       <yawGaussianNoise>0.0</yawGaussianNoise>
+       <!-- angular velocities parameters -->
+       <rateOffset>0.0 0.0 0.0</rateOffset>
+       <rateDrift>0.0 0.0 0.0</rateDrift>
+       <rateGaussianNoise>0.0 0.0 0.0</rateGaussianNoise>
+       <!-- linear accelerations parameters -->
+       <accelOffset>0.0 0.0 0.0</accelOffset>
+       <accelDrift>0.0 0.0 0.0</accelDrift>
+       <accelGaussianNoise>0.0 0.0 0.0</accelGaussianNoise>
 	    </plugin>
 	  </gazebo>

Commit message: Update imu inertia

File: urdf/imu.urdf.xacro (robot description, xacro)
@@ -11,8 +11,8 @@
 	  <link name="${prefix}_link">
 	      <inertial>
-	        <mass value="0.001"/>
-	        <origin rpy="0 0 0" xyz="0 0 0"/>
-	        <inertia ixx="0.00000000167" ixy="0" ixz="0" iyy="0.00000000167" iyz="0" izz="0.00000000167"/>
-	      </inertial>
+			<origin xyz="0.0 0 0.01" rpy="0 0 0" />
+			<mass value="0.005" />
+			<xacro:solid_cuboid_inertia m="0.005" w="0.001" h="0.001" d="0.001" />
+		  </inertial>
 	      <visual>
 	        <origin rpy="0 0 0" xyz="0 0 0"/>

Commit message: Add an argument to set the topic name in the imu plugins

File: urdf/imu.urdf.xacro (robot description, xacro)
@@ -1,5 +1,5 @@
 <?xml version="1.0"?>
 <robot name="sensor_imu" xmlns:xacro="http://wiki.ros.org/xacro">
-  <xacro:macro name="sensor_imu" params="prefix ns:='' parent *origin">
+  <xacro:macro name="sensor_imu" params="prefix ns:='' topic:='imu/data' parent *origin">
 	  <joint name="${prefix}_joint" type="fixed">
 	      <axis xyz="1 0 0"/>
@@ -45,5 +45,5 @@
       <topic>__default_topic__</topic>
       <plugin filename="libgazebo_ros_imu_sensor.so" name="${prefix}_imu_plugin">
-        <topicName>imu/data</topicName>
+        <topicName>${topic}</topicName>
 		<bodyName>${prefix}_link</bodyName>
         <updateRateHZ>100.0</updateRateHZ>
