Commit message: Fix zed urdf optical frames

File: urdf/zed.urdf.xacro (robot description, xacro)
@@ -51,5 +51,5 @@
     <!-- Left camera -->
     <joint name="${prefix}_rgb_left_joint" type="fixed">
-      <origin xyz="0.0 -0.06 0.0" rpy="0.0 0.0 0.0" />
+      <origin xyz="0.0 0.06 0.0" rpy="0.0 0.0 0.0" />
       <parent link="${prefix}_link" />
       <child link="${prefix}_left_rgb_frame" />
@@ -57,5 +57,5 @@
     <link name="${prefix}_left_rgb_frame"/>
     <joint name="${prefix}_rgb_left_optical_joint" type="fixed">
-      <origin xyz="0.0 0.06 0.0" rpy="${-M_PI/2} 0.0 ${-M_PI/2}" />
+      <origin xyz="0.0 0.0 0.0" rpy="${-M_PI/2} 0.0 ${-M_PI/2}" />
       <parent link="${prefix}_left_rgb_frame" />
       <child link="${prefix}_left_rgb_optical_frame" />
@@ -64,5 +64,5 @@
     <!-- Right camera-->
     <joint name="${prefix}_rgb_right_joint" type="fixed">
-      <origin xyz="0.0 0.06 0.0" rpy="0.0 0.0 0.0" />
+      <origin xyz="0.0 -0.06 0.0" rpy="0.0 0.0 0.0" />
       <parent link="${prefix}_link" />
       <child link="${prefix}_right_rgb_frame" />
@@ -70,5 +70,5 @@
     <link name="${prefix}_right_rgb_frame"/>
     <joint name="${prefix}_rgb_right_optical_joint" type="fixed">
-      <origin xyz="0.0 -0.06 0.0" rpy="${-M_PI/2} 0.0 ${-M_PI/2}" />
+      <origin xyz="0.0 0 0.0" rpy="${-M_PI/2} 0.0 ${-M_PI/2}" />
       <parent link="${prefix}_right_rgb_frame" />
       <child link="${prefix}_right_rgb_optical_frame" />

Commit message: Update zed inertia

File: urdf/zed.urdf.xacro (robot description, xacro)
@@ -11,9 +11,10 @@
     <link name="${prefix}_rgb_base_link">
       <inertial>
-        <mass value="0.001" />
+        <mass value="0.135" />
         <origin xyz="0 0 0" />
-        <inertia ixx="0.0001" ixy="0.0" ixz="0.0"
+        <xacro:solid_cuboid_inertia m="0.135" w="0.033" h="0.175" d="0.03" />
+        <!--inertia ixx="0.0001" ixy="0.0" ixz="0.0"
           iyy="0.0001" iyz="0.0"
-          izz="0.0001" />
+          izz="0.0001" /-->
       </inertial>
     </link>
@@ -42,9 +43,10 @@
       </collision>
       <inertial>
-        <mass value="0.564" />
+        <mass value="0.135" />
         <origin xyz="0 0 0" />
-        <inertia ixx="0.003881243" ixy="0.0" ixz="0.0"
+        <xacro:solid_cuboid_inertia m="0.135" w="0.033" h="0.175" d="0.03" />
+        <!--inertia ixx="0.003881243" ixy="0.0" ixz="0.0"
                   iyy="0.000498940" iyz="0.0"
-                  izz="0.003879257" />
+                  izz="0.003879257" /-->
       </inertial>
     </link>

Commit message: added gazebo stereo cam plugin

File: urdf/zed.urdf.xacro (robot description, xacro)
@@ -1,37 +1,86 @@
 <?xml version="1.0"?>
-<robot name="sensor_zed" xmlns:xacro="http://wiki.ros.org/xacro">
-  <!-- Xacro properties -->
-  <xacro:property name="M_PI" value="3.1415926535897931" />
-  <xacro:macro name="sensor_zed" params="prefix parent prefix_topic:='front_rgbd_camera' *origin">
-    <joint name="${prefix}_rgb_joint" type="fixed">
-	    <xacro:insert_block name="origin" />
+<robot xmlns:xacro="http://wiki.ros.org/xacro">
+  <xacro:macro name="stereo_camera"
+    params="prefix fps baseline hfov width height format near far">
+    <gazebo reference="${prefix}_base_link">
+      <visual>
+        <material>
+          <ambient>0.35 0.35 0.35 1.0</ambient>
+          <diffuse>0.350754 0.350754 0.350754 1.0</diffuse>
+          <specular>0.308273 0.3508273 0.3508273 1.0</specular>
+          <emissive>0.0 0.0 0.0 0.0</emissive>
+        </material>
+      </visual>
+      <sensor type="multicamera" name="stereo_camera">
+        <update_rate>${fps}</update_rate>
+        <camera name="left">
+          <pose>0 0 0 0 0 0 </pose>
+          <horizontal_fov>${hfov}</horizontal_fov>
+          <image>
+            <width>${width}</width>
+            <height>${height}</height>
+            <format>${format}</format>
+          </image>
+          <clip>
+            <near>${near}</near>
+            <far>${far}</far>
+          </clip>
+          <noise>
+            <type>gaussian</type>
+            <mean>0.0</mean>
+            <stddev>0.007</stddev>
+          </noise>
+        </camera>
+        <camera name="right">
+          <pose>${baseline} 0 0 0 0 0</pose>
+          <horizontal_fov>${hfov}</horizontal_fov>
+          <image>
+            <width>${width}</width>
+            <height>${height}</height>
+            <format>${format}</format>
+          </image>
+          <clip>
+            <near>${near}</near>
+            <far>${far}</far>
+          </clip>
+          <noise>
+            <type>gaussian</type>
+            <mean>0.0</mean>
+            <stddev>0.007</stddev>
+          </noise>
+        </camera>
+        <plugin name="stereo_camera_controller" filename="libgazebo_ros_multicamera.so">
+          <alwaysOn>true</alwaysOn>
+          <cameraName>${prefix}</cameraName>
+          <imageTopicName>image_raw</imageTopicName>
+          <cameraInfoTopicName>camera_info</cameraInfoTopicName>
+          <frameName>${prefix}_base_link</frameName>
+          <hackBaseline>${baseline}</hackBaseline>
+          <!-- NOTE: Distortion is currently unused -->
+          <distortionK1>0.0</distortionK1>
+          <distortionK2>0.0</distortionK2>
+          <distortionK3>0.0</distortionK3>
+          <distortionT1>0.0</distortionT1>
+          <distortionT2>0.0</distortionT2>
+          <ignoreTfPrefix>1</ignoreTfPrefix>
+        </plugin>
+      </sensor>
+    </gazebo>
+  </xacro:macro>
+  <xacro:macro name="stereolabs_zed"
+    params="prefix:=zed parent *origin format:=R8G8B8 near:=0.05 far:=2500">
+    <joint name="${prefix}_base_joint" type="fixed">
+      <xacro:insert_block name="origin" />
       <parent link="${parent}"/>
-      <child link="${prefix}_rgb_base_link" />
+      <child link="${prefix}_base_link" />
     </joint>
-    <link name="${prefix}_rgb_base_link">
-      <inertial>
-        <mass value="0.135" />
-        <origin xyz="0 0 0" />
-        <xacro:solid_cuboid_inertia m="0.135" w="0.033" h="0.175" d="0.03" />
-        <!--inertia ixx="0.0001" ixy="0.0" ixz="0.0"
-          iyy="0.0001" iyz="0.0"
-          izz="0.0001" /-->
-      </inertial>
-    </link>
-    <!-- Camera center -->
-    <joint name="${prefix}_joint" type="fixed">
-      <origin xyz="0.0 0.0 0.0"
-              rpy="0.0 0.0 0.0"/>
-      <parent link="${prefix}_rgb_base_link"/>
-      <child link="${prefix}_link"/>
-    </joint>
-    <link name="${prefix}_link">
-      <visual>
+    <link name="${prefix}_base_link">
+       <visual>
         <origin xyz="0 0 0" rpy="0 0 0"/>
         <geometry>
           <mesh filename="package://robotnik_sensors/meshes/zed.stl"/>
         </geometry>
-        <material name="light_grey">
-          <color rgba="0.8 0.8 0.8 0.8"/>
+        <material name="light_zed_grey">
+          <color rgba="0.35 0.35 0.35 1"/>
         </material>
       </visual>
@@ -46,13 +95,10 @@
         <origin xyz="0 0 0" />
         <xacro:solid_cuboid_inertia m="0.135" w="0.033" h="0.175" d="0.03" />
-        <!--inertia ixx="0.003881243" ixy="0.0" ixz="0.0"
-                  iyy="0.000498940" iyz="0.0"
-                  izz="0.003879257" /-->
       </inertial>
     </link>
-    <!-- Left camera -->
+   <!-- Left camera -->
     <joint name="${prefix}_rgb_left_joint" type="fixed">
       <origin xyz="0.0 0.06 0.0" rpy="0.0 0.0 0.0" />
-      <parent link="${prefix}_link" />
+      <parent link="${prefix}_base_link" />
       <child link="${prefix}_left_rgb_frame" />
     </joint>
@@ -67,5 +113,5 @@
     <joint name="${prefix}_rgb_right_joint" type="fixed">
       <origin xyz="0.0 -0.06 0.0" rpy="0.0 0.0 0.0" />
-      <parent link="${prefix}_link" />
+      <parent link="${prefix}_base_link" />
       <child link="${prefix}_right_rgb_frame" />
     </joint>
@@ -77,5 +123,19 @@
     </joint>
     <link name="${prefix}_right_rgb_optical_frame"/>
-  <!-- TODO: simulation -->
+      <xacro:stereo_camera
+        prefix="${prefix}"
+        hfov="1.2217"
+        baseline="0.12"
+        fps="40"
+        width="640"
+        height="480"
+        format="${format}"
+        near="${near}"
+        far="${far}"/>
+  </xacro:macro>
+  <xacro:macro name="sensor_zed" params="prefix:=myzed parent *origin" >
+    <stereolabs_zed prefix="${prefix}" parent="${parent}">
+      <xacro:insert_block name="origin" />
+    </stereolabs_zed>
   </xacro:macro>
 </robot>

Commit message: added zed2 and zedm models

File: urdf/zed.urdf.xacro (robot description, xacro)
@@ -69,5 +69,14 @@
   </xacro:macro>
   <xacro:macro name="stereolabs_zed"
-    params="prefix:=zed parent *origin format:=R8G8B8 near:=0.05 far:=2500">
+    params="prefix:=zed parent *origin model:=zed format:=R8G8B8 near:=0.05 far:=2500">
+    <xacro:if value="${model == 'zed'}">
+        <xacro:property name="baseline" value="0.12" />
+    </xacro:if>
+    <xacro:if value="${model == 'zedm'}">
+        <xacro:property name="baseline" value="0.06" />
+    </xacro:if>
+    <xacro:if value="${model == 'zed2'}">
+        <xacro:property name="baseline" value="0.12" />
+    </xacro:if>
     <joint name="${prefix}_base_joint" type="fixed">
       <xacro:insert_block name="origin" />
@@ -79,5 +88,5 @@
         <origin xyz="0 0 0" rpy="0 0 0"/>
         <geometry>
-          <mesh filename="package://robotnik_sensors/meshes/zed.stl"/>
+          <mesh filename="package://robotnik_sensors/meshes/${model}.stl"/>
         </geometry>
         <material name="light_zed_grey">
@@ -88,5 +97,5 @@
         <origin xyz="0.0 0.0 0.0" rpy="0 0 0" />
         <geometry>
-          <mesh filename="package://robotnik_sensors/meshes/zed.stl" />
+          <mesh filename="package://robotnik_sensors/meshes/${model}.stl" />
         </geometry>
       </collision>
@@ -126,5 +135,5 @@
         prefix="${prefix}"
         hfov="1.2217"
-        baseline="0.12"
+        baseline="${baseline}"
         fps="40"
         width="640"
@@ -134,6 +143,6 @@
         far="${far}"/>
   </xacro:macro>
-  <xacro:macro name="sensor_zed" params="prefix:=myzed parent *origin" >
-    <stereolabs_zed prefix="${prefix}" parent="${parent}">
+  <xacro:macro name="sensor_zed" params="prefix:=myzed parent *origin model:=zed" >
+    <stereolabs_zed prefix="${prefix}" parent="${parent}" model="${model}">
       <xacro:insert_block name="origin" />
     </stereolabs_zed>

Commit message: Update Zed model - Naming of the links didn't fit the ones published by the driver

File: urdf/zed.urdf.xacro (robot description, xacro)
@@ -1,79 +1,88 @@
 <?xml version="1.0"?>
 <robot name="sensor_zed" xmlns:xacro="http://wiki.ros.org/xacro">
-  <!-- Xacro properties -->
-  <xacro:property name="M_PI" value="3.1415926535897931" />
-  <xacro:macro name="sensor_zed" params="prefix parent prefix_topic:='front_rgbd_camera' *origin">
-    <joint name="${prefix}_rgb_joint" type="fixed">
-	    <xacro:insert_block name="origin" />
-      <parent link="${parent}"/>
-      <child link="${prefix}_rgb_base_link" />
+	<!-- Xacro properties -->
+	<xacro:property name="M_PI" value="3.1415926535897931" />
+  <xacro:macro name="sensor_zed" params="prefix parent prefix_topic:='front_rgbd_camera' *origin camera_model:='zed'">
+	<xacro:if value="${camera_model == 'zed'}">
+        <xacro:property name="baseline" value="0.12" />
+    </xacro:if>
+    <xacro:if value="${camera_model == 'zedm'}">
+		<xacro:property name="baseline" value="0.06" />
+    </xacro:if>
+	<xacro:if value="${camera_model == 'zed2'}">
+		<xacro:property name="baseline" value="0.12" />
+	</xacro:if>
+    <joint name="${prefix}_camera_center_joint" type="fixed">
+        <parent link="${parent}"/>
+        <child link="${prefix}_camera_center"/>
+        <xacro:insert_block name="origin" />
     </joint>
-    <link name="${prefix}_rgb_base_link">
-      <inertial>
-        <mass value="0.001" />
-        <origin xyz="0 0 0" />
-        <inertia ixx="0.0001" ixy="0.0" ixz="0.0"
-          iyy="0.0001" iyz="0.0"
-          izz="0.0001" />
-      </inertial>
+    <link name="${prefix}_camera_center">
+        <visual>
+            <origin xyz="0 0 0" rpy="0 0 0"/>
+            <geometry>
+                <mesh filename="package://robotnik_sensors/meshes/${camera_model}.stl"/>
+            </geometry>
+        </visual>
+        <collision>
+			<origin xyz="0.0 0.0 0.0" rpy="0 0 0" />
+			<geometry>
+			  <mesh filename="package://robotnik_sensors/meshes/${camera_model}.stl"/>
+			</geometry>
+      </collision>
     </link>
-    <!-- Camera center -->
-    <joint name="${prefix}_joint" type="fixed">
-      <origin xyz="0.0 0.0 0.0"
-              rpy="0.0 0.0 0.0"/>
-      <parent link="${prefix}_rgb_base_link"/>
-      <child link="${prefix}_link"/>
+	<!-- Left Camera -->
+    <joint name="${prefix}_left_camera_joint" type="fixed">
+        <parent link="${prefix}_camera_center"/>
+        <child link="${prefix}_left_camera_frame"/>
+        <origin xyz="0 ${baseline/2} 0" rpy="0 0 0" />
     </joint>
-    <link name="${prefix}_link">
-      <visual>
-        <origin xyz="0 0 0" rpy="0 0 0"/>
-        <geometry>
-          <mesh filename="package://robotnik_sensors/meshes/zed.stl"/>
-        </geometry>
-        <material name="light_grey">
-          <color rgba="0.8 0.8 0.8 0.8"/>
-        </material>
-      </visual>
-      <collision>
-        <origin xyz="0.0 0.0 0.0" rpy="0 0 0" />
-        <geometry>
-          <mesh filename="package://robotnik_sensors/meshes/zed.stl" />
-        </geometry>
-      </collision>
-      <inertial>
-        <mass value="0.564" />
-        <origin xyz="0 0 0" />
-        <inertia ixx="0.003881243" ixy="0.0" ixz="0.0"
-                  iyy="0.000498940" iyz="0.0"
-                  izz="0.003879257" />
-      </inertial>
-    </link>
-    <!-- Left camera -->
-    <joint name="${prefix}_rgb_left_joint" type="fixed">
-      <origin xyz="0.0 0.06 0.0" rpy="0.0 0.0 0.0" />
-      <parent link="${prefix}_link" />
-      <child link="${prefix}_left_rgb_frame" />
+    <link name="${prefix}_left_camera_frame" />
+    <joint name="${prefix}_left_camera_optical_joint" type="fixed">
+        <origin xyz="0 0 0" rpy="-${M_PI/2} 0.0 -${M_PI/2}"/>
+        <parent link="${prefix}_left_camera_frame"/>
+        <child link="${prefix}_left_camera_optical_frame"/>
     </joint>
-    <link name="${prefix}_left_rgb_frame"/>
-    <joint name="${prefix}_rgb_left_optical_joint" type="fixed">
-      <origin xyz="0.0 0.0 0.0" rpy="${-M_PI/2} 0.0 ${-M_PI/2}" />
-      <parent link="${prefix}_left_rgb_frame" />
-      <child link="${prefix}_left_rgb_optical_frame" />
+    <link name="${prefix}_left_camera_optical_frame"/>
+	<!-- Right Camera -->
+    <joint name="${prefix}_right_camera_joint" type="fixed">
+        <parent link="${prefix}_camera_center"/>
+        <child link="${prefix}_right_camera_frame"/>
+        <origin xyz="0 -${baseline/2} 0" rpy="0 0 0" />
     </joint>
-    <link name="${prefix}_left_rgb_optical_frame"/>
-    <!-- Right camera-->
-    <joint name="${prefix}_rgb_right_joint" type="fixed">
-      <origin xyz="0.0 -0.06 0.0" rpy="0.0 0.0 0.0" />
-      <parent link="${prefix}_link" />
-      <child link="${prefix}_right_rgb_frame" />
+    <link name="${prefix}_right_camera_frame" />
+    <joint name="${prefix}_right_camera_optical_joint" type="fixed">
+        <origin xyz="0 0 0" rpy="-${M_PI/2} 0.0 -${M_PI/2}"/>
+        <parent link="${prefix}_right_camera_frame"/>
+        <child link="${prefix}_right_camera_optical_frame"/>
     </joint>
-    <link name="${prefix}_right_rgb_frame"/>
-    <joint name="${prefix}_rgb_right_optical_joint" type="fixed">
-      <origin xyz="0.0 0 0.0" rpy="${-M_PI/2} 0.0 ${-M_PI/2}" />
-      <parent link="${prefix}_right_rgb_frame" />
-      <child link="${prefix}_right_rgb_optical_frame" />
-    </joint>
-    <link name="${prefix}_right_rgb_optical_frame"/>
-  <!-- TODO: simulation -->
+    <link name="${prefix}_right_camera_optical_frame"/>
+	<!-- ZED2 Sensors -->
+    <xacro:if value="${camera_model == 'zed2'}">
+        <joint name="${prefix}_mag_joint" type="fixed">
+            <parent link="${prefix}_camera_center"/>
+            <child link="${prefix}_mag_link"/>
+            <origin xyz="0 0 0" rpy="0 0 0" />
+        </joint>
+        <link name="${prefix}_mag_link" />
+        <joint name="${prefix}_baro_joint" type="fixed">
+            <parent link="${prefix}_camera_center"/>
+            <child link="${prefix}_baro_link"/>
+            <origin xyz="0 0 0" rpy="0 0 0" />
+        </joint>
+        <link name="${prefix}_baro_link" />
+        <joint name="${prefix}_temp_left_joint" type="fixed">
+            <parent link="${prefix}_left_camera_frame"/>
+            <child link="${prefix}_temp_left_link"/>
+            <origin xyz="0 0 0" rpy="0 0 0" />
+        </joint>
+        <link name="${prefix}_temp_left_link" />
+        <joint name="${prefix}_temp_right_joint" type="fixed">
+            <parent link="${prefix}_right_camera_frame"/>
+            <child link="${prefix}_temp_right_link"/>
+            <origin xyz="0 0 0" rpy="0 0 0" />
+        </joint>
+        <link name="${prefix}_temp_right_link" />
+    </xacro:if>
   </xacro:macro>
 </robot>

Commit message: update zed urdf to be closer to the zed package urdf

File: urdf/zed.urdf.xacro (robot description, xacro)
@@ -106,30 +106,37 @@
       </inertial>
     </link>
+   <!-- Center camera -->
+   <joint name="${prefix}_camera_center_joint" type="fixed">
+        <parent link="${prefix}_base_link"/>
+        <child link="${prefix}_camera_center"/>
+        <origin xyz="0.0 0.0 0.0" rpy="0.0 0.0 0.0" />
+    </joint>
+   <link name="${prefix}_camera_center"/>
    <!-- Left camera -->
-    <joint name="${prefix}_rgb_left_joint" type="fixed">
-      <origin xyz="0.0 0.06 0.0" rpy="0.0 0.0 0.0" />
-      <parent link="${prefix}_base_link" />
-      <child link="${prefix}_left_rgb_frame" />
+    <joint name="${prefix}_camera_left_joint" type="fixed">
+        <origin xyz="0 ${baseline/2} 0" rpy="0 0 0" />
+      <parent link="${prefix}_camera_center" />
+      <child link="${prefix}_left_camera_frame" />
     </joint>
-    <link name="${prefix}_left_rgb_frame"/>
-    <joint name="${prefix}_rgb_left_optical_joint" type="fixed">
+    <link name="${prefix}_left_camera_frame"/>
+    <joint name="${prefix}_camera_left_optical_joint" type="fixed">
       <origin xyz="0.0 0.0 0.0" rpy="${-M_PI/2} 0.0 ${-M_PI/2}" />
-      <parent link="${prefix}_left_rgb_frame" />
-      <child link="${prefix}_left_rgb_optical_frame" />
+      <parent link="${prefix}_left_camera_frame" />
+      <child link="${prefix}_left_camera_optical_frame" />
     </joint>
-    <link name="${prefix}_left_rgb_optical_frame"/>
+    <link name="${prefix}_left_camera_optical_frame"/>
     <!-- Right camera-->
-    <joint name="${prefix}_rgb_right_joint" type="fixed">
-      <origin xyz="0.0 -0.06 0.0" rpy="0.0 0.0 0.0" />
-      <parent link="${prefix}_base_link" />
-      <child link="${prefix}_right_rgb_frame" />
+    <joint name="${prefix}_camera_right_joint" type="fixed">
+      <origin xyz="0 -${baseline/2} 0" rpy="0 0 0" />
+      <parent link="${prefix}_camera_center" />
+      <child link="${prefix}_right_camera_frame" />
     </joint>
-    <link name="${prefix}_right_rgb_frame"/>
-    <joint name="${prefix}_rgb_right_optical_joint" type="fixed">
+    <link name="${prefix}_right_camera_frame"/>
+    <joint name="${prefix}_camera_right_optical_joint" type="fixed">
       <origin xyz="0.0 0 0.0" rpy="${-M_PI/2} 0.0 ${-M_PI/2}" />
-      <parent link="${prefix}_right_rgb_frame" />
-      <child link="${prefix}_right_rgb_optical_frame" />
+      <parent link="${prefix}_right_camera_frame" />
+      <child link="${prefix}_right_camera_optical_frame" />
     </joint>
-    <link name="${prefix}_right_rgb_optical_frame"/>
+    <link name="${prefix}_right_camera_optical_frame"/>
       <xacro:stereo_camera
         prefix="${prefix}"
