Commit message: Add outdoorscan3 stl and dae

File: urdf/sick_outdoorscan3.urdf.xacro (robot description, xacro)
@@ -14,5 +14,5 @@
 					<!--<box size="0.106 0.094 0.152"/>-->
 					<!--<cylinder radius="0.058" length="0.152"/>-->
-					<mesh filename="package://robotnik_sensors/meshes/sick_microscan3.dae"/>
+					<mesh filename="package://robotnik_sensors/meshes/sick_outdoorscan3.dae"/>
 				</geometry>
 			</collision>
@@ -20,5 +20,5 @@
 				<origin xyz="0 0 0" rpy="0 0 0"/>
 				<geometry>
-					<mesh filename="package://robotnik_sensors/meshes/sick_microscan3.dae"/>
+					<mesh filename="package://robotnik_sensors/meshes/sick_outdoorscan3.dae"/>
 				</geometry>
 			</visual>
