Commit message: collision model of sick s300 corrected

File: urdf/sick_s300.urdf.xacro (robot description, xacro)
@@ -9,5 +9,5 @@
 	<link name="${prefix}_base_link">
 		<collision>
-			<origin xyz="0 0 0.076" rpy="0 0 0"/>
+			<origin xyz="0 0 0" rpy="0 0 0"/>
 			<geometry>
 				<!--<box size="0.106 0.094 0.152"/>-->

Commit message: sick s300 has configurable min and max angles

File: urdf/sick_s300.urdf.xacro (robot description, xacro)
@@ -1,5 +1,5 @@
 <?xml version="1.0"?>
 <robot name="sensor_sick_s300" xmlns:xacro="http://wiki.ros.org/xacro">
-  <xacro:macro name="sensor_sick_s300" params="prefix parent prefix_topic:='front_laser' *origin">
+  <xacro:macro name="sensor_sick_s300" params="prefix parent prefix_topic:='front_laser' *origin min_angle:=-2.3562 max_angle:=2.3562">
     <joint name="${prefix}_base_joint" type="fixed">
       <xacro:insert_block name="origin" />
@@ -48,6 +48,6 @@
 							<samples>541</samples>
 							<resolution>1</resolution>
-							<min_angle>-2.3562</min_angle>
-							<max_angle>2.3562</max_angle>
+							<min_angle>${min_angle}</min_angle>
+							<max_angle>${max_angle}</max_angle>
 						</horizontal>
 					</scan>

Commit message: sick_s300.urdf.xacro: added inertia values that fits better the shape of the sensor
+ changed joint type to revolute with upper and down limits equal to 0

File: urdf/sick_s300.urdf.xacro (robot description, xacro)
@@ -2,8 +2,9 @@
 <robot name="sensor_sick_s300" xmlns:xacro="http://wiki.ros.org/xacro">
   <xacro:macro name="sensor_sick_s300" params="prefix parent prefix_topic:='front_laser' *origin min_angle:=-2.3562 max_angle:=2.3562 gpu:=^|true">
-    <joint name="${prefix}_base_joint" type="fixed">
+    <joint name="${prefix}_base_joint" type="revolute">
       <xacro:insert_block name="origin" />
       <parent link="${parent}"/>
       <child link="${prefix}_base_link"/>
+      <limit effort="100" velocity="100" lower="0.0" upper="0.0"/>
 	</joint>
 	<link name="${prefix}_base_link">
@@ -22,8 +23,13 @@
 			</geometry>
 		</visual>
-		<inertial>
+		<!--inertial>
 			<mass value="1e-5" />
 			<origin xyz="0 0 0" rpy="0 0 0"/>
 			<inertia ixx="1e-6" ixy="0" ixz="0" iyy="1e-6" iyz="0" izz="1e-6" />
+		</inertial-->
+		<inertial>
+			<mass value="0.1" />
+			<origin xyz="0 0 0" rpy="0 0 0"/>
+			<inertia ixx="0.0002708333" ixy="0" ixz="0" iyy="0.0002708333" iyz="0" izz="0.00009434" />
 		</inertial>
 	</link>
@@ -34,4 +40,14 @@
 	</joint>
 	<link name="${prefix}_link" />
+	<transmission name="${prefix}_base_trans">
+      <type>transmission_interface/SimpleTransmission</type>
+      <joint name="${prefix}_base_joint">
+        <hardwareInterface>hardware_interface/VelocityJointInterface</hardwareInterface>
+      </joint>
+      <actuator name="sick_motor">
+        <hardwareInterface>hardware_interface/VelocityJointInterface</hardwareInterface>
+        <mechanicalReduction>${ptz_mechanical_reduction}</mechanicalReduction>
+      </actuator>
+    </transmission>
 	<!-- Sick sensor sensor for simulation -->
 	<sensor_sick_s300_gazebo />

Commit message: sick_s300: switch back joint to fixed
it was causing problems with moveit. joint was simulated, small
move happened and joint went off limits.

File: urdf/sick_s300.urdf.xacro (robot description, xacro)
@@ -2,5 +2,5 @@
 <robot name="sensor_sick_s300" xmlns:xacro="http://wiki.ros.org/xacro">
   <xacro:macro name="sensor_sick_s300" params="prefix parent prefix_topic:='front_laser' *origin min_angle:=-2.3562 max_angle:=2.3562 gpu:=^|true">
-    <joint name="${prefix}_base_joint" type="revolute">
+    <joint name="${prefix}_base_joint" type="fixed">
       <xacro:insert_block name="origin" />
       <parent link="${parent}"/>
@@ -40,14 +40,4 @@
 	</joint>
 	<link name="${prefix}_link" />
-	<transmission name="${prefix}_base_trans">
-      <type>transmission_interface/SimpleTransmission</type>
-      <joint name="${prefix}_base_joint">
-        <hardwareInterface>hardware_interface/VelocityJointInterface</hardwareInterface>
-      </joint>
-      <actuator name="sick_motor">
-        <hardwareInterface>hardware_interface/VelocityJointInterface</hardwareInterface>
-        <mechanicalReduction>${ptz_mechanical_reduction}</mechanicalReduction>
-      </actuator>
-    </transmission>
 	<!-- Sick sensor sensor for simulation -->
 	<sensor_sick_s300_gazebo />

Commit message: Fix sick s300 inertia

File: urdf/sick_s300.urdf.xacro (robot description, xacro)
@@ -29,7 +29,8 @@
 		</inertial-->
 		<inertial>
-			<mass value="0.1" />
-			<origin xyz="0 0 0" rpy="0 0 0"/>
-			<inertia ixx="0.0002708333" ixy="0" ixz="0" iyy="0.0002708333" iyz="0" izz="0.00009434" />
+			<mass value="1.2" />
+			<origin xyz="0 0.0 0.0751" rpy="0 0 0"/>
+            <xacro:solid_cuboid_inertia m="1.2" w="0.102" h="0.106" d="0.152" />
+			<!--inertia ixx="0.0002708333" ixy="0" ixz="0" iyy="0.0002708333" iyz="0" izz="0.00009434" /-->
 		</inertial>
 	</link>

Commit message: sick_s300 fixed joint instead of revolute

File: urdf/sick_s300.urdf.xacro (robot description, xacro)
@@ -2,9 +2,8 @@
 <robot name="sensor_sick_s300" xmlns:xacro="http://wiki.ros.org/xacro">
   <xacro:macro name="sensor_sick_s300" params="prefix parent prefix_topic:='front_laser' *origin min_angle:=-2.3562 max_angle:=2.3562 gpu:=^|true">
-    <joint name="${prefix}_base_joint" type="revolute">
+    <joint name="${prefix}_base_joint" type="fixed">
       <xacro:insert_block name="origin" />
       <parent link="${parent}"/>
       <child link="${prefix}_base_link"/>
-      <limit effort="100" velocity="100" lower="0.0" upper="0.0"/>
 	</joint>
 	<link name="${prefix}_base_link">
@@ -40,14 +39,4 @@
 	</joint>
 	<link name="${prefix}_link" />
-	<transmission name="${prefix}_base_trans">
-      <type>transmission_interface/SimpleTransmission</type>
-      <joint name="${prefix}_base_joint">
-        <hardwareInterface>hardware_interface/VelocityJointInterface</hardwareInterface>
-      </joint>
-      <actuator name="sick_motor">
-        <hardwareInterface>hardware_interface/VelocityJointInterface</hardwareInterface>
-        <mechanicalReduction>${ptz_mechanical_reduction}</mechanicalReduction>
-      </actuator>
-    </transmission>
 	<!-- Sick sensor sensor for simulation -->
 	<sensor_sick_s300_gazebo />

Commit message: Added gazebo models and paint sick_s300

File: urdf/sick_s300.urdf.xacro (robot description, xacro)
@@ -1,5 +1,12 @@
 <?xml version="1.0"?>
 <robot name="sensor_sick_s300" xmlns:xacro="http://wiki.ros.org/xacro">
-  <xacro:macro name="sensor_sick_s300" params="prefix parent prefix_topic:='front_laser' *origin min_angle:=-2.3562 max_angle:=2.3562 gpu:=^|true">
+  <xacro:macro name="sensor_sick_s300"
+               params="prefix
+			           parent
+					   prefix_topic:='front_laser'
+					   *origin
+					   min_angle:=-2.3562
+					   max_angle:=2.3562
+					   gpu:=^|true">
     <joint name="${prefix}_base_joint" type="fixed">
       <xacro:insert_block name="origin" />
@@ -18,19 +25,13 @@
 		</collision>
 		<visual>
-			<origin xyz="0 0 0" rpy="0 0 0"/>
+			<origin xyz="0 0 0" rpy="${-M_PI/2} 0 0"/>
 			<geometry>
-	     		<mesh filename="package://robotnik_sensors/meshes/sick_s300.dae"/>
+	     		<mesh filename="package://robotnik_sensors/meshes/sick_s300_color.dae"/>
 			</geometry>
 		</visual>
-		<!--inertial>
-			<mass value="1e-5" />
-			<origin xyz="0 0 0" rpy="0 0 0"/>
-			<inertia ixx="1e-6" ixy="0" ixz="0" iyy="1e-6" iyz="0" izz="1e-6" />
-		</inertial-->
 		<inertial>
 			<mass value="1.2" />
 			<origin xyz="0 0.0 0.0751" rpy="0 0 0"/>
             <xacro:solid_cuboid_inertia m="1.2" w="0.102" h="0.106" d="0.152" />
-			<!--inertia ixx="0.0002708333" ixy="0" ixz="0" iyy="0.0002708333" iyz="0" izz="0.00009434" /-->
 		</inertial>
 	</link>
@@ -78,7 +79,11 @@
 				</noise>
 			</ray>
-			<plugin name="${prefix}_controller" filename="${plugin_lib}">
-				<topicName>${prefix_topic}/scan</topicName>
-				<frameName>/${prefix}_link</frameName><!-- if not global (leading /) sets the current namespace as a prefix (/ns/name_laser_link) -->
+			<plugin name="${prefix}_controller" filename="libgazebo_ros_ray_sensor.so">
+				<ros>
+				  <remapping>~/out:=${prefix_topic}/scan</remapping>
+				</ros>
+				<!-- when leaving away frame_name it defaults to base_footprint instead-->
+				<frame_name>${prefix}_link</frame_name>
+				<output_type>sensor_msgs/LaserScan</output_type>
 			</plugin>
 		</sensor>

File: urdf/vectornav.urdf.xacro (robot description, xacro)
@@ -112,7 +112,7 @@
 			<plugin name="${prefix}imu_controller" filename="libgazebo_ros_imu_sensor.so">
 				<initial_orientation_as_reference>false</initial_orientation_as_reference>
-				<frame_name>${prefix}imu_link</frame_name>
+				<frame_name>${prefix}</frame_name>
 				<ros>
-					<remapping>~/out:=imu/data</remapping>
+					<remapping>~/out:=${topic}</remapping>
 				</ros>
 			</plugin>
