Commit message: intel_d435 updated to run in gazebo

File: urdf/intel_d435.urdf.xacro (robot description, xacro)
@@ -12,7 +12,5 @@
   <xacro:property name="r430_cam_width" value="0.105"/>
   <xacro:property name="r430_cam_depth" value="0.019"/>
-  <!-- xacro:property name="r430_cam_height" value="0.039"/>
-  <xacro:property name="r430_cam_mount_from_center_offset" value=".0275"/ -->
-  <xacro:property name="r430_cam_height" value="0.0"/>
+  <xacro:property name="r430_cam_height" value="0.020"/>
   <xacro:property name="r430_cam_mount_from_center_offset" value="0.0"/>
   <!-- The following offset is relative the the physical R430 camera peripherial
@@ -34,5 +32,5 @@
       <visual>
       <!-- origin xyz="0 ${-r430_cam_mount_from_center_offset} ${r430_cam_height/2}" rpy="${M_PI/2} 0 ${M_PI/2}"/ -->
-      <origin xyz="0 ${-r430_cam_mount_from_center_offset} ${r430_cam_height/2}" rpy="0 0 0"/>
+      <origin xyz="0 ${-r430_cam_mount_from_center_offset} 0" rpy="0 0 0"/>
         <geometry>
           <!-- box size="${r430_cam_width} ${r430_cam_height} ${r430_cam_depth}"/ -->
@@ -110,10 +108,11 @@
   </xacro:macro>
    <xacro:macro name="sensor_r430_gazebo">
-    <gazebo reference="${prefix}_rgb_base_link">
+    <!-- gazebo reference="${prefix}_rgb_base_link" -->
+    <gazebo reference="${prefix}_camera_link">
       <sensor type="depth" name="${prefix}_depth_sensor">
         <always_on>true</always_on>
-        <update_rate>20.0</update_rate>
+        <update_rate>15.0</update_rate>
         <camera>
-          <horizontal_fov>${60.0*M_PI/180.0}</horizontal_fov>
+          <horizontal_fov>${91.2*M_PI/180.0}</horizontal_fov>
           <image>
             <format>R8G8B8</format>
@@ -135,5 +134,5 @@
           <cameraInfoTopicName>rgb/camera_info</cameraInfoTopicName>
           <depthImageCameraInfoTopicName>depth/camera_info</depthImageCameraInfoTopicName>
-          <frameName>/${prefix}_depth_optical_frame</frameName>
+          <frameName>/${prefix}_camera_depth_optical_frame</frameName>
           <baseline>0.1</baseline>
           <distortion_k1>0.0</distortion_k1>

Commit message: corrected collision box d435

File: urdf/intel_d435.urdf.xacro (robot description, xacro)
@@ -10,7 +10,7 @@
     R430 camera, with the camera joint represented by the actual
     peripherial camera tripod mount -->
-  <xacro:property name="r430_cam_width" value="0.105"/>
-  <xacro:property name="r430_cam_depth" value="0.019"/>
-  <xacro:property name="r430_cam_height" value="0.020"/>
+  <xacro:property name="r430_cam_width" value="0.100"/>
+  <xacro:property name="r430_cam_depth" value="0.025"/>
+  <xacro:property name="r430_cam_height" value="0.025"/>
   <xacro:property name="r430_cam_mount_from_center_offset" value="0.0"/>
   <!-- The following offset is relative the the physical R430 camera peripherial
@@ -40,5 +40,5 @@
       </visual>
       <collision>
-        <origin xyz="0.0 0.0 ${r430_cam_height/2}" rpy="0 0 0"/>
+        <origin xyz="${-r430_cam_depth/2} 0.0 0.0" rpy="0 0 0"/>
         <geometry>
         <box size="${r430_cam_depth} ${r430_cam_width} ${r430_cam_height}"/>
@@ -121,6 +121,6 @@
           </image>
           <clip>
-            <near>0.05</near>
-            <far>3.5</far>
+            <near>0.3</near>
+            <far>10.0</far>
           </clip>
         </camera>

Commit message: Define aluminum material in place to avoid duplicate declarations

File: urdf/intel_d435.urdf.xacro (robot description, xacro)
@@ -19,7 +19,4 @@
   <xacro:property name="r430_cam_depth_py" value="-0.0115"/>
   <xacro:property name="r430_cam_depth_pz" value="0.0"/>
-  <material name="aluminum">
-    <color rgba="0.5 0.5 0.5 1"/>
-  </material>
   <xacro:macro name="sensor_r430" params="prefix parent prefix_topic:='front_rgbd_camera' *origin">
     <!-- camera body, with origin at bottom screw mount -->
@@ -37,5 +34,7 @@
           <mesh filename="package://robotnik_sensors/meshes/intel_realsense_depth_camera_d435.dae" />
         </geometry>
-        <material name="aluminum"/>
+        <material name="aluminum">
+          <color rgba="0.5 0.5 0.5 1"/>
+        </material>
       </visual>
       <collision>

Commit message: corrected positioning of intel d435

File: urdf/intel_d435.urdf.xacro (robot description, xacro)
@@ -28,4 +28,5 @@
     <xacro:property name="d435_cam_depth_pz" value="${d435_cam_height/2}"/>
     <joint name="${prefix}_base_joint" type="fixed">
+      <xacro:insert_block name="origin" />
       <parent link="${parent}"/>
       <child link="${prefix}_base_link" />
@@ -34,15 +35,10 @@
     <!-- camera body, with origin at bottom screw mount -->
     <joint name="${prefix}_joint" type="fixed">
-      <xacro:insert_block name="origin" />
       <parent link="${prefix}_base_link" />
-      <child link="${prefix}_bottom_screw_frame" />
-    </joint>
-    <link name="${prefix}_bottom_screw_frame"/>
-    <joint name="${prefix}_link_joint" type="fixed">
-      <origin xyz="0 ${d435_cam_depth_py} ${d435_cam_depth_pz}" rpy="0 0 0"/>
-      <parent link="${prefix}_bottom_screw_frame"/>
+      <child link="${prefix}_link" />
+      <origin xyz="0.01 0.02 0" rpy="0 0 0"/>
       <child link="${prefix}_link" />
     </joint>
-    <link name="${prefix}_link">
+    <link name="${prefix}_link"> <!-- camera link is aligned with the infrared sensor 1 that is "in the middle of the camera", not the one in the edge -->
       <visual>
         <origin xyz="${d435_cam_mount_from_center_offset} ${-d435_cam_depth_py} 0" rpy="${M_PI/2} 0 ${M_PI/2}"/>

Commit message: updated intel mesh

File: urdf/intel_d435.urdf.xacro (robot description, xacro)
@@ -45,5 +45,5 @@
         <geometry>
           <!-- <box size="${d435_cam_width} ${d435_cam_height} ${d435_cam_depth}"/> -->
-          <mesh filename="package://realsense2_description/meshes/d435.dae" />
+	  <mesh filename="package://robotnik_sensors/meshes/intel_d435.dae" />
         </geometry>
       </visual>

Commit message: intel_d435.urdf.xacro corrected possition of inertia

File: urdf/intel_d435.urdf.xacro (robot description, xacro)
@@ -57,5 +57,5 @@
         <!-- The following are not reliable values, and should not be used for modeling -->
         <mass value="0.564" />
-        <origin xyz="0 0 0" />
+        <origin xyz="-0.01 -0.02 0" />
         <inertia ixx="0.003881243" ixy="0.0" ixz="0.0" iyy="0.000498940" iyz="0.0" izz="0.003879257" />
       </inertial>

Commit message: Update intel_d435 inertia

File: urdf/intel_d435.urdf.xacro (robot description, xacro)
@@ -45,5 +45,5 @@
         <geometry>
           <!-- <box size="${d435_cam_width} ${d435_cam_height} ${d435_cam_depth}"/> -->
-	  <mesh filename="package://robotnik_sensors/meshes/intel_d435.dae" />
+          <mesh filename="package://robotnik_sensors/meshes/intel_d435.dae" />
         </geometry>
       </visual>
@@ -55,8 +55,7 @@
       </collision>
       <inertial>
-        <!-- The following are not reliable values, and should not be used for modeling -->
-        <mass value="0.564" />
-        <origin xyz="-0.01 -0.02 0" />
-        <inertia ixx="0.003881243" ixy="0.0" ixz="0.0" iyy="0.000498940" iyz="0.0" izz="0.003879257" />
+        <origin xyz="0.0025 -0.015 0.0" rpy="0 0 0" />
+        <mass value="0.1" />
+        <xacro:solid_cuboid_inertia m="0.1" w="0.025" h="0.09" d="0.025" />
       </inertial>
     </link>

Commit message: Intel d435 publish under namespace, accept arg update_rate for depth&image

File: urdf/intel_d435.urdf.xacro (robot description, xacro)
@@ -8,5 +8,5 @@
   xmlns:xacro="http://wiki.ros.org/xacro">
   <!-- Includes -->
-  <xacro:macro name="sensor_intel_d435" params="prefix parent *origin prefix_topic:='front_rgbd_camera' use_nominal_extrinsics:=false">
+  <xacro:macro name="sensor_intel_d435" params="prefix parent *origin prefix_topic:='front_rgbd_camera' use_nominal_extrinsics:=true update_rate:=7">
     <xacro:property name="M_PI" value="3.1415926535897931" />
     <!-- The following values are approximate, and the camera node
@@ -115,7 +115,7 @@
       <link name="${prefix}_color_optical_frame"/>
     </xacro:if>
-    <xacro:gazebo_d435 camera_name="${prefix}" reference_link="${prefix}_link" topics_ns="${prefix_topic}" depth_optical_frame="${prefix}_depth_optical_frame" color_optical_frame="${prefix}_color_optical_frame" infrared1_optical_frame="${prefix}_left_ir_optical_frame" infrared2_optical_frame="${prefix}_right_ir_optical_frame"/>
+    <xacro:gazebo_d435 update_rate="${update_rate}" camera_name="${prefix}" reference_link="${prefix}_link" topics_ns="${prefix_topic}" depth_optical_frame="${prefix}_depth_optical_frame" color_optical_frame="${prefix}_color_optical_frame" infrared1_optical_frame="${prefix}_left_ir_optical_frame" infrared2_optical_frame="${prefix}_right_ir_optical_frame"/>
   </xacro:macro>
-  <xacro:macro name="gazebo_d435" params="camera_name reference_link topics_ns depth_optical_frame color_optical_frame infrared1_optical_frame infrared2_optical_frame" >
+  <xacro:macro name="gazebo_d435" params="camera_name reference_link topics_ns depth_optical_frame color_optical_frame infrared1_optical_frame infrared2_optical_frame update_rate" >
    <!-- Load parameters to model's main link-->
    <xacro:property name="deg_to_rad" value="0.01745329251994329577" />
@@ -153,12 +153,12 @@
        </camera>
        <always_on>1</always_on>
-       <update_rate>30</update_rate>
+       <update_rate>${update_rate}</update_rate>
        <visualize>1</visualize>
        <plugin name="${prefix}kortex_vision_controller" filename="libgazebo_ros_camera.so">
           <alwaysOn>true</alwaysOn>
-          <updateRate>30.0</updateRate>
-          <cameraName>${prefix_topic}/color</cameraName>
-          <imageTopicName>image_raw</imageTopicName>
-          <cameraInfoTopicName>camera_info</cameraInfoTopicName>
+          <updateRate>${update_rate}</updateRate>
+          <cameraName>${camera_name}_color</cameraName>
+          <imageTopicName>${prefix_topic}/color/image_raw</imageTopicName>
+          <cameraInfoTopicName>${prefix_topic}/camera_info</cameraInfoTopicName>
           <frameName>/${prefix}_color_optical_frame</frameName>
           <!-- this is just which name the Image msg will have, it does not affect the simulation.
@@ -192,5 +192,5 @@
        </camera>
        <always_on>1</always_on>
-       <update_rate>90</update_rate>
+       <update_rate>${update_rate}</update_rate>
        <visualize>0</visualize>
      </sensor>
@@ -214,5 +214,5 @@
        </camera>
        <always_on>1</always_on>
-       <update_rate>90</update_rate>
+       <update_rate>${update_rate}</update_rate>
        <visualize>0</visualize>
      </sensor>
@@ -235,31 +235,31 @@
        </camera>
        <always_on>1</always_on>
-       <update_rate>90</update_rate>
+       <update_rate>${update_rate}</update_rate>
        <visualize>0</visualize>
      </sensor>
    </gazebo>
    <gazebo>
-     <plugin name="${topics_ns}" filename="librealsense_gazebo_plugin.so">
+     <plugin name="${camera_name}_controller" filename="librealsense_gazebo_plugin.so">
        <prefix>${camera_name}</prefix>
-       <depthUpdateRate>60.0</depthUpdateRate>
-       <colorUpdateRate>60.0</colorUpdateRate>
-       <infraredUpdateRate>60.0</infraredUpdateRate>
-       <depthTopicName>depth/image_raw</depthTopicName>
-       <depthCameraInfoTopicName>depth/camera_info</depthCameraInfoTopicName>
-       <colorTopicName>color/image_raw</colorTopicName>
-       <colorCameraInfoTopicName>color/camera_info</colorCameraInfoTopicName>
-       <infrared1TopicName>infra1/image_raw</infrared1TopicName>
-       <infrared1CameraInfoTopicName>infra1/camera_info</infrared1CameraInfoTopicName>
-       <infrared2TopicName>infra2/image_raw</infrared2TopicName>
-       <infrared2CameraInfoTopicName>infra2/camera_info</infrared2CameraInfoTopicName>
+       <depthUpdateRate>${update_rate}</depthUpdateRate>
+       <colorUpdateRate>${update_rate}</colorUpdateRate>
+       <infraredUpdateRate>${update_rate}</infraredUpdateRate>
+       <depthTopicName>${prefix_topic}/depth/image_raw</depthTopicName>
+       <depthCameraInfoTopicName>${prefix_topic}/depth/camera_info</depthCameraInfoTopicName>
+       <colorTopicName>${prefix_topic}/color/image_raw</colorTopicName>
+       <colorCameraInfoTopicName>${prefix_topic}/color/camera_info</colorCameraInfoTopicName>
+       <infrared1TopicName>${prefix_topic}/infra1/image_raw</infrared1TopicName>
+       <infrared1CameraInfoTopicName>${prefix_topic}/infra1/camera_info</infrared1CameraInfoTopicName>
+       <infrared2TopicName>${prefix_topic}/infra2/image_raw</infrared2TopicName>
+       <infrared2CameraInfoTopicName>${prefix_topic}/infra2/camera_info</infrared2CameraInfoTopicName>
        <colorOpticalframeName>${color_optical_frame}</colorOpticalframeName>
        <depthOpticalframeName>${depth_optical_frame}</depthOpticalframeName>
        <infrared1OpticalframeName>${infrared1_optical_frame}</infrared1OpticalframeName>
        <infrared2OpticalframeName>${infrared2_optical_frame}</infrared2OpticalframeName>
-       <rangeMinDepth>0.2</rangeMinDepth>
+       <rangeMinDepth>0.105</rangeMinDepth>
        <rangeMaxDepth>10.0</rangeMaxDepth>
-       <pointCloud>false</pointCloud>
-       <pointCloudTopicName>depth/points</pointCloudTopicName>
-       <pointCloudCutoff>0.5</pointCloudCutoff>
+       <pointCloud>true</pointCloud>
+       <pointCloudTopicName>${prefix_topic}/depth/points</pointCloudTopicName>
+       <pointCloudCutoff>0.105</pointCloudCutoff>
      </plugin>
    </gazebo>

Commit message: Ported intel realsense 435d to ROS2

File: urdf/intel_d435.urdf.xacro (robot description, xacro)
@@ -45,5 +45,5 @@
         <geometry>
           <!-- <box size="${d435_cam_width} ${d435_cam_height} ${d435_cam_depth}"/> -->
-          <mesh filename="package://robotnik_sensors/meshes/intel_d435.dae" />
+          <mesh filename="package://robotnik_sensors/meshes/intel_d435_color.dae" />
         </geometry>
       </visual>
@@ -115,5 +115,11 @@
       <link name="${prefix}_color_optical_frame"/>
     </xacro:if>
-    <xacro:gazebo_d435 camera_name="${prefix}" reference_link="${prefix}_link" topics_ns="${prefix_topic}" depth_optical_frame="${prefix}_depth_optical_frame" color_optical_frame="${prefix}_color_optical_frame" infrared1_optical_frame="${prefix}_left_ir_optical_frame" infrared2_optical_frame="${prefix}_right_ir_optical_frame"/>
+    <xacro:gazebo_d435 camera_name="${prefix}"
+                       reference_link="${prefix}_link"
+                       topics_ns="${prefix_topic}"
+                       depth_optical_frame="${prefix}_depth_optical_frame"
+                       color_optical_frame="${prefix}_color_optical_frame"
+                       infrared1_optical_frame="${prefix}_left_ir_optical_frame"
+                       infrared2_optical_frame="${prefix}_right_ir_optical_frame"/>
   </xacro:macro>
   <xacro:macro name="gazebo_d435" params="camera_name reference_link topics_ns depth_optical_frame color_optical_frame infrared1_optical_frame infrared2_optical_frame" >
@@ -154,22 +160,5 @@
        <always_on>1</always_on>
        <update_rate>30</update_rate>
-       <visualize>1</visualize>
-       <plugin name="${prefix}kortex_vision_controller" filename="libgazebo_ros_camera.so">
-          <alwaysOn>true</alwaysOn>
-          <updateRate>30.0</updateRate>
-          <cameraName>${prefix_topic}/color</cameraName>
-          <imageTopicName>image_raw</imageTopicName>
-          <cameraInfoTopicName>camera_info</cameraInfoTopicName>
-          <frameName>/${prefix}_color_optical_frame</frameName>
-          <!-- this is just which name the Image msg will have, it does not affect the simulation.
-                However must be set to the optical_frame,  -->
-          <hackBaseline>0.07</hackBaseline>
-          <distortionK1>0.0</distortionK1>
-          <distortionK2>0.0</distortionK2>
-          <distortionK3>0.0</distortionK3>
-          <distortionT1>0.0</distortionT1>
-          <distortionT2>0.0</distortionT2>
-          <ignoreTfPrefix>1</ignoreTfPrefix>
-        </plugin>
+       <visualize>false</visualize>
      </sensor>
      <sensor name="${camera_name}ired1" type="camera">
@@ -193,5 +182,5 @@
        <always_on>1</always_on>
        <update_rate>90</update_rate>
-       <visualize>0</visualize>
+       <visualize>false</visualize>
      </sensor>
      <sensor name="${camera_name}ired2" type="camera">
@@ -215,5 +204,5 @@
        <always_on>1</always_on>
        <update_rate>90</update_rate>
-       <visualize>0</visualize>
+       <visualize>false</visualize>
      </sensor>
      <sensor name="${camera_name}depth" type="depth">
@@ -236,5 +225,5 @@
        <always_on>1</always_on>
        <update_rate>90</update_rate>
-       <visualize>0</visualize>
+       <visualize>false</visualize>
      </sensor>
    </gazebo>
@@ -245,12 +234,12 @@
        <colorUpdateRate>60.0</colorUpdateRate>
        <infraredUpdateRate>60.0</infraredUpdateRate>
-       <depthTopicName>depth/image_raw</depthTopicName>
-       <depthCameraInfoTopicName>depth/camera_info</depthCameraInfoTopicName>
-       <colorTopicName>color/image_raw</colorTopicName>
-       <colorCameraInfoTopicName>color/camera_info</colorCameraInfoTopicName>
-       <infrared1TopicName>infra1/image_raw</infrared1TopicName>
-       <infrared1CameraInfoTopicName>infra1/camera_info</infrared1CameraInfoTopicName>
-       <infrared2TopicName>infra2/image_raw</infrared2TopicName>
-       <infrared2CameraInfoTopicName>infra2/camera_info</infrared2CameraInfoTopicName>
+       <depthTopicName>${prefix_topic}/depth/image_raw</depthTopicName>
+       <depthCameraInfoTopicName>${prefix_topic}/depth/camera_info</depthCameraInfoTopicName>
+       <colorTopicName>${prefix_topic}/color/image_raw</colorTopicName>
+       <colorCameraInfoTopicName>${prefix_topic}/color/camera_info</colorCameraInfoTopicName>
+       <infrared1TopicName>${prefix_topic}/infra1/image_rect_raw</infrared1TopicName>
+       <infrared1CameraInfoTopicName>${prefix_topic}/infra1/camera_info</infrared1CameraInfoTopicName>
+       <infrared2TopicName>${prefix_topic}/infra2/image_rect_raw</infrared2TopicName>
+       <infrared2CameraInfoTopicName>${prefix_topic}/infra2/camera_info</infrared2CameraInfoTopicName>
        <colorOpticalframeName>${color_optical_frame}</colorOpticalframeName>
        <depthOpticalframeName>${depth_optical_frame}</depthOpticalframeName>
@@ -260,5 +249,5 @@
        <rangeMaxDepth>10.0</rangeMaxDepth>
        <pointCloud>false</pointCloud>
-       <pointCloudTopicName>depth/points</pointCloudTopicName>
+       <pointCloudTopicName>${prefix_topic}/depth/color/points</pointCloudTopicName>
        <pointCloudCutoff>0.5</pointCloudCutoff>
      </plugin>
