Commit message: Modified mockup of intel d405

File: urdf/intel_d405.urdf.xacro (robot description, xacro)
@@ -13,6 +13,6 @@
      publishing TF values with actual calibrated camera extrinsic values -->
     <xacro:property name="d405_cam_depth_to_infra1_offset" value="0.0"/>
-    <xacro:property name="d405_cam_depth_to_infra2_offset" value="-0.050"/>
-    <xacro:property name="d405_cam_depth_to_color_offset" value="0.015"/>
+    <xacro:property name="d405_cam_depth_to_infra2_offset" value="0.0"/>
+    <xacro:property name="d405_cam_depth_to_color_offset" value="0.0"/>
     <!-- The following values model the aluminum peripherial case for the
     D405 camera, with the camera joint represented by the actual
@@ -21,5 +21,5 @@
     <xacro:property name="d405_cam_height" value="0.042"/>
     <xacro:property name="d405_cam_depth" value="0.023"/>
-    <xacro:property name="d405_cam_mount_from_center_offset" value="0.0149"/>
+    <xacro:property name="d405_cam_mount_from_center_offset" value="0.0"/>
     <!-- The following offset is relative the the physical D405 camera peripherial
     camera tripod mount -->
@@ -37,5 +37,5 @@
       <parent link="${prefix}_base_link" />
       <child link="${prefix}_link" />
-      <origin xyz="0.01 0.02 0" rpy="0 0 0"/>
+      <origin xyz="0.0 0.0 0" rpy="0 0 0"/>
       <child link="${prefix}_link" />
     </joint>

Commit message: intel_d405 add collision to urdf

File: urdf/intel_d405.urdf.xacro (robot description, xacro)
@@ -49,10 +49,10 @@
         </geometry>
       </visual>
-      <!--<collision>-->
-        <!--<origin xyz="0 ${-d405_cam_depth_py} 0" rpy="0 0 0"/>-->
-        <!--<geometry>-->
-          <!--<box size="${d405_cam_depth} ${d405_cam_width} ${d405_cam_height}"/>-->
-        <!--</geometry>-->
-      <!--</collision>-->
+      <collision>
+        <origin xyz="${d405_cam_width/2.0} ${d405_cam_height/2.0} ${d405_cam_depth/2.0}" rpy="${M_PI/2} 0 ${M_PI/2}"/>
+        <geometry>
+          <box size="${d405_cam_width} ${d405_cam_height} ${d405_cam_depth}"/>
+        </geometry>
+      </collision>
       <inertial>
         <origin xyz="0.0025 -0.015 0.0" rpy="0 0 0" />

Commit message: intel_d405 update intertia

File: urdf/intel_d405.urdf.xacro (robot description, xacro)
@@ -56,7 +56,7 @@
       </collision>
       <inertial>
-        <origin xyz="0.0025 -0.015 0.0" rpy="0 0 0" />
-        <mass value="0.1" />
-        <xacro:solid_cuboid_inertia m="0.1" w="0.025" h="0.09" d="0.025" />
+        <origin xyz="${d405_cam_width/2.0} ${d405_cam_height/2.0} ${d405_cam_depth/2.0}" rpy="${M_PI/2} 0 ${M_PI/2}" />
+        <mass value="0.01" />
+        <xacro:solid_cuboid_inertia m="0.01" w="${d405_cam_height}" h="${d405_cam_depth}" d="${d405_cam_width}" />
       </inertial>
     </link>
