Commit message: add lidar_m10_p

File: urdf/lidar_m10_p.urdf.xacro (robot description, xacro)
@@ -11,5 +11,5 @@
         <origin xyz="0 0 0" rpy="0 0 0"/>
         <geometry>
-         <mesh filename="package://robotnik_sensors/meshes/lidar_m10_p.dae"/>
+         <mesh filename="package://robotnik_sensors/meshes/lidar_m10_p.STL"/>
         </geometry>
       </collision>
@@ -17,5 +17,5 @@
         <origin xyz="0 0 0" rpy="0 0 0"/>
         <geometry>
-            <mesh filename="package://robotnik_sensors/meshes/lidar_m10_p.dae" scale="0.001 0.001 0.001"/>
+            <mesh filename="package://robotnik_sensors/meshes/lidar_m10_p.STL" />
         </geometry>
       </visual>
@@ -27,5 +27,5 @@
     </link>
     <joint name="${prefix}_joint" type="fixed">
-      <origin xyz="0 0 0.0461" rpy="0 0 0"/>
+      <origin xyz="0 0 0.02305" rpy="0 0 0"/>
       <parent link="${prefix}_base_link"/>
       <child link="${prefix}_link"/>

Commit message: Update lidar_m10_p: Added gazebo plugin to publish the laser in simulation.

File: urdf/lidar_m10_p.urdf.xacro (robot description, xacro)
@@ -33,4 +33,48 @@
     <link name="${prefix}_link">
     </link>
+    <!-- Hokuyo sensor for simulation -->
+    <xacro:sensor_lidar_m10_p_gazebo/>
+  </xacro:macro>
+  <xacro:macro name="sensor_lidar_m10_p_gazebo">
+    <gazebo reference="${prefix}_link">
+      <xacro:if value="${gpu}">
+        <xacro:property name="ray_type" value="gpu_ray" />
+        <xacro:property name="plugin_lib" value="libgazebo_ros_gpu_laser.so" />
+      </xacro:if>
+      <xacro:unless value="${gpu}">
+        <xacro:property name="ray_type" value="ray" />
+        <xacro:property name="plugin_lib" value="libgazebo_ros_laser.so" />
+      </xacro:unless>
+      <sensor type="${ray_type}" name="${prefix}_sensor">
+        <pose>0 0 0 0 0 0</pose>
+        <visualize>false</visualize>
+        <update_rate>12</update_rate>
+        <ray>
+          <scan>
+            <horizontal>
+              <samples>1636</samples>
+              <resolution>1</resolution>
+              <min_angle>${min_angle}</min_angle>
+              <max_angle>${max_angle}</max_angle>
+            </horizontal>
+          </scan>
+          <range>
+            <min>0.06</min>
+            <max>10.0</max>
+            <resolution>0.03</resolution>
+          </range>
+          <noise>
+            <type>gaussian</type>
+            <mean>0.0</mean>
+            <stddev>0.01</stddev>
+          </noise>
+        </ray>
+        <plugin name="${prefix}_controller" filename="${plugin_lib}">
+          <topicName>${prefix_topic}/scan</topicName>
+          <frameName>/${prefix}_link</frameName>
+          <ignoreTfPrefix>1</ignoreTfPrefix>
+        </plugin>
+      </sensor>
+    </gazebo>
   </xacro:macro>
 </robot>
