Commit message: Update hokuyo_ust20lx
- Fixes inertias
- Sets links correctly based on datasheet

File: urdf/hokuyo_ust20lx.urdf.xacro (robot description, xacro)
@@ -10,5 +10,5 @@
     <link name="${prefix}_base_link">
       <collision>
-        <origin xyz="0 0 -0.05" rpy="0 0 0"/>
+        <origin xyz="0 0 0.0" rpy="0 0 0"/>
         <geometry>
           <box size="0.010 0.010 0.010"/>
@@ -16,5 +16,5 @@
       </collision>
       <visual>
-        <origin xyz="0 0 -0.05" rpy="0 0 0"/>
+        <origin xyz="0 0 0.0" rpy="0 0 0"/>
         <geometry>
             <mesh filename="package://robotnik_sensors/meshes/hokuyo_ust_20lx.dae"/>
@@ -22,7 +22,7 @@
       </visual>
       <inertial>
-        <mass value="1e-5" />
-        <origin xyz="0 0 0" rpy="0 0 0"/>
-        <inertia ixx="1e-6" ixy="0" ixz="0" iyy="1e-6" iyz="0" izz="1e-6" />
+        <origin xyz="0.0 0 0.035" rpy="0 0 0" />
+        <mass value="0.130" />
+        <xacro:solid_cuboid_inertia m="0.130" w="0.05" h="0.05" d="0.07" />
       </inertial>
     </link>
@@ -32,5 +32,5 @@
       <parent link="${prefix}_base_link"/>
       <child link="${prefix}_link"/>
-      <origin xyz="0.00 0 0.0" rpy="0 0 0"/>
+      <origin xyz="0.00 0.0 0.0474" rpy="0 0 0"/>
 	</joint>
     <!-- Hokuyo sensor for simulation -->

Commit message: Export hokuyo_ust20lx to ROS2

File: urdf/hokuyo_ust20lx.urdf.xacro (robot description, xacro)
@@ -18,5 +18,5 @@
         <origin xyz="0 0 0.0" rpy="0 0 0"/>
         <geometry>
-            <mesh filename="package://robotnik_sensors/meshes/hokuyo_ust_20lx.dae"/>
+            <mesh filename="file://$(find robotnik_sensors)/meshes/hokuyo_ust_20lx.dae"/>
         </geometry>
       </visual>
@@ -41,9 +41,7 @@
 			<xacro:if value="${gpu}">
         <xacro:property name="ray_type" value="gpu_ray" />
-        <xacro:property name="plugin_lib" value="libgazebo_ros_gpu_laser.so" />
       </xacro:if>
       <xacro:unless value="${gpu}">
         <xacro:property name="ray_type" value="ray" />
-        <xacro:property name="plugin_lib" value="libgazebo_ros_laser.so" />
       </xacro:unless>
 			<sensor type="${ray_type}" name="${prefix}_sensor">
@@ -73,7 +71,10 @@
 					</noise>
 				</ray>
-				<plugin name="${prefix}_controller" filename="${plugin_lib}">
-					<topicName>${prefix_topic}/scan</topicName>
-					<frameName>/${prefix}_link</frameName>
+				<plugin name="${prefix}_controller" filename="libgazebo_ros_ray_sensor.so">
+          <ros>
+            <remapping>~/out:=${prefix_topic}/scan</remapping>
+          </ros>
+          <output_type>sensor_msgs/LaserScan</output_type>
+          <frame_name>${prefix}_link</frame_name>
 				</plugin>
 			</sensor>

Commit message: Updated xacro hokuyo_ust20lx. Gazebo and colision

File: urdf/hokuyo_ust20lx.urdf.xacro (robot description, xacro)
@@ -1,6 +1,5 @@
 <?xml version="1.0"?>
 <robot name="sensor_hokuyo_ust20lx" xmlns:xacro="http://wiki.ros.org/xacro">
-  <xacro:macro name="sensor_hokuyo_ust20lx" params="prefix parent prefix_topic:='front_laser' *origin min_angle:=-2.3562 max_angle:=2.3562 gpu:=^|true">
-			<!--arg name="namespace" value="$(arg namespace)"/-->
+  <xacro:macro name="sensor_hokuyo_ust20lx" params="ns prefix parent *origin min_angle:=-2.3562 max_angle:=2.3562">
     <joint name="${prefix}_base_joint" type="fixed">
       <xacro:insert_block name="origin" />
@@ -10,40 +9,32 @@
     <link name="${prefix}_base_link">
       <collision>
-        <origin xyz="0 0 0.0" rpy="0 0 0"/>
+        <origin xyz="0 0 0.036" rpy="0 0 0"/>
         <geometry>
-          <box size="0.010 0.010 0.010"/>
+          <cylinder length="0.072" radius="0.022"/>
         </geometry>
       </collision>
       <visual>
-        <origin xyz="0 0 0.0" rpy="0 0 0"/>
+        <origin xyz="0 0 0" rpy="0 0 0"/>
         <geometry>
-            <mesh filename="file://$(find robotnik_sensors)/meshes/hokuyo_ust_20lx.dae"/>
+          <mesh filename="file://$(find robotnik_sensors)/meshes/hokuyo_ust_20lx.dae"/>
         </geometry>
       </visual>
       <inertial>
-        <origin xyz="0.0 0 0.035" rpy="0 0 0" />
+        <origin xyz="0.0 0 0.036" rpy="0 0 0" />
         <mass value="0.130" />
         <xacro:solid_cuboid_inertia m="0.130" w="0.05" h="0.05" d="0.07" />
       </inertial>
     </link>
-    <link name="${prefix}_link">
-	</link>
     <joint name="${prefix}_joint" type="fixed">
       <parent link="${prefix}_base_link"/>
       <child link="${prefix}_link"/>
       <origin xyz="0.00 0.0 0.0474" rpy="0 0 0"/>
-	</joint>
-    <!-- Hokuyo sensor for simulation -->
+	  </joint>
+    <link name="${prefix}_link"/>
     <xacro:sensor_hokuyo_ust20_gazebo/>
   </xacro:macro>
   <xacro:macro name="sensor_hokuyo_ust20_gazebo">
     <gazebo reference="${prefix}_link">
-			<xacro:if value="${gpu}">
-        <xacro:property name="ray_type" value="gpu_ray" />
-      </xacro:if>
-      <xacro:unless value="${gpu}">
-        <xacro:property name="ray_type" value="ray" />
-      </xacro:unless>
-			<sensor type="${ray_type}" name="${prefix}_sensor">
+			<sensor type="ray" name="${prefix}_sensor">
 				<pose>0 0 0 0 0 0</pose>
 				<visualize>false</visualize>
@@ -61,7 +52,5 @@
 						<min>0.06</min>
 						<max>20.0</max>
-						<!-- resolution>0.004363323</resolution -->
 						<resolution>0.004359297</resolution>
-						<!-- resolution>0.001</resolution -->
 					</range>
 					<noise>
@@ -71,13 +60,14 @@
 					</noise>
 				</ray>
-				<plugin name="${prefix}_controller" filename="libgazebo_ros_ray_sensor.so">
+				<plugin name="${prefix}" filename="libgazebo_ros_ray_sensor.so">
           <ros>
-            <remapping>~/out:=${prefix_topic}/scan</remapping>
+            <namespace>${ns}</namespace>
+            <remapping>~/out:=~/scan</remapping>
           </ros>
           <output_type>sensor_msgs/LaserScan</output_type>
-          <frame_name>${prefix}_link</frame_name>
+          <frame_name>${ns}/${prefix}_link</frame_name>
 				</plugin>
 			</sensor>
-	</gazebo>
+	  </gazebo>
   </xacro:macro>
 </robot>
