Commit message: standarized all sensors: frames, joints, topics and params

File: urdf/imu_hector_plugin.urdf.xacro (robot description, xacro)
@@ -29,10 +29,11 @@
 	  </link>
 	  <gazebo>
-	    <plugin name="ros_imu_hector" filename="libhector_gazebo_ros_imu.so">
+	    <plugin name="${name}_controller" filename="libhector_gazebo_ros_imu.so">
 	       <alwaysOn>true</alwaysOn>
-	       <topicName>imu_data</topicName>
-	       <bodyName>imu_link</bodyName>
+	       <topicName>${name}/data</topicName>
+		   <serviceName>${name}/service</serviceName>
+		   <bodyName>${name}_link</bodyName>
 	       <updateRate>50.0</updateRate>
-	       <serviceName>imu_service</serviceName>
+	       <gaussianNoise>0.005</gaussianNoise>
 	       <!-- orientation parameters -->
            <yawOffset>0.0</yawOffset>

File: urdf/orbbec_astra.urdf.xacro (robot description, xacro)
@@ -4,7 +4,7 @@
   <xacro:property name="orbbec_astra_scale" value="1.0"/>
   <!-- RGB sensor - cam -->
-  <xacro:property name="orbbec_astra_cam_rel_rgb_px"   value="0.0" />
-  <xacro:property name="orbbec_astra_cam_rel_rgb_py"   value="-0.0125" />
-  <xacro:property name="orbbec_astra_cam_rel_rgb_pz"   value="-0.0150" />
+  <xacro:property name="orbbec_astra_rel_rgb_px"   value="0.0" />
+  <xacro:property name="orbbec_astra_rel_rgb_py"   value="-0.0125" />
+  <xacro:property name="orbbec_astra_rel_rgb_pz"   value="-0.0150" />
   <!-- IR sensor - depth -->
   <xacro:property name="orbbec_astra_depth_rel_rgb_px" value="0.0" />
@@ -13,10 +13,10 @@
   <xacro:property name="M_PI" value="3.1415926535897931" />
   <xacro:macro name="sensor_orbbec_astra" params="name parent *origin">
-    <joint name="${name}_cam_rgb_joint" type="fixed">
+    <joint name="${name}_rgb_joint" type="fixed">
 	  <xacro:insert_block name="origin" />
       <parent link="${parent}"/>
-      <child link="${name}_cam_rgb_frame" />
+      <child link="${name}_rgb_frame" />
     </joint>
-    <link name="${name}_cam_rgb_frame">
+    <link name="${name}_rgb_frame">
       <inertial>
         <mass value="0.001" />
@@ -27,10 +27,10 @@
       </inertial>
     </link>
-    <joint name="${name}_cam_rgb_optical_joint" type="fixed">
+    <joint name="${name}_rgb_optical_joint" type="fixed">
       <origin xyz="0.0 0.0 0.0" rpy="${-M_PI/2} 0 ${-M_PI/2}" />
-      <parent link="${name}_cam_rgb_frame" />
-      <child link="${name}_cam_rgb_optical_frame" />
+      <parent link="${name}_rgb_frame" />
+      <child link="${name}_rgb_optical_frame" />
     </joint>
-    <link name="${name}_cam_rgb_optical_frame">
+    <link name="${name}_rgb_optical_frame">
       <inertial>
         <mass value="0.001" />
@@ -41,11 +41,11 @@
       </inertial>
     </link>
-    <joint name="${name}_cam_joint" type="fixed">
-      <origin xyz="${orbbec_astra_cam_rel_rgb_px} ${orbbec_astra_cam_rel_rgb_py} ${orbbec_astra_cam_rel_rgb_pz}"
+    <joint name="${name}_joint" type="fixed">
+      <origin xyz="${orbbec_astra_rel_rgb_px} ${orbbec_astra_rel_rgb_py} ${orbbec_astra_rel_rgb_pz}"
               rpy="0 0 0"/>
-      <parent link="${name}_cam_rgb_frame"/>
-      <child link="${name}_cam_link"/>
+      <parent link="${name}_rgb_frame"/>
+      <child link="${name}_link"/>
     </joint>
-    <link name="${name}_cam_link">
+    <link name="${name}_link">
       <visual>
         <origin xyz="0 0 0" rpy="0 0 0"/>
@@ -68,10 +68,10 @@
       </inertial>
     </link>
-    <joint name="${name}_cam_depth_joint" type="fixed">
+    <joint name="${name}_depth_joint" type="fixed">
       <origin xyz="${orbbec_astra_depth_rel_rgb_px} ${orbbec_astra_depth_rel_rgb_py} ${orbbec_astra_depth_rel_rgb_pz}" rpy="0 0 0" />
-      <parent link="${name}_cam_rgb_frame" />
-      <child link="${name}_cam_depth_frame" />
+      <parent link="${name}_rgb_frame" />
+      <child link="${name}_depth_frame" />
     </joint>
-    <link name="${name}_cam_depth_frame">
+    <link name="${name}_depth_frame">
       <inertial>
         <mass value="0.01" />
@@ -82,10 +82,10 @@
       </inertial>
     </link>
-    <joint name="${name}_cam_depth_optical_joint" type="fixed">
+    <joint name="${name}_depth_optical_joint" type="fixed">
       <origin xyz="0 0 0" rpy="${-M_PI/2} 0 ${-M_PI/2}" />
-      <parent link="${name}_cam_depth_frame" />
-      <child link="${name}_cam_depth_optical_frame" />
+      <parent link="${name}_depth_frame" />
+      <child link="${name}_depth_optical_frame" />
     </joint>
-    <link name="${name}_cam_depth_optical_frame">
+    <link name="${name}_depth_optical_frame">
       <inertial>
         <mass value="0.001" />
@@ -100,6 +100,6 @@
   </xacro:macro>
    <xacro:macro name="sensor_orbbec_astra_gazebo">
-    <gazebo reference="${name}_cam_rgb_optical_frame">
-      <sensor type="depth" name="cam">
+    <gazebo reference="${name}_rgb_optical_frame">
+      <sensor type="depth" name="${name}_controller">
         <always_on>true</always_on>
         <update_rate>20.0</update_rate>
@@ -116,5 +116,5 @@
           </clip>
         </camera>
-        <plugin name="orbbec_astra_cam_controller" filename="libgazebo_ros_openni_kinect.so">
+        <plugin name="${name}_controller" filename="libgazebo_ros_openni_kinect.so">
           <cameraName>${name}</cameraName>
           <alwaysOn>true</alwaysOn>
@@ -125,5 +125,5 @@
           <cameraInfoTopicName>rgb/camera_info</cameraInfoTopicName>
           <depthImageCameraInfoTopicName>depth/camera_info</depthImageCameraInfoTopicName>
-          <frameName>${name}_cam_depth_optical_frame</frameName>
+          <frameName>${name}_depth_optical_frame</frameName>
           <baseline>0.1</baseline>
           <distortion_k1>0.0</distortion_k1>

Commit message: adding prefix_frame and prefix_topic

File: urdf/imu_hector_plugin.urdf.xacro (robot description, xacro)
@@ -1,13 +1,13 @@
 <?xml version="1.0"?>
 <robot name="sensor_imu" xmlns:xacro="http://www.ros.org/wiki/xacro">
-  <xacro:macro name="sensor_imu_hector" params="name parent *origin">
-	  <joint name="${name}_joint" type="fixed">
+  <xacro:macro name="sensor_imu_hector" params="prefix_frame prefix_topic parent *origin">
+	  <joint name="${prefix_frame}_joint" type="fixed">
 	      <axis xyz="1 0 0"/>
 	      <!--origin xyz="0 0 0.2825"/-->
 	      <xacro:insert_block name="origin"/>
 	      <parent link="${parent}"/>
-	      <child link="${name}_link"/>
+	      <child link="${prefix_frame}_link"/>
 	  </joint>
-	  <link name="${name}_link">
+	  <link name="${prefix_frame}_link">
 	      <inertial>
 	        <mass value="0.001"/>
@@ -29,9 +29,9 @@
 	  </link>
 	  <gazebo>
-	    <plugin name="${name}_controller" filename="libhector_gazebo_ros_imu.so">
+	    <plugin name="${prefix_frame}_controller" filename="libhector_gazebo_ros_imu.so">
 	       <alwaysOn>true</alwaysOn>
-	       <topicName>${name}/data</topicName>
-		   <serviceName>${name}/service</serviceName>
-		   <bodyName>${name}_link</bodyName>
+	       <topicName>${prefix_topic}imu/data</topicName>
+		   <serviceName>${prefix_topic}imu/service</serviceName>
+		   <bodyName>${prefix_frame}_link</bodyName>
 	       <updateRate>50.0</updateRate>
 	       <gaussianNoise>0.005</gaussianNoise>

Commit message: prefix added to imu hector urdf

File: urdf/imu_hector_plugin.urdf.xacro (robot description, xacro)
@@ -7,5 +7,5 @@
 	      <xacro:insert_block name="origin"/>
 	      <parent link="${parent}"/>
-	      <child link="${prefix_frame}_link"/>
+	      <child link="${prefix}_link"/>
 	  </joint>
 	  <link name="${prefix}_link">

Commit message: Update imu_hector inertia

File: urdf/imu_hector_plugin.urdf.xacro (robot description, xacro)
@@ -11,8 +11,8 @@
 	  <link name="${prefix}_link">
 	      <inertial>
-	        <mass value="0.001"/>
-	        <origin rpy="0 0 0" xyz="0 0 0"/>
-	        <inertia ixx="0.0001" ixy="0" ixz="0" iyy="0.000001" iyz="0" izz="0.0001"/>
-	      </inertial>
+			<origin xyz="0.0 0 0.01" rpy="0 0 0" />
+			<mass value="0.05" />
+			<xacro:solid_cuboid_inertia m="0.05" w="0.02" h="0.02" d="0.02" />
+		  </inertial>
 	      <visual>
 	        <origin rpy="0 0 0" xyz="0 0 0"/>

Commit message: Updated imu hector to ros2

File: urdf/imu_hector_plugin.urdf.xacro (robot description, xacro)
@@ -1,53 +1,121 @@
 <?xml version="1.0"?>
 <robot name="sensor_imu" xmlns:xacro="http://wiki.ros.org/xacro">
-  <xacro:macro name="sensor_imu_hector" params="prefix topic:='imu/data' parent *origin">
-	  <joint name="${prefix}_joint" type="fixed">
-	      <axis xyz="1 0 0"/>
-	      <!--origin xyz="0 0 0.2825"/-->
-	      <xacro:insert_block name="origin"/>
-	      <parent link="${parent}"/>
-	      <child link="${prefix}_link"/>
-	  </joint>
-	  <link name="${prefix}_link">
-	      <inertial>
-			<origin xyz="0.0 0 0.01" rpy="0 0 0" />
-			<mass value="0.05" />
-			<xacro:solid_cuboid_inertia m="0.05" w="0.02" h="0.02" d="0.02" />
-		  </inertial>
-	      <visual>
-	        <origin rpy="0 0 0" xyz="0 0 0"/>
-	        <geometry>
-	          <box size="0.001 0.001 0.001"/>
-	        </geometry>
-	      </visual>
-	      <collision>
-	        <origin rpy="0 0 0" xyz="0 0 0"/>
-	        <geometry>
-	          <box size=".001 .001 .001"/>
-	        </geometry>
-	      </collision>
-	  </link>
-	  <gazebo>
-	    <plugin name="${prefix}_controller" filename="libhector_gazebo_ros_imu.so">
-	       <alwaysOn>true</alwaysOn>
-	       <topicName>${topic}</topicName>
-		   <serviceName>${prefix}imu/service</serviceName>
-		   <bodyName>${prefix}_link</bodyName>
-		   <frameId>${prefix}_link</frameId>
-	       <updateRate>50.0</updateRate>
-	       <gaussianNoise>0.00</gaussianNoise>
-           <yawOffset>0.0</yawOffset>
-           <yawDrift>0.0</yawDrift>
-           <yawGaussianNoise>0.0</yawGaussianNoise>
-           <!-- angular velocities parameters -->
-           <rateOffset>0.0 0.0 0.0</rateOffset>
-           <rateDrift>0.0 0.0 0.0</rateDrift>
-           <rateGaussianNoise>0.0 0.0 0.0</rateGaussianNoise>
-           <!-- linear accelerations parameters -->
-           <accelOffset>0.0 0.0 0.0</accelOffset>
-           <accelDrift>0.0 0.0 0.0</accelDrift>
-           <accelGaussianNoise>0.0 0.0 0.0</accelGaussianNoise>
-	    </plugin>
-	  </gazebo>
+  <xacro:macro name="sensor_imu_hector" params="ns prefix topic:='imu/data' parent *origin">
+    <joint name="${prefix}_joint" type="fixed">
+      <axis xyz="1 0 0"/>
+      <xacro:insert_block name="origin"/>
+      <parent link="${parent}"/>
+      <child link="${prefix}_link"/>
+    </joint>
+    <link name="${prefix}_link">
+      <inertial>
+        <origin xyz="0 0 0" rpy="0 0 0" />
+        <mass value="0.05" />
+        <xacro:solid_cuboid_inertia m="0.05" w="0.021" h="0.027" d="0.003" />
+      </inertial>
+      <visual>
+        <origin rpy="0 0 0" xyz="0 0 0"/>
+        <geometry>
+          <box size="0.021 0.027 0.003"/>
+        </geometry>
+      </visual>
+      <collision>
+        <origin rpy="0 0 0" xyz="0 0 0"/>
+        <geometry>
+          <box size=".001 .001 .001"/>
+        </geometry>
+      </collision>
+    </link>
+    <xacro:sensor_imu_hector_gazebo/>
+  </xacro:macro>
+  <xacro:macro name="sensor_imu_hector_gazebo">
+    <gazebo reference="${prefix}_link">
+      <gravity>true</gravity>
+      <sensor name="imu_sensor" type="imu">
+        <pose>0 0 0 0 0 0</pose>
+        <visualize>true</visualize>
+        <update_rate>100</update_rate>
+        <imu>
+          <topic>__default_topic__</topic>
+          <angular_velocity>
+            <x>
+              <noise type="gaussian">
+	    					<type>gaussian</type>
+                <mean>0</mean>
+                <stddev>0.2</stddev>
+                <bias_mean>0</bias_mean>
+                <bias_stddev>0</bias_stddev>
+                <dynamic_bias_stddev>0</dynamic_bias_stddev>
+                <dynamic_bias_correlation_time>0</dynamic_bias_correlation_time>
+              </noise>
+            </x>
+            <y>
+              <noise type="gaussian">
+	    					<type>gaussian</type>
+                <mean>0</mean>
+                <stddev>0.2</stddev>
+                <bias_mean>0</bias_mean>
+                <bias_stddev>0</bias_stddev>
+                <dynamic_bias_stddev>0</dynamic_bias_stddev>
+                <dynamic_bias_correlation_time>0</dynamic_bias_correlation_time>
+              </noise>
+            </y>
+            <z>
+              <noise type="gaussian">
+	    					<type>gaussian</type>
+                <mean>0</mean>
+                <stddev>0.2</stddev>
+                <bias_mean>0</bias_mean>
+                <bias_stddev>0</bias_stddev>
+                <dynamic_bias_stddev>0</dynamic_bias_stddev>
+                <dynamic_bias_correlation_time>0</dynamic_bias_correlation_time>
+              </noise>
+            </z>
+          </angular_velocity>
+          <linear_acceleration>
+            <x>
+              <noise type="gaussian">
+	    					<type>gaussian</type>
+                <mean>0</mean>
+                <stddev>0.2</stddev>
+                <bias_mean>0</bias_mean>
+                <bias_stddev>0</bias_stddev>
+                <dynamic_bias_stddev>0</dynamic_bias_stddev>
+                <dynamic_bias_correlation_time>0</dynamic_bias_correlation_time>
+              </noise>
+            </x>
+            <y>
+              <noise type="gaussian">
+	    					<type>gaussian</type>
+                <mean>0</mean>
+                <stddev>0.2</stddev>
+                <bias_mean>0</bias_mean>
+                <bias_stddev>0</bias_stddev>
+                <dynamic_bias_stddev>0</dynamic_bias_stddev>
+                <dynamic_bias_correlation_time>0</dynamic_bias_correlation_time>
+              </noise>
+            </y>
+            <z>
+              <noise type="gaussian">
+	    					<type>gaussian</type>
+                <mean>0</mean>
+                <stddev>0.2</stddev>
+                <bias_mean>0</bias_mean>
+                <bias_stddev>0</bias_stddev>
+                <dynamic_bias_stddev>0</dynamic_bias_stddev>
+                <dynamic_bias_correlation_time>0</dynamic_bias_correlation_time>
+              </noise>
+            </z>
+          </linear_acceleration>
+        </imu>
+        <plugin name="imu" filename="libgazebo_ros_imu_sensor.so">
+          <ros>
+            <namespace>${ns}</namespace>
+            <remapping>~/out:=~/data</remapping>
+          </ros>
+          <initial_orientation_as_reference>initial_orientation_as_reference</initial_orientation_as_reference>
+        </plugin>
+      </sensor>
+    </gazebo>
   </xacro:macro>
 </robot>
