Commit message: minor change names

File: urdf/orbbec_astra.urdf.xacro (robot description, xacro)
@@ -93,5 +93,5 @@
   <sensor_xtion_pro_gazebo/>
   </xacro:macro>
-   <xacro:macro name="sensor_xtion_pro_gazebo">
+   <xacro:macro name="sensor_orbbec_astra_gazebo">
     <gazebo reference="${name}_cam_depth_frame">
       <sensor type="depth" name="cam">
@@ -110,5 +110,5 @@
           </clip>
         </camera>
-        <plugin name="xtion_pro_cam_controller" filename="libgazebo_ros_openni_kinect.so">
+        <plugin name="orbbec_astra_cam_controller" filename="libgazebo_ros_openni_kinect.so">
           <cameraName>${name}</cameraName>
           <alwaysOn>true</alwaysOn>

Commit message: corrected scale and positions of optical frames

File: urdf/orbbec_astra.urdf.xacro (robot description, xacro)
@@ -2,7 +2,15 @@
 <robot name="sensor_orbbec_astra" xmlns:xacro="http://ros.org/wiki/xacro">
   <!-- Xacro properties -->
-  <xacro:property name="M_SCALE" value="0.001"/>
-  <xacro:property name="orbbec_astra_depth_rel_rgb_py" value="0.0270" />
-  <xacro:property name="orbbec_astra_cam_rel_rgb_py"   value="-0.0220" />
+  <xacro:property name="M_SCALE" value="1.0"/>
+  <!-- RGB sensor - cam -->
+  <xacro:property name="orbbec_astra_cam_rel_rgb_px"   value="0.015" />
+  <xacro:property name="orbbec_astra_cam_rel_rgb_py"   value="0.0" />
+  <xacro:property name="orbbec_astra_cam_rel_rgb_pz"   value="0.0125" />
+  <!-- IR sensor - depth -->
+  <xacro:property name="orbbec_astra_depth_rel_rgb_px" value="0.015" />
+  <xacro:property name="orbbec_astra_depth_rel_rgb_py" value="0.0" />
+  <xacro:property name="orbbec_astra_depth_rel_rgb_pz" value="0.0375" />
+  <!-- xacro:property name="orbbec_astra_px" value="-0.010" />
+  <xacro:property name="orbbec_astra_pz" value="0.015" / -->
   <xacro:property name="M_PI" value="3.1415926535897931" />
   <xacro:macro name="sensor_orbbec_astra" params="name parent *origin">
@@ -22,5 +30,5 @@
     </link>
     <joint name="${name}_cam_rgb_optical_joint" type="fixed">
-      <origin xyz="0 0 0" rpy="${-M_PI/2} 0 ${-M_PI/2}" />
+      <origin xyz="${orbbec_astra_cam_rel_rgb_px} ${orbbec_astra_cam_rel_rgb_py} ${orbbec_astra_cam_rel_rgb_pz}" rpy="0.0 ${M_PI/2} ${M_PI/2}" />
       <parent link="${name}_cam_rgb_frame" />
       <child link="${name}_cam_rgb_optical_frame" />
@@ -36,5 +44,5 @@
     </link>
     <joint name="${name}_cam_joint" type="fixed">
-      <origin xyz="0 ${orbbec_astra_cam_rel_rgb_py} 0"
+      <origin xyz="0.0 0.0 0.0"
               rpy="0 0 0"/>
       <parent link="${name}_cam_rgb_frame"/>
@@ -43,5 +51,5 @@
     <link name="${name}_cam_link">
       <visual>
-        <origin xyz="-0.01 0 0" rpy="${-M_PI/2} -${M_PI} ${-M_PI/2}"/>
+        <origin xyz="0 0 0" rpy="${-M_PI/2} -${M_PI} ${-M_PI/2}"/>
         <geometry>
           <mesh filename="package://robotnik_sensors/meshes/orbbec_astra.dae" scale="${M_SCALE} ${M_SCALE} ${M_SCALE}"/>
@@ -63,5 +71,5 @@
     </link>
     <joint name="${name}_cam_depth_joint" type="fixed">
-      <origin xyz="0 ${orbbec_astra_depth_rel_rgb_py} 0" rpy="0 0 0" />
+      <origin xyz="${orbbec_astra_depth_rel_rgb_px} ${orbbec_astra_depth_rel_rgb_py} ${orbbec_astra_depth_rel_rgb_pz}" rpy="0 0 0" />
       <parent link="${name}_cam_rgb_frame" />
       <child link="${name}_cam_depth_frame" />
@@ -77,5 +85,6 @@
     </link>
     <joint name="${name}_cam_depth_optical_joint" type="fixed">
-      <origin xyz="0 0 0" rpy="${-M_PI/2} 0 ${-M_PI/2}" />
+      <!-- origin xyz="0 0 0" rpy="${-M_PI/2} 0 ${-M_PI/2}" / -->
+      <origin xyz="0 0 0" rpy="0 ${M_PI/2} ${M_PI/2}" />
       <parent link="${name}_cam_depth_frame" />
       <child link="${name}_cam_depth_optical_frame" />

Commit message: orbbec_astra frames updated to be compatible with gazebo plugin

File: urdf/orbbec_astra.urdf.xacro (robot description, xacro)
@@ -4,13 +4,11 @@
   <xacro:property name="M_SCALE" value="1.0"/>
   <!-- RGB sensor - cam -->
-  <xacro:property name="orbbec_astra_cam_rel_rgb_px"   value="0.015" />
+  <xacro:property name="orbbec_astra_cam_rel_rgb_px"   value="0.0" />
   <xacro:property name="orbbec_astra_cam_rel_rgb_py"   value="0.0" />
-  <xacro:property name="orbbec_astra_cam_rel_rgb_pz"   value="0.0125" />
+  <xacro:property name="orbbec_astra_cam_rel_rgb_pz"   value="0.015" />
   <!-- IR sensor - depth -->
-  <xacro:property name="orbbec_astra_depth_rel_rgb_px" value="0.015" />
-  <xacro:property name="orbbec_astra_depth_rel_rgb_py" value="0.0" />
-  <xacro:property name="orbbec_astra_depth_rel_rgb_pz" value="0.0375" />
-  <!-- xacro:property name="orbbec_astra_px" value="-0.010" />
-  <xacro:property name="orbbec_astra_pz" value="0.015" / -->
+  <xacro:property name="orbbec_astra_depth_rel_rgb_px" value="0.0" />
+  <xacro:property name="orbbec_astra_depth_rel_rgb_py" value="0.0250" />
+  <xacro:property name="orbbec_astra_depth_rel_rgb_pz" value="0.0" />
   <xacro:property name="M_PI" value="3.1415926535897931" />
   <xacro:macro name="sensor_orbbec_astra" params="name parent *origin">
@@ -30,5 +28,5 @@
     </link>
     <joint name="${name}_cam_rgb_optical_joint" type="fixed">
-      <origin xyz="${orbbec_astra_cam_rel_rgb_px} ${orbbec_astra_cam_rel_rgb_py} ${orbbec_astra_cam_rel_rgb_pz}" rpy="0.0 ${M_PI/2} ${M_PI/2}" />
+      <origin xyz="0.0 0.0 0.0" rpy="${-M_PI/2} 0 ${-M_PI/2}" />
       <parent link="${name}_cam_rgb_frame" />
       <child link="${name}_cam_rgb_optical_frame" />
@@ -44,5 +42,5 @@
     </link>
     <joint name="${name}_cam_joint" type="fixed">
-      <origin xyz="0.0 0.0 0.0"
+      <origin xyz="0 0 0"
               rpy="0 0 0"/>
       <parent link="${name}_cam_rgb_frame"/>
@@ -51,5 +49,5 @@
     <link name="${name}_cam_link">
       <visual>
-        <origin xyz="0 0 0" rpy="${-M_PI/2} -${M_PI} ${-M_PI/2}"/>
+        <origin xyz="0 0 0" rpy="0 0 0"/>
         <geometry>
           <mesh filename="package://robotnik_sensors/meshes/orbbec_astra.dae" scale="${M_SCALE} ${M_SCALE} ${M_SCALE}"/>
@@ -85,6 +83,5 @@
     </link>
     <joint name="${name}_cam_depth_optical_joint" type="fixed">
-      <!-- origin xyz="0 0 0" rpy="${-M_PI/2} 0 ${-M_PI/2}" / -->
-      <origin xyz="0 0 0" rpy="0 ${M_PI/2} ${M_PI/2}" />
+      <origin xyz="0 0 0" rpy="${-M_PI/2} 0 ${-M_PI/2}" />
       <parent link="${name}_cam_depth_frame" />
       <child link="${name}_cam_depth_optical_frame" />
@@ -103,5 +100,5 @@
   </xacro:macro>
    <xacro:macro name="sensor_orbbec_astra_gazebo">
-    <gazebo reference="${name}_cam_depth_frame">
+    <gazebo reference="${name}_cam_rgb_optical_frame">
       <sensor type="depth" name="cam">
         <always_on>true</always_on>

Commit message: changed cam_link to have a reference frame for mounting in robot, not very useful at al...

File: urdf/orbbec_astra.urdf.xacro (robot description, xacro)
@@ -5,6 +5,6 @@
   <!-- RGB sensor - cam -->
   <xacro:property name="orbbec_astra_cam_rel_rgb_px"   value="0.0" />
-  <xacro:property name="orbbec_astra_cam_rel_rgb_py"   value="0.0" />
-  <xacro:property name="orbbec_astra_cam_rel_rgb_pz"   value="0.015" />
+  <xacro:property name="orbbec_astra_cam_rel_rgb_py"   value="-0.0125" />
+  <xacro:property name="orbbec_astra_cam_rel_rgb_pz"   value="-0.0150" />
   <!-- IR sensor - depth -->
   <xacro:property name="orbbec_astra_depth_rel_rgb_px" value="0.0" />
@@ -42,5 +42,5 @@
     </link>
     <joint name="${name}_cam_joint" type="fixed">
-      <origin xyz="0 0 0"
+      <origin xyz="${orbbec_astra_cam_rel_rgb_px} ${orbbec_astra_cam_rel_rgb_py} ${orbbec_astra_cam_rel_rgb_pz}"
               rpy="0 0 0"/>
       <parent link="${name}_cam_rgb_frame"/>

Commit message: MOD: Fixed problem with rotations

File: urdf/orbbec_astra.urdf.xacro (robot description, xacro)
@@ -2,4 +2,5 @@
 <robot name="sensor_orbbec_astra" xmlns:xacro="http://www.ros.org/wiki/xacro">
   <!-- Xacro properties -->
+  <!--xacro:property name="orbbec_astra_scale" value="0.015"/-->
   <xacro:property name="orbbec_astra_scale" value="1.0"/>
   <!-- RGB sensor - cam -->
@@ -33,5 +34,5 @@
     </joint>
     <link name="${name}_rgb_optical_frame">
-      <inertial>
+      <!--inertial>
         <mass value="0.001" />
         <origin xyz="0 0 0" />
@@ -39,9 +40,9 @@
           iyy="0.0001" iyz="0.0"
           izz="0.0001" />
-      </inertial>
+      </inertial-->
     </link>
     <joint name="${name}_joint" type="fixed">
       <origin xyz="${orbbec_astra_rel_rgb_px} ${orbbec_astra_rel_rgb_py} ${orbbec_astra_rel_rgb_pz}"
-              rpy="0 0 0"/>
+              rpy="0.0 0 0"/>
       <parent link="${name}_rgb_frame"/>
       <child link="${name}_link"/>
@@ -61,10 +62,15 @@
       </collision>
       <inertial>
-        <mass value="0.01" />
+        <!--mass value="0.01" />
         <origin xyz="0 0 0" />
         <inertia ixx="0.001" ixy="0.0" ixz="0.0"
           iyy="0.001" iyz="0.0"
-          izz="0.001" />
-      </inertial>
+          izz="0.001" /-->
+          <mass value="0.564" />
+          <origin xyz="0 0 0" />
+          <inertia ixx="0.003881243" ixy="0.0" ixz="0.0"
+                   iyy="0.000498940" iyz="0.0"
+                   izz="0.003879257" />
+       </inertial>
     </link>
     <joint name="${name}_depth_joint" type="fixed">
@@ -74,5 +80,5 @@
     </joint>
     <link name="${name}_depth_frame">
-      <inertial>
+      <!--inertial>
         <mass value="0.01" />
         <origin xyz="0 0 0" />
@@ -80,5 +86,5 @@
           iyy="0.001" iyz="0.0"
           izz="0.001" />
-      </inertial>
+      </inertial-->
     </link>
     <joint name="${name}_depth_optical_joint" type="fixed">
@@ -88,5 +94,5 @@
     </joint>
     <link name="${name}_depth_optical_frame">
-      <inertial>
+      <!--inertial>
         <mass value="0.001" />
         <origin xyz="0 0 0" />
@@ -94,5 +100,5 @@
           iyy="0.0001" iyz="0.0"
           izz="0.0001" />
-      </inertial>
+      </inertial-->
     </link>
   <!-- RGBD sensor for simulation, same as Kinect -->
@@ -100,6 +106,6 @@
   </xacro:macro>
    <xacro:macro name="sensor_orbbec_astra_gazebo">
-    <gazebo reference="${name}_rgb_optical_frame">
-      <sensor type="depth" name="${name}_controller">
+    <gazebo reference="${name}_link">
+      <sensor type="depth" name="${name}">
         <always_on>true</always_on>
         <update_rate>20.0</update_rate>
@@ -119,5 +125,5 @@
           <cameraName>${name}</cameraName>
           <alwaysOn>true</alwaysOn>
-          <updateRate>15</updateRate>
+          <updateRate>10</updateRate>
           <imageTopicName>rgb/image_raw</imageTopicName>
           <depthImageTopicName>depth/image_raw</depthImageTopicName>

Commit message: orbbec_astra: removing the suffix link from frame links

File: urdf/orbbec_astra.urdf.xacro (robot description, xacro)
@@ -31,7 +31,7 @@
       <origin xyz="0.0 0.0 0.0" rpy="${-M_PI/2} 0 ${-M_PI/2}" />
       <parent link="${prefix}_rgb_base_link" />
-      <child link="${prefix}_rgb_optical_frame_link" />
+      <child link="${prefix}_rgb_optical_frame" />
     </joint>
-    <link name="${prefix}_rgb_optical_frame_link">
+    <link name="${prefix}_rgb_optical_frame">
       <!--inertial>
         <mass value="0.001" />
@@ -77,7 +77,7 @@
       <origin xyz="${orbbec_astra_depth_rel_rgb_px} ${orbbec_astra_depth_rel_rgb_py} ${orbbec_astra_depth_rel_rgb_pz}" rpy="0 0 0" />
       <parent link="${prefix}_rgb_base_link" />
-      <child link="${prefix}_depth_frame_link" />
+      <child link="${prefix}_depth_frame" />
     </joint>
-    <link name="${prefix}_depth_frame_link">
+    <link name="${prefix}_depth_frame">
       <!--inertial>
         <mass value="0.01" />
@@ -90,8 +90,8 @@
     <joint name="${prefix}_depth_optical_joint" type="fixed">
       <origin xyz="0 0 0" rpy="${-M_PI/2} 0 ${-M_PI/2}" />
-      <parent link="${prefix}_depth_frame_link" />
-      <child link="${prefix}_depth_optical_frame_link" />
+      <parent link="${prefix}_depth_frame" />
+      <child link="${prefix}_depth_optical_frame" />
     </joint>
-    <link name="${prefix}_depth_optical_frame_link">
+    <link name="${prefix}_depth_optical_frame">
       <!--inertial>
         <mass value="0.001" />
@@ -131,5 +131,5 @@
           <cameraInfoTopicName>rgb/camera_info</cameraInfoTopicName>
           <depthImageCameraInfoTopicName>depth/camera_info</depthImageCameraInfoTopicName>
-          <frameName>${prefix}_depth_optical_frame_link</frameName>
+          <frameName>${prefix}_depth_optical_frame</frameName>
           <baseline>0.1</baseline>
           <distortion_k1>0.0</distortion_k1>

Commit message: adding prefix topic for the orbbec astra

File: urdf/orbbec_astra.urdf.xacro (robot description, xacro)
@@ -13,5 +13,5 @@
   <xacro:property name="orbbec_astra_depth_rel_rgb_pz" value="0.0" />
   <xacro:property name="M_PI" value="3.1415926535897931" />
-  <xacro:macro name="sensor_orbbec_astra" params="prefix parent *origin">
+  <xacro:macro name="sensor_orbbec_astra" params="prefix parent prefix_topic *origin">
     <joint name="${prefix}_rgb_joint" type="fixed">
 	  <xacro:insert_block name="origin" />
@@ -123,5 +123,5 @@
         </camera>
         <plugin name="${prefix}_controller" filename="libgazebo_ros_openni_kinect.so">
-          <cameraName>orbbec_astra</cameraName>
+          <cameraName>${prefix_topic}</cameraName>
           <alwaysOn>true</alwaysOn>
           <updateRate>10</updateRate>

Commit message: changing collision geometry for the orbbec

File: urdf/orbbec_astra.urdf.xacro (robot description, xacro)
@@ -57,7 +57,10 @@
       <collision>
         <origin xyz="0.0 0.0 0.0" rpy="0 0 0" />
-        <geometry>
+        <!--geometry>
         <box size="0.0730 .2760 0.0720"/>
-      </geometry>
+      </geometry-->
+      <geometry>
+          <mesh filename="package://robotnik_sensors/meshes/orbbec_astra.dae" scale="${orbbec_astra_scale} ${orbbec_astra_scale} ${orbbec_astra_scale}"/>
+        </geometry>
       </collision>
       <inertial>

Commit message: Fix orbbec astra inertia

File: urdf/orbbec_astra.urdf.xacro (robot description, xacro)
@@ -21,9 +21,7 @@
     <link name="${prefix}_rgb_base_link">
       <inertial>
-        <mass value="0.001" />
-        <origin xyz="0 0 0" />
-        <inertia ixx="0.0001" ixy="0.0" ixz="0.0"
-          iyy="0.0001" iyz="0.0"
-          izz="0.0001" />
+        <mass value="0.297" />
+        <origin xyz="-0.02 -0.0125 0.0" />
+        <xacro:solid_cuboid_inertia m="0.297" w="0.04" h="0.165" d="0.03" />
       </inertial>
     </link>
@@ -34,11 +32,9 @@
     </joint>
     <link name="${prefix}_rgb_optical_frame">
-      <!--inertial>
+      <inertial>
         <mass value="0.001" />
-        <origin xyz="0 0 0" />
-        <inertia ixx="0.0001" ixy="0.0" ixz="0.0"
-          iyy="0.0001" iyz="0.0"
-          izz="0.0001" />
-      </inertial-->
+        <origin xyz="0 0 0" rpy="${M_PI/2} 0 ${M_PI/2}"/>
+        <xacro:solid_cuboid_inertia m="0.001" w="0.04" h="0.165" d="0.03" />
+      </inertial>
     </link>
     <joint name="${prefix}_joint" type="fixed">
@@ -56,23 +52,12 @@
       </visual>
       <collision>
-        <origin xyz="0.0 0.0 0.0" rpy="0 0 0" />
-        <!--geometry>
-        <box size="0.0730 .2760 0.0720"/>
-      </geometry-->
-      <geometry>
+        <geometry>
           <mesh filename="package://robotnik_sensors/meshes/orbbec_astra.dae" scale="${orbbec_astra_scale} ${orbbec_astra_scale} ${orbbec_astra_scale}"/>
         </geometry>
       </collision>
       <inertial>
-        <!--mass value="0.01" />
-        <origin xyz="0 0 0" />
-        <inertia ixx="0.001" ixy="0.0" ixz="0.0"
-          iyy="0.001" iyz="0.0"
-          izz="0.001" /-->
-          <mass value="0.564" />
-          <origin xyz="0 0 0" />
-          <inertia ixx="0.003881243" ixy="0.0" ixz="0.0"
-                   iyy="0.000498940" iyz="0.0"
-                   izz="0.003879257" />
+        <mass value="0.001" />
+        <origin xyz="0.0 0.0 0.0" />
+        <xacro:solid_cuboid_inertia m="0.001" w="0.04" h="0.165" d="0.03" />
        </inertial>
     </link>
@@ -83,11 +68,9 @@
     </joint>
     <link name="${prefix}_depth_frame">
-      <!--inertial>
-        <mass value="0.01" />
+      <inertial>
+        <mass value="0.001" />
         <origin xyz="0 0 0" />
-        <inertia ixx="0.001" ixy="0.0" ixz="0.0"
-          iyy="0.001" iyz="0.0"
-          izz="0.001" />
-      </inertial-->
+        <xacro:solid_cuboid_inertia m="0.001" w="0.04" h="0.165" d="0.03" />
+      </inertial>
     </link>
     <joint name="${prefix}_depth_optical_joint" type="fixed">
@@ -97,14 +80,12 @@
     </joint>
     <link name="${prefix}_depth_optical_frame">
-      <!--inertial>
+      <inertial>
         <mass value="0.001" />
         <origin xyz="0 0 0" />
-        <inertia ixx="0.0001" ixy="0.0" ixz="0.0"
-          iyy="0.0001" iyz="0.0"
-          izz="0.0001" />
-      </inertial-->
+        <xacro:solid_cuboid_inertia m="0.001" w="0.04" h="0.165" d="0.03" />
+      </inertial>
     </link>
   <!-- RGBD sensor for simulation, same as Kinect -->
-  <sensor_orbbec_astra_gazebo/>
+  <!--sensor_orbbec_astra_gazebo/-->
   </xacro:macro>
    <xacro:macro name="sensor_orbbec_astra_gazebo">

Commit message: changed orbbec astra tf tree, the transformations between final frames have been preserved

File: urdf/orbbec_astra.urdf.xacro (robot description, xacro)
@@ -1,23 +1,34 @@
 <?xml version="1.0"?>
-<robot name="sensor_orbbec_astra" xmlns:xacro="http://wiki.ros.org/xacro">
-  <!-- Xacro properties -->
-  <!--xacro:property name="orbbec_astra_scale" value="0.015"/-->
-  <xacro:property name="orbbec_astra_scale" value="1.0"/>
-  <!-- RGB sensor - cam -->
-  <xacro:property name="orbbec_astra_rel_rgb_px"   value="0.0" />
-  <xacro:property name="orbbec_astra_rel_rgb_py"   value="-0.0125" />
-  <xacro:property name="orbbec_astra_rel_rgb_pz"   value="-0.0150" />
-  <!-- IR sensor - depth -->
-  <xacro:property name="orbbec_astra_depth_rel_rgb_px" value="0.0" />
-  <xacro:property name="orbbec_astra_depth_rel_rgb_py" value="0.0250" />
-  <xacro:property name="orbbec_astra_depth_rel_rgb_pz" value="0.0" />
-  <xacro:property name="M_PI" value="3.1415926535897931" />
+<robot name="sensor_orbbec_astra" xmlns:xacro="http://wiki.ros.org/Sensors/OrbbecAstra">
   <xacro:macro name="sensor_orbbec_astra" params="prefix parent prefix_topic:='front_rgbd_camera' *origin">
+    <joint name="${prefix}_joint" type="fixed">
+    	<xacro:insert_block name="origin" />
+      <parent link="${parent}"/>
+      <child link="${prefix}_link"/>
+    </joint>
+    <link name="${prefix}_link">
+      <visual>
+        <origin xyz="0 0 0" rpy="0 0 0"/>
+        <geometry>
+          <mesh filename="package://robotnik_sensors/meshes/orbbec_astra.dae"/>
+        </geometry>
+      </visual>
+      <collision>
+        <geometry>
+          <mesh filename="package://robotnik_sensors/meshes/orbbec_astra.dae"/>
+        </geometry>
+      </collision>
+      <inertial>
+        <mass value="0.001" />
+        <origin xyz="0.0 0.0 0.0" />
+        <xacro:solid_cuboid_inertia m="0.001" w="0.04" h="0.165" d="0.03" />
+      </inertial>
+    </link>
     <joint name="${prefix}_rgb_joint" type="fixed">
-	  <xacro:insert_block name="origin" />
-      <parent link="${parent}"/>
-      <child link="${prefix}_rgb_base_link" />
+      <origin xyz="0.0 0.0125 0.0150" rpy="0.0 0.0 0.0"/>
+      <parent link="${prefix}_link"/>
+      <child link="${prefix}_rgb_frame" />
     </joint>
-    <link name="${prefix}_rgb_base_link">
+    <link name="${prefix}_rgb_frame">
       <inertial>
         <mass value="0.297" />
@@ -28,5 +39,5 @@
     <joint name="${prefix}_rgb_optical_joint" type="fixed">
       <origin xyz="0.0 0.0 0.0" rpy="${-M_PI/2} 0 ${-M_PI/2}" />
-      <parent link="${prefix}_rgb_base_link" />
+      <parent link="${prefix}_rgb_frame" />
       <child link="${prefix}_rgb_optical_frame" />
     </joint>
@@ -38,31 +49,7 @@
       </inertial>
     </link>
-    <joint name="${prefix}_joint" type="fixed">
-      <origin xyz="${orbbec_astra_rel_rgb_px} ${orbbec_astra_rel_rgb_py} ${orbbec_astra_rel_rgb_pz}"
-              rpy="0.0 0 0"/>
-      <parent link="${prefix}_rgb_base_link"/>
-      <child link="${prefix}_link"/>
-    </joint>
-    <link name="${prefix}_link">
-      <visual>
-        <origin xyz="0 0 0" rpy="0 0 0"/>
-        <geometry>
-          <mesh filename="package://robotnik_sensors/meshes/orbbec_astra.dae" scale="${orbbec_astra_scale} ${orbbec_astra_scale} ${orbbec_astra_scale}"/>
-        </geometry>
-      </visual>
-      <collision>
-        <geometry>
-          <mesh filename="package://robotnik_sensors/meshes/orbbec_astra.dae" scale="${orbbec_astra_scale} ${orbbec_astra_scale} ${orbbec_astra_scale}"/>
-        </geometry>
-      </collision>
-      <inertial>
-        <mass value="0.001" />
-        <origin xyz="0.0 0.0 0.0" />
-        <xacro:solid_cuboid_inertia m="0.001" w="0.04" h="0.165" d="0.03" />
-       </inertial>
-    </link>
     <joint name="${prefix}_depth_joint" type="fixed">
-      <origin xyz="${orbbec_astra_depth_rel_rgb_px} ${orbbec_astra_depth_rel_rgb_py} ${orbbec_astra_depth_rel_rgb_pz}" rpy="0 0 0" />
-      <parent link="${prefix}_rgb_base_link" />
+      <origin xyz="0.0 0.0375 0.0150" rpy="0 0 0" />
+      <parent link="${prefix}_link" />
       <child link="${prefix}_depth_frame" />
     </joint>
@@ -87,5 +74,5 @@
     </link>
   <!-- RGBD sensor for simulation, same as Kinect -->
-  <!--sensor_orbbec_astra_gazebo/-->
+  <sensor_orbbec_astra_gazebo/>
   </xacro:macro>
    <xacro:macro name="sensor_orbbec_astra_gazebo">

Commit message: Adds offset to the orbec depth

File: urdf/orbbec_astra.urdf.xacro (robot description, xacro)
@@ -1,5 +1,5 @@
 <?xml version="1.0"?>
 <robot name="sensor_orbbec_astra" xmlns:xacro="http://wiki.ros.org/Sensors/OrbbecAstra">
-  <xacro:macro name="sensor_orbbec_astra" params="prefix parent prefix_topic:='front_rgbd_camera' *origin">
+  <xacro:macro name="sensor_orbbec_astra" params="prefix parent prefix_topic:='front_rgbd_camera' *origin depth_offset_x:=0 depth_offset_y:=0 depth_offset_z:=0">
     <joint name="${prefix}_joint" type="fixed">
     	<xacro:insert_block name="origin" />
@@ -62,5 +62,5 @@
     </link>
     <joint name="${prefix}_depth_optical_joint" type="fixed">
-      <origin xyz="0 0 0" rpy="${-M_PI/2} 0 ${-M_PI/2}" />
+      <origin xyz="${depth_offset_x} ${depth_offset_y} ${depth_offset_z}" rpy="${-M_PI/2} 0 ${-M_PI/2}" />
       <parent link="${prefix}_depth_frame" />
       <child link="${prefix}_depth_optical_frame" />
