Commit message: Updated orbbec_astra gazebo and namespace

File: urdf/orbbec_astra.urdf.xacro (robot description, xacro)
@@ -1,5 +1,5 @@
 <?xml version="1.0"?>
 <robot name="sensor_orbbec_astra" xmlns:xacro="http://wiki.ros.org/Sensors/OrbbecAstra">
-  <xacro:macro name="sensor_orbbec_astra" params="prefix parent prefix_topic:='front_rgbd_camera' *origin depth_offset_x:=0 depth_offset_y:=0 depth_offset_z:=0">
+  <xacro:macro name="sensor_orbbec_astra" params="ns prefix parent *origin">
     <joint name="${prefix}_joint" type="fixed">
     	<xacro:insert_block name="origin" />
@@ -11,16 +11,16 @@
         <origin xyz="0 0 0" rpy="0 0 0"/>
         <geometry>
-          <mesh filename="package://robotnik_sensors/meshes/orbbec_astra.dae"/>
+          <mesh filename="file://$(find robotnik_sensors)/meshes/orbbec_astra.dae"/>
         </geometry>
       </visual>
       <collision>
         <geometry>
-          <mesh filename="package://robotnik_sensors/meshes/orbbec_astra.dae"/>
+          <box size="0.1 0.1 0.1"/>
         </geometry>
       </collision>
       <inertial>
-        <mass value="0.001" />
+        <mass value="0.3" />
         <origin xyz="0.0 0.0 0.0" />
-        <xacro:solid_cuboid_inertia m="0.001" w="0.04" h="0.165" d="0.03" />
+        <xacro:solid_cuboid_inertia m="0.3" w="0.04" h="0.165" d="0.03" />
       </inertial>
     </link>
@@ -62,5 +62,5 @@
     </link>
     <joint name="${prefix}_depth_optical_joint" type="fixed">
-      <origin xyz="${depth_offset_x} ${depth_offset_y} ${depth_offset_z}" rpy="${-M_PI/2} 0 ${-M_PI/2}" />
+      <origin xyz="0 0 0" rpy="${-M_PI/2} 0 ${-M_PI/2}" />
       <parent link="${prefix}_depth_frame" />
       <child link="${prefix}_depth_optical_frame" />
@@ -73,14 +73,97 @@
       </inertial>
     </link>
-  <!-- RGBD sensor for simulation, same as Kinect -->
   <xacro:sensor_orbbec_astra_gazebo/>
+  <xacro:sensor_orbbec_astra_gazebo/>
+    <xacro:sensor_orbbec_astra_gazebo/>
   </xacro:macro>
-   <xacro:macro name="sensor_orbbec_astra_gazebo">
+  <xacro:macro name="sensor_orbbec_astra_gazebo">
+    <xacro:property name="deg_to_rad" value="0.01745329251994329577" />
     <gazebo reference="${prefix}_link">
-      <sensor type="depth" name="${prefix}_depth_sensor">
-        <always_on>true</always_on>
-        <update_rate>20.0</update_rate>
-        <camera>
-          <horizontal_fov>${60.0*M_PI/180.0}</horizontal_fov>
+      <self_collide>0</self_collide>
+      <enable_wind>0</enable_wind>
+      <kinematic>0</kinematic>
+      <gravity>1</gravity>
+      <!--<mu>1</mu>-->
+      <mu2>1</mu2>
+      <fdir1>0 0 0</fdir1>
+      <!--<slip1>0</slip1>
+      <slip2>0</slip2>-->
+      <kp>1e+13</kp>
+      <kd>1</kd>
+      <!--<max_vel>0.01</max_vel>
+      <min_depth>0</min_depth>-->
+      <sensor name="${prefix}color" type="camera">
+        <camera name="${prefix}">
+          <vertical_fov>${49.5*deg_to_rad}</vertical_fov>
+          <horizontal_fov>${60*deg_to_rad}</horizontal_fov>
+          <image>
+            <format>RGB_INT8</format>
+            <width>1280</width>
+            <height>960</height>
+          </image>
+          <clip>
+            <near>0.1</near>
+            <far>100</far>
+          </clip>
+          <noise>
+            <type>gaussian</type>
+            <mean>0.0</mean>
+            <stddev>0.004</stddev>
+          </noise>
+        </camera>
+        <always_on>1</always_on>
+        <update_rate>10</update_rate>
+        <visualize>false</visualize>
+      </sensor>
+      <sensor name="${prefix}ired1" type="camera">
+        <camera name="${prefix}">
+          <vertical_fov>${49.5*deg_to_rad}</vertical_fov>
+          <horizontal_fov>${60*deg_to_rad}</horizontal_fov>
+          <image>
+            <format>L_INT8</format>
+            <width>640</width>
+            <height>480</height>
+          </image>
+          <clip>
+            <near>0.1</near>
+            <far>100</far>
+          </clip>
+          <noise>
+            <type>gaussian</type>
+            <mean>0.0</mean>
+            <stddev>0.004</stddev>
+          </noise>
+        </camera>
+        <always_on>1</always_on>
+        <update_rate>10</update_rate>
+        <visualize>false</visualize>
+      </sensor>
+      <sensor name="${prefix}ired2" type="camera">
+        <camera name="${prefix}">
+          <vertical_fov>${49.5*deg_to_rad}</vertical_fov>
+          <horizontal_fov>${60*deg_to_rad}</horizontal_fov>
+          <image>
+            <format>L_INT8</format>
+            <width>640</width>
+            <height>480</height>
+          </image>
+          <clip>
+            <near>0.1</near>
+            <far>100</far>
+          </clip>
+          <noise>
+            <type>gaussian</type>
+            <mean>0.0</mean>
+            <stddev>0.004</stddev>
+          </noise>
+        </camera>
+        <always_on>1</always_on>
+        <update_rate>30</update_rate>
+        <visualize>false</visualize>
+      </sensor>
+      <sensor name="${prefix}depth" type="depth">
+        <camera name="${prefix}">
+          <vertical_fov>${49.5*deg_to_rad}</vertical_fov>
+          <horizontal_fov>${60*deg_to_rad}</horizontal_fov>
           <image>
             <format>R8G8B8</format>
@@ -89,27 +172,42 @@
           </image>
           <clip>
-            <near>0.05</near>
-            <far>3.5</far>
-          </clip>
-        </camera>
-        <plugin name="${prefix}_controller" filename="libgazebo_ros_openni_kinect.so">
-          <cameraName>${prefix_topic}</cameraName>
-          <alwaysOn>true</alwaysOn>
-          <updateRate>10</updateRate>
-          <imageTopicName>rgb/image_raw</imageTopicName>
-          <depthImageTopicName>depth/image_raw</depthImageTopicName>
-          <pointCloudTopicName>depth/points</pointCloudTopicName>
-          <cameraInfoTopicName>rgb/camera_info</cameraInfoTopicName>
-          <depthImageCameraInfoTopicName>depth/camera_info</depthImageCameraInfoTopicName>
-          <frameName>/${prefix}_depth_optical_frame</frameName>
-          <baseline>0.1</baseline>
-          <distortion_k1>0.0</distortion_k1>
-          <distortion_k2>0.0</distortion_k2>
-          <distortion_k3>0.0</distortion_k3>
-          <distortion_t1>0.0</distortion_t1>
-          <distortion_t2>0.0</distortion_t2>
-          <pointCloudCutoff>0.4</pointCloudCutoff>
-        </plugin>
-      </sensor>
+            <near>0.1</near>
+            <far>100</far>
+          </clip>
+          <noise>
+            <type>gaussian</type>
+            <mean>0.0</mean>
+            <stddev>0.004</stddev>
+          </noise>
+        </camera>
+        <always_on>1</always_on>
+        <update_rate>10</update_rate>
+        <visualize>false</visualize>
+      </sensor>
+    </gazebo>
+    <gazebo>
+      <plugin name="${ns}" filename="librealsense_gazebo_plugin.so">
+        <prefix>${prefix}</prefix>
+        <depthUpdateRate>60.0</depthUpdateRate>
+        <colorUpdateRate>60.0</colorUpdateRate>
+        <infraredUpdateRate>60.0</infraredUpdateRate>
+        <depthTopicName>${ns}/${prefix}/depth/image_raw</depthTopicName>
+        <depthCameraInfoTopicName>${ns}/${prefix}/depth/camera_info</depthCameraInfoTopicName>
+        <colorTopicName>${ns}/${prefix}/color/image_raw</colorTopicName>
+        <colorCameraInfoTopicName>${ns}/${prefix}/color/camera_info</colorCameraInfoTopicName>
+        <infrared1TopicName>${ns}/${prefix}/infra1/image_rect_raw</infrared1TopicName>
+        <infrared1CameraInfoTopicName>${ns}/${prefix}/infra1/camera_info</infrared1CameraInfoTopicName>
+        <infrared2TopicName>${ns}/${prefix}/infra2/image_rect_raw</infrared2TopicName>
+        <infrared2CameraInfoTopicName>${ns}/${prefix}/infra2/camera_info</infrared2CameraInfoTopicName>
+        <colorOpticalframeName>${ns}/${prefix}_rgb_optical_frame</colorOpticalframeName>
+        <depthOpticalframeName>${ns}/${prefix}_depth_optical_frame</depthOpticalframeName>
+        <infrared1OpticalframeName>${ns}/${prefix}_left_ir_optical_frame</infrared1OpticalframeName>
+        <infrared2OpticalframeName>${ns}/${prefix}_right_ir_optical_frame</infrared2OpticalframeName>
+        <rangeMinDepth>0.4</rangeMinDepth>
+        <rangeMaxDepth>6.0</rangeMaxDepth>
+        <pointCloud>true</pointCloud>
+        <pointCloudTopicName>${ns}/${prefix}/depth/color/points</pointCloudTopicName>
+        <pointCloudCutoff>0.5</pointCloudCutoff>
+      </plugin>
     </gazebo>
   </xacro:macro>
