Commit message: Add params to set laser angle limits for sick_microscan

File: urdf/sick_microscan3.urdf.xacro (robot description, xacro)
@@ -2,5 +2,5 @@
 <robot name="sensor_sick_microscan3"
 	xmlns:xacro="http://www.ros.org/wiki/xacro">
-	<xacro:macro name="sensor_sick_microscan3" params="prefix parent prefix_topic:='front_laser' *origin">
+	<xacro:macro name="sensor_sick_microscan3" params="prefix parent prefix_topic:='front_laser' *origin max_angle:=2.3562 min_angle:=-2.3562">
 		<joint name="${prefix}_base_joint" type="fixed">
 			<xacro:insert_block name="origin" />
@@ -49,6 +49,6 @@
 							<samples>541</samples>
 							<resolution>1</resolution>
-							<min_angle>-2.3562</min_angle>
-							<max_angle>2.3562</max_angle>
+							<min_angle>${min_angle}</min_angle>
+							<max_angle>${max_angle}</max_angle>
 						</horizontal>
 					</scan>

Commit message: Fix sick microscan3 inertia

File: urdf/sick_microscan3.urdf.xacro (robot description, xacro)
@@ -24,7 +24,7 @@
 			</visual>
 			<inertial>
-				<mass value="1e-5" />
-				<origin xyz="0 0 0" rpy="0 0 0"/>
-				<inertia ixx="1e-6" ixy="0" ixz="0" iyy="1e-6" iyz="0" izz="1e-6" />
+				<mass value="1.15" />
+				<origin xyz="0 0 0.075" rpy="0 0 0"/>
+				<xacro:solid_cuboid_inertia m="1.15" w="0.112" h="0.111" d="0.15" />
 			</inertial>
 		</link>

Commit message: sick_microscan3: Simplified collision

File: urdf/sick_microscan3.urdf.xacro (robot description, xacro)
@@ -10,9 +10,9 @@
 		<link name="${prefix}_base_link">
 			<collision>
-				<origin xyz="0 0 0" rpy="0 0 0"/>
+				<origin xyz="0 0 0.075" rpy="0 0 0"/>
 				<geometry>
-					<!--<box size="0.106 0.094 0.152"/>-->
+					<box size="0.106 0.094 0.152"/>
 					<!--<cylinder radius="0.058" length="0.152"/>-->
-					<mesh filename="package://robotnik_sensors/meshes/sick_microscan3.dae"/>
+					<!--<mesh filename="package://robotnik_sensors/meshes/sick_microscan3.dae"/>-->
 				</geometry>
 			</collision>

Commit message: changed the angle_max and angle_min parameters of the lidar

File: urdf/sick_microscan3.urdf.xacro (robot description, xacro)
@@ -2,5 +2,5 @@
 <robot name="sensor_sick_microscan3"
 	xmlns:xacro="http://wiki.ros.org/xacro">
-	<xacro:macro name="sensor_sick_microscan3" params="prefix parent prefix_topic:='front_laser' *origin max_angle:=2.3562 min_angle:=-2.3562 gpu:=^|true">
+	<xacro:macro name="sensor_sick_microscan3" params="prefix parent prefix_topic:='front_laser' *origin max_angle:=2.2465 min_angle:=-2.2465 gpu:=^|true">
 		<joint name="${prefix}_base_joint" type="fixed">
 			<xacro:insert_block name="origin" />
