Commit message: Add ouster mesh

File: urdf/ouster1.urdf.xacro (robot description, xacro)
@@ -15,5 +15,5 @@
         <origin xyz="0 0 0" rpy="0 0 0"/>
         <geometry>
-          <mesh filename="package://robotnik_sensors/meshes/rslidar.stl"/>
+          <mesh filename="package://robotnik_sensors/meshes/ouster1.STL"/>
         </geometry>
         <material name="black_alu"/>
@@ -22,5 +22,5 @@
         <origin xyz="0 0 0" rpy="0 0 0"/>
         <geometry>
-          <mesh filename="package://robotnik_sensors/meshes/rslidar.stl"/>
+          <mesh filename="package://robotnik_sensors/meshes/ouster1.STL"/>
         </geometry>
       </collision>

Commit message: Update ouster1 inertia

File: urdf/ouster1.urdf.xacro (robot description, xacro)
@@ -26,8 +26,7 @@
       </collision>
       <inertial>
-        <mass value="0.380" />
-        <origin xyz="0 0 0" />
-        <!-- The following are not reliable values, and should not be used for modeling -->
-        <inertia ixx="0.003881243" ixy="0.0" ixz="0.0" iyy="0.000498940" iyz="0.0" izz="0.003879257" />
+        <origin xyz="-0.0 0.0 0.029" rpy="0 0 0" />
+        <mass value="3.5" />
+        <xacro:solid_cuboid_inertia m="3.5" w="0.06" h="0.06" d="0.058" />
       </inertial>
     </link>

Commit message: Update ouster lidar stl

File: urdf/ouster1.urdf.xacro (robot description, xacro)
@@ -12,5 +12,6 @@
         <origin xyz="0 0 0" rpy="0 0 0"/>
         <geometry>
-          <mesh filename="package://robotnik_sensors/meshes/ouster1.STL"/>
+	  <mesh filename="package://robotnik_sensors/meshes/lidar3d_os1.stl"/>
+          <!--mesh filename="package://robotnik_sensors/meshes/ouster1.STL"/-->
         </geometry>
         <material name="black_alu"/>
@@ -19,5 +20,5 @@
         <origin xyz="0 0 0" rpy="0 0 0"/>
         <geometry>
-          <mesh filename="package://robotnik_sensors/meshes/ouster1.STL"/>
+          <mesh filename="package://robotnik_sensors/meshes/lidar3d_os1.stl"/>
         </geometry>
       </collision>
