Commit message: Setting TIM571 params

File: urdf/sick_tim571.urdf.xacro (robot description, xacro)
@@ -1,5 +1,5 @@
 <?xml version="1.0"?>
 <robot xmlns:xacro="http://ros.org/wiki/xacro">
-  <xacro:macro name="sensor_sick_tim571" params="prefix parent *origin min_angle:=-0.785398 max_angle:=3.92699">
+  <xacro:macro name="sensor_sick_tim571" params="prefix parent *origin min_angle:=-2.36 max_angle:=2.36">
     <joint name="${prefix}laser_base_joint" type="fixed">
       <insert_block name="origin" />
@@ -40,9 +40,9 @@
 				<pose>0 0 0 0 0 0</pose>
 				<visualize>false</visualize>
-				<update_rate>10</update_rate>
+				<update_rate>15</update_rate>
 				<ray>
 					<scan>
 						<horizontal>
-							<samples>361</samples>
+							<samples>819</samples>
 							<resolution>1</resolution>
 							<min_angle>${min_angle}</min_angle>
@@ -51,7 +51,7 @@
 					</scan>
 					<range>
-						<min>0.15</min>
-						<max>6.0</max>
-						<resolution>0.0174</resolution>
+						<min>0.05</min>
+						<max>25.0</max>
+						<resolution>0.00575</resolution>
 					</range>
 					<noise>

Commit message: Update sick tim571 inertia

File: urdf/sick_tim571.urdf.xacro (robot description, xacro)
@@ -21,7 +21,7 @@
       </visual>
       <inertial>
-        <mass value="1e-5" />
-        <origin xyz="0 0 0" rpy="0 0 0"/>
-        <inertia ixx="1e-6" ixy="0" ixz="0" iyy="1e-6" iyz="0" izz="1e-6" />
+        <mass value="0.25" />
+        <origin xyz="0 0 0.042875" rpy="0 0 0"/>
+        <xacro:solid_cuboid_inertia m="0.25" w="0.061" h="0.06" d="0.08575" />
       </inertial>
     </link>

Commit message: Fix sick tim571 inertia

File: urdf/sick_tim571.urdf.xacro (robot description, xacro)
@@ -22,5 +22,5 @@
       <inertial>
         <mass value="0.25" />
-        <origin xyz="0 0 0.042875" rpy="0 0 0"/>
+        <origin xyz="-0.0017 0 0.042875" rpy="0 0 0"/>
         <xacro:solid_cuboid_inertia m="0.25" w="0.061" h="0.06" d="0.08575" />
       </inertial>

Commit message: Added gpu functionality laser and 3D lidar velodyne

File: urdf/sick_tim571.urdf.xacro (robot description, xacro)
@@ -1,5 +1,5 @@
 <?xml version="1.0"?>
 <robot xmlns:xacro="http://wiki.ros.org/xacro">
-  <xacro:macro name="sensor_sick_tim571" params="ns prefix parent *origin min_angle:=-2.3562 max_angle:=2.3562">
+  <xacro:macro name="sensor_sick_tim571" params="ns prefix parent *origin min_angle:=-2.3562 max_angle:=2.3562 gpu:=false">
     <joint name="${prefix}_base_joint" type="fixed">
       <xacro:insert_block name="origin" />
@@ -32,42 +32,48 @@
     </joint>
     <link name="${prefix}_link"/>
-    <xacro:sensor_sick_tim571_gazebo/>
+    <xacro:sensor_sick_tim571_gazebo ns="${ns}" prefix="${prefix}" min_angle="${min_angle}" max_angle="${max_angle}" gpu="${gpu}"/>
   </xacro:macro>
-  <xacro:macro name="sensor_sick_tim571_gazebo">
+  <xacro:macro name="sensor_sick_tim571_gazebo" params="ns prefix min_angle max_angle gpu">
+    <xacro:if value="${gpu}">
+      <xacro:property name="ray_type" value="gpu_ray" />
+    </xacro:if>
+    <xacro:unless value="${gpu}">
+      <xacro:property name="ray_type" value="ray" />
+    </xacro:unless>
     <gazebo reference="${prefix}_link">
-    <sensor type="ray" name="${prefix}_sensor">
-      <pose>0 0 0 0 0 0</pose>
-      <visualize>false</visualize>
-      <update_rate>15</update_rate>
-      <ray>
-        <scan>
-          <horizontal>
-            <samples>819</samples>
-            <resolution>1</resolution>
-            <min_angle>${min_angle}</min_angle>
-            <max_angle>${max_angle}</max_angle>
-          </horizontal>
-        </scan>
-        <range>
-          <min>0.05</min>
-          <max>25.0</max>
-          <resolution>0.00575</resolution>
-        </range>
-        <noise>
-          <type>gaussian</type>
-          <mean>0.0</mean>
-          <stddev>0.01</stddev>
-        </noise>
-      </ray>
-      <plugin name="${prefix}" filename="libgazebo_ros_ray_sensor.so">
-        <ros>
-          <namespace>${ns}</namespace>
-          <remapping>~/out:=~/scan</remapping>
-        </ros>
-        <output_type>sensor_msgs/LaserScan</output_type>
-        <frame_name>${ns}/${prefix}_link</frame_name>
-      </plugin>
-    </sensor>
-  </gazebo>
+      <sensor type="${ray_type}" name="${prefix}_sensor">
+        <pose>0 0 0 0 0 0</pose>
+        <visualize>false</visualize>
+        <update_rate>15</update_rate>
+        <ray>
+          <scan>
+            <horizontal>
+              <samples>819</samples>
+              <resolution>1</resolution>
+              <min_angle>${min_angle}</min_angle>
+              <max_angle>${max_angle}</max_angle>
+            </horizontal>
+          </scan>
+          <range>
+            <min>0.05</min>
+            <max>25.0</max>
+            <resolution>0.00575</resolution>
+          </range>
+          <noise>
+            <type>gaussian</type>
+            <mean>0.0</mean>
+            <stddev>0.01</stddev>
+          </noise>
+        </ray>
+        <plugin name="${prefix}" filename="libgazebo_ros_ray_sensor.so">
+          <ros>
+            <namespace>${ns}</namespace>
+            <remapping>~/out:=~/scan</remapping>
+          </ros>
+          <output_type>sensor_msgs/LaserScan</output_type>
+          <frame_name>${ns}/${prefix}_link</frame_name>
+        </plugin>
+      </sensor>
+    </gazebo>
   </xacro:macro>
 </robot>

File: urdf/velodyne_vlp16.urdf.xacro (robot description, xacro)
@@ -1,5 +1,5 @@
 <?xml version="1.0"?>
 <robot name="sensor_velodyne_vlp16" xmlns:xacro="http://wiki.ros.org/xacro">
-  <xacro:macro name="sensor_velodyne_vlp16" params="prefix parent prefix_topic:='velodyne' *origin range_min range_max gpu:=^|true">
+  <xacro:macro name="sensor_velodyne_vlp16" params="ns prefix parent *origin range_min:=0.1 range_max:=20.0 gpu:=false">
     <joint name="${prefix}_base_joint" type="fixed">
       <xacro:insert_block name="origin" />
@@ -8,21 +8,21 @@
     </joint>
     <link name="${prefix}_base_link">
-        <collision>
-            <origin xyz="0 0 0" rpy="0 0 0"/>
-            <geometry>
-                <mesh filename="file://$(find robotnik_sensors)/meshes/velodyne_vlp16.dae"/>
-            </geometry>
-        </collision>
-        <visual>
-            <origin xyz="0 0 0" rpy="0 0 0"/>
-            <geometry>
-                <mesh filename="file://$(find robotnik_sensors)/meshes/velodyne_vlp16.dae"/>
-            </geometry>
-        </visual>
-        <inertial>
-            <mass value="0.830" />
-            <origin xyz="0 0 0.03555" rpy="0 0 0"/>
-            <xacro:solid_cuboid_inertia m="0.830" w="0.1033" h="0.1033" d="0.0711" />
-        </inertial>
+      <collision>
+        <origin xyz="0 0 0" rpy="0 0 0"/>
+        <geometry>
+          <mesh filename="file://$(find robotnik_sensors)/meshes/velodyne_vlp16.dae"/>
+        </geometry>
+      </collision>
+      <visual>
+        <origin xyz="0 0 0" rpy="0 0 0"/>
+        <geometry>
+          <mesh filename="file://$(find robotnik_sensors)/meshes/velodyne_vlp16.dae"/>
+        </geometry>
+      </visual>
+      <inertial>
+        <mass value="0.830" />
+        <origin xyz="0 0 0.03555" rpy="0 0 0"/>
+        <xacro:solid_cuboid_inertia m="0.830" w="0.1033" h="0.1033" d="0.0711" />
+      </inertial>
     </link>
     <joint name="${prefix}_joint" type="fixed">
@@ -31,55 +31,52 @@
       <origin xyz="0.0 0 0.035" rpy="0 0 0"/>
     </joint>
-    <link name="${prefix}_link">
-    </link>
-    <!-- Velodyne sensor for simulation -->
-    <xacro:sensor_velodyne_vlp16_gazebo range_min="${range_min}" range_max="${range_max}" gpu="${gpu}" />
+    <link name="${prefix}_link"/>
+    <xacro:sensor_velodyne_vlp16_gazebo ns="${ns}" prefix="${prefix}" range_min="${range_min}" range_max="${range_max}" gpu="${gpu}"/>
   </xacro:macro>
-  <xacro:macro name="sensor_velodyne_vlp16_gazebo" params="range_min range_max gpu">
+  <xacro:macro name="sensor_velodyne_vlp16_gazebo" params="ns prefix range_min range_max gpu">
+    <xacro:if value="${gpu}">
+      <xacro:property name="ray_type" value="gpu_ray" />
+    </xacro:if>
+    <xacro:unless value="${gpu}">
+      <xacro:property name="ray_type" value="ray" />
+    </xacro:unless>
     <gazebo reference="${prefix}_link">
-      <xacro:if value="${gpu}">
-        <!-- Using GPU needs: https://github.com/RobotnikAutomation/velodyne_simulator -->
-        <xacro:property name="ray_type" value="gpu_ray" />
-        <xacro:property name="plugin_lib" value="libgazebo_ros_velodyne_gpu_laser.so" />
-      </xacro:if>
-      <xacro:unless value="${gpu}">
-        <xacro:property name="ray_type" value="ray" />
-        <xacro:property name="plugin_lib" value="libgazebo_ros_velodyne_laser.so" />
-      </xacro:unless>
       <sensor type="${ray_type}" name="${prefix}_sensor">
-          <pose>0 0 0 0 0 0</pose>
-          <visualize>false</visualize>
-          <update_rate>15</update_rate>
-          <ray>
-              <scan>
-                  <horizontal>
-                      <samples>300</samples>
-                      <resolution>1.0</resolution>
-                      <min_angle>-1.83591184</min_angle>
-                      <max_angle>1.83591184</max_angle>
-                  </horizontal>
-                  <vertical>
-                      <samples>100</samples>
-                      <resolution>1.0</resolution>
-                      <min_angle>-0.610865238</min_angle>
-                      <max_angle>1.83591184</max_angle>
-                  </vertical>
-              </scan>
-              <range>
-              <min>${range_min}</min>
-              <max>${range_max}</max>
-                  <resolution>0.01</resolution>
-              </range>
-              <noise>
-                  <type>gaussian</type>
-                  <mean>0.0</mean>
-                  <stddev>0.01</stddev>
-              </noise>
-          </ray>
-          <plugin name="${prefix}_controller" filename="${plugin_lib}">
-              <topicName>${prefix_topic}/point_cloud</topicName>
-              <frameName>/${prefix}_link</frameName>
-              <ignoreTfPrefix>1</ignoreTfPrefix>
-          </plugin>
+        <pose>0 0 0 0 0 0</pose>
+        <visualize>false</visualize>
+        <update_rate>10</update_rate>
+        <ray>
+          <scan>
+            <horizontal>
+              <samples>300</samples>
+              <resolution>1.0</resolution>
+              <min_angle>-1.83591184</min_angle>
+              <max_angle>1.83591184</max_angle>
+            </horizontal>
+            <vertical>
+              <samples>100</samples>
+              <resolution>1.0</resolution>
+              <min_angle>-0.610865238</min_angle>
+              <max_angle>1.83591184</max_angle>
+            </vertical>
+          </scan>
+          <range>
+            <min>${range_min}</min>
+            <max>${range_max}</max>
+            <resolution>0.001</resolution>
+          </range>
+          <noise>
+            <type>gaussian</type>
+            <mean>0.0</mean>
+            <stddev>0.00</stddev>
+          </noise>
+        </ray>
+        <plugin name="gazebo_ros_laser_controller" filename="libgazebo_ros_velodyne_laser.so">
+          <topicName>${ns}/point_cloud</topicName>
+          <frameName>${ns}/${prefix}_link</frameName>
+          <min_range>${range_min}</min_range>
+          <max_range>${range_max}</max_range>
+          <gaussianNoise>0.01</gaussianNoise>
+        </plugin>
       </sensor>
     </gazebo>
