Commit message: fixing 'scale' variable name. It was colliding between asus_xtion and orbec_astra sensors

File: urdf/asus_xtion_pro.urdf.xacro (robot description, xacro)
@@ -2,7 +2,7 @@
 <robot name="sensor_asus_xtion_pro" xmlns:xacro="http://ros.org/wiki/xacro">
   <!-- Xacro properties -->
-  <xacro:property name="M_SCALE" value="0.001"/>
+  <xacro:property name="asus_xtion_scale" value="0.001"/>
   <xacro:property name="asus_xtion_pro_depth_rel_rgb_py" value="0.0270" />
-  <xacro:property name="asus_xtion_pro_cam_rel_rgb_py"   value="-0.0220" />
+  <xacro:property name="asus_xtion_pro_cam_rel_rgb_py"   value="-0.0220" />z
   <xacro:property name="M_PI" value="3.1415926535897931" />
   <xacro:macro name="sensor_asus_xtion_pro" params="name parent *origin">
@@ -45,5 +45,5 @@
         <origin xyz="-0.01 0 0" rpy="${-M_PI/2} -${M_PI} ${-M_PI/2}"/>
         <geometry>
-          <mesh filename="package://robotnik_sensors/meshes/asus_xtion_pro_live.dae" scale="${M_SCALE} ${M_SCALE} ${M_SCALE}"/>
+          <mesh filename="package://robotnik_sensors/meshes/asus_xtion_pro_live.dae" scale="${asus_xtion_scale} ${asus_xtion_scale} ${asus_xtion_scale}"/>
         </geometry>
       </visual>

File: urdf/orbbec_astra.urdf.xacro (robot description, xacro)
@@ -2,5 +2,5 @@
 <robot name="sensor_orbbec_astra" xmlns:xacro="http://ros.org/wiki/xacro">
   <!-- Xacro properties -->
-  <xacro:property name="M_SCALE" value="1.0"/>
+  <xacro:property name="orbbec_astra_scale" value="1.0"/>
   <!-- RGB sensor - cam -->
   <xacro:property name="orbbec_astra_cam_rel_rgb_px"   value="0.0" />
@@ -51,5 +51,5 @@
         <origin xyz="0 0 0" rpy="0 0 0"/>
         <geometry>
-          <mesh filename="package://robotnik_sensors/meshes/orbbec_astra.dae" scale="${M_SCALE} ${M_SCALE} ${M_SCALE}"/>
+          <mesh filename="package://robotnik_sensors/meshes/orbbec_astra.dae" scale="${orbbec_astra_scale} ${orbbec_astra_scale} ${orbbec_astra_scale}"/>
         </geometry>
       </visual>

Commit message: changed scale in asus_xtion_pro.urdf.xacro for new dae

File: urdf/asus_xtion_pro.urdf.xacro (robot description, xacro)
@@ -2,4 +2,6 @@
 <robot name="sensor_asus_xtion_pro" xmlns:xacro="http://ros.org/wiki/xacro">
   <!-- Xacro properties -->
+  <!-- xacro:property name="M_SCALE" value="0.001"/ -->
+  <xacro:property name="M_SCALE" value="1.0"/>
   <xacro:property name="asus_xtion_scale" value="0.001"/>
   <xacro:property name="asus_xtion_pro_depth_rel_rgb_py" value="0.0270" />

Commit message: changed scale to 1 as the meshes were updated to scale 1

File: urdf/asus_xtion_pro.urdf.xacro (robot description, xacro)
@@ -4,5 +4,6 @@
   <!-- xacro:property name="M_SCALE" value="0.001"/ -->
   <xacro:property name="M_SCALE" value="1.0"/>
-  <xacro:property name="asus_xtion_scale" value="0.001"/>
+  <!-- xacro:property name="asus_xtion_scale" value="0.001"/ -->
+  <xacro:property name="asus_xtion_scale" value="1.0"/>
   <xacro:property name="asus_xtion_pro_depth_rel_rgb_py" value="0.0270" />
   <xacro:property name="asus_xtion_pro_cam_rel_rgb_py"   value="-0.0220" />z

Commit message: Modified .xacro files

File: urdf/asus_xtion_pro.urdf.xacro (robot description, xacro)
@@ -11,5 +11,5 @@
   <xacro:macro name="sensor_asus_xtion_pro" params="name parent *origin">
     <joint name="${name}_cam_rgb_joint" type="fixed">
-	  <insert_block name="origin" />
+	  <xacro:insert_block name="origin" />
       <parent link="${parent}"/>
       <child link="${name}_cam_rgb_frame" />

File: urdf/axis.urdf.xacro (robot description, xacro)
@@ -12,5 +12,5 @@
 	      <origin xyz="0.180 0.0 0.270"/>
 -->
-				<insert_block name="origin"/>
+				<xacro:insert_block name="origin"/>
 	      <parent link="${parent}"/>
 	      <child link="${name}_link"/>

File: urdf/axis_m5013.urdf.xacro (robot description, xacro)
@@ -12,5 +12,5 @@
 	      <origin xyz="0.180 0.0 0.270"/>
 -->
-		  <insert_block name="origin"/>
+		  <xacro:insert_block name="origin"/>
 	      <parent link="${parent}"/>
 	      <child link="${name}_link"/>

File: urdf/fotonic.urdf.xacro (robot description, xacro)
@@ -3,5 +3,5 @@
   <xacro:macro name="sensor_fotonic" params="name parent *origin">
     <joint name="${name}_joint" type="fixed">
-			<insert_block name="origin"/>
+			<xacro:insert_block name="origin"/>
       <parent link="${parent}"/>
       <child link="${name}_link"/>

File: urdf/gps.urdf.xacro (robot description, xacro)
@@ -5,5 +5,5 @@
 	  <joint name="${name}_joint" type="fixed">
 	    <axis xyz="0 1 0"/>
-	    <insert_block name="origin"/>
+	    <xacro:insert_block name="origin"/>
 	    <parent link="${parent}"/>
 	    <child link="${name}_link"/>

File: urdf/gps_with_mast.urdf.xacro (robot description, xacro)
@@ -1,11 +1,11 @@
 <?xml version="1.0"?>
 <robot name="sensor_gps_with_mast" xmlns:xacro="http://ros.org/wiki/xacro">
-  <property name="mast_height" value="0.5" />
-  <property name="mast_radius" value="0.010" />
+  <xacro:property name="mast_height" value="0.5" />
+  <xacro:property name="mast_radius" value="0.010" />
   <xacro:macro name="sensor_gps_with_mast" params="name parent *origin">
 	  <!-- MAST OF THE ANTENNA GPS -->
 	  <joint name="${name}_joint" type="fixed">
 	    <axis xyz="0 1 0"/>
-	    <insert_block name="origin"/>
+	    <xacro:insert_block name="origin"/>
 	    <parent link="${parent}"/>
 	    <child link="${name}_mast_link"/>

File: urdf/hokuyo3d.urdf.xacro (robot description, xacro)
@@ -3,5 +3,5 @@
   <xacro:macro name="sensor_hokuyo3d" params="name parent *origin">
     <joint name="${name}_laser_fix_joint" type="fixed">
-      <insert_block name="origin" />
+      <xacro:insert_block name="origin" />
       <parent link="${parent}"/>
       <child link="${name}_laser_fix_link"/>

File: urdf/hokuyo_urg04lx.urdf.xacro (robot description, xacro)
@@ -7,5 +7,5 @@
       <!-- TOP MOUNT -->
       <!-- origin xyz="0.0 0.0 0.325"-->
-      <insert_block name="origin" />
+      <xacro:insert_block name="origin" />
       <parent link="${parent}"/>
       <child link="${name}_laser_link"/>

File: urdf/hokuyo_ust10lx.urdf.xacro (robot description, xacro)
@@ -3,5 +3,5 @@
   <xacro:macro name="sensor_hokuyo_ust10lx" params="name parent *origin min_angle:=2.3562 max_angle:=-2.3562">
     <joint name="${name}_laser_joint" type="fixed">
-      <insert_block name="origin" />
+      <xacro:insert_block name="origin" />
       <parent link="${parent}"/>
       <child link="${name}_laser_link"/>

File: urdf/hokuyo_utm30lx.urdf.xacro (robot description, xacro)
@@ -7,5 +7,5 @@
       <!-- TOP MOUNT -->
       <!-- origin xyz="0.0 0.0 0.325"-->
-      <insert_block name="origin" />
+      <xacro:insert_block name="origin" />
       <parent link="${parent}"/>
       <child link="${name}_laser_link"/>

File: urdf/imu.urdf.xacro (robot description, xacro)
@@ -5,5 +5,5 @@
 	      <axis xyz="1 0 0"/>
 	      <!--origin xyz="0 0 0.2825"/-->
-	      <insert_block name="origin"/>
+	      <xacro:insert_block name="origin"/>
 	      <parent link="${parent}"/>
 	      <child link="${name}_link"/>

File: urdf/imu_hector_plugin.urdf.xacro (robot description, xacro)
@@ -5,5 +5,5 @@
 	      <axis xyz="1 0 0"/>
 	      <!--origin xyz="0 0 0.2825"/-->
-	      <insert_block name="origin"/>
+	      <xacro:insert_block name="origin"/>
 	      <parent link="${parent}"/>
 	      <child link="${name}_link"/>

File: urdf/kinect.urdf.xacro (robot description, xacro)
@@ -10,5 +10,5 @@
   <xacro:macro name="sensor_kinect" params="name parent *origin">
     <joint name="${name}_rgb_joint" type="fixed">
-      <insert_block name="origin" />
+      <xacro:insert_block name="origin" />
       <parent link="${parent}"/>
       <child link="${name}_rgb_frame" />

File: urdf/kinectv2.urdf.xacro (robot description, xacro)
@@ -10,5 +10,5 @@
   <xacro:macro name="sensor_kinectv2" params="name parent base:=true *origin">
     <joint name="${name}_rgb_joint" type="fixed">
-      <insert_block name="origin" />
+      <xacro:insert_block name="origin" />
       <parent link="${parent}"/>
       <child link="${name}_rgb_frame" />

File: urdf/orbbec_astra.urdf.xacro (robot description, xacro)
@@ -14,5 +14,5 @@
   <xacro:macro name="sensor_orbbec_astra" params="name parent *origin">
     <joint name="${name}_cam_rgb_joint" type="fixed">
-	  <insert_block name="origin" />
+	  <xacro:insert_block name="origin" />
       <parent link="${parent}"/>
       <child link="${name}_cam_rgb_frame" />

File: urdf/rplidar.urdf.xacro (robot description, xacro)
@@ -3,5 +3,5 @@
   <xacro:macro name="sensor_rplidar" params="prefix parent *origin min_angle:=3.14159 max_angle:=-3.14159">
     <joint name="${prefix}_laser_base_joint" type="fixed">
-      <insert_block name="origin" />
+      <xacro:insert_block name="origin" />
       <parent link="${parent}"/>
       <child link="${prefix}_laser_base_link"/>

File: urdf/sick_s300.urdf.xacro (robot description, xacro)
@@ -3,5 +3,5 @@
   <xacro:macro name="sensor_sick_s300" params="name parent *origin">
     <joint name="${name}_laser_fix_joint" type="fixed">
-      <insert_block name="origin" />
+      <xacro:insert_block name="origin" />
       <parent link="${parent}"/>
       <child link="${name}_laser_fix_link"/>

File: urdf/sick_s3000.urdf.xacro (robot description, xacro)
@@ -3,5 +3,5 @@
   <xacro:macro name="sensor_sick_s3000" params="name parent *origin">
     <joint name="${name}_laser_joint" type="fixed">
-      <insert_block name="origin" />
+      <xacro:insert_block name="origin" />
       <parent link="${parent}"/>
       <child link="${name}_laser_link"/>

File: urdf/sick_tim571.urdf.xacro (robot description, xacro)
@@ -3,5 +3,5 @@
   <xacro:macro name="sensor_sick_tim571" params="prefix parent *origin min_angle:=-2.36 max_angle:=2.36">
     <joint name="${prefix}laser_base_joint" type="fixed">
-      <insert_block name="origin" />
+      <xacro:insert_block name="origin" />
       <parent link="${parent}"/>
       <child link="${prefix}laser_base_link"/>
