Commit message: adding prefix_topic and prefix_frame for multirobot

File: urdf/asus_xtion_pro.urdf.xacro (robot description, xacro)
@@ -9,5 +9,5 @@
   <xacro:property name="asus_xtion_pro_rgb_rel_rgb_py"   value="-0.0220" />
   <xacro:property name="M_PI" value="3.1415926535897931" />
-  <xacro:macro name="sensor_asus_xtion_pro" params="name parent *origin">
+  <xacro:macro name="sensor_asus_xtion_pro" params="name prefix_frame prefix_topic parent *origin">
     <joint name="${name}_rgb_joint" type="fixed">
 	  <xacro:insert_block name="origin" />
@@ -117,10 +117,10 @@
           <alwaysOn>true</alwaysOn>
           <updateRate>15</updateRate>
-          <imageTopicName>rgb/image_raw</imageTopicName>
-          <depthImageTopicName>depth/image_raw</depthImageTopicName>
-          <pointCloudTopicName>depth/points</pointCloudTopicName>
-          <cameraInfoTopicName>rgb/camera_info</cameraInfoTopicName>
-          <depthImageCameraInfoTopicName>depth/camera_info</depthImageCameraInfoTopicName>
-          <frameName>${name}_depth_optical_frame</frameName>
+          <imageTopicName>{prefix_topic}rgb/image_raw</imageTopicName>
+          <depthImageTopicName>{prefix_topic}depth/image_raw</depthImageTopicName>
+          <pointCloudTopicName>{prefix_topic}depth/points</pointCloudTopicName>
+          <cameraInfoTopicName>{prefix_topic}rgb/camera_info</cameraInfoTopicName>
+          <depthImageCameraInfoTopicName>{prefix_topic}depth/camera_info</depthImageCameraInfoTopicName>
+          <frameName>${prefix_frame}_${name}_depth_optical_frame</frameName>
           <baseline>0.1</baseline>
           <distortion_k1>0.0</distortion_k1>

File: urdf/axis.urdf.xacro (robot description, xacro)
@@ -6,5 +6,5 @@
   <xacro:property name="ptz_joint_damping" value="0.1"/>
   <xacro:property name="ptz_mechanical_reduction" value="1.0"/>
-  <xacro:macro name="sensor_axis" params="name parent *origin">
+  <xacro:macro name="sensor_axis" params="name prefix_frame prefix_topic parent *origin">
     <joint name="${name}_joint" type="fixed">
       <axis xyz="0 1 0"/>
@@ -140,7 +140,7 @@
           <updateRate>0.0</updateRate>
           <cameraName>${name}</cameraName>
-          <imageTopicName>image_raw</imageTopicName>
-          <cameraInfoTopicName>camera_info</cameraInfoTopicName>
-          <frameName>${name}_optical_frame</frameName>
+          <imageTopicName>${prefix_topic}image_raw</imageTopicName>
+          <cameraInfoTopicName>${prefix_topic}camera_info</cameraInfoTopicName>
+          <frameName>${prefix_frame}_${name}_optical_frame</frameName>
           <hackBaseline>0.0</hackBaseline>
           <distortionK1>0.0</distortionK1>

File: urdf/axis_m5013.urdf.xacro (robot description, xacro)
@@ -6,5 +6,5 @@
   <xacro:property name="ptz_joint_damping" value="0.1"/>
   <xacro:property name="ptz_mechanical_reduction" value="1.0"/>
-  <xacro:macro name="sensor_axis_m5013" params="name parent *origin">
+  <xacro:macro name="sensor_axis_m5013" params="name prefix_frame prefix_topic parent *origin">
     <joint name="${name}_joint" type="fixed">
       <axis xyz="0 1 0"/>
@@ -143,7 +143,7 @@
 					<updateRate>0.0</updateRate>
 					<cameraName>${name}</cameraName>
-					<imageTopicName>image_raw</imageTopicName>
-					<cameraInfoTopicName>camera_info</cameraInfoTopicName>
-					<frameName>${name}_optical_frame</frameName>
+					<imageTopicName>${prefix_topic}image_raw</imageTopicName>
+					<cameraInfoTopicName>${prefix_topic}camera_info</cameraInfoTopicName>
+					<frameName>${prefix_frame}_${name}_optical_frame</frameName>
 					<!-- this is just which name the Image msg will have, it does not affect the simulation.
 					     However must be set to the optical_frame,  -->

File: urdf/fotonic_e.urdf.xacro (robot description, xacro)
@@ -1,5 +1,5 @@
 <?xml version="1.0"?>
 <robot name="sensor_fotonic" xmlns:xacro="http://www.ros.org/wiki/xacro">
-  <xacro:macro name="sensor_fotonic" params="name parent *origin">
+  <xacro:macro name="sensor_fotonic" params="name prefix_frame prefix_topic parent *origin">
     <joint name="${name}_joint" type="fixed">
 			<xacro:insert_block name="origin"/>
@@ -91,10 +91,10 @@
 					<updateRate>10.0</updateRate>
 					<cameraName>${name}</cameraName>
-					<imageTopicName>ir/image_raw</imageTopicName>
-					<cameraInfoTopicName>ir/camera_info</cameraInfoTopicName>
-					<depthImageTopicName>depth/image_raw</depthImageTopicName>
-					<depthImageCameraInfoTopicName>depth/camera_info</depthImageCameraInfoTopicName>
-					<pointCloudTopicName>points</pointCloudTopicName>
-					<frameName>${name}_depth_optical_frame</frameName>
+					<imageTopicName>${prefix_topic}ir/image_raw</imageTopicName>
+					<cameraInfoTopicName>${prefix_topic}ir/camera_info</cameraInfoTopicName>
+					<depthImageTopicName>${prefix_topic}depth/image_raw</depthImageTopicName>
+					<depthImageCameraInfoTopicName>${prefix_topic}depth/camera_info</depthImageCameraInfoTopicName>
+					<pointCloudTopicName>${prefix_topic}points</pointCloudTopicName>
+					<frameName>${prefix_frame}_${name}_depth_optical_frame</frameName>
 					<pointCloudCutoff>0.5</pointCloudCutoff>
 					<distortionK1>0</distortionK1>

File: urdf/gps.urdf.xacro (robot description, xacro)
@@ -1,5 +1,5 @@
 <?xml version="1.0"?>
 <robot name="sensor_gps" xmlns:xacro="http://www.ros.org/wiki/xacro">
-  <xacro:macro name="sensor_gps" params="name parent *origin">
+  <xacro:macro name="sensor_gps" params="name prefix_frame prefix_topic parent *origin">
 	  <!-- ANTENNA GPS -->
 	  <joint name="${name}_joint" type="fixed">
@@ -40,6 +40,6 @@
         <updateRate>5</updateRate>
         <bodyName>${name}_link</bodyName> <!-- must be the link of the gps device, not the base_link or base_footprint -->
-        <frameId>${name}_link</frameId>
-        <topicName>${name}/fix</topicName>
+        <frameId>${prefix_frame}_${name}_link</frameId>
+        <topicName>${prefix_topic}${name}/fix</topicName>
         <!-- Robotnik position at Fuente del Jarro -->
         <referenceLatitude>39.5080331</referenceLatitude>
@@ -47,5 +47,5 @@
         <!-- To set heading in ENU orientation (degrees) -->
         <referenceHeading>90</referenceHeading>
-        <velocityTopicName>${name}/fix_velocity</velocityTopicName>
+        <velocityTopicName>${prefix_topic}${name}/fix_velocity</velocityTopicName>
         <drift>0.0 0.0 0.0</drift>
         <!--<drift>0.0001 0.0001 0.0001</drift>-->

File: urdf/gps_with_mast.urdf.xacro (robot description, xacro)
@@ -3,5 +3,5 @@
   <xacro:property name="mast_height" value="0.5" />
   <xacro:property name="mast_radius" value="0.010" />
-  <xacro:macro name="sensor_gps_with_mast" params="name parent *origin">
+  <xacro:macro name="sensor_gps_with_mast" params="name prefix_frame prefix_topic parent *origin">
 	  <!-- MAST OF THE ANTENNA GPS -->
 	  <joint name="${name}_joint" type="fixed">
@@ -75,6 +75,6 @@
         <updateRate>5</updateRate>
         <bodyName>${name}_link</bodyName> <!-- must be the link of the gps device, not the base_link or base_footprint -->
-        <frameId>${name}_link</frameId>   <!-- which frame_id would be on the published message -->
-        <topicName>${name}/fix</topicName>
+        <frameId>${prefix_frame}_${name}_link</frameId>   <!-- which frame_id would be on the published message -->
+        <topicName>${prefix_topic}${name}/fix</topicName>
         <!-- Robotnik position at Fuente del Jarro -->
         <referenceLatitude>39.5080331</referenceLatitude>
@@ -82,5 +82,5 @@
         <!-- To set heading in ENU orientation (degrees) -->
         <referenceHeading>90</referenceHeading>
-        <velocityTopicName>${name}/fix_velocity</velocityTopicName>
+        <velocityTopicName>${prefix_topic}${name}/fix_velocity</velocityTopicName>
         <drift>0.0 0.0 0.0</drift>
         <!--<drift>0.0001 0.0001 0.0001</drift>-->

File: urdf/hokuyo3d.urdf.xacro (robot description, xacro)
@@ -1,5 +1,5 @@
 <?xml version="1.0"?>
 <robot name="sensor_hokuyo3d" xmlns:xacro="http://www.ros.org/wiki/xacro">
-  <xacro:macro name="sensor_hokuyo3d" params="name parent *origin">
+  <xacro:macro name="sensor_hokuyo3d" params="name prefix_frame prefix_topic parent *origin">
     <joint name="${name}_fix_joint" type="fixed">
       <xacro:insert_block name="origin" />
@@ -69,6 +69,6 @@
 				</ray>
 				<plugin name="${name}_controller" filename="libgazebo_ros_block_laser.so">
-					<topicName>${name}/points</topicName>
-					<frameName>${name}_link</frameName>
+					<topicName>${prefix_topic}${name}/points</topicName>
+					<frameName>${prefix_frame}_${name}_link</frameName>
 				</plugin>
 			</sensor>

File: urdf/hokuyo_urg04lx.urdf.xacro (robot description, xacro)
@@ -1,5 +1,5 @@
 <?xml version="1.0"?>
 <robot name="sensor_hokuyo_urg04lx" xmlns:xacro="http://www.ros.org/wiki/xacro">
-  <xacro:macro name="sensor_hokuyo_urg04lx" params="name parent *origin min_angle:=-2.0943 max_angle:=2.0943">
+  <xacro:macro name="sensor_hokuyo_urg04lx" params="name prefix_frame prefix_topic parent *origin min_angle:=-2.0943 max_angle:=2.0943">
     <joint name="${name}_joint" type="fixed">
       <!-- FRONT MOUNT  -->
@@ -60,6 +60,6 @@
 				</ray>
 				<plugin name="${name}_controller" filename="libgazebo_ros_laser.so">
-					<topicName>${name}/scan</topicName>
-					<frameName>${name}_link</frameName>
+					<topicName>${prefix_topic}${name}/scan</topicName>
+					<frameName>${prefix_frame}_${name}_link</frameName>
 				</plugin>
 			</sensor>

File: urdf/hokuyo_ust10lx.urdf.xacro (robot description, xacro)
@@ -60,5 +60,5 @@
 				<plugin name="${prefix_frame}_controller" filename="libgazebo_ros_laser.so">
 					<topicName>${prefix_topic}hokuyo_base/scan</topicName>
-					<frameName>${prefix_frame}_link</frameName>
+					<frameName>${prefix_frame}_${name}_link</frameName>
 					<ignoreTfPrefix>1</ignoreTfPrefix>
 				</plugin>

File: urdf/hokuyo_utm30lx.urdf.xacro (robot description, xacro)
@@ -1,5 +1,5 @@
 <?xml version="1.0"?>
 <robot name="sensor_hokuyo_utm30lx" xmlns:xacro="http://www.ros.org/wiki/xacro">
-  <xacro:macro name="sensor_hokuyo_utm30lx" params="name parent *origin min_angle:=-2.35 max_angle:=2.35">
+  <xacro:macro name="sensor_hokuyo_utm30lx" params="name prefix_frame prefix_topic parent *origin min_angle:=-2.35 max_angle:=2.35">
     <joint name="${name}_joint" type="fixed">
       <!-- FRONT MOUNT  -->
@@ -54,6 +54,6 @@
 				</ray>
 				<plugin name="${name}_controller" filename="libgazebo_ros_laser.so">
-					<topicName>${name}/scan</topicName>
-					<frameName>${name}_link</frameName>
+					<topicName>${prefix_topic}${name}/scan</topicName>
+					<frameName>${prefix_frame}_${name}_link</frameName>
 				</plugin>
 			</sensor>

File: urdf/imu.urdf.xacro (robot description, xacro)
@@ -30,6 +30,6 @@
 	  <gazebo>
 	    <plugin name="${name}_controller" filename="libgazebo_ros_imu.so">
-	       <topicName>${prefix_topic}/data</topicName>
-		   <serviceName>${prefix_topic}/service</serviceName>
+	       <topicName>${prefix_topic}data</topicName>
+		   <serviceName>${prefix_topic}service</serviceName>
 		   <bodyName>${prefix_frame}_link</bodyName>
 	       <gaussianNoise>0.005</gaussianNoise>

File: urdf/kinect.urdf.xacro (robot description, xacro)
@@ -8,5 +8,5 @@
 	<xacro:property name="cam_op" value="0" />
 	<xacro:property name="cam_oy" value="0" />
-  <xacro:macro name="sensor_kinect" params="name parent *origin">
+  <xacro:macro name="sensor_kinect" params="name prefix_frame prefix_topic parent *origin">
     <joint name="${name}_rgb_joint" type="fixed">
       <xacro:insert_block name="origin" />
@@ -118,10 +118,10 @@
           <alwaysOn>true</alwaysOn>
           <updateRate>10</updateRate>
-          <imageTopicName>rgb/image_raw</imageTopicName>
-          <depthImageTopicName>depth/image_raw</depthImageTopicName>
-          <pointCloudTopicName>depth/points</pointCloudTopicName>
-          <cameraInfoTopicName>rgb/camera_info</cameraInfoTopicName>
-          <depthImageCameraInfoTopicName>depth/camera_info</depthImageCameraInfoTopicName>
-          <frameName>${name}_depth_optical_frame</frameName>
+          <imageTopicName>${prefix_topic}rgb/image_raw</imageTopicName>
+          <depthImageTopicName>${prefix_topic}depth/image_raw</depthImageTopicName>
+          <pointCloudTopicName>${prefix_topic}depth/points</pointCloudTopicName>
+          <cameraInfoTopicName>${prefix_topic}rgb/camera_info</cameraInfoTopicName>
+          <depthImageCameraInfoTopicName>${prefix_topic}depth/camera_info</depthImageCameraInfoTopicName>
+          <frameName>${prefix_frame}_${name}_depth_optical_frame</frameName>
           <baseline>0.1</baseline>
           <distortion_k1>0.0</distortion_k1>

File: urdf/kinectv2.urdf.xacro (robot description, xacro)
@@ -8,5 +8,5 @@
     <xacro:property name="cam_op" value="0" />
     <xacro:property name="cam_oy" value="0" />
-  <xacro:macro name="sensor_kinectv2" params="name parent base:=true *origin">
+  <xacro:macro name="sensor_kinectv2" params="name prefix_frame prefix_topic parent base:=true *origin">
     <joint name="${name}_rgb_joint" type="fixed">
       <xacro:insert_block name="origin" />
@@ -138,10 +138,10 @@
           <alwaysOn>true</alwaysOn>
           <updateRate>10</updateRate>
-          <imageTopicName>rgb/image_raw</imageTopicName>
-          <depthImageTopicName>depth/image_raw</depthImageTopicName>
-          <pointCloudTopicName>depth/points</pointCloudTopicName>
-          <cameraInfoTopicName>rgb/camera_info</cameraInfoTopicName>
-          <depthImageCameraInfoTopicName>depth/camera_info</depthImageCameraInfoTopicName>
-          <frameName>${name}_depth_optical_frame</frameName>
+          <imageTopicName>${prefix_topic}rgb/image_raw</imageTopicName>
+          <depthImageTopicName>${prefix_topic}depth/image_raw</depthImageTopicName>
+          <pointCloudTopicName>${prefix_topic}depth/points</pointCloudTopicName>
+          <cameraInfoTopicName>${prefix_topic}rgb/camera_info</cameraInfoTopicName>
+          <depthImageCameraInfoTopicName>${prefix_topic}depth/camera_info</depthImageCameraInfoTopicName>
+          <frameName>${prefix_frame}_${name}_depth_optical_frame</frameName>
           <baseline>0.1</baseline>
           <distortion_k1>0.0</distortion_k1>

File: urdf/orbbec_astra.urdf.xacro (robot description, xacro)
@@ -13,5 +13,5 @@
   <xacro:property name="orbbec_astra_depth_rel_rgb_pz" value="0.0" />
   <xacro:property name="M_PI" value="3.1415926535897931" />
-  <xacro:macro name="sensor_orbbec_astra" params="name parent *origin">
+  <xacro:macro name="sensor_orbbec_astra" params="name prefix_frame prefix_topic parent *origin">
     <joint name="${name}_rgb_joint" type="fixed">
 	  <xacro:insert_block name="origin" />
@@ -126,10 +126,10 @@
           <alwaysOn>true</alwaysOn>
           <updateRate>10</updateRate>
-          <imageTopicName>rgb/image_raw</imageTopicName>
-          <depthImageTopicName>depth/image_raw</depthImageTopicName>
-          <pointCloudTopicName>depth/points</pointCloudTopicName>
-          <cameraInfoTopicName>rgb/camera_info</cameraInfoTopicName>
-          <depthImageCameraInfoTopicName>depth/camera_info</depthImageCameraInfoTopicName>
-          <frameName>${name}_depth_optical_frame</frameName>
+          <imageTopicName>${prefix_topic}rgb/image_raw</imageTopicName>
+          <depthImageTopicName>${prefix_topic}depth/image_raw</depthImageTopicName>
+          <pointCloudTopicName>${prefix_topic}depth/points</pointCloudTopicName>
+          <cameraInfoTopicName>${prefix_topic}rgb/camera_info</cameraInfoTopicName>
+          <depthImageCameraInfoTopicName>${prefix_topic}depth/camera_info</depthImageCameraInfoTopicName>
+          <frameName>${prefix_frame}_${name}_depth_optical_frame</frameName>
           <baseline>0.1</baseline>
           <distortion_k1>0.0</distortion_k1>

File: urdf/rplidar.urdf.xacro (robot description, xacro)
@@ -1,11 +1,11 @@
 <?xml version="1.0"?>
 <robot xmlns:xacro="http://www.ros.org/wiki/xacro">
-  <xacro:macro name="sensor_rplidar" params="prefix parent *origin min_angle:=3.14159 max_angle:=-3.14159">
-    <joint name="${prefix}_laser_base_joint" type="fixed">
+  <xacro:macro name="sensor_rplidar" params="name prefix_frame prefix_topic parent *origin min_angle:=3.14159 max_angle:=-3.14159">
+    <joint name="${name}_laser_base_joint" type="fixed">
       <xacro:insert_block name="origin" />
       <parent link="${parent}"/>
-      <child link="${prefix}_laser_base_link"/>
+      <child link="${name}_laser_base_link"/>
     </joint>
-    <link name="${prefix}_laser_base_link">
+    <link name="${name}_laser_base_link">
       <collision>
         <origin xyz="0 0 0" rpy="0 0 0"/>
@@ -26,16 +26,16 @@
       </inertial>
     </link>
-    <joint name="${prefix}_laser_joint" type="fixed">
+    <joint name="${name}_laser_joint" type="fixed">
       <origin xyz="0 0 0.0461" rpy="0 0 0"/>
-      <parent link="${prefix}_laser_base_link"/>
-      <child link="${prefix}_laser_link"/>
+      <parent link="${name}_laser_base_link"/>
+      <child link="${name}_laser_link"/>
     </joint>
-    <link name="${prefix}_laser_link">
+    <link name="${name}_laser_link">
     </link>
     <sensor_rplidar_gazebo/>
   </xacro:macro>
   <xacro:macro name="sensor_rplidar_gazebo">
-    <gazebo reference="${prefix}_laser_link">
-			<sensor type="ray" name="${prefix}_rplidar_sensor">
+    <gazebo reference="${name}_laser_link">
+			<sensor type="ray" name="${name}_rplidar_sensor">
 				<pose>0 0 0 0 0 0</pose>
 				<visualize>false</visualize>
@@ -62,6 +62,6 @@
 				</ray>
 				<plugin name="gazebo_ros_rplidar_controller" filename="libgazebo_ros_laser.so">
-					<topicName>${prefix}/scan</topicName>
-					<frameName>${prefix}_laser_link</frameName>
+					<topicName>${prefix_topic}${name}/scan</topicName>
+					<frameName>${prefix_frame}_${name}_laser_link</frameName>
 				</plugin>
 			</sensor>

File: urdf/sick_s300.urdf.xacro (robot description, xacro)
@@ -1,5 +1,5 @@
 <?xml version="1.0"?>
 <robot name="sensor_sick_s300" xmlns:xacro="http://www.ros.org/wiki/xacro">
-  <xacro:macro name="sensor_sick_s300" params="name parent *origin">
+  <xacro:macro name="sensor_sick_s300" params="name prefix_frame prefix_topic parent *origin">
     <joint name="${name}_fix_joint" type="fixed">
       <xacro:insert_block name="origin" />
@@ -64,6 +64,6 @@
 				</ray>
 				<plugin name="${name}_controller" filename="libgazebo_ros_laser.so">
-					<topicName>${name}/scan</topicName>
-					<frameName>/${name}_link</frameName><!-- if not global (leading /) sets the current namespace as a prefix (/ns/name_laser_link) -->
+					<topicName>${prefix_topic}${name}/scan</topicName>
+					<frameName>${prefix_frame}_${name}_link</frameName><!-- if not global (leading /) sets the current namespace as a prefix (/ns/name_laser_link) -->
 				</plugin>
 			</sensor>

File: urdf/sick_s3000.urdf.xacro (robot description, xacro)
@@ -1,5 +1,5 @@
 <?xml version="1.0"?>
 <robot name="sensor_sick_s3000" xmlns:xacro="http://www.ros.org/wiki/xacro">
-  <xacro:macro name="sensor_sick_s3000" params="name parent *origin">
+  <xacro:macro name="sensor_sick_s3000" params="name prefix_frame prefix_topic parent *origin">
     <joint name="${name}_joint" type="fixed">
       <xacro:insert_block name="origin" />
@@ -56,6 +56,6 @@
 				</ray>
 				<plugin name="${name}_controller" filename="libgazebo_ros_laser.so">
-					<topicName>${name}/scan</topicName>
-					<frameName>${name}_link</frameName>
+					<topicName>${prefix_topic}${name}/scan</topicName>
+					<frameName>${prefix_frame}_${name}_link</frameName>
 				</plugin>
 			</sensor>

File: urdf/sick_tim571.urdf.xacro (robot description, xacro)
@@ -1,11 +1,11 @@
 <?xml version="1.0"?>
 <robot xmlns:xacro="http://www.ros.org/wiki/xacro">
-  <xacro:macro name="sensor_sick_tim571" params="prefix parent *origin min_angle:=-2.36 max_angle:=2.36">
-    <joint name="${prefix}_base_joint" type="fixed">
+  <xacro:macro name="sensor_sick_tim571" params="name prefix_frame prefix_topic parent *origin min_angle:=-2.36 max_angle:=2.36">
+    <joint name="${name}_base_joint" type="fixed">
       <xacro:insert_block name="origin" />
       <parent link="${parent}"/>
-      <child link="${prefix}_base_link"/>
+      <child link="${name}_base_link"/>
     </joint>
-    <link name="${prefix}_base_link">
+    <link name="${name}_base_link">
       <collision>
         <origin xyz="0 0 0" rpy="0 0 0"/>
@@ -26,16 +26,16 @@
       </inertial>
     </link>
-    <joint name="${prefix}_joint" type="fixed">
+    <joint name="${name}_joint" type="fixed">
       <origin xyz="0 0 0.06246" rpy="0 0 0"/>
-      <parent link="${prefix}_base_link"/>
-      <child link="${prefix}_link"/>
+      <parent link="${name}_base_link"/>
+      <child link="${name}_link"/>
     </joint>
-    <link name="${prefix}_link">
+    <link name="${name}_link">
     </link>
     <sensor_sick_tim571_gazebo/>
   </xacro:macro>
   <xacro:macro name="sensor_sick_tim571_gazebo">
-    <gazebo reference="${prefix}_link">
-			<sensor type="ray" name="${prefix}_sensor">
+    <gazebo reference="${name}_link">
+			<sensor type="ray" name="${name}_sensor">
 				<pose>0 0 0 0 0 0</pose>
 				<visualize>false</visualize>
@@ -61,7 +61,7 @@
 					</noise>
 				</ray>
-				<plugin name="${prefix}_controller" filename="libgazebo_ros_laser.so">
-					<topicName>${prefix}/scan</topicName>
-					<frameName>${prefix}_link</frameName>
+				<plugin name="${name}_controller" filename="libgazebo_ros_laser.so">
+					<topicName>${prefix_topic}${name}/scan</topicName>
+					<frameName>${prefix_frame}_${name}_link</frameName>
 				</plugin>
 			</sensor>

File: urdf/ueye_cp_gige.urdf.xacro (robot description, xacro)
@@ -1,5 +1,5 @@
 <?xml version="1.0"?>
 <robot xmlns:xacro="http://www.ros.org/wiki/xacro">
-  <xacro:macro name="sensor_ueye_cp_gige" params="name parent *origin">
+  <xacro:macro name="sensor_ueye_cp_gige" params="name prefix_frame prefix_topic parent *origin">
     <joint name="${name}_joint" type="fixed">
       <insert_block name="origin"/>
@@ -86,7 +86,7 @@
           <updateRate>0.0</updateRate>
           <cameraName>${name}</cameraName>
-          <imageTopicName>image_raw</imageTopicName>
-          <cameraInfoTopicName>camera_info</cameraInfoTopicName>
-          <frameName>${name}_rgb_frame</frameName>
+          <imageTopicName>${prefix_topic}${name}/image_raw</imageTopicName>
+          <cameraInfoTopicName>${prefix_topic}${name}/camera_info</cameraInfoTopicName>
+          <frameName>${prefix_frame}_${name}_rgb_frame</frameName>
           <distortionK1>0.0</distortionK1>
           <distortionK2>0.0</distortionK2>
