Commit message: links of xacro file renamed

File: urdf/asus_xtion_pro.urdf.xacro (robot description, xacro)
@@ -13,7 +13,7 @@
 	  <xacro:insert_block name="origin" />
       <parent link="${parent}"/>
-      <child link="${prefix}_rgb_frame" />
+      <child link="${prefix}_rgb_base_link" />
     </joint>
-    <link name="${prefix}_rgb_frame">
+    <link name="${prefix}_rgb_base_link">
       <inertial>
         <mass value="0.001" />
@@ -26,8 +26,8 @@
     <joint name="${prefix}_rgb_optical_joint" type="fixed">
       <origin xyz="0 0 0" rpy="${-M_PI/2} 0 ${-M_PI/2}" />
-      <parent link="${prefix}_rgb_frame" />
-      <child link="${prefix}_rgb_optical_frame" />
+      <parent link="${prefix}_rgb_base_link" />
+      <child link="${prefix}_rgb_optical_link" />
     </joint>
-    <link name="${prefix}_rgb_optical_frame">
+    <link name="${prefix}_rgb_optical_link">
       <inertial>
         <mass value="0.001" />
@@ -41,5 +41,5 @@
       <origin xyz="0 ${asus_xtion_pro_rgb_rel_rgb_py} 0"
               rpy="0 0 0"/>
-      <parent link="${prefix}_rgb_frame"/>
+      <parent link="${prefix}_rgb_link"/>
       <child link="${prefix}_link"/>
     </joint>
@@ -67,8 +67,8 @@
     <joint name="${prefix}_depth_joint" type="fixed">
       <origin xyz="0 ${asus_xtion_pro_depth_rel_rgb_py} 0" rpy="0 0 0" />
-      <parent link="${name}_rgb_frame" />
-      <child link="${name}_depth_frame" />
+      <parent link="${name}_rgb_base_link" />
+      <child link="${name}_depth_link" />
     </joint>
-    <link name="${prefix}_depth_frame">
+    <link name="${prefix}_depth_link">
       <inertial>
         <mass value="0.01" />
@@ -81,8 +81,8 @@
     <joint name="${prefix}_depth_optical_joint" type="fixed">
       <origin xyz="0 0 0" rpy="${-M_PI/2} 0 ${-M_PI/2}" />
-      <parent link="${prefix}_depth_frame" />
-      <child link="${prefix}_depth_optical_frame" />
+      <parent link="${prefix}_depth_link" />
+      <child link="${prefix}_depth_optical_link" />
     </joint>
-    <link name="${prefix}_depth_optical_frame">
+    <link name="${prefix}_depth_optical_link">
       <inertial>
         <mass value="0.001" />
@@ -97,5 +97,5 @@
   </xacro:macro>
    <xacro:macro name="sensor_xtion_pro_gazebo">
-    <gazebo reference="${prefix}_depth_frame">
+    <gazebo reference="${prefix}_depth_link">
       <sensor type="depth" name="${prefix}_sensor">
         <always_on>true</always_on>
@@ -122,5 +122,5 @@
           <cameraInfoTopicName>rgb/camera_info</cameraInfoTopicName>
           <depthImageCameraInfoTopicName>depth/camera_info</depthImageCameraInfoTopicName>
-          <frameName>${prefix}_depth_optical_frame</frameName>
+          <frameName>${prefix}_depth_optical_link</frameName>
           <baseline>0.1</baseline>
           <distortion_k1>0.0</distortion_k1>

Commit message: Changed optical_link reference to optical_frame in remaining cameras

File: urdf/asus_xtion_pro.urdf.xacro (robot description, xacro)
@@ -27,7 +27,7 @@
       <origin xyz="0 0 0" rpy="${-M_PI/2} 0 ${-M_PI/2}" />
       <parent link="${prefix}_rgb_base_link" />
-      <child link="${prefix}_rgb_optical_link" />
+      <child link="${prefix}_rgb_optical_frame" />
     </joint>
-    <link name="${prefix}_rgb_optical_link">
+    <link name="${prefix}_rgb_optical_frame">
       <inertial>
         <mass value="0.001" />
@@ -82,7 +82,7 @@
       <origin xyz="0 0 0" rpy="${-M_PI/2} 0 ${-M_PI/2}" />
       <parent link="${prefix}_depth_link" />
-      <child link="${prefix}_depth_optical_link" />
+      <child link="${prefix}_depth_optical_frame" />
     </joint>
-    <link name="${prefix}_depth_optical_link">
+    <link name="${prefix}_depth_optical_frame">
       <inertial>
         <mass value="0.001" />
@@ -122,5 +122,5 @@
           <cameraInfoTopicName>rgb/camera_info</cameraInfoTopicName>
           <depthImageCameraInfoTopicName>depth/camera_info</depthImageCameraInfoTopicName>
-          <frameName>${prefix}_depth_optical_link</frameName>
+          <frameName>${prefix}_depth_optical_frame</frameName>
           <baseline>0.1</baseline>
           <distortion_k1>0.0</distortion_k1>

File: urdf/kinect.urdf.xacro (robot description, xacro)
@@ -26,7 +26,7 @@
       <origin xyz="0 0 0" rpy="${-M_PI/2} 0 ${-M_PI/2}" />
       <parent link="${prefix}_rgb_base_link" />
-      <child link="${prefix}_rgb_optical_link" />
+      <child link="${prefix}_rgb_optical_frame" />
     </joint>
-    <link name="${prefix}_rgb_optical_link">
+    <link name="${prefix}_rgb_optical_frame">
       <inertial>
         <mass value="0.001" />
@@ -83,7 +83,7 @@
 	  <origin xyz="0 0 0" rpy="${-M_PI/2} 0 ${-M_PI/2}" />
 	  <parent link="${prefix}_depth_link" />
-	  <child link="${prefix}_depth_optical_link" />
+	  <child link="${prefix}_depth_optical_frame" />
 	</joint>
-	<link name="${prefix}_depth_optical_link">
+	<link name="${prefix}_depth_optical_frame">
     <inertial>
       <mass value="0.001" />
@@ -123,5 +123,5 @@
           <cameraInfoTopicName>rgb/camera_info</cameraInfoTopicName>
           <depthImageCameraInfoTopicName>depth/camera_info</depthImageCameraInfoTopicName>
-          <frameName>/${prefix}_depth_optical_link</frameName>
+          <frameName>/${prefix}_depth_optical_frame</frameName>
           <baseline>0.1</baseline>
           <distortion_k1>0.0</distortion_k1>

File: urdf/kinectv2.urdf.xacro (robot description, xacro)
@@ -26,7 +26,7 @@
       <origin xyz="0 0 0" rpy="${-M_PI/2} 0 ${-M_PI/2}" />
       <parent link="${prefix}_rgb_base_link" />
-      <child link="${prefix}_rgb_optical_link" />
+      <child link="${prefix}_rgb_optical_frame" />
     </joint>
-    <link name="${prefix}_rgb_optical_link">
+    <link name="${prefix}_rgb_optical_frame">
       <inertial>
         <mass value="0.001" />
@@ -103,7 +103,7 @@
       <origin xyz="0 0 0" rpy="${-M_PI/2} 0 ${-M_PI/2}" />
       <parent link="${prefix}_depth_link" />
-      <child link="${prefix}_depth_optical_link" />
+      <child link="${prefix}_depth_optical_frame" />
     </joint>
-    <link name="${prefix}_depth_optical_link">
+    <link name="${prefix}_depth_optical_frame">
     <inertial>
       <mass value="0.001" />
@@ -143,5 +143,5 @@
           <cameraInfoTopicName>rgb/camera_info</cameraInfoTopicName>
           <depthImageCameraInfoTopicName>depth/camera_info</depthImageCameraInfoTopicName>
-          <frameName>/${prefix}_depth_optical_link</frameName>
+          <frameName>/${prefix}_depth_optical_frame</frameName>
           <baseline>0.1</baseline>
           <distortion_k1>0.0</distortion_k1>

File: urdf/pointgrey_bumblebee2.urdf.xacro (robot description, xacro)
@@ -83,5 +83,5 @@
       </inertial>
     </link>
-    <link name="${prefix}_optical_link">
+    <link name="${prefix}_optical_frame">
       <inertial>
         <mass value="1E-5" />
@@ -95,9 +95,9 @@
       <origin xyz="0 0 0" rpy="-1.570796 0 -1.570796" />
       <parent link="${prefix}_base_link" />
-      <child link="${prefix}_optical_link" />
+      <child link="${prefix}_optical_frame" />
     </joint>
     <xacro:if value="${high_res}">
       <xacro:stereo_camera
-        frame="${prefix}_optical_link"
+        frame="${prefix}_optical_frame"
         name="${prefix}"
         hfov="${hfov}"
@@ -112,5 +112,5 @@
     <xacro:unless value="${high_res}">
       <xacro:stereo_camera
-        frame="${prefix}_optical_link"
+        frame="${prefix}_optical_frame"
         name="${prefix}"
         hfov="${hfov}"

Commit message: urdf: updated asus xtion pro inertia and fixed some incompatibilities

File: urdf/asus_xtion_pro.urdf.xacro (robot description, xacro)
@@ -1,4 +1,4 @@
 <?xml version="1.0"?>
-<robot name="sensor_asus_xtion_pro" xmlns:xacro="http://wiki.ros.org/xacro">
+<robot xmlns:xacro="http://wiki.ros.org/xacro" name="sensor_asus_xtion_pro">
   <!-- Xacro properties -->
   <!-- xacro:property name="M_SCALE" value="0.001"/ -->
@@ -10,39 +10,35 @@
   <xacro:property name="M_PI" value="3.1415926535897931" />
   <xacro:macro name="sensor_asus_xtion_pro" params="prefix parent *origin">
-    <joint name="${prefix}_rgb_joint" type="fixed">
+    <joint name="${prefix}rgb_joint" type="fixed">
 	  <xacro:insert_block name="origin" />
       <parent link="${parent}"/>
-      <child link="${prefix}_rgb_base_link" />
+      <child link="${prefix}rgb_base_link" />
     </joint>
-    <link name="${prefix}_rgb_base_link">
+    <link name="${prefix}rgb_base_link">
       <inertial>
-        <mass value="0.001" />
-        <origin xyz="0 0 0" />
-        <inertia ixx="0.0001" ixy="0.0" ixz="0.0"
-          iyy="0.0001" iyz="0.0"
-          izz="0.0001" />
+        <mass value="0.01" />
+        <origin xyz="-0.0175 0 0" />
+        <xacro:solid_cuboid_inertia m="0.01" w="0.035" h="0.180" d="0.05" />
       </inertial>
     </link>
-    <joint name="${prefix}_rgb_optical_joint" type="fixed">
+    <joint name="${prefix}rgb_optical_joint" type="fixed">
       <origin xyz="0 0 0" rpy="${-M_PI/2} 0 ${-M_PI/2}" />
-      <parent link="${prefix}_rgb_base_link" />
-      <child link="${prefix}_rgb_optical_frame" />
+      <parent link="${prefix}rgb_base_link" />
+      <child link="${prefix}rgb_optical_frame" />
     </joint>
-    <link name="${prefix}_rgb_optical_frame">
+    <link name="${prefix}rgb_optical_frame">
       <inertial>
-        <mass value="0.001" />
+        <mass value="0.01" />
         <origin xyz="0 0 0" />
-        <inertia ixx="0.0001" ixy="0.0" ixz="0.0"
-          iyy="0.0001" iyz="0.0"
-          izz="0.0001" />
+        <xacro:solid_cuboid_inertia m="0.01" w="0.180" h="0.035" d="0.05" />
       </inertial>
     </link>
-    <joint name="${prefix}_joint" type="fixed">
+    <joint name="${prefix}joint" type="fixed">
       <origin xyz="0 ${asus_xtion_pro_rgb_rel_rgb_py} 0"
               rpy="0 0 0"/>
-      <parent link="${prefix}_rgb_link"/>
-      <child link="${prefix}_link"/>
+      <parent link="${prefix}rgb_base_link"/>
+      <child link="${prefix}link"/>
     </joint>
-    <link name="${prefix}_link">
+    <link name="${prefix}link">
       <visual>
         <origin xyz="-0.01 0 0" rpy="${-M_PI/2} -${M_PI} ${-M_PI/2}"/>
@@ -59,36 +55,30 @@
       <inertial>
         <mass value="0.01" />
-        <origin xyz="0 0 0" />
-        <inertia ixx="0.001" ixy="0.0" ixz="0.0"
-          iyy="0.001" iyz="0.0"
-          izz="0.001" />
+        <origin xyz="-0.0175 0.0025 0" rpy="0 0 0"/>
+        <xacro:solid_cuboid_inertia m="0.01" w="0.035" h="0.180" d="0.05" />
       </inertial>
     </link>
-    <joint name="${prefix}_depth_joint" type="fixed">
+    <joint name="${prefix}depth_joint" type="fixed">
       <origin xyz="0 ${asus_xtion_pro_depth_rel_rgb_py} 0" rpy="0 0 0" />
-      <parent link="${name}_rgb_base_link" />
-      <child link="${name}_depth_link" />
+      <parent link="${prefix}rgb_base_link" />
+      <child link="${prefix}depth_link" />
     </joint>
-    <link name="${prefix}_depth_link">
+    <link name="${prefix}depth_link">
       <inertial>
         <mass value="0.01" />
-        <origin xyz="0 0 0" />
-        <inertia ixx="0.001" ixy="0.0" ixz="0.0"
-          iyy="0.001" iyz="0.0"
-          izz="0.001" />
+        <origin xyz="-0.0175 -${asus_xtion_pro_depth_rel_rgb_py} 0" />
+        <xacro:solid_cuboid_inertia m="0.01" w="0.035" h="0.180" d="0.05" />
       </inertial>
     </link>
-    <joint name="${prefix}_depth_optical_joint" type="fixed">
+    <joint name="${prefix}depth_optical_joint" type="fixed">
       <origin xyz="0 0 0" rpy="${-M_PI/2} 0 ${-M_PI/2}" />
-      <parent link="${prefix}_depth_link" />
-      <child link="${prefix}_depth_optical_frame" />
+      <parent link="${prefix}depth_link" />
+      <child link="${prefix}depth_optical_frame" />
     </joint>
-    <link name="${prefix}_depth_optical_frame">
+    <link name="${prefix}depth_optical_frame">
       <inertial>
-        <mass value="0.001" />
-        <origin xyz="0 0 0" />
-        <inertia ixx="0.0001" ixy="0.0" ixz="0.0"
-          iyy="0.0001" iyz="0.0"
-          izz="0.0001" />
+        <mass value="0.01" />
+        <origin xyz="${asus_xtion_pro_depth_rel_rgb_py} 0 -0.0175" />
+        <xacro:solid_cuboid_inertia m="0.01" w="0.18" h="0.05" d="0.035" />
       </inertial>
     </link>
@@ -97,6 +87,6 @@
   </xacro:macro>
    <xacro:macro name="sensor_xtion_pro_gazebo">
-    <gazebo reference="${prefix}_depth_link">
-      <sensor type="depth" name="${prefix}_sensor">
+    <gazebo reference="${prefix}depth_link">
+      <sensor type="depth" name="${prefix}sensor">
         <always_on>true</always_on>
         <update_rate>20.0</update_rate>
@@ -113,5 +103,5 @@
           </clip>
         </camera>
-        <plugin name="${prefix}_controller" filename="libgazebo_ros_openni_kinect.so">
+        <plugin name="${prefix}controller" filename="libgazebo_ros_openni_kinect.so">
           <cameraName>${prefix}</cameraName>
           <alwaysOn>true</alwaysOn>
@@ -122,5 +112,5 @@
           <cameraInfoTopicName>rgb/camera_info</cameraInfoTopicName>
           <depthImageCameraInfoTopicName>depth/camera_info</depthImageCameraInfoTopicName>
-          <frameName>${prefix}_depth_optical_frame</frameName>
+          <frameName>${prefix}depth_optical_frame</frameName>
           <baseline>0.1</baseline>
           <distortion_k1>0.0</distortion_k1>
