Commit message: Ported tim571 humble, remove package:// in xacro

File: urdf/asus_xtion_pro.urdf.xacro (robot description, xacro)
@@ -44,5 +44,5 @@
         <origin xyz="-0.01 0 0" rpy="${-M_PI/2} -${M_PI} ${-M_PI/2}"/>
         <geometry>
-          <mesh filename="package://robotnik_sensors/meshes/asus_xtion_pro_live.dae" scale="${asus_xtion_scale} ${asus_xtion_scale} ${asus_xtion_scale}"/>
+          <mesh filename="file://$(find robotnik_sensors)/meshes/asus_xtion_pro_live.dae" scale="${asus_xtion_scale} ${asus_xtion_scale} ${asus_xtion_scale}"/>
         </geometry>
       </visual>

File: urdf/axis.urdf.xacro (robot description, xacro)
@@ -26,5 +26,5 @@
         </material>
         <geometry>
-          <mesh filename="package://robotnik_sensors/meshes/axis_p5514.stl" scale="1.0 1.0 1.0"/>
+          <mesh filename="file://$(find robotnik_sensors)/meshes/axis_p5514.stl" scale="1.0 1.0 1.0"/>
         </geometry>
       </visual>
@@ -33,5 +33,5 @@
         <!-- because the origin of the mesh file is not at the "center" of the model-->
         <geometry>
-          <mesh filename="package://robotnik_sensors/meshes/axis_p5514.stl" scale="1.0 1.0 1.0"/>
+          <mesh filename="file://$(find robotnik_sensors)/meshes/axis_p5514.stl" scale="1.0 1.0 1.0"/>
         </geometry>
       </collision>

File: urdf/axis_m5013.urdf.xacro (robot description, xacro)
@@ -27,5 +27,5 @@
         </material>
         <geometry>
-          <mesh filename="package://robotnik_sensors/meshes/axis_m5013.dae" scale="1.0 1.0 1.0"/>
+          <mesh filename="file://$(find robotnik_sensors)/meshes/axis_m5013.dae" scale="1.0 1.0 1.0"/>
         </geometry>
       </visual>
@@ -33,5 +33,5 @@
         <origin xyz="0.0 0.0 0" rpy="0 ${M_PI/2} 0"/>
         <geometry>
-          <mesh filename="package://robotnik_sensors/meshes/axis_m5013.stl" scale="1.0 1.0 1.0"/>
+          <mesh filename="file://$(find robotnik_sensors)/meshes/axis_m5013.stl" scale="1.0 1.0 1.0"/>
         </geometry>
       </collision>

File: urdf/axis_m5525.urdf.xacro (robot description, xacro)
@@ -30,5 +30,5 @@
         </material>
         <geometry>
-          <mesh filename="package://robotnik_sensors/meshes/axis_m5525.dae" scale="1.0 1.0 1.0"/>
+          <mesh filename="file://$(find robotnik_sensors)/meshes/axis_m5525.dae" scale="1.0 1.0 1.0"/>
         </geometry>
       </visual>
@@ -36,5 +36,5 @@
         <origin xyz="0.0 0.0 0" rpy="0 ${M_PI/2} 0"/>
         <geometry>
-          <mesh filename="package://robotnik_sensors/meshes/axis_m5525.stl" scale="1.0 1.0 1.0"/>
+          <mesh filename="file://$(find robotnik_sensors)/meshes/axis_m5525.stl" scale="1.0 1.0 1.0"/>
         </geometry>
       </collision>

File: urdf/axis_q8641.urdf.xacro (robot description, xacro)
@@ -30,5 +30,5 @@
         </material>
         <geometry>
-          <mesh filename="package://robotnik_sensors/meshes/axis_q8641_n1-1.STL" scale="1.0 1.0 1.0"/>
+          <mesh filename="file://$(find robotnik_sensors)/meshes/axis_q8641_n1-1.STL" scale="1.0 1.0 1.0"/>
         </geometry>
       </visual>
@@ -37,5 +37,5 @@
         <!-- because the origin of the mesh file is not at the "center" of the model-->
         <geometry>
-          <mesh filename="package://robotnik_sensors/meshes/axis_q8641_n1-1.STL" scale="1.0 1.0 1.0"/>
+          <mesh filename="file://$(find robotnik_sensors)/meshes/axis_q8641_n1-1.STL" scale="1.0 1.0 1.0"/>
         </geometry>
       </collision>
@@ -67,5 +67,5 @@
         </material>
         <geometry>
-          <mesh filename="package://robotnik_sensors/meshes/axis_q8641_n2-1.STL" scale="1.0 1.0 1.0"/>
+          <mesh filename="file://$(find robotnik_sensors)/meshes/axis_q8641_n2-1.STL" scale="1.0 1.0 1.0"/>
         </geometry>
       </visual>
@@ -74,5 +74,5 @@
         <!-- because the origin of the mesh file is not at the "center" of the model-->
         <geometry>
-          <mesh filename="package://robotnik_sensors/meshes/axis_q8641_n2-1.STL" scale="1.0 1.0 1.0"/>
+          <mesh filename="file://$(find robotnik_sensors)/meshes/axis_q8641_n2-1.STL" scale="1.0 1.0 1.0"/>
         </geometry>
       </collision>
@@ -113,5 +113,5 @@
         </material>
         <geometry>
-          <mesh filename="package://robotnik_sensors/meshes/camera_axis_q8641.STL" scale="1.0 1.0 1.0"/>
+          <mesh filename="file://$(find robotnik_sensors)/meshes/camera_axis_q8641.STL" scale="1.0 1.0 1.0"/>
         </geometry>
       </visual>
@@ -120,5 +120,5 @@
         <!-- because the origin of the mesh file is not at the "center" of the model-->
         <geometry>
-          <mesh filename="package://robotnik_sensors/meshes/camera_axis_q8641.STL" scale="1.0 1.0 1.0"/>
+          <mesh filename="file://$(find robotnik_sensors)/meshes/camera_axis_q8641.STL" scale="1.0 1.0 1.0"/>
         </geometry>
       </collision>

File: urdf/benewake_ce30.urdf.xacro (robot description, xacro)
@@ -16,5 +16,5 @@
       <origin xyz="0 0 0" rpy="0 0 0"/>
         <geometry>
-          <mesh filename="package://robotnik_sensors/meshes/benewake_ce30.stl" />
+          <mesh filename="file://$(find robotnik_sensors)/meshes/benewake_ce30.stl" />
         </geometry>
         <material name="black_alu"/>
@@ -23,5 +23,5 @@
         <origin xyz="0 0 0" rpy="0 0 0"/>
         <geometry>
-          <mesh filename="package://robotnik_sensors/meshes/benewake_ce30.stl" />
+          <mesh filename="file://$(find robotnik_sensors)/meshes/benewake_ce30.stl" />
         </geometry>
       </collision>

File: urdf/benewake_ce30d.urdf.xacro (robot description, xacro)
@@ -16,5 +16,5 @@
       <origin xyz="0 0 0" rpy="1.5708 0 1.5708"/>
         <geometry>
-          <mesh filename="package://robotnik_sensors/meshes/benewake_ce30d.stl" />
+          <mesh filename="file://$(find robotnik_sensors)/meshes/benewake_ce30d.stl" />
           <!--box size="${ce30d_length} ${ce30d_width} ${ce30d_height}"/-->
         </geometry>
@@ -24,5 +24,5 @@
         <origin xyz="0 0 0" rpy="0 0 0"/>
         <geometry>
-          <mesh filename="package://robotnik_sensors/meshes/benewake_ce30d.stl" />
+          <mesh filename="file://$(find robotnik_sensors)/meshes/benewake_ce30d.stl" />
         </geometry>
       </collision>

File: urdf/embedded_s.urdf.xacro (robot description, xacro)
@@ -11,5 +11,5 @@
         <origin xyz="0 0 0" rpy="0 0 0"/>
         <geometry>
-          <mesh filename="package://robotnik_sensors/meshes/orbbec_astra_embedded_s.stl"/>
+          <mesh filename="file://$(find robotnik_sensors)/meshes/orbbec_astra_embedded_s.stl"/>
           <!--box size="0.0148 0.0686 0.02235"/-->
         </geometry>
@@ -20,5 +20,5 @@
       <collision>
         <geometry>
-          <mesh filename="package://robotnik_sensors/meshes/orbbec_astra_embedded_s.stl"/>
+          <mesh filename="file://$(find robotnik_sensors)/meshes/orbbec_astra_embedded_s.stl"/>
           <!--box size="0.0148 0.0686 0.02235"/-->
         </geometry>

File: urdf/fotonic_e.urdf.xacro (robot description, xacro)
@@ -19,5 +19,5 @@
         </material>
         <geometry>
-          <mesh filename= "package://robotnik_sensors/meshes/fotonic_e.stl" scale="1.0 1.0 1.0"/>
+          <mesh filename= "file://$(find robotnik_sensors)/meshes/fotonic_e.stl" scale="1.0 1.0 1.0"/>
         </geometry>
       </visual>
@@ -25,5 +25,5 @@
         <origin xyz="0.0 0 -0.04" rpy="0 0 0" />
         <geometry>
-          <mesh filename= "package://robotnik_sensors/meshes/fotonic_e.stl" scale="1.0 1.0 1.0"/>
+          <mesh filename= "file://$(find robotnik_sensors)/meshes/fotonic_e.stl" scale="1.0 1.0 1.0"/>
         </geometry>
       </collision>

File: urdf/gps.urdf.xacro (robot description, xacro)
@@ -22,5 +22,5 @@
         </material>
 	      <geometry>
-	        <mesh filename="package://robotnik_sensors/meshes/antenna_3GO16.stl" scale="1.0 1.0 1.0"/>
+	        <mesh filename="file://$(find robotnik_sensors)/meshes/antenna_3GO16.stl" scale="1.0 1.0 1.0"/>
 	      </geometry>
 	    </visual>
@@ -28,5 +28,5 @@
 	      <origin rpy="0 0 0" xyz="0 0 0"/>
 	      <geometry>
-	        <mesh filename="package://robotnik_sensors/meshes/antenna_3GO16.stl" scale="1.0 1.0 1.0"/>
+	        <mesh filename="file://$(find robotnik_sensors)/meshes/antenna_3GO16.stl" scale="1.0 1.0 1.0"/>
 	      </geometry>
 	    </collision>

File: urdf/gps_with_mast.urdf.xacro (robot description, xacro)
@@ -57,5 +57,5 @@
         </material>
 	      <geometry>
-	        <mesh filename="package://robotnik_sensors/meshes/antenna_3GO16.stl" scale="1.0 1.0 1.0"/>
+	        <mesh filename="file://$(find robotnik_sensors)/meshes/antenna_3GO16.stl" scale="1.0 1.0 1.0"/>
 	      </geometry>
 	    </visual>
@@ -63,5 +63,5 @@
 	      <origin rpy="0 0 0" xyz="0 0 0"/>
 	      <geometry>
-	        <mesh filename="package://robotnik_sensors/meshes/antenna_3GO16.stl" scale="1.0 1.0 1.0"/>
+	        <mesh filename="file://$(find robotnik_sensors)/meshes/antenna_3GO16.stl" scale="1.0 1.0 1.0"/>
 	      </geometry>
 	    </collision>

File: urdf/hokuyo3d.urdf.xacro (robot description, xacro)
@@ -17,5 +17,5 @@
             <origin xyz="0 0 0" rpy="0 0 0"/>
             <geometry>
-                <mesh filename="package://robotnik_sensors/meshes/hokuyo3d.stl"/>
+                <mesh filename="file://$(find robotnik_sensors)/meshes/hokuyo3d.stl"/>
             </geometry>
         </visual>

File: urdf/hokuyo_urg04lx.urdf.xacro (robot description, xacro)
@@ -15,5 +15,5 @@
         <origin xyz="0.0 0.0 0.0" rpy="0 0 0"/>
         <geometry>
-            <mesh filename="package://robotnik_sensors/meshes/hokuyo_urg_04lx.dae"/>
+            <mesh filename="file://$(find robotnik_sensors)/meshes/hokuyo_urg_04lx.dae"/>
         </geometry>
       </visual>

File: urdf/hokuyo_ust10lx.urdf.xacro (robot description, xacro)
@@ -17,5 +17,5 @@
         <origin xyz="0 0 0.0" rpy="0 0 0"/>
         <geometry>
-            <mesh filename="package://robotnik_sensors/meshes/hokuyo_ust_10lx.dae"/>
+            <mesh filename="file://$(find robotnik_sensors)/meshes/hokuyo_ust_10lx.dae"/>
         </geometry>
       </visual>

File: urdf/hokuyo_utm30lx.urdf.xacro (robot description, xacro)
@@ -15,5 +15,5 @@
         <origin xyz="0 0 0.055" rpy="0 0 0"/>
         <geometry>
-            <mesh filename="package://robotnik_sensors/meshes/hokuyo_utm_30lx.dae"/>
+            <mesh filename="file://$(find robotnik_sensors)/meshes/hokuyo_utm_30lx.dae"/>
         </geometry>
       </visual>

File: urdf/intel_d435.urdf.xacro (robot description, xacro)
@@ -45,5 +45,5 @@
         <geometry>
           <!-- <box size="${d435_cam_width} ${d435_cam_height} ${d435_cam_depth}"/> -->
-          <mesh filename="package://robotnik_sensors/meshes/intel_d435_color.dae" />
+          <mesh filename="file://$(find robotnik_sensors)/meshes/intel_d435_color.dae" />
         </geometry>
       </visual>

File: urdf/intel_r430.urdf.xacro (robot description, xacro)
@@ -32,5 +32,5 @@
         <geometry>
           <!-- box size="${r430_cam_width} ${r430_cam_height} ${r430_cam_depth}"/ -->
-          <mesh filename="package://robotnik_sensors/meshes/intel_r430.dae" />
+          <mesh filename="file://$(find robotnik_sensors)/meshes/intel_r430.dae" />
         </geometry>
         <material name="aluminum">

File: urdf/kinect.urdf.xacro (robot description, xacro)
@@ -32,5 +32,5 @@
      <origin xyz="0 0 0" rpy="0 0 ${M_PI/2}"/>
       <geometry>
-       <mesh filename="package://robotnik_sensors/meshes/kinect.dae"/>
+       <mesh filename="file://$(find robotnik_sensors)/meshes/kinect.dae"/>
       </geometry>
     </visual>

File: urdf/kinectv2.urdf.xacro (robot description, xacro)
@@ -39,8 +39,8 @@
       <geometry>
         <xacro:if value="${base}">
-          <mesh filename="package://robotnik_sensors/meshes/kinectv2.dae"/>
+          <mesh filename="file://$(find robotnik_sensors)/meshes/kinectv2.dae"/>
         </xacro:if>
         <xacro:unless value="${base}">
-          <mesh filename="package://robotnik_sensors/meshes/kinectv2_nobase.dae"/>
+          <mesh filename="file://$(find robotnik_sensors)/meshes/kinectv2_nobase.dae"/>
         </xacro:unless>
       </geometry>

File: urdf/lidar_mast.urdf.xacro (robot description, xacro)
@@ -12,5 +12,5 @@
         <origin xyz="0 0 0" rpy="0 0 0"/>
         <geometry>
-          <mesh filename="package://robotnik_sensors/meshes/lidar_mast.STL"/>
+          <mesh filename="file://$(find robotnik_sensors)/meshes/lidar_mast.STL"/>
         </geometry>
         <material name="light_zed_grey">
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