Commit message: Update oak_d_pro_poe to match the real driver

File: urdf/oak_d_pro_poe.urdf.xacro (robot description, xacro)
@@ -65,7 +65,7 @@
       <origin xyz="0 0 0" rpy="${-M_PI/2} 0 ${-M_PI/2}" />
       <parent link="${prefix}_rgb_camera_frame" />
-      <child link="${prefix}_rgb_optical_frame" />
+      <child link="${prefix}_rgb_camera_optical_frame" />
     </joint>
-    <link name="${prefix}_rgb_optical_frame"/>
+    <link name="${prefix}_rgb_camera_optical_frame"/>
     <!-- Left camera joints and links -->
     <joint name="${prefix}_left_camera_joint" type="fixed">

Commit message: Update oak_d_pro_poe.urdf.xacro
correct "grey" material issue.

File: urdf/oak_d_pro_poe.urdf.xacro (robot description, xacro)
@@ -7,7 +7,4 @@
 <robot name="sensor_oak_d_pro_poe" xmlns:xacro="http://wiki.ros.org/xacro">
   <!-- Includes -->
-  <material name="grey">
-    <color rgba="0.75 0.75 0.75 1"/>
-  </material>
   <xacro:macro name="sensor_oak_d_pro_poe" params="prefix parent *origin prefix_topic:='front_rgbd_camera' use_nominal_extrinsics:=true update_rate:=7">
     <xacro:property name="M_PI" value="3.1415926535897931" />
@@ -41,5 +38,7 @@
           <mesh filename="package://robotnik_sensors/meshes/oak_d_pro_poe.stl" />
         </geometry>
-        <material name="grey"/>
+        <material name="grey">
+          <color rgba="0.75 0.75 0.75 1"/>
+        </material>
       </visual>
       <collision>

Commit message: Update oak_d_pro_poe.urdf.xacro
Change "grey" material name to "grey_oak"

File: urdf/oak_d_pro_poe.urdf.xacro (robot description, xacro)
@@ -38,5 +38,5 @@
           <mesh filename="package://robotnik_sensors/meshes/oak_d_pro_poe.stl" />
         </geometry>
-        <material name="grey">
+        <material name="grey_oak">
           <color rgba="0.75 0.75 0.75 1"/>
         </material>
