Commit message: bpearl: correct link and joint names

File: urdf/rs_bpearl.urdf.xacro (robot description, xacro)
@@ -6,10 +6,10 @@
       <color rgba="0.9 0.9 0.9 1"/>
     </material>
-    <joint name="${prefix}bpearl_base_joint" type="fixed">
+    <joint name="${prefix}_base_joint" type="fixed">
       <xacro:insert_block name="origin" />
       <parent link="${parent}"/>
-      <child link="${prefix}bpearl_base_link" />
+      <child link="${prefix}_base_link" />
     </joint>
-    <link name="${prefix}bpearl_base_link">
+    <link name="${prefix}_base_link">
       <visual>
       <!-- origin xyz="0 0 0" rpy="0 0 1.5708"/ -->
@@ -33,10 +33,10 @@
       </inertial>
     </link>
-    <joint name="${prefix}bpearl_joint" type="fixed">
-      <parent link="${prefix}bpearl_base_link"/>
-      <child link="${prefix}bpearl_link" />
+    <joint name="${prefix}_joint" type="fixed">
+      <parent link="${prefix}_base_link"/>
+      <child link="${prefix}_link" />
       <origin xyz="0 0 0.06" rpy="0 0 0"/>
     </joint>
-    <link name="${prefix}bpearl_link"/>
+    <link name="${prefix}_link"/>
   <sensor_rs_bpearl_gazebo range_min="${range_min}" range_max="${range_max}" hfov="${hfov}" samples="${samples}" vfov="${vfov}" lasers="${lasers}" fps="${fps}" gpu="${gpu}"/>
   </xacro:macro>

Commit message: Fix rs bpearl inertia

File: urdf/rs_bpearl.urdf.xacro (robot description, xacro)
@@ -28,7 +28,7 @@
       <inertial>
         <!-- The following are not reliable values, and should not be used for modeling -->
-        <mass value="0.564" />
-        <origin xyz="0 0 0" />
-        <inertia ixx="0.003881243" ixy="0.0" ixz="0.0" iyy="0.000498940" iyz="0.0" izz="0.003879257" />
+        <mass value="0.92" />
+        <origin xyz="0 0 0.055" />
+        <xacro:solid_cuboid_inertia m="0.92" w="0.111" h="0.111" d="0.11" />
       </inertial>
     </link>

Commit message: color added

File: urdf/rs_bpearl.urdf.xacro (robot description, xacro)
@@ -3,7 +3,4 @@
   <xacro:property name="M_PI" value="3.1415926535897931" />
   <xacro:macro name="sensor_rs_bpearl" params="prefix parent prefix_topic *origin range_min range_max hfov samples vfov lasers fps gpu:=^|true">
-    <material name="black_alu">
-      <color rgba="0.9 0.9 0.9 1"/>
-    </material>
     <joint name="${prefix}_base_joint" type="fixed">
       <xacro:insert_block name="origin" />
@@ -18,5 +15,7 @@
           <mesh filename="package://robotnik_sensors/meshes/rs_bpearl.stl" />
         </geometry>
-        <material name="black_alu"/>
+        <material name="blackgray_color">
+          <color rgba="0.25 0.25 0.25 1"/>
+        </material>
       </visual>
       <collision>
@@ -42,5 +41,23 @@
   </xacro:macro>
   <xacro:macro name="sensor_rs_bpearl_gazebo" params="range_min range_max hfov samples vfov lasers fps gpu">
+    <gazebo reference="${prefix}_base_link">
+      <visual>
+        <material>
+          <ambient>0.5 0.5 0.5 1.0</ambient>
+          <diffuse>0.250754 0.250754 0.250754 1.0</diffuse>
+          <specular>0.2508273 0.2508273 0.2508273 1.0</specular>
+          <emissive>0.0 0.0 0.0 0.0</emissive>
+        </material>
+      </visual>
+    </gazebo>
     <gazebo reference="${prefix}_link">
+      <visual>
+        <material>
+          <ambient>1.2 0.2 0.2 1.0</ambient>
+          <diffuse>0.250754 0.250754 0.250754 1.0</diffuse>
+          <specular>0.2508273 0.2508273 0.2508273 1.0</specular>
+          <emissive>0.0 0.0 0.0 0.0</emissive>
+        </material>
+      </visual>
       <xacro:if value="${gpu}">
         <!-- Using GPU needs: https://github.com/RobotnikAutomation/velodyne_simulator -->

Commit message: use of gpu/cpu parametrized, set to gpu by default

File: urdf/rs_bpearl.urdf.xacro (robot description, xacro)
@@ -2,5 +2,5 @@
 <robot name="sensor_rs_bpearl" xmlns:xacro="http://wiki.ros.org/xacro">
   <xacro:property name="M_PI" value="3.1415926535897931" />
-  <xacro:macro name="sensor_rs_bpearl" params="prefix parent prefix_topic *origin range_min range_max hfov samples vfov lasers fps gpu:=^|true">
+  <xacro:macro name="sensor_rs_bpearl" params="prefix parent prefix_topic *origin range_min range_max hfov samples vfov lasers fps gpu:=true">
     <joint name="${prefix}_base_joint" type="fixed">
       <xacro:insert_block name="origin" />

File: urdf/sick_microscan3.urdf.xacro (robot description, xacro)
@@ -2,5 +2,5 @@
 <robot name="sensor_sick_microscan3"
 	xmlns:xacro="http://wiki.ros.org/xacro">
-	<xacro:macro name="sensor_sick_microscan3" params="prefix parent prefix_topic:='front_laser' *origin max_angle:=2.3562 min_angle:=-2.3562">
+	<xacro:macro name="sensor_sick_microscan3" params="prefix parent prefix_topic:='front_laser' *origin max_angle:=2.3562 min_angle:=-2.3562 gpu:=^|true">
 		<joint name="${prefix}_base_joint" type="fixed">
 			<xacro:insert_block name="origin" />
@@ -40,5 +40,13 @@
 	<xacro:macro name="sensor_sick_microscan3_gazebo">
 		<gazebo reference="${prefix}_link">
-			<sensor type="gpu_ray" name="${prefix}_sensor">
+			<xacro:if value="${gpu}">
+				<xacro:property name="ray_type" value="gpu_ray" />
+				<xacro:property name="plugin_lib" value="libgazebo_ros_gpu_laser.so" />
+			</xacro:if>
+			<xacro:unless value="${gpu}">
+				<xacro:property name="ray_type" value="ray" />
+				<xacro:property name="plugin_lib" value="libgazebo_ros_laser.so" />
+			</xacro:unless>
+			<sensor type="${ray_type}" name="${prefix}_sensor">
 				<pose>0 0 0 0 0 0</pose>
 				<visualize>false</visualize>
@@ -64,5 +72,5 @@
 					</noise>
 				</ray>
-				<plugin name="${prefix}_controller" filename="libgazebo_ros_gpu_laser.so">
+				<plugin name="${prefix}_controller" filename="${plugin_lib}">
 					<topicName>${prefix_topic}/scan</topicName>
 					<frameName>/${prefix}_link</frameName>					<!-- if not global (leading /) sets the current namespace as a prefix (/ns/name_laser_link) -->

Commit message: rs_bpearl: Move link origin to match the user manual specs

File: urdf/rs_bpearl.urdf.xacro (robot description, xacro)
@@ -35,5 +35,5 @@
       <parent link="${prefix}_base_link"/>
       <child link="${prefix}_link" />
-      <origin xyz="0 0 0.06" rpy="0 0 0"/>
+      <origin xyz="0 0 0.09427" rpy="0 0 0"/>
     </joint>
     <link name="${prefix}_link"/>

Commit message: Add suffix_topic to rs_bpearl

File: urdf/rs_bpearl.urdf.xacro (robot description, xacro)
@@ -2,5 +2,5 @@
 <robot name="sensor_rs_bpearl" xmlns:xacro="http://wiki.ros.org/xacro">
   <xacro:property name="M_PI" value="3.1415926535897931" />
-  <xacro:macro name="sensor_rs_bpearl" params="prefix parent prefix_topic *origin range_min range_max hfov samples vfov lasers fps gpu:=true">
+  <xacro:macro name="sensor_rs_bpearl" params="prefix parent prefix_topic suffix_topic *origin range_min range_max hfov samples vfov lasers fps gpu:=true">
     <joint name="${prefix}_base_joint" type="fixed">
       <xacro:insert_block name="origin" />
@@ -97,5 +97,5 @@
           </ray>
           <plugin name="${prefix}_controller" filename="${plugin_lib}">
-            <topicName>${prefix_topic}/points</topicName>
+            <topicName>${prefix_topic}/points${suffix_topic}</topicName>
             <frameName>/${prefix}_link</frameName>
             <gaussianNoise>0.008</gaussianNoise>

Commit message: Update visual tf for rs_bpearl

File: urdf/rs_bpearl.urdf.xacro (robot description, xacro)
@@ -11,5 +11,5 @@
       <visual>
       <!-- origin xyz="0 0 0" rpy="0 0 1.5708"/ -->
-      <origin xyz="0 0 0" rpy="0 0 0"/>
+      <origin xyz="0 0 0" rpy="0 0 1.5708"/>
         <geometry>
           <mesh filename="package://robotnik_sensors/meshes/rs_bpearl.stl" />
@@ -20,5 +20,5 @@
       </visual>
       <collision>
-        <origin xyz="0 0 0" rpy="0 0 0"/>
+        <origin xyz="0 0 0" rpy="0 0 1.5708"/>
         <geometry>
           <mesh filename="package://robotnik_sensors/meshes/rs_bpearl.stl" />

Commit message: rs_bpearl: Set suffix_topic to '' as default

File: urdf/rs_bpearl.urdf.xacro (robot description, xacro)
@@ -2,5 +2,5 @@
 <robot name="sensor_rs_bpearl" xmlns:xacro="http://wiki.ros.org/xacro">
   <xacro:property name="M_PI" value="3.1415926535897931" />
-  <xacro:macro name="sensor_rs_bpearl" params="prefix parent prefix_topic suffix_topic *origin range_min range_max hfov samples vfov lasers fps gpu:=true">
+  <xacro:macro name="sensor_rs_bpearl" params="prefix parent prefix_topic suffix_topic:='' *origin range_min range_max hfov samples vfov lasers fps gpu:=true">
     <joint name="${prefix}_base_joint" type="fixed">
       <xacro:insert_block name="origin" />
