Commit message: compliant with new tag hardwareInterface requirement in joint

File: urdf/axis.urdf.xacro (robot description, xacro)
@@ -56,5 +56,7 @@
 	  <transmission name="${name}_pan_trans">
 		 <type>transmission_interface/SimpleTransmission</type>
-	     <joint name="joint_${name}_pan" />
+	     <joint name="joint_${name}_pan">
+			<hardwareInterface>EffortJointInterface</hardwareInterface>
+	     </joint>
 	     <actuator name="pan_motor">
 			   <hardwareInterface>EffortJointInterface</hardwareInterface>
@@ -79,5 +81,7 @@
 	  <transmission name="${name}_tilt_trans">
 		 <type>transmission_interface/SimpleTransmission</type>
-	     <joint name="joint_${name}_tilt" />
+	     <joint name="joint_${name}_tilt">
+	     	<hardwareInterface>EffortJointInterface</hardwareInterface>
+		 </joint>
 	     <actuator name="tilt_motor">
 				 <hardwareInterface>EffortJointInterface</hardwareInterface>

File: urdf/axis_m5013.urdf.xacro (robot description, xacro)
@@ -56,5 +56,7 @@
 	  <transmission name="${name}_pan_trans">
 		 <type>transmission_interface/SimpleTransmission</type>
-	     <joint name="joint_${name}_pan" />
+	     <joint name="joint_${name}_pan">
+			<hardwareInterface>EffortJointInterface</hardwareInterface>
+		 </joint>
 	     <actuator name="pan_motor">
 			   <hardwareInterface>EffortJointInterface</hardwareInterface>
@@ -79,8 +81,10 @@
 	  <transmission name="${name}_tilt_trans">
 		 <type>transmission_interface/SimpleTransmission</type>
-	     <joint name="joint_${name}_tilt" />
+	     <joint name="joint_${name}_tilt">
+			 <hardwareInterface>EffortJointInterface</hardwareInterface>
+		 </joint>
 	     <actuator name="tilt_motor">
-				 <hardwareInterface>EffortJointInterface</hardwareInterface>
-				 <mechanicalReduction>${ptz_mechanical_reduction}</mechanicalReduction>
+			<hardwareInterface>EffortJointInterface</hardwareInterface>
+			<mechanicalReduction>${ptz_mechanical_reduction}</mechanicalReduction>
 	     </actuator>
 	  </transmission>

Commit message: updated model of axis camera

File: urdf/axis.urdf.xacro (robot description, xacro)
@@ -15,5 +15,5 @@
     <link name="${name}_link">
       <inertial>
-        <origin xyz="-0.3 0.0 -0.03" rpy="0 ${M_PI/2} 0"/>
+        <origin xyz="0.0 0.0 0.0" rpy="0 0 0"/>
         <mass value="0.1"/>
         <origin xyz="0 0 0" rpy="0 0 0"/>
@@ -21,5 +21,5 @@
       </inertial>
       <visual>
-        <origin xyz="-0.3 0.0 -0.03" rpy="0 ${M_PI/2} 0"/>
+        <origin xyz="0.0 0.0 0.0" rpy="0 0 0"/>
         <!-- because the origin of the mesh file is not at the "center" of the model-->
         <material name="axis_color">
@@ -27,12 +27,12 @@
         </material>
         <geometry>
-          <mesh filename="package://robotnik_sensors/meshes/axis_p5512.stl" scale="1.0 1.0 1.0"/>
+          <mesh filename="package://robotnik_sensors/meshes/camera_axis_p5514.stl" scale="1.0 1.0 1.0"/>
         </geometry>
       </visual>
       <collision>
-        <origin xyz="-0.3 0.0 -0.03" rpy="0 ${M_PI/2} 0"/>
+        <origin xyz="0.0 0.0 0.0" rpy="0 0 0"/>
         <!-- because the origin of the mesh file is not at the "center" of the model-->
         <geometry>
-          <mesh filename="package://robotnik_sensors/meshes/axis_p5512.stl" scale="1.0 1.0 1.0"/>
+          <mesh filename="package://robotnik_sensors/meshes/camera_axis_p5514.stl" scale="1.0 1.0 1.0"/>
         </geometry>
       </collision>
@@ -40,5 +40,5 @@
     <joint name="joint_${name}_pan" type="revolute">
       <axis xyz="0 0 -1"/>
-      <origin xyz="0.1 0.0 0.0" rpy="0 0 0"/>
+      <origin xyz="0.0 0.0 0.0" rpy="0 0 0"/>
       <!-- check the displacement -->
       <parent link="${name}_link"/>

Commit message: links of xacro file renamed

File: urdf/axis.urdf.xacro (robot description, xacro)
@@ -11,7 +11,7 @@
       <xacro:insert_block name="origin"/>
       <parent link="${parent}"/>
-      <child link="${prefix}_link"/>
+      <child link="${prefix}_base_link"/>
     </joint>
-    <link name="${prefix}_link">
+    <link name="${prefix}_base_link">
       <inertial>
         <origin xyz="0.0 0.0 0.0" rpy="0 0 0"/>
@@ -42,5 +42,5 @@
       <origin xyz="0.0 0.0 0.0" rpy="0 0 0"/>
       <!-- check the displacement -->
-      <parent link="${prefix}_link"/>
+      <parent link="${prefix}_base_link"/>
       <child link="${prefix}_pan_link"/>
       <limit effort="${ptz_joint_effort_limit}" velocity="${ptz_joint_velocity_limit}" lower="-3.1416" upper="3.1416"/>
@@ -92,7 +92,7 @@
       <origin xyz="0.0 0 0" rpy="0 0 0"/>
       <parent link="${prefix}_tilt_link"/>
-      <child link="${prefix}_frame"/>
+      <child link="${prefix}_frame_link"/>
     </joint>
-    <link name="${prefix}_frame">
+    <link name="${prefix}_frame_link">
       <inertial>
         <mass value="0.001"/>
@@ -104,8 +104,8 @@
     <joint name="${prefix}_optical_joint" type="fixed">
       <origin xyz="0 0 0" rpy="${-M_PI/2} 0 ${-M_PI/2}"/>
-      <parent link="${prefix}_frame"/>
-      <child link="${prefix}_optical_frame"/>
+      <parent link="${prefix}_frame_link"/>
+      <child link="${prefix}_optical_frame_link"/>
     </joint>
-    <link name="${prefix}_optical_frame">
+    <link name="${prefix}_optical_frame_link">
       <inertial>
         <mass value="0.001"/>
@@ -114,5 +114,5 @@
       </inertial>
     </link>
-    <gazebo reference="${prefix}_link">
+    <gazebo reference="${prefix}_base_link">
       <material>Gazebo/FlatBlack</material>
     </gazebo>
@@ -121,5 +121,5 @@
   </xacro:macro>
   <xacro:macro name="sensor_axis_gazebo">
-    <gazebo reference="${prefix}_frame">
+    <gazebo reference="${prefix}_frame_link">
       <sensor type="camera" name="${prefix}_sensor">
         <update_rate>30.0</update_rate>
@@ -142,5 +142,5 @@
           <imageTopicName>image_raw</imageTopicName>
           <cameraInfoTopicName>camera_info</cameraInfoTopicName>
-          <frameName>${prefix}_optical_frame</frameName>
+          <frameName>${prefix}_optical_frame_link</frameName>
           <hackBaseline>0.0</hackBaseline>
           <distortionK1>0.0</distortionK1>

Commit message: Fixed bug in limits of velocity controller, also changed controller type from position to velocity position controller

File: urdf/axis.urdf.xacro (robot description, xacro)
@@ -44,5 +44,5 @@
       <parent link="${prefix}_base_link"/>
       <child link="${prefix}_pan_link"/>
-      <limit effort="${ptz_joint_effort_limit}" velocity="${ptz_joint_velocity_limit}" lower="-3.1416" upper="3.1416"/>
+      <limit effort="${ptz_joint_effort_limit}" velocity="${ptz_joint_velocity_limit}" lower="-3.1415" upper="3.1415"/>
       <joint_properties damping="${ptz_joint_damping}" friction="{ptz_joint_friction}"/>
     </joint>
@@ -57,8 +57,8 @@
       <type>transmission_interface/SimpleTransmission</type>
       <joint name="${prefix}_pan_joint">
-        <hardwareInterface>hardware_interface/PositionJointInterface</hardwareInterface>
+        <hardwareInterface>hardware_interface/VelocityJointInterface</hardwareInterface>
       </joint>
       <actuator name="pan_motor">
-        <hardwareInterface>hardware_interface/PositionJointInterface</hardwareInterface>
+        <hardwareInterface>hardware_interface/VelocityJointInterface</hardwareInterface>
         <mechanicalReduction>${ptz_mechanical_reduction}</mechanicalReduction>
       </actuator>
@@ -82,8 +82,8 @@
       <type>transmission_interface/SimpleTransmission</type>
       <joint name="${prefix}_tilt_joint">
-        <hardwareInterface>hardware_interface/PositionJointInterface</hardwareInterface>
+        <hardwareInterface>hardware_interface/VelocityJointInterface</hardwareInterface>
       </joint>
       <actuator name="tilt_motor">
-        <hardwareInterface>hardware_interface/PositionJointInterface</hardwareInterface>
+        <hardwareInterface>hardware_interface/VelocityJointInterface</hardwareInterface>
         <mechanicalReduction>${ptz_mechanical_reduction}</mechanicalReduction>
       </actuator>

Commit message: added the capability to set the Axis camera far and near from params

File: urdf/axis.urdf.xacro (robot description, xacro)
@@ -6,5 +6,5 @@
   <xacro:property name="ptz_joint_damping" value="0.1"/>
   <xacro:property name="ptz_mechanical_reduction" value="1.0"/>
-  <xacro:macro name="sensor_axis" params="prefix parent *origin">
+  <xacro:macro name="sensor_axis" params="prefix parent *origin far:=^|8.0 near:=^|0.05">
     <joint name="${prefix}_joint" type="fixed">
       <axis xyz="0 1 0"/>
@@ -132,6 +132,6 @@
           </image>
           <clip>
-            <near>0.05</near>
-            <far>8.0</far>
+            <near>${near}</near>
+            <far>${far}</far>
           </clip>
         </camera>

File: urdf/axis_m5013.urdf.xacro (robot description, xacro)
@@ -7,5 +7,5 @@
   <xacro:property name="ptz_mechanical_reduction" value="1.0"/>
   <xacro:property name="PI" value="3.14159265359"/>
-  <xacro:macro name="sensor_axis_m5013" params="prefix parent *origin">
+  <xacro:macro name="sensor_axis_m5013" params="prefix parent *origin far:=^|8.0 near:=^|0.05">
     <joint name="${prefix}_joint" type="fixed">
       <axis xyz="0 1 0"/>
@@ -132,6 +132,6 @@
 					</image>
 					<clip>
-						<near>0.05</near>
-						<far>8.0</far>
+						<near>${near}</near>
+						<far>${far}</far>
 					</clip>
 				</camera>

File: urdf/axis_m5525.urdf.xacro (robot description, xacro)
@@ -7,5 +7,5 @@
   <xacro:property name="ptz_mechanical_reduction" value="1.0"/>
   <xacro:property name="PI" value="3.14159265359"/>
-  <xacro:macro name="sensor_axis_m5525" params="prefix parent *origin">
+  <xacro:macro name="sensor_axis_m5525" params="prefix parent *origin far:=^|8.0 near:=^|0.05">
     <joint name="${prefix}_joint" type="fixed">
       <axis xyz="0 1 0"/>
@@ -135,6 +135,6 @@
 					</image>
 					<clip>
-						<near>0.05</near>
-						<far>8.0</far>
+						<near>${near}</near>
+						<far>${far}</far>
 					</clip>
 				</camera>

Commit message: Update axis inertia

File: urdf/axis.urdf.xacro (robot description, xacro)
@@ -15,8 +15,7 @@
     <link name="${prefix}_base_link">
       <inertial>
-        <origin xyz="0.0 0.0 0.0" rpy="0 0 0"/>
-        <mass value="0.1"/>
-        <origin xyz="0 0 0" rpy="0 0 0"/>
-        <inertia ixx="0.1" ixy="0" ixz="0" iyy="0.1" iyz="0" izz="0.1"/>
+        <origin xyz="0.0  0.0 -0.015" rpy="0 ${M_PI/2} 0"/>
+        <mass value="0.8"/>
+        <xacro:solid_cuboid_inertia m="0.8" w="0.152" h="0.132" d="0.132" />
       </inertial>
       <visual>
@@ -51,5 +50,5 @@
         <mass value="0.1"/>
         <origin xyz="0 0 0" rpy="0 0 0"/>
-        <inertia ixx="0.1" ixy="0" ixz="0" iyy="0.1" iyz="0" izz="0.1"/>
+        <xacro:solid_cuboid_inertia m="0.1" w="0.1" h="0.11" d="0.11" />
       </inertial>
     </link>
@@ -76,5 +75,5 @@
         <mass value="0.1"/>
         <origin xyz="0 0 0" rpy="0 0 0"/>
-        <inertia ixx="0.1" ixy="0" ixz="0" iyy="0.1" iyz="0" izz="0.1"/>
+        <xacro:solid_cuboid_inertia m="0.1" w="0.11" h="0.11" d="0.1" />
       </inertial>
     </link>
@@ -96,7 +95,7 @@
     <link name="${prefix}_frame_link">
       <inertial>
-        <mass value="0.001"/>
+        <mass value="0.1"/>
         <origin xyz="0 0 0"/>
-        <inertia ixx="0.0001" ixy="0.0" ixz="0.0" iyy="0.0001" iyz="0.0" izz="0.0001"/>
+        <xacro:solid_cuboid_inertia m="0.1" w="0.11" h="0.11" d="0.1" />
       </inertial>
     </link>
@@ -109,7 +108,7 @@
     <link name="${prefix}_optical_frame_link">
       <inertial>
-        <mass value="0.001"/>
+        <mass value="0.1"/>
         <origin xyz="0 0 0"/>
-        <inertia ixx="0.0001" ixy="0.0" ixz="0.0" iyy="0.0001" iyz="0.0" izz="0.0001"/>
+        <xacro:solid_cuboid_inertia m="0.1" w="0.11" h="0.11" d="0.1" />
       </inertial>
     </link>

Commit message: Normalize the rotation axis of the axis urdf camera

File: urdf/axis.urdf.xacro (robot description, xacro)
@@ -38,5 +38,5 @@
     </link>
     <joint name="${prefix}_pan_joint" type="revolute">
-      <axis xyz="0 0 -1"/>
+      <axis xyz="0 0 1"/>
       <origin xyz="0.0 0.0 0.0" rpy="0 0 0"/>
       <!-- check the displacement -->
@@ -64,6 +64,7 @@
     </transmission>
     <joint name="${prefix}_tilt_joint" type="revolute">
-      <axis xyz="0 -1 0"/>
-      <origin xyz="0.0 0.0 0.0"/>
+      <axis xyz="0 0 1"/>
+      <!--origin xyz="0.0 0.0 0.0"/-->
+      <origin xyz="0.0 0.0 0.0" rpy="${-PI/2} 0 0"/>
       <parent link="${prefix}_pan_link"/>
       <child link="${prefix}_tilt_link"/>

Commit message: axis: Normalize the axis of the camear ptz models

File: urdf/axis.urdf.xacro (robot description, xacro)
@@ -8,5 +8,5 @@
   <xacro:macro name="sensor_axis" params="prefix parent *origin far:=^|8.0 near:=^|0.05">
     <joint name="${prefix}_joint" type="fixed">
-      <axis xyz="0 1 0"/>
+      <axis xyz="0 0 1"/>
       <xacro:insert_block name="origin"/>
       <parent link="${parent}"/>
@@ -65,5 +65,4 @@
     <joint name="${prefix}_tilt_joint" type="revolute">
       <axis xyz="0 0 1"/>
-      <!--origin xyz="0.0 0.0 0.0"/-->
       <origin xyz="0.0 0.0 0.0" rpy="${-PI/2} 0 0"/>
       <parent link="${prefix}_pan_link"/>

File: urdf/axis_m5013.urdf.xacro (robot description, xacro)
@@ -9,5 +9,5 @@
   <xacro:macro name="sensor_axis_m5013" params="prefix parent *origin far:=^|8.0 near:=^|0.05">
     <joint name="${prefix}_joint" type="fixed">
-      <axis xyz="0 1 0"/>
+      <axis xyz="0 0 1"/>
       <xacro:insert_block name="origin"/>
       <parent link="${parent}"/>
@@ -38,6 +38,6 @@
     </link>
     <joint name="${prefix}_pan_joint" type="revolute">
-      <axis xyz="1 0 0"/>
-      <origin xyz="0.04 0.0 0.0" rpy="0 0 0"/>
+      <axis xyz="0 0 1"/>
+      <origin xyz="1 0.0 0.04" rpy="0 0 0"/>
       <!-- check the displacement -->
       <parent link="${prefix}_base_link"/>
@@ -64,6 +64,6 @@
     </transmission>
     <joint name="${prefix}_tilt_joint" type="revolute">
-      <axis xyz="0 -1 0"/>
-      <origin xyz="0.0 0.0 0.0" rpy="0 ${-PI/2} 0"/>
+      <axis xyz="0 0 1"/>
+      <origin xyz="0.0 0.0 0.0" rpy="${-PI/2} 0 0"/>
       <parent link="${prefix}_pan_link"/>
       <child link="${prefix}_tilt_link"/>

File: urdf/axis_m5525.urdf.xacro (robot description, xacro)
@@ -9,8 +9,5 @@
   <xacro:macro name="sensor_axis_m5525" params="prefix parent *origin far:=^|8.0 near:=^|0.05 prefix_topic:=^ptz_camera">
     <joint name="${prefix}_joint" type="fixed">
-      <axis xyz="0 1 0"/>
-      <!--
-	      <origin xyz="0.180 0.0 0.270"/>
--->
+      <axis xyz="0 0 1"/>
       <xacro:insert_block name="origin"/>
       <parent link="${parent}"/>
@@ -19,10 +16,10 @@
     <link name="${prefix}_base_link">
       <inertial>
-        <origin xyz="0.066 0 0" rpy="0 ${M_PI/2} 0"/>
+        <origin xyz="0.066 0 0" rpy="0 0 0"/>
         <mass value="0.8"/>
         <xacro:solid_cuboid_inertia m="0.8" w="0.165" h="0.165" d="0.132" />
       </inertial>
       <visual>
-        <origin xyz="0 0 0" rpy="0 ${M_PI/2} 0"/>
+        <origin xyz="0 0 0" rpy="0 0 0"/>
         <!-- to center the axis model -->
         <material name="axis_color">
@@ -34,5 +31,5 @@
       </visual>
       <collision>
-        <origin xyz="0.0 0.0 0" rpy="0 ${M_PI/2} 0"/>
+        <origin xyz="0.0 0.0 0" rpy="0 0 0"/>
         <geometry>
           <mesh filename="package://robotnik_sensors/meshes/axis_m5525.stl" scale="1.0 1.0 1.0"/>
@@ -41,6 +38,6 @@
     </link>
     <joint name="${prefix}_pan_joint" type="revolute">
-      <axis xyz="1 0 0"/>
-      <origin xyz="0.087 0.0 0.0" rpy="0 0 0"/>
+      <axis xyz="0 0 1"/>
+      <origin xyz="0 0.0 0.087" rpy="0 0 0"/>
       <!-- check the displacement -->
       <parent link="${prefix}_base_link"/>
@@ -67,6 +64,6 @@
     </transmission>
     <joint name="${prefix}_tilt_joint" type="revolute">
-      <axis xyz="0 -1 0"/>
-      <origin xyz="0.0 0.0 0.0" rpy="0 ${-PI/2} 0"/>
+      <axis xyz="0 0 1"/>
+      <origin xyz="0.0 0.0 0.0" rpy="${-PI/2} 0 0"/>
       <parent link="${prefix}_pan_link"/>
       <child link="${prefix}_tilt_link"/>
