Commit message: Create variable include_inertial to be able to deactivate all sensors inertia

File: urdf/a21_ultrasonic_sensor.urdf.xacro (robot description, xacro)
@@ -1,5 +1,5 @@
 <?xml version="1.0"?>
 <robot name="sensor_ultrasonic_a21" xmlns:xacro="http://wiki.ros.org/xacro">
-  <xacro:macro name="sensor_ultrasonic_a21" params="prefix parent prefix_topic:='front_ultrasonic' *origin gpu:=^|true">
+  <xacro:macro name="sensor_ultrasonic_a21" params="prefix parent prefix_topic:='front_ultrasonic' *origin gpu:=^|true include_inertial:=^|true">
     <joint name="${prefix}_base_joint" type="fixed">
       <xacro:insert_block name="origin" />
@@ -20,9 +20,11 @@
         </geometry>
       </visual>
-      <inertial>
-        <origin xyz="0.0 0 0.035" rpy="0 0 0" />
-        <mass value="0.130" />
-        <xacro:solid_cuboid_inertia m="0.130" w="0.05" h="0.05" d="0.07" />
-      </inertial>
+      <xacro:if value="$(include_inertial)">
+        <inertial>
+          <origin xyz="0.0 0 0.035" rpy="0 0 0" />
+          <mass value="0.130" />
+          <xacro:solid_cuboid_inertia m="0.130" w="0.05" h="0.05" d="0.07" />
+        </inertial>
+      </xacro:if>
     </link>
     <link name="${prefix}_link">

File: urdf/asus_xtion_pro.urdf.xacro (robot description, xacro)
@@ -9,5 +9,5 @@
   <xacro:property name="asus_xtion_pro_rgb_rel_rgb_py"   value="-0.0220" />
   <xacro:property name="M_PI" value="3.1415926535897931" />
-  <xacro:macro name="sensor_asus_xtion_pro" params="prefix parent *origin">
+  <xacro:macro name="sensor_asus_xtion_pro" params="prefix parent *origin include_inertial:=^|true">
     <joint name="${prefix}rgb_joint" type="fixed">
 	  <xacro:insert_block name="origin" />
@@ -16,9 +16,11 @@
     </joint>
     <link name="${prefix}rgb_base_link">
-      <inertial>
-        <mass value="0.01" />
-        <origin xyz="-0.0175 0 0" />
-        <xacro:solid_cuboid_inertia m="0.01" w="0.035" h="0.180" d="0.05" />
-      </inertial>
+      <xacro:if value="${include_inertial}">
+        <inertial>
+          <mass value="0.01" />
+          <origin xyz="-0.0175 0 0" />
+          <xacro:solid_cuboid_inertia m="0.01" w="0.035" h="0.180" d="0.05" />
+        </inertial>
+      </xacro:if>
     </link>
     <joint name="${prefix}rgb_optical_joint" type="fixed">
@@ -28,9 +30,11 @@
     </joint>
     <link name="${prefix}rgb_optical_frame">
-      <inertial>
-        <mass value="0.01" />
-        <origin xyz="0 0 0" />
-        <xacro:solid_cuboid_inertia m="0.01" w="0.180" h="0.035" d="0.05" />
-      </inertial>
+      <xacro:if value="${include_inertial}">
+        <inertial>
+          <mass value="0.01" />
+          <origin xyz="0 0 0" />
+          <xacro:solid_cuboid_inertia m="0.01" w="0.180" h="0.035" d="0.05" />
+        </inertial>
+      </xacro:if>
     </link>
     <joint name="${prefix}joint" type="fixed">
@@ -53,9 +57,11 @@
       </geometry>
       </collision>
-      <inertial>
-        <mass value="0.01" />
-        <origin xyz="-0.0175 0.0025 0" rpy="0 0 0"/>
-        <xacro:solid_cuboid_inertia m="0.01" w="0.035" h="0.180" d="0.05" />
-      </inertial>
+      <xacro:if value="${include_inertial}">
+        <inertial>
+          <mass value="0.01" />
+          <origin xyz="-0.0175 0.0025 0" rpy="0 0 0"/>
+          <xacro:solid_cuboid_inertia m="0.01" w="0.035" h="0.180" d="0.05" />
+        </inertial>
+      </xacro:if>
     </link>
     <joint name="${prefix}depth_joint" type="fixed">
@@ -65,9 +71,11 @@
     </joint>
     <link name="${prefix}depth_link">
-      <inertial>
-        <mass value="0.01" />
-        <origin xyz="-0.0175 -${asus_xtion_pro_depth_rel_rgb_py} 0" />
-        <xacro:solid_cuboid_inertia m="0.01" w="0.035" h="0.180" d="0.05" />
-      </inertial>
+      <xacro:if value="${include_inertial}">
+        <inertial>
+          <mass value="0.01" />
+          <origin xyz="-0.0175 -${asus_xtion_pro_depth_rel_rgb_py} 0" />
+          <xacro:solid_cuboid_inertia m="0.01" w="0.035" h="0.180" d="0.05" />
+        </inertial>
+      </xacro:if>
     </link>
     <joint name="${prefix}depth_optical_joint" type="fixed">
@@ -77,9 +85,11 @@
     </joint>
     <link name="${prefix}depth_optical_frame">
-      <inertial>
-        <mass value="0.01" />
-        <origin xyz="${asus_xtion_pro_depth_rel_rgb_py} 0 -0.0175" />
-        <xacro:solid_cuboid_inertia m="0.01" w="0.18" h="0.05" d="0.035" />
-      </inertial>
+      <xacro:if value="${include_inertial}">
+        <inertial>
+          <mass value="0.01" />
+          <origin xyz="${asus_xtion_pro_depth_rel_rgb_py} 0 -0.0175" />
+          <xacro:solid_cuboid_inertia m="0.01" w="0.18" h="0.05" d="0.035" />
+        </inertial>
+      </xacro:if>
     </link>
   <!-- RGBD sensor for simulation, same as Kinect -->

File: urdf/axis.urdf.xacro (robot description, xacro)
@@ -6,5 +6,5 @@
   <xacro:property name="ptz_joint_damping" value="0.1"/>
   <xacro:property name="ptz_mechanical_reduction" value="1.0"/>
-  <xacro:macro name="sensor_axis" params="prefix parent *origin far:=^|8.0 near:=^|0.05">
+  <xacro:macro name="sensor_axis" params="prefix parent *origin far:=^|8.0 near:=^|0.05 include_inertial:=^|true">
     <joint name="${prefix}_joint" type="fixed">
       <axis xyz="0 0 1"/>
@@ -14,9 +14,11 @@
     </joint>
     <link name="${prefix}_base_link">
-      <inertial>
-        <origin xyz="0.0  0.0 -0.015" rpy="0 ${M_PI/2} 0"/>
-        <mass value="0.8"/>
-        <xacro:solid_cuboid_inertia m="0.8" w="0.152" h="0.132" d="0.132" />
-      </inertial>
+      <xacro:if value="${include_inertial}">
+        <inertial>
+          <origin xyz="0.0  0.0 -0.015" rpy="0 ${M_PI/2} 0"/>
+          <mass value="0.8"/>
+          <xacro:solid_cuboid_inertia m="0.8" w="0.152" h="0.132" d="0.132" />
+        </inertial>
+      </xacro:if>
       <visual>
         <origin xyz="0.0 0.0 0.0" rpy="0 0 0"/>
@@ -47,9 +49,11 @@
     </joint>
     <link name="${prefix}_pan_link">
-      <inertial>
-        <mass value="0.1"/>
-        <origin xyz="0 0 0" rpy="0 0 0"/>
-        <xacro:solid_cuboid_inertia m="0.1" w="0.1" h="0.11" d="0.11" />
-      </inertial>
+      <xacro:if value="${include_inertial}">
+        <inertial>
+          <mass value="0.1"/>
+          <origin xyz="0 0 0" rpy="0 0 0"/>
+          <xacro:solid_cuboid_inertia m="0.1" w="0.1" h="0.11" d="0.11" />
+        </inertial>
+      </xacro:if>
     </link>
     <transmission name="${prefix}_pan_trans">
@@ -72,9 +76,11 @@
     </joint>
     <link name="${prefix}_tilt_link">
-      <inertial>
-        <mass value="0.1"/>
-        <origin xyz="0 0 0" rpy="0 0 0"/>
-        <xacro:solid_cuboid_inertia m="0.1" w="0.11" h="0.11" d="0.1" />
-      </inertial>
+      <xacro:if value="${include_inertial}">
+        <inertial>
+          <mass value="0.1"/>
+          <origin xyz="0 0 0" rpy="0 0 0"/>
+          <xacro:solid_cuboid_inertia m="0.1" w="0.11" h="0.11" d="0.1" />
+        </inertial>
+      </xacro:if>
     </link>
     <transmission name="${prefix}_tilt_trans">
@@ -94,9 +100,11 @@
     </joint>
     <link name="${prefix}_frame_link">
-      <inertial>
-        <mass value="0.1"/>
-        <origin xyz="0 0 0"/>
-        <xacro:solid_cuboid_inertia m="0.1" w="0.11" h="0.11" d="0.1" />
-      </inertial>
+      <xacro:if value="${include_inertial}">
+        <inertial>
+          <mass value="0.1"/>
+          <origin xyz="0 0 0"/>
+          <xacro:solid_cuboid_inertia m="0.1" w="0.11" h="0.11" d="0.1" />
+        </inertial>
+      </xacro:if>
     </link>
     <!-- Optical frame -->
@@ -107,9 +115,11 @@
     </joint>
     <link name="${prefix}_optical_frame_link">
-      <inertial>
-        <mass value="0.1"/>
-        <origin xyz="0 0 0"/>
-        <xacro:solid_cuboid_inertia m="0.1" w="0.11" h="0.11" d="0.1" />
-      </inertial>
+      <xacro:if value="${include_inertial}">
+        <inertial>
+          <mass value="0.1"/>
+          <origin xyz="0 0 0"/>
+          <xacro:solid_cuboid_inertia m="0.1" w="0.11" h="0.11" d="0.1" />
+        </inertial>
+      </xacro:if>
     </link>
     <gazebo reference="${prefix}_base_link">

File: urdf/axis_m5013.urdf.xacro (robot description, xacro)
@@ -7,5 +7,5 @@
   <xacro:property name="ptz_mechanical_reduction" value="1.0"/>
   <xacro:property name="PI" value="3.14159265359"/>
-  <xacro:macro name="sensor_axis_m5013" params="prefix parent *origin far:=^|8.0 near:=^|0.05">
+  <xacro:macro name="sensor_axis_m5013" params="prefix parent *origin far:=^|8.0 near:=^|0.05 include_inertial:=^|true">
     <joint name="${prefix}_joint" type="fixed">
       <axis xyz="0 0 1"/>
@@ -15,9 +15,11 @@
     </joint>
     <link name="${prefix}_base_link">
-      <inertial>
-        <origin xyz="0.0175 0 0" rpy="0 ${M_PI/2} 0"/>
-        <mass value="0.3"/>
-        <xacro:solid_cuboid_inertia m="0.3" w="0.130" h="0.130" d="0.035" /> <!-- Data from axis M5013 datasheet -->
-      </inertial>
+      <xacro:if value="${include_inertial}">
+        <inertial>
+          <origin xyz="0.0175 0 0" rpy="0 ${M_PI/2} 0"/>
+          <mass value="0.3"/>
+          <xacro:solid_cuboid_inertia m="0.3" w="0.130" h="0.130" d="0.035" /> <!-- Data from axis M5013 datasheet -->
+        </inertial>
+      </xacro:if>
       <visual>
         <origin xyz="0 0 0" rpy="0 ${M_PI/2} 0"/>
@@ -47,9 +49,11 @@
     </joint>
     <link name="${prefix}_pan_link">
-      <inertial>
-        <mass value="0.01"/>
-        <origin xyz="0 0 0" rpy="0 0 0"/>
-        <xacro:solid_cuboid_inertia m="0.01" w="0.03" h="0.06" d="0.06" />
-      </inertial>
+      <xacro:if value="${include_inertial}">
+        <inertial>
+          <mass value="0.01"/>
+          <origin xyz="0 0 0" rpy="0 0 0"/>
+          <xacro:solid_cuboid_inertia m="0.01" w="0.03" h="0.06" d="0.06" />
+        </inertial>
+      </xacro:if>
     </link>
     <transmission name="${prefix}_pan_trans">
@@ -72,9 +76,11 @@
     </joint>
     <link name="${prefix}_tilt_link">
-      <inertial>
-        <mass value="0.01"/>
-        <origin xyz="0 0 0" rpy="0 0 0"/>
-        <xacro:solid_cuboid_inertia m="0.01" w="0.06" h="0.06" d="0.03" />
-      </inertial>
+      <xacro:if value="${include_inertial}">
+        <inertial>
+          <mass value="0.01"/>
+          <origin xyz="0 0 0" rpy="0 0 0"/>
+          <xacro:solid_cuboid_inertia m="0.01" w="0.06" h="0.06" d="0.03" />
+        </inertial>
+      </xacro:if>
     </link>
     <transmission name="${prefix}_tilt_trans">
@@ -94,9 +100,11 @@
     </joint>
     <link name="${prefix}_frame_link">
-      <inertial>
-        <mass value="0.01"/>
-        <origin xyz="0 0 0" rpy="0 0 0"/>
-        <xacro:solid_cuboid_inertia m="0.01" w="0.06" h="0.06" d="0.03" />
-      </inertial>
+      <xacro:if value="${include_inertial}">
+        <inertial>
+          <mass value="0.01"/>
+          <origin xyz="0 0 0" rpy="0 0 0"/>
+          <xacro:solid_cuboid_inertia m="0.01" w="0.06" h="0.06" d="0.03" />
+        </inertial>
+      </xacro:if>
     </link>
     <!-- Optical frame -->
@@ -107,9 +115,11 @@
     </joint>
     <link name="${prefix}_optical_frame_link">
-      <inertial>
-        <mass value="0.01"/>
-        <origin xyz="0 0 0" rpy="0 0 0"/>
-        <xacro:solid_cuboid_inertia m="0.01" w="0.06" h="0.03" d="0.06" />
-      </inertial>
+      <xacro:if value="${include_inertial}">
+        <inertial>
+          <mass value="0.01"/>
+          <origin xyz="0 0 0" rpy="0 0 0"/>
+          <xacro:solid_cuboid_inertia m="0.01" w="0.06" h="0.03" d="0.06" />
+        </inertial>
+      </xacro:if>
     </link>
     <gazebo reference="${prefix}_base_link">

File: urdf/axis_m5525.urdf.xacro (robot description, xacro)
@@ -7,5 +7,5 @@
   <xacro:property name="ptz_mechanical_reduction" value="1.0"/>
   <xacro:property name="PI" value="3.14159265359"/>
-  <xacro:macro name="sensor_axis_m5525" params="prefix parent *origin far:=^|8.0 near:=^|0.05 prefix_topic:=^ptz_camera">
+  <xacro:macro name="sensor_axis_m5525" params="prefix parent *origin far:=^|8.0 near:=^|0.05 prefix_topic:=^ptz_camera include_inertial:=^|true">
     <joint name="${prefix}_joint" type="fixed">
       <axis xyz="0 0 1"/>
@@ -15,9 +15,11 @@
     </joint>
     <link name="${prefix}_base_link">
-      <inertial>
-        <origin xyz="0.066 0 0" rpy="0 0 0"/>
-        <mass value="0.8"/>
-        <xacro:solid_cuboid_inertia m="0.8" w="0.165" h="0.165" d="0.132" />
-      </inertial>
+      <xacro:if value="${include_inertial}">
+        <inertial>
+          <origin xyz="0.066 0 0" rpy="0 0 0"/>
+          <mass value="0.8"/>
+          <xacro:solid_cuboid_inertia m="0.8" w="0.165" h="0.165" d="0.132" />
+        </inertial>
+      </xacro:if>
       <visual>
         <origin xyz="0 0 0" rpy="0 0 0"/>
@@ -47,9 +49,11 @@
     </joint>
     <link name="${prefix}_pan_link">
-      <inertial>
-        <mass value="0.1"/>
-        <origin xyz="0 0 0" rpy="0 0 0"/>
-        <xacro:solid_cuboid_inertia m="0.1" w="0.1" h="0.11" d="0.11" />
-      </inertial>
+      <xacro:if value="${include_inertial}">
+        <inertial>
+          <mass value="0.1"/>
+          <origin xyz="0 0 0" rpy="0 0 0"/>
+          <xacro:solid_cuboid_inertia m="0.1" w="0.1" h="0.11" d="0.11" />
+        </inertial>
+      </xacro:if>
     </link>
     <transmission name="${prefix}_pan_trans">
@@ -72,9 +76,11 @@
     </joint>
     <link name="${prefix}_tilt_link">
-      <inertial>
-        <mass value="0.1"/>
-        <origin xyz="0 0 0" rpy="0 0 0"/>
-        <xacro:solid_cuboid_inertia m="0.1" w="0.11" h="0.11" d="0.1" />
-      </inertial>
+      <xacro:if value="${include_inertial}">
+        <inertial>
+          <mass value="0.1"/>
+          <origin xyz="0 0 0" rpy="0 0 0"/>
+          <xacro:solid_cuboid_inertia m="0.1" w="0.11" h="0.11" d="0.1" />
+        </inertial>
+      </xacro:if>
     </link>
     <transmission name="${prefix}_tilt_trans">
@@ -94,9 +100,11 @@
     </joint>
     <link name="${prefix}_frame_link">
-      <inertial>
-        <mass value="0.1"/>
-        <origin xyz="0 0 0"/>
-        <xacro:solid_cuboid_inertia m="0.1" w="0.11" h="0.11" d="0.1" />
-      </inertial>
+      <xacro:if value="${include_inertial}">
+        <inertial>
+          <mass value="0.1"/>
+          <origin xyz="0 0 0"/>
+          <xacro:solid_cuboid_inertia m="0.1" w="0.11" h="0.11" d="0.1" />
+        </inertial>
+      </xacro:if>
     </link>
     <!-- Optical frame -->
@@ -107,9 +115,11 @@
     </joint>
     <link name="${prefix}_optical_frame_link">
-      <inertial>
-        <mass value="0.1"/>
-        <origin xyz="0 0 0"/>
-        <xacro:solid_cuboid_inertia m="0.1" w="0.11" h="0.11" d="0.1" />
-      </inertial>
+      <xacro:if value="${include_inertial}">
+        <inertial>
+          <mass value="0.1"/>
+          <origin xyz="0 0 0"/>
+          <xacro:solid_cuboid_inertia m="0.1" w="0.11" h="0.11" d="0.1" />
+        </inertial>
+      </xacro:if>
     </link>
     <gazebo reference="${prefix}_base_link">

File: urdf/axis_q8641.urdf.xacro (robot description, xacro)
@@ -6,5 +6,5 @@
   <xacro:property name="ptz_joint_damping" value="0.1"/>
   <xacro:property name="ptz_mechanical_reduction" value="1.0"/>
-  <xacro:macro name="sensor_axis_q8641" params="prefix parent *origin far:=^|8.0 near:=^|0.05">
+  <xacro:macro name="sensor_axis_q8641" params="prefix parent *origin far:=^|8.0 near:=^|0.05 include_inertial:=^|true">
     <joint name="${prefix}_joint" type="fixed">
       <axis xyz="0 1 0"/>
@@ -19,8 +19,10 @@
         <xacro:solid_cuboid_inertia m="2" w="0.175" h="0.175" d="0.12" />
       </inertial-->
-      <inertial>
-        <mass value="0.001"/>
-        <inertia ixx="0.001" ixy="0" ixz="0" iyy="0.001" iyz="0" izz="0.001"/>
-      </inertial>
+      <xacro:if value="${include_inertial}">
+        <inertial>
+          <mass value="0.001"/>
+          <inertia ixx="0.001" ixy="0" ixz="0" iyy="0.001" iyz="0" izz="0.001"/>
+        </inertial>
+      </xacro:if>
       <visual>
         <origin xyz="0.0 0.0 0.0" rpy="0 0 0"/>
@@ -56,8 +58,10 @@
         <xacro:solid_cuboid_inertia m="5.0" w="0.175" h="0.175" d="0.24" />
       </inertial-->
-      <inertial>
-        <mass value="0.001"/>
-        <inertia ixx="0.001" ixy="0" ixz="0" iyy="0.001" iyz="0" izz="0.001"/>
-      </inertial>
+      <xacro:if value="${include_inertial}">
+        <inertial>
+          <mass value="0.001"/>
+          <inertia ixx="0.001" ixy="0" ixz="0" iyy="0.001" iyz="0" izz="0.001"/>
+        </inertial>
+      </xacro:if>
       <visual>
         <origin xyz="0.0 0.0 0.0" rpy="0 0 0"/>
@@ -102,8 +106,10 @@
         <xacro:solid_cuboid_inertia m="5.0" w="0.24" h="0.09" d="0.09" />
       </inertial-->
-      <inertial>
-        <mass value="0.001"/>
-        <inertia ixx="0.001" ixy="0" ixz="0" iyy="0.001" iyz="0" izz="0.001"/>
-      </inertial>
+      <xacro:if value="${include_inertial}">
+       <inertial>
+         <mass value="0.001"/>
+         <inertia ixx="0.001" ixy="0" ixz="0" iyy="0.001" iyz="0" izz="0.001"/>
+       </inertial>
+      </xacro:if>
       <visual>
         <origin xyz="0.0 0.0 0.0" rpy="0 0 0"/>

File: urdf/benewake_ce30.urdf.xacro (robot description, xacro)
@@ -2,5 +2,5 @@
 <robot name="sensor_benewake_ce30" xmlns:xacro="http://wiki.ros.org/xacro">
   <xacro:property name="M_PI" value="3.1415926535897931" />
-  <xacro:macro name="sensor_benewake_ce30" params="prefix parent prefix_topic *origin range_min range_max hfov vfov fps gpu:=^|true">
+  <xacro:macro name="sensor_benewake_ce30" params="prefix parent prefix_topic *origin range_min range_max hfov vfov fps gpu:=^|true include_inertial:=^|true">
     <joint name="${prefix}_base_joint" type="fixed">
       <xacro:insert_block name="origin" />
@@ -23,10 +23,12 @@
         </geometry>
       </collision>
-      <inertial>
-        <!-- The following are not reliable values, and should not be used for modeling -->
-        <mass value="0.219" />
-        <origin xyz="0 0 0.025" />
-        <xacro:solid_cuboid_inertia m="0.219" w="0.047" h="0.079" d="0.05" />
-      </inertial>
+      <xacro:if value="${include_inertial}">
+        <inertial>
+          <!-- The following are not reliable values, and should not be used for modeling -->
+          <mass value="0.219" />
+          <origin xyz="0 0 0.025" />
+          <xacro:solid_cuboid_inertia m="0.219" w="0.047" h="0.079" d="0.05" />
+        </inertial>
+      </xacro:if>
     </link>
     <joint name="${prefix}_joint" type="fixed">
@@ -84,11 +86,11 @@
     </gazebo>
   </xacro:macro>
-  <xacro:macro name="sensor_benewake_ce30a" params="prefix parent prefix_topic:='lidar_3d' *origin gpu:=false">
-    <xacro:sensor_benewake_ce30 prefix="${prefix}" parent="${parent}" prefix_topic="${prefix_topic}" range_min="0.1" range_max="4.0" hfov="132.0" vfov="9.0" fps="20.0" gpu="${gpu}" >
+  <xacro:macro name="sensor_benewake_ce30a" params="prefix parent prefix_topic:='lidar_3d' *origin gpu:=false include_inertial:=^|true">
+    <xacro:sensor_benewake_ce30 prefix="${prefix}" parent="${parent}" prefix_topic="${prefix_topic}" range_min="0.1" range_max="4.0" hfov="132.0" vfov="9.0" fps="20.0" gpu="${gpu}" include_inertial="${include_inertial}" >
       <xacro:insert_block name="origin" />
     </xacro:sensor_benewake_ce30>
   </xacro:macro>
-  <xacro:macro name="sensor_benewake_ce30c" params="prefix parent prefix_topic:='lidar_3d' *origin gpu:=false">
-    <xacro:sensor_benewake_ce30 prefix="${prefix}" parent="${parent}" prefix_topic="${prefix_topic}" range_min="0.1" range_max="4.0" hfov="132.0" vfov="9.0" fps="20.0" gpu="${gpu}" >
+  <xacro:macro name="sensor_benewake_ce30c" params="prefix parent prefix_topic:='lidar_3d' *origin gpu:=false include_inertial:=^|true">
+    <xacro:sensor_benewake_ce30 prefix="${prefix}" parent="${parent}" prefix_topic="${prefix_topic}" range_min="0.1" range_max="4.0" hfov="132.0" vfov="9.0" fps="20.0" gpu="${gpu}" include_inertial="${include_inertial}" >
       <xacro:insert_block name="origin" />
     </xacro:sensor_benewake_ce30>

File: urdf/benewake_ce30d.urdf.xacro (robot description, xacro)
@@ -2,5 +2,5 @@
 <robot name="sensor_benewake_ce30d" xmlns:xacro="http://wiki.ros.org/xacro">
   <xacro:property name="M_PI" value="3.1415926535897931" />
-  <xacro:macro name="sensor_benewake_ce30d" params="prefix parent prefix_topic:='lidar_3d' *origin range_min:=0.4 range_max:=28.0 hfov:=60.0 vfov:=4.0 fps:=30.0 gpu:=^|true">
+  <xacro:macro name="sensor_benewake_ce30d" params="prefix parent prefix_topic:='lidar_3d' *origin range_min:=0.4 range_max:=28.0 hfov:=60.0 vfov:=4.0 fps:=30.0 gpu:=^|true include_inertial:=^|true">
     <joint name="${prefix}_base_joint" type="fixed">
       <xacro:insert_block name="origin" />
@@ -23,10 +23,12 @@
         </geometry>
       </collision>
-      <inertial>
-        <!-- The following are not reliable values, and should not be used for modeling -->
-        <mass value="0.336" />
-        <origin xyz="0 0 0.027" rpy="0 0 ${M_PI/2}" />
-        <xacro:solid_cuboid_inertia m="0.336" w="0.057" h="0.083" d="0.054" />
-      </inertial>
+      <xacro:if value="${include_inertial}">
+        <inertial>
+          <!-- The following are not reliable values, and should not be used for modeling -->
+          <mass value="0.336" />
+          <origin xyz="0 0 0.027" rpy="0 0 ${M_PI/2}" />
+          <xacro:solid_cuboid_inertia m="0.336" w="0.057" h="0.083" d="0.054" />
+        </inertial>
+      </xacro:if>
     </link>
     <joint name="${prefix}_joint" type="fixed">

File: urdf/blk_arc.urdf.xacro (robot description, xacro)
@@ -1,5 +1,5 @@
 <?xml version="1.0"?>
 <robot name="sensor_blk_arc" xmlns:xacro="http://wiki.ros.org/xacro">
-  <xacro:macro name="sensor_blk_arc" params="prefix parent *origin">
+  <xacro:macro name="sensor_blk_arc" params="prefix parent *origin include_inertial:=^|true">
     <joint name="${prefix}_joint" type="fixed">
       <xacro:insert_block name="origin"/>
@@ -8,9 +8,11 @@
     </joint>
     <link name="${prefix}_link">
-      <inertial>
-        <origin xyz="0.0 0 0.0" rpy="0 0 0" />
-        <mass value="0.79" />
-        <xacro:solid_cuboid_inertia m="0.125" w="0.025" h="0.054" d="0.079" />
-      </inertial>
+      <xacro:if value="${include_inertial}">
+        <inertial>
+          <origin xyz="0.0 0 0.0" rpy="0 0 0" />
+          <mass value="0.79" />
+          <xacro:solid_cuboid_inertia m="0.125" w="0.025" h="0.054" d="0.079" />
+        </inertial>
+      </xacro:if>
       <visual>
         <origin xyz="0.0 0 0" rpy="0 0 0" /> <!-- to center the .dae model -->
