Commit message: Create variable include_inertial to be able to deactivate all sensors inertia

File: urdf/embedded_s.urdf.xacro (robot description, xacro)
@@ -1,5 +1,5 @@
 <?xml version="1.0"?>
 <robot name="sensor_orbbec_astra_embedded_s" xmlns:xacro="http://wiki.ros.org/Sensors/OrbbecAstra">
-  <xacro:macro name="sensor_orbbec_astra_embedded_s" params="prefix parent prefix_topic:='front_rgbd_camera' *origin">
+  <xacro:macro name="sensor_orbbec_astra_embedded_s" params="prefix parent prefix_topic:='front_rgbd_camera' *origin include_inertial:=^|true">
     <joint name="${prefix}_joint" type="fixed">
 	  <xacro:insert_block name="origin" />
@@ -24,9 +24,11 @@
         </geometry>
       </collision>
-      <inertial>
-        <mass value="0.001" />
-        <origin xyz="0.0 0.0 0.0" />
-        <xacro:solid_cuboid_inertia m="0.001" w="0.04" h="0.165" d="0.03" />
-      </inertial>
+      <xacro:if value="${include_inertial}">
+        <inertial>
+          <mass value="0.001" />
+          <origin xyz="0.0 0.0 0.0" />
+          <xacro:solid_cuboid_inertia m="0.001" w="0.04" h="0.165" d="0.03" />
+        </inertial>
+      </xacro:if>
     </link>
     <joint name="${prefix}_rgb_joint" type="fixed">

File: urdf/flir_ax8.urdf.xacro (robot description, xacro)
@@ -1,5 +1,5 @@
 <?xml version="1.0"?>
 <robot name="sensor_flir_ax8" xmlns:xacro="http://wiki.ros.org/xacro">
-  <xacro:macro name="sensor_flir_ax8" params="prefix parent *origin">
+  <xacro:macro name="sensor_flir_ax8" params="prefix parent *origin include_inertial:=^|true">
     <joint name="${prefix}_joint" type="fixed">
       <xacro:insert_block name="origin"/>
@@ -8,9 +8,11 @@
     </joint>
     <link name="${prefix}_link">
-      <inertial>
-        <origin xyz="0.0 0 0.0" rpy="0 0 0" />
-        <mass value="0.79" />
-        <xacro:solid_cuboid_inertia m="0.125" w="0.025" h="0.054" d="0.079" />
-      </inertial>
+      <xacro:if value="${include_inertial}">
+        <inertial>
+          <origin xyz="0.0 0 0.0" rpy="0 0 0" />
+          <mass value="0.79" />
+          <xacro:solid_cuboid_inertia m="0.125" w="0.025" h="0.054" d="0.079" />
+        </inertial>
+      </xacro:if>
       <visual>
         <origin xyz="0.0125 0 0" rpy="0 0 0" /> <!-- to center the .dae model -->

File: urdf/fotonic_e.urdf.xacro (robot description, xacro)
@@ -1,5 +1,5 @@
 <?xml version="1.0"?>
 <robot name="sensor_fotonic" xmlns:xacro="http://wiki.ros.org/xacro">
-  <xacro:macro name="sensor_fotonic" params="prefix parent *origin">
+  <xacro:macro name="sensor_fotonic" params="prefix parent *origin include_inertial:=^|true">
     <joint name="${prefix}_joint" type="fixed">
       <xacro:insert_block name="origin"/>
@@ -8,9 +8,11 @@
     </joint>
     <link name="${prefix}_base_link">
-      <inertial>
-        <origin xyz="0.0 0 0.0" rpy="0 0 0" />
-        <mass value="0.79" />
-        <xacro:solid_cuboid_inertia m="0.79" w="0.08" h="0.0863" d="0.08" />
-      </inertial>
+      <xacro:if value="${include_inertial}">
+        <inertial>
+          <origin xyz="0.0 0 0.0" rpy="0 0 0" />
+          <mass value="0.79" />
+          <xacro:solid_cuboid_inertia m="0.79" w="0.08" h="0.0863" d="0.08" />
+        </inertial>
+      </xacro:if>
       <visual>
         <origin xyz="0.0 0.0 -0.04" rpy="0 0 0" /> <!-- to center the .dae model -->
@@ -35,9 +37,11 @@
     </joint>
     <link name="${prefix}_depth_frame_link">
-      <inertial>
-        <origin xyz="-0.0375 0 0.0" rpy="0 0 0" />
-        <mass value="0.01" />
-        <xacro:solid_cuboid_inertia m="0.01" w="0.08" h="0.0863" d="0.08" />
-      </inertial>
+      <xacro:if value="${include_inertial}">
+        <inertial>
+          <origin xyz="-0.0375 0 0.0" rpy="0 0 0" />
+          <mass value="0.01" />
+          <xacro:solid_cuboid_inertia m="0.01" w="0.08" h="0.0863" d="0.08" />
+        </inertial>
+      </xacro:if>
     </link>
     <joint name="${prefix}_depth_optical_joint" type="fixed">

File: urdf/gps.urdf.xacro (robot description, xacro)
@@ -2,5 +2,5 @@
 <robot name="sensor_gps" xmlns:xacro="http://wiki.ros.org/xacro">
   <!-- if no latitude/longitud is specified, then use Fuente del Jarro as default -->
-  <xacro:macro name="sensor_gps" params="prefix parent *origin gps_latitude:=^|39.5080331 gps_longitude:=^|-0.4619816 update_rate:=^|5">
+  <xacro:macro name="sensor_gps" params="prefix parent *origin gps_latitude:=^|39.5080331 gps_longitude:=^|-0.4619816 update_rate:=^|5 include_inertial:=^|true">
 	  <!-- ANTENNA GPS -->
 	  <joint name="${prefix}_joint" type="fixed">
@@ -11,9 +11,11 @@
 	  </joint>
 	  <link name="${prefix}_base_link">
-		<inertial>
-			<origin xyz="0.0 0 0.015" rpy="0 0 0" />
-			<mass value="0.2" />
-			<xacro:solid_cuboid_inertia m="0.2" w="0.081" h="0.081" d="0.03" />
-      </inertial>
+		<xacro:if value="$(include_inertial)">
+			<inertial>
+				<origin xyz="0.0 0 0.015" rpy="0 0 0" />
+				<mass value="0.2" />
+				<xacro:solid_cuboid_inertia m="0.2" w="0.081" h="0.081" d="0.03" />
+      		</inertial>
+	  	</xacro:if>
 	    <visual>
 	      <origin rpy="0 0 0" xyz="0 0 0"/>

File: urdf/gps_with_mast.urdf.xacro (robot description, xacro)
@@ -4,5 +4,5 @@
   <xacro:property name="mast_radius" value="0.010" />
   <!-- if no latitude/longitud is specified, then use Fuente del Jarro as default -->
-  <xacro:macro name="sensor_gps_with_mast" params="prefix parent *origin gps_latitude:=^|39.5080331 gps_longitude:=^|-0.4619816 update_rate:=^|5">
+  <xacro:macro name="sensor_gps_with_mast" params="prefix parent *origin gps_latitude:=^|39.5080331 gps_longitude:=^|-0.4619816 update_rate:=^|5 include_inertial:=^|true">
 	  <!-- MAST OF THE ANTENNA GPS -->
 	  <joint name="${prefix}_joint" type="fixed">
@@ -13,9 +13,11 @@
 	  </joint>
 	  <link name="${prefix}_mast_base_link">
-		<inertial>
-			<origin xyz="0.0 0 0.0" rpy="0 0 0" />
-			<mass value="1.0" />
-			<xacro:solid_cuboid_inertia m="1.0" w="${mast_radius}" h="${mast_radius}" d="${mast_height}" />
-		</inertial>
+		<xacro:if value="$(include_inertial)">
+			<inertial>
+				<origin xyz="0.0 0 0.0" rpy="0 0 0" />
+				<mass value="1.0" />
+				<xacro:solid_cuboid_inertia m="1.0" w="${mast_radius}" h="${mast_radius}" d="${mast_height}" />
+			</inertial>
+	  	</xacro:if>
 	    <visual>
 	      <origin rpy="0 0 0" xyz="0 0 0"/>
@@ -46,9 +48,11 @@
       <!-- ANTENNA GPS -->
 	  <link name="${prefix}_base_link">
-	    <inertial>
-			<origin xyz="0.0 0 0.015" rpy="0 0 0" />
-			<mass value="0.2" />
-			<xacro:solid_cuboid_inertia m="0.2" w="0.081" h="0.081" d="0.03" />
-      	</inertial>
+		<xacro:if value="$(include_inertial)">
+	    	<inertial>
+				<origin xyz="0.0 0 0.015" rpy="0 0 0" />
+				<mass value="0.2" />
+				<xacro:solid_cuboid_inertia m="0.2" w="0.081" h="0.081" d="0.03" />
+      		</inertial>
+		</xacro:if>
 	    <visual>
 	      <origin rpy="0 0 0" xyz="0 0 0"/>

File: urdf/hokuyo3d.urdf.xacro (robot description, xacro)
@@ -1,5 +1,5 @@
 <?xml version="1.0"?>
 <robot name="sensor_hokuyo3d" xmlns:xacro="http://wiki.ros.org/xacro">
-  <xacro:macro name="sensor_hokuyo3d" params="prefix parent *origin gpu:=^|true">
+  <xacro:macro name="sensor_hokuyo3d" params="prefix parent *origin gpu:=^|true include_inertial:=^|true">
     <joint name="${prefix}_fix_joint" type="fixed">
       <xacro:insert_block name="origin" />
@@ -20,9 +20,11 @@
             </geometry>
         </visual>
-        <inertial>
-            <mass value="0.65" />
-            <origin xyz="0.0475 0.0 0.053" rpy="0 0 0"/>
-            <xacro:solid_cuboid_inertia m="0.65" w="0.095" h="0.07" d="0.106" />
-        </inertial>
+        <xacro:if value="$(include_inertial)">
+          <inertial>
+              <mass value="0.65" />
+              <origin xyz="0.0475 0.0 0.053" rpy="0 0 0"/>
+              <xacro:solid_cuboid_inertia m="0.65" w="0.095" h="0.07" d="0.106" />
+          </inertial>
+        </xacro:if>
     </link>
     <link name="${prefix}_link">

File: urdf/hokuyo_uam05lp.urdf.xacro (robot description, xacro)
@@ -1,5 +1,5 @@
 <?xml version="1.0"?>
 <robot name="sensor_hokuyo_uam" xmlns:xacro="http://wiki.ros.org/xacro">
-  <xacro:macro name="sensor_hokuyo_uam" params="prefix parent prefix_topic:='front_laser' *origin min_angle:=-2.3562 max_angle:=2.3562  gpu:=^|true">
+  <xacro:macro name="sensor_hokuyo_uam" params="prefix parent prefix_topic:='front_laser' *origin min_angle:=-2.3562 max_angle:=2.3562  gpu:=^|true include_inertial:=^|true">
     <joint name="${prefix}_base_joint" type="fixed">
       <xacro:insert_block name="origin" />
@@ -14,9 +14,11 @@
         </geometry>
       </visual>
-      <inertial>
-        <origin xyz="0.0 0 0.035" rpy="0 0 0" />
-        <mass value="0.8" />
-        <xacro:solid_cuboid_inertia m="0.8" w="0.08" h="0.095" d="0.08" />
-      </inertial>
+      <xacro:if value="$(include_inertial)">
+        <inertial>
+          <origin xyz="0.0 0 0.035" rpy="0 0 0" />
+          <mass value="0.8" />
+          <xacro:solid_cuboid_inertia m="0.8" w="0.08" h="0.095" d="0.08" />
+        </inertial>
+      </xacro:if>
     </link>
     <link name="${prefix}_link">

File: urdf/hokuyo_urg04lx.urdf.xacro (robot description, xacro)
@@ -1,5 +1,5 @@
 <?xml version="1.0"?>
 <robot name="sensor_hokuyo_urg04lx" xmlns:xacro="http://wiki.ros.org/xacro">
-  <xacro:macro name="sensor_hokuyo_urg04lx" params="prefix parent prefix_topic:='front_laser' *origin min_angle:=-2.0943 max_angle:=2.0943  gpu:=^|true">
+  <xacro:macro name="sensor_hokuyo_urg04lx" params="prefix parent prefix_topic:='front_laser' *origin min_angle:=-2.0943 max_angle:=2.0943  gpu:=^|true include_inertial:=^|true">
     <joint name="${prefix}_base_joint" type="fixed">
       <!-- FRONT MOUNT  -->
@@ -18,9 +18,11 @@
         </geometry>
       </visual>
-      <inertial>
-        <origin xyz="0.0 0 0.035" rpy="0 0 0" />
-        <mass value="0.160" />
-        <xacro:solid_cuboid_inertia m="0.160" w="0.05" h="0.05" d="0.07" />
-      </inertial>
+      <xacro:if value="$(include_inertial)">
+        <inertial>
+          <origin xyz="0.0 0 0.035" rpy="0 0 0" />
+          <mass value="0.160" />
+          <xacro:solid_cuboid_inertia m="0.160" w="0.05" h="0.05" d="0.07" />
+        </inertial>
+      </xacro:if>
     </link>
     <link name="${prefix}_link">

File: urdf/hokuyo_ust10lx.urdf.xacro (robot description, xacro)
@@ -1,5 +1,5 @@
 <?xml version="1.0"?>
 <robot name="sensor_hokuyo_ust10lx" xmlns:xacro="http://wiki.ros.org/xacro">
-  <xacro:macro name="sensor_hokuyo_ust10lx" params="prefix parent prefix_topic:='front_laser' *origin min_angle:=-2.3562 max_angle:=2.3562 gpu:=^|true">
+  <xacro:macro name="sensor_hokuyo_ust10lx" params="prefix parent prefix_topic:='front_laser' *origin min_angle:=-2.3562 max_angle:=2.3562 gpu:=^|true include_inertial:=^|true">
     <joint name="${prefix}_base_joint" type="fixed">
       <xacro:insert_block name="origin" />
@@ -20,9 +20,11 @@
         </geometry>
       </visual>
-      <inertial>
-        <origin xyz="0.0 0 0.035" rpy="0 0 0" />
-        <mass value="0.130" />
-        <xacro:solid_cuboid_inertia m="0.130" w="0.05" h="0.05" d="0.07" />
-      </inertial>
+      <xacro:if value="$(include_inertial)">
+        <inertial>
+          <origin xyz="0.0 0 0.035" rpy="0 0 0" />
+          <mass value="0.130" />
+          <xacro:solid_cuboid_inertia m="0.130" w="0.05" h="0.05" d="0.07" />
+        </inertial>
+      </xacro:if>
     </link>
     <joint name="${prefix}_joint" type="fixed">

File: urdf/hokuyo_ust20lx.urdf.xacro (robot description, xacro)
@@ -1,5 +1,5 @@
 <?xml version="1.0"?>
 <robot name="sensor_hokuyo_ust20lx" xmlns:xacro="http://wiki.ros.org/xacro">
-  <xacro:macro name="sensor_hokuyo_ust20lx" params="prefix parent prefix_topic:='front_laser' *origin min_angle:=-2.3562 max_angle:=2.3562 gpu:=^|true">
+  <xacro:macro name="sensor_hokuyo_ust20lx" params="prefix parent prefix_topic:='front_laser' *origin min_angle:=-2.3562 max_angle:=2.3562 gpu:=^|true include_inertial:=^|true">
     <joint name="${prefix}_base_joint" type="fixed">
       <xacro:insert_block name="origin" />
@@ -20,9 +20,11 @@
         </geometry>
       </visual>
-      <inertial>
-        <origin xyz="0.0 0 0.035" rpy="0 0 0" />
-        <mass value="0.130" />
-        <xacro:solid_cuboid_inertia m="0.130" w="0.05" h="0.05" d="0.07" />
-      </inertial>
+      <xacro:if value="$(include_inertial)">
+        <inertial>
+          <origin xyz="0.0 0 0.035" rpy="0 0 0" />
+          <mass value="0.130" />
+          <xacro:solid_cuboid_inertia m="0.130" w="0.05" h="0.05" d="0.07" />
+        </inertial>
+      </xacro:if>
     </link>
     <link name="${prefix}_link">

File: urdf/hokuyo_ust30lx.urdf.xacro (robot description, xacro)
@@ -1,5 +1,5 @@
 <?xml version="1.0"?>
 <robot name="sensor_hokuyo_ust30lx" xmlns:xacro="http://wiki.ros.org/xacro">
-  <xacro:macro name="sensor_hokuyo_ust30lx" params="prefix parent prefix_topic:='front_laser' *origin min_angle:=-2.3562 max_angle:=2.3562 gpu:=^|true">
+  <xacro:macro name="sensor_hokuyo_ust30lx" params="prefix parent prefix_topic:='front_laser' *origin min_angle:=-2.3562 max_angle:=2.3562 gpu:=^|true include_inertial:=^|true">
     <joint name="${prefix}_base_joint" type="fixed">
       <xacro:insert_block name="origin" />
@@ -20,9 +20,11 @@
         </geometry>
       </visual>
-      <inertial>
-        <origin xyz="0.0 0 0.035" rpy="0 0 0" />
-        <mass value="0.130" />
-        <xacro:solid_cuboid_inertia m="0.130" w="0.05" h="0.05" d="0.07" />
-      </inertial>
+      <xacro:if value="$(include_inertial)">
+        <inertial>
+          <origin xyz="0.0 0 0.035" rpy="0 0 0" />
+          <mass value="0.130" />
+          <xacro:solid_cuboid_inertia m="0.130" w="0.05" h="0.05" d="0.07" />
+        </inertial>
+      </xacro:if>
     </link>
     <link name="${prefix}_link">
