Commit message: axis_m5013 collision pos corrected

File: urdf/axis_m5013.urdf.xacro (robot description, xacro)
@@ -33,5 +33,5 @@
 	    </visual>
 	    <collision>
-	      <origin xyz="0.03 0.0 -0.3" rpy="0 0 0"/>
+	      <origin xyz="0.0 0.0 0" rpy="0 0 0"/>
 	      <geometry>
 	        <mesh filename= "package://robotnik_sensors/meshes/axis_m5013.stl" scale="1.0 1.0 1.0"/>

Commit message: Added optical frame and modified parameters to axis_m5013.urdf.xacro

File: urdf/axis_m5013.urdf.xacro (robot description, xacro)
@@ -89,4 +89,19 @@
 	     </actuator>
 	  </transmission>
+		<!-- Optical frame -->
+		<joint name="${name}_depth_optical_joint" type="fixed">
+			<origin xyz="0 0 0" rpy="${-M_PI/2} 0 ${-M_PI/2}" />
+			<parent link="${name}_link"/>
+			<child link="${name}_depth_optical_frame" />
+		</joint>
+		<link name="${name}_depth_optical_frame">
+			<inertial>
+				<mass value="0.001" />
+				<origin xyz="0 0 0" />
+				<inertia ixx="0.0001" ixy="0.0" ixz="0.0"
+								 iyy="0.0001" iyz="0.0"
+								 izz="0.0001" />
+			</inertial>
+		</link>
 	  <gazebo reference="${name}_link">
       <material>Gazebo/FlatBlack</material>
@@ -95,41 +110,36 @@
 		<sensor_axis_m5013_gazebo/>
   </xacro:macro>
-  <xacro:macro name="sensor_axis_m5013_gazebo">
-    <gazebo reference="${name}_tilt_link">
-	    <sensor type="camera" name="camera1">
-	      <update_rate>30.0</update_rate>
-	      <camera name="head">
-	        <horizontal_fov>1.3962634</horizontal_fov>
-	        <image>
-	          <width>800</width>
-	          <height>800</height>
-	          <format>R8G8B8</format>
-	        </image>
-	        <clip>
-	          <near>0.03</near>
-	          <far>300</far>
-	        </clip>
-	        <noise>
-	          <type>gaussian</type>
-	          <mean>0.0</mean>
-	          <stddev>0.007</stddev>
-	        </noise>
-	      </camera>
-	      <plugin name="camera_controller" filename="libgazebo_ros_camera.so">
-	        <alwaysOn>true</alwaysOn>
-	        <updateRate>0.0</updateRate>
-	        <cameraName>${name}</cameraName>
-	        <imageTopicName>image_raw</imageTopicName>
-	        <cameraInfoTopicName>camera_info</cameraInfoTopicName>
-	        <frameName>${name}_tilt_link</frameName>
-	        <hackBaseline>0.07</hackBaseline>
-	        <distortionK1>0.0</distortionK1>
-	        <distortionK2>0.0</distortionK2>
-	        <distortionK3>0.0</distortionK3>
-	        <distortionT1>0.0</distortionT1>
-	        <distortionT2>0.0</distortionT2>
-	      </plugin>
-	    </sensor>
-	  </gazebo>
-  </xacro:macro>
+	<xacro:macro name="sensor_axis_m5013_gazebo">
+		<gazebo reference="${name}_tilt_link">
+			<sensor type="camera" name="camera1">
+				<update_rate>30.0</update_rate>
+				<camera name="head">
+					<horizontal_fov>${60.0*M_PI/180.0}</horizontal_fov>
+					<image>
+						<format>R8G8B8</format>
+						<width>640</width>
+						<height>480</height>
+					</image>
+					<clip>
+						<near>0.05</near>
+						<far>8.0</far>
+					</clip>
+				</camera>
+				<plugin name="camera_controller" filename="libgazebo_ros_camera.so">
+					<alwaysOn>true</alwaysOn>
+					<updateRate>0.0</updateRate>
+					<cameraName>${name}</cameraName>
+					<imageTopicName>image_raw</imageTopicName>
+					<cameraInfoTopicName>camera_info</cameraInfoTopicName>
+					<frameName>${name}_depth_optical_frame</frameName>
+					<hackBaseline>0.07</hackBaseline>
+					<distortionK1>0.0</distortionK1>
+					<distortionK2>0.0</distortionK2>
+					<distortionK3>0.0</distortionK3>
+					<distortionT1>0.0</distortionT1>
+					<distortionT2>0.0</distortionT2>
+				</plugin>
+			</sensor>
+		</gazebo>
+	</xacro:macro>
 </robot>

Commit message: axis sensor: corrected pan tilt joints positions

File: urdf/axis_m5013.urdf.xacro (robot description, xacro)
@@ -40,6 +40,6 @@
     </link>
 	  <joint name="joint_${name}_pan" type="continuous">
-	     <axis xyz="0 0 1" />
-	     <origin xyz="0.0 0.0 0.1"/>
+	     <axis xyz="0 0 -1" />
+	     <origin xyz="0.0 0.0 0.03"/>
 	     <parent link="${name}_link"/>
 	     <child link="${name}_pan_link"/>
@@ -65,5 +65,5 @@
 	  </transmission>
 	  <joint name="joint_${name}_tilt" type="continuous">
-	     <axis xyz="0 1 0" />
+	     <axis xyz="0 -1 0" />
 	     <origin xyz="0.0 0.0 0.0"/>
 	     <parent link="${name}_pan_link"/>
@@ -89,24 +89,24 @@
 	     </actuator>
 	  </transmission>
-		<!-- Optical frame -->
-		<joint name="${name}_depth_optical_joint" type="fixed">
-			<origin xyz="0 0 0" rpy="${-M_PI/2} 0 ${-M_PI/2}" />
-			<parent link="${name}_link"/>
-			<child link="${name}_depth_optical_frame" />
-		</joint>
-		<link name="${name}_depth_optical_frame">
-			<inertial>
-				<mass value="0.001" />
-				<origin xyz="0 0 0" />
-				<inertia ixx="0.0001" ixy="0.0" ixz="0.0"
-								 iyy="0.0001" iyz="0.0"
-								 izz="0.0001" />
-			</inertial>
-		</link>
-	  <gazebo reference="${name}_link">
+	  <!-- Optical frame -->
+	  <joint name="${name}_depth_optical_joint" type="fixed">
+		  <origin xyz="0 0 0" rpy="${-M_PI/2} 0 ${-M_PI/2}" />
+		  <parent link="${name}_tilt_link"/>
+		  <child link="${name}_depth_optical_frame" />
+	  </joint>
+	  <link name="${name}_depth_optical_frame">
+	    <inertial>
+	      <mass value="0.001" />
+	      <origin xyz="0 0 0" />
+	      <inertia ixx="0.0001" ixy="0.0" ixz="0.0"
+					       iyy="0.0001" iyz="0.0"
+					       izz="0.0001" />
+	    </inertial>
+	  </link>
+    <gazebo reference="${name}_link">
       <material>Gazebo/FlatBlack</material>
     </gazebo>
-		<!-- Axis sensor for simulation -->
-		<sensor_axis_m5013_gazebo/>
+    <!-- Axis sensor for simulation -->
+    <sensor_axis_m5013_gazebo/>
   </xacro:macro>
 	<xacro:macro name="sensor_axis_m5013_gazebo">

Commit message: axis_m5013: changing joint names and new position adjustments

File: urdf/axis_m5013.urdf.xacro (robot description, xacro)
@@ -6,4 +6,5 @@
   <xacro:property name="ptz_joint_damping" value="0.1"/>
   <xacro:property name="ptz_mechanical_reduction" value="1.0"/>
+  <xacro:property name="PI" value="3.14159265359"/>
   <xacro:macro name="sensor_axis_m5013" params="name parent *origin">
     <joint name="${name}_joint" type="fixed">
@@ -40,6 +41,6 @@
       </collision>
     </link>
-    <joint name="joint_${name}_pan" type="revolute">
-      <axis xyz="0 0 -1"/>
+    <joint name="${name}_pan_joint" type="revolute">
+      <axis xyz="1 0 0"/>
       <origin xyz="0.04 0.0 0.0" rpy="0 0 0"/>
       <!-- check the displacement -->
@@ -58,5 +59,5 @@
     <transmission name="${name}_pan_trans">
       <type>transmission_interface/SimpleTransmission</type>
-      <joint name="joint_${name}_pan">
+      <joint name="${name}_pan_joint">
         <hardwareInterface>PositionJointInterface</hardwareInterface>
       </joint>
@@ -66,7 +67,7 @@
       </actuator>
     </transmission>
-    <joint name="joint_${name}_tilt" type="revolute">
+    <joint name="${name}_tilt_joint" type="revolute">
       <axis xyz="0 -1 0"/>
-      <origin xyz="0.0 0.0 0.0"/>
+      <origin xyz="0.0 0.0 0.0" rpy="0 ${-PI/2} 0"/>
       <parent link="${name}_pan_link"/>
       <child link="${name}_tilt_link"/>
@@ -83,5 +84,5 @@
     <transmission name="${name}_tilt_trans">
       <type>transmission_interface/SimpleTransmission</type>
-      <joint name="joint_${name}_tilt">
+      <joint name="${name}_tilt_joint">
         <hardwareInterface>PositionJointInterface</hardwareInterface>
       </joint>
