Commit message: links of xacro files renamed

File: urdf/axis_m5013.urdf.xacro (robot description, xacro)
@@ -15,7 +15,7 @@
       <xacro:insert_block name="origin"/>
       <parent link="${parent}"/>
-      <child link="${prefix}_link"/>
+      <child link="${prefix}_base_link"/>
     </joint>
-    <link name="${prefix}_link">
+    <link name="${prefix}_base_link">
       <inertial>
         <origin xyz="0 0 0" rpy="0 0 0"/>
@@ -45,5 +45,5 @@
       <origin xyz="0.04 0.0 0.0" rpy="0 0 0"/>
       <!-- check the displacement -->
-      <parent link="${prefix}_link"/>
+      <parent link="${prefix}_base_link"/>
       <child link="${prefix}_pan_link"/>
       <limit effort="${ptz_joint_effort_limit}" velocity="${ptz_joint_velocity_limit}" lower="-3.1416" upper="3.1416"/>
@@ -95,7 +95,7 @@
       <origin xyz="0 0 0" rpy="0 0 0"/>
       <parent link="${prefix}_tilt_link"/>
-      <child link="${prefix}_frame"/>
+      <child link="${prefix}_frame_link"/>
     </joint>
-    <link name="${prefix}_frame">
+    <link name="${prefix}_frame_link">
       <inertial>
         <mass value="0.001"/>
@@ -107,8 +107,8 @@
     <joint name="${prefix}_optical_joint" type="fixed">
       <origin xyz="0 0 0" rpy="${-M_PI/2} 0 ${-M_PI/2}"/>
-      <parent link="${prefix}_frame"/>
-      <child link="${prefix}_optical_frame"/>
+      <parent link="${prefix}_frame_link"/>
+      <child link="${prefix}_optical_frame_link"/>
     </joint>
-    <link name="${prefix}_optical_frame">
+    <link name="${prefix}_optical_frame_link">
       <inertial>
         <mass value="0.001"/>
@@ -117,5 +117,5 @@
       </inertial>
     </link>
-    <gazebo reference="${prefix}_link">
+    <gazebo reference="${prefix}_base_link">
       <material>Gazebo/FlatBlack</material>
     </gazebo>
@@ -124,5 +124,5 @@
   </xacro:macro>
 	<xacro:macro name="sensor_axis_m5013_gazebo">
-		<gazebo reference="${prefix}_frame"> <!-- the image will be generated from this (${name}_frame) point of view, with the front being the X axis -->
+		<gazebo reference="${prefix}_frame_link"> <!-- the image will be generated from this (${name}_frame) point of view, with the front being the X axis -->
 			<sensor type="camera" name="${prefix}_sensor">
 				<update_rate>30.0</update_rate>
@@ -146,5 +146,5 @@
 					<imageTopicName>image_raw</imageTopicName>
 					<cameraInfoTopicName>camera_info</cameraInfoTopicName>
-					<frameName>${prefix}_optical_frame</frameName>
+					<frameName>${prefix}_optical_frame_link</frameName>
 					<!-- this is just which name the Image msg will have, it does not affect the simulation.
 					     However must be set to the optical_frame,  -->

File: urdf/fotonic_e.urdf.xacro (robot description, xacro)
@@ -5,7 +5,7 @@
 			<xacro:insert_block name="origin"/>
       <parent link="${parent}"/>
-      <child link="${prefix}_link"/>
+      <child link="${prefix}_base_link"/>
 	  </joint>
-	  <link name="${prefix}_link">
+	  <link name="${prefix}_base_link">
 	    <inertial>
 			<origin xyz="0.0 0 0.0" rpy="0 0 0" />
@@ -34,8 +34,8 @@
 	  <joint name="${prefix}_depth_joint" type="fixed">
 			<origin xyz="0.0375 0 0" rpy="0 0 0" />
-	    <parent link="${prefix}_link" />
-	    <child link="${prefix}_depth_frame" />
+	    <parent link="${prefix}_base_link" />
+	    <child link="${prefix}_depth_frame_link" />
 	  </joint>
-	  <link name="${prefix}_depth_frame">
+	  <link name="${prefix}_depth_frame_link">
 	    <inertial>
 	      <mass value="0.0001" />
@@ -48,8 +48,8 @@
 	  <joint name="${prefix}_depth_optical_joint" type="fixed">
 	    <origin xyz="0 0 0" rpy="-1.5708 0 -1.5708" />
-	    <parent link="${prefix}_depth_frame" />
-	    <child link="${prefix}_depth_optical_frame" />
+	    <parent link="${prefix}_depth_frame_link" />
+	    <child link="${prefix}_depth_optical_frame_link" />
 	  </joint>
-	  <link name="${prefix}_depth_optical_frame">
+	  <link name="${prefix}_depth_optical_frame_link">
 	    <inertial>
 	      <mass value="0.0001" />
@@ -64,8 +64,8 @@
   </xacro:macro>
   <xacro:macro name="sensor_fotonic_gazebo">
-		<gazebo reference="${prefix}_link">
+		<gazebo reference="${prefix}_base_link">
       <material>Gazebo/Grey</material>
     </gazebo>
-    <gazebo reference="${prefix}_depth_frame">
+    <gazebo reference="${prefix}_depth_frame_link">
 	    <sensor type="depth" name="${prefix}_sensor">
 	      <update_rate>30.0</update_rate>
@@ -96,5 +96,5 @@
 					<depthImageCameraInfoTopicName>depth/camera_info</depthImageCameraInfoTopicName>
 					<pointCloudTopicName>points</pointCloudTopicName>
-					<frameName>${prefix}_depth_optical_frame</frameName>
+					<frameName>${prefix}_depth_optical_frame_link</frameName>
 					<pointCloudCutoff>0.5</pointCloudCutoff>
 					<distortionK1>0</distortionK1>

File: urdf/gps.urdf.xacro (robot description, xacro)
@@ -7,7 +7,7 @@
 	    <xacro:insert_block name="origin"/>
 	    <parent link="${parent}"/>
-	    <child link="${prefix}_link"/>
+	    <child link="${prefix}_base_link"/>
 	  </joint>
-	  <link name="${prefix}_link">
+	  <link name="${prefix}_base_link">
 	    <inertial>
 	      <mass value="0.001"/>
@@ -31,5 +31,5 @@
 	    </collision>
 	  </link>
-	  <gazebo reference="${prefix}_link">
+	  <gazebo reference="${prefix}_base_link">
 	    <material>Gazebo/White</material>
 	    <gravity>true</gravity>
@@ -39,6 +39,6 @@
         <alwaysOn>1</alwaysOn>
         <updateRate>5</updateRate>
-        <bodyName>${prefix}_link</bodyName> <!-- must be the link of the gps device, not the base_link or base_footprint -->
-        <frameId>${prefix}_link</frameId>
+        <bodyName>${prefix}_base_link</bodyName> <!-- must be the link of the gps device, not the base_link or base_footprint -->
+        <frameId>${prefix}_base_link</frameId>
         <topicName>fix</topicName>
         <!-- Robotnik position at Fuente del Jarro -->

File: urdf/gps_with_mast.urdf.xacro (robot description, xacro)
@@ -9,7 +9,7 @@
 	    <xacro:insert_block name="origin"/>
 	    <parent link="${parent}"/>
-	    <child link="${prefix}_mast_link"/>
+	    <child link="${prefix}_mast_base_link"/>
 	  </joint>
-	  <link name="${prefix}_mast_link">
+	  <link name="${prefix}_mast_base_link">
 	    <inertial>
 	      <mass value="0.001"/>
@@ -35,9 +35,9 @@
 	  <joint name="${prefix}_mast_joint" type="fixed">
 	    <axis xyz="0 1 0"/>
-	    <parent link="${prefix}_mast_link"/>
+	    <parent link="${prefix}_mast_base_link"/>
 	    <child link="${prefix}_link"/>
 	    <origin xyz="0 0 ${mast_height/2.0}" rpy="0 0 0" />
 	  </joint>
-	  <gazebo reference="${prefix}_mast_link">
+	  <gazebo reference="${prefix}_mast_base_link">
 	    <material>Gazebo/Black</material>
 	    <gravity>true</gravity>

File: urdf/hokuyo3d.urdf.xacro (robot description, xacro)
@@ -5,7 +5,7 @@
       <xacro:insert_block name="origin" />
       <parent link="${parent}"/>
-      <child link="${prefix}_fix_link"/>
+      <child link="${prefix}_base_link"/>
 	</joint>
-	<link name="${prefix}_fix_link">
+	<link name="${prefix}_base_link">
 		<collision>
 			<origin xyz="0 0 0" rpy="0 0 0"/>
@@ -29,5 +29,5 @@
 	</link>
     <joint name="${prefix}_joint" type="fixed">
-      <parent link="${prefix}_fix_link"/>
+      <parent link="${prefix}_base_link"/>
       <child link="${prefix}_link"/>
       <origin xyz="0.08 0 0.08" rpy="0 0 0"/>

File: urdf/hokuyo_urg04lx.urdf.xacro (robot description, xacro)
@@ -2,5 +2,5 @@
 <robot name="sensor_hokuyo_urg04lx" xmlns:xacro="http://www.ros.org/wiki/xacro">
   <xacro:macro name="sensor_hokuyo_urg04lx" params="prefix parent *origin min_angle:=-2.0943 max_angle:=2.0943">
-    <joint name="${prefix}_joint" type="fixed">
+    <joint name="${prefix}_base_joint" type="fixed">
       <!-- FRONT MOUNT  -->
       <!-- origin xyz="0.29 0 0.1" -->
@@ -9,7 +9,7 @@
       <xacro:insert_block name="origin" />
       <parent link="${parent}"/>
-      <child link="${prefix}_link"/>
+      <child link="${prefix}_base_link"/>
     </joint>
-    <link name="${prefix}_link">
+    <link name="${prefix}_base_link">
       <collision>
         <origin xyz="0 0 -0.05" rpy="0 0 0"/>
@@ -34,5 +34,5 @@
   </xacro:macro>
   <xacro:macro name="sensor_hokuyo_urg_gazebo">
-    <gazebo reference="${prefix}_link">
+    <gazebo reference="${prefix}_base_link">
 			<sensor type="ray" name="${prefix}_sensor">
 				<pose>0 0 0 0 0 0</pose>
@@ -61,5 +61,5 @@
 				<plugin name="${name}_controller" filename="libgazebo_ros_laser.so">
 					<topicName>scan</topicName>
-					<frameName>${prefix}_link</frameName>
+					<frameName>${prefix}_base_link</frameName>
 					<ignoreTfPrefix>1</ignoreTfPrefix>
 				</plugin>

File: urdf/hokuyo_ust10lx.urdf.xacro (robot description, xacro)
@@ -3,10 +3,10 @@
   <xacro:macro name="sensor_hokuyo_ust10lx" params="prefix parent *origin min_angle:=-2.3562 max_angle:=2.3562">
 			<!--arg name="namespace" value="$(arg namespace)"/-->
-    <joint name="${prefix}_joint" type="fixed">
+    <joint name="${prefix}_base_joint" type="fixed">
       <xacro:insert_block name="origin" />
       <parent link="${parent}"/>
-      <child link="${prefix}_link"/>
+      <child link="${prefix}_base_link"/>
     </joint>
-    <link name="${prefix}_link">
+    <link name="${prefix}_base_link">
       <collision>
         <origin xyz="0 0 -0.05" rpy="0 0 0"/>
@@ -31,5 +31,5 @@
   </xacro:macro>
   <xacro:macro name="sensor_hokuyo_ust_gazebo">
-    <gazebo reference="${prefix}_link">
+    <gazebo reference="${prefix}_base_link">
 			<sensor type="ray" name="${prefix}_sensor">
 				<pose>0 0 0 0 0 0</pose>
@@ -60,5 +60,5 @@
 				<plugin name="${prefix}_controller" filename="libgazebo_ros_laser.so">
 					<topicName>scan</topicName>
-					<frameName>${prefix}_link</frameName>
+					<frameName>${prefix}_base_link</frameName>
 					<ignoreTfPrefix>1</ignoreTfPrefix>
 				</plugin>

File: urdf/hokuyo_utm30lx.urdf.xacro (robot description, xacro)
@@ -2,5 +2,5 @@
 <robot name="sensor_hokuyo_utm30lx" xmlns:xacro="http://www.ros.org/wiki/xacro">
   <xacro:macro name="sensor_hokuyo_utm30lx" params="prefix parent *origin min_angle:=-2.35 max_angle:=2.35">
-    <joint name="${prefix}_joint" type="fixed">
+    <joint name="${prefix}_base_joint" type="fixed">
       <!-- FRONT MOUNT  -->
       <!-- origin xyz="0.29 0 0.1" -->
@@ -9,7 +9,7 @@
       <xacro:insert_block name="origin" />
       <parent link="${parent}"/>
-      <child link="${prefix}_link"/>
+      <child link="${prefix}_base_link"/>
     </joint>
-    <link name="${prefix}_link">
+    <link name="${prefix}_base_link">
       <visual>
         <origin xyz="0 0 0" rpy="0 0 0"/>
@@ -28,5 +28,5 @@
   </xacro:macro>
   <xacro:macro name="sensor_hokuyo_utm_gazebo">
-    <gazebo reference="${prefix}_link">
+    <gazebo reference="${prefix}_base_link">
 			<sensor type="ray" name="${prefix}_sensor">
 				<pose>0 0 0 0 0 0</pose>
@@ -55,5 +55,5 @@
 				<plugin name="${prefix}_controller" filename="libgazebo_ros_laser.so">
 					<topicName>scan</topicName>
-					<frameName>${prefix}_link</frameName>
+					<frameName>${prefix}_base_link</frameName>
 					<ignoreTfPrefix>1</ignoreTfPrefix>
 				</plugin>

File: urdf/imu.urdf.xacro (robot description, xacro)
@@ -2,12 +2,12 @@
 <robot name="sensor_imu" xmlns:xacro="http://www.ros.org/wiki/xacro">
   <xacro:macro name="sensor_imu" params="prefix parent *origin">
-	  <joint name="${prefix}_joint" type="fixed">
+	  <joint name="${prefix}_base_joint" type="fixed">
 	      <axis xyz="1 0 0"/>
 	      <!--origin xyz="0 0 0.2825"/-->
 	      <xacro:insert_block name="origin"/>
 	      <parent link="${parent}"/>
-	      <child link="${prefix}_link"/>
+	      <child link="${prefix}_base_link"/>
 	  </joint>
-	  <link name="${prefix}_link">
+	  <link name="${prefix}_base_link">
 	      <inertial>
 	        <mass value="0.001"/>
@@ -32,5 +32,5 @@
 	       <topicName>data</topicName>
 		   <serviceName>${prefix}service</serviceName>
-		   <bodyName>${prefix}_link</bodyName>
+		   <bodyName>${prefix}_base_link</bodyName>
 	       <gaussianNoise>0.005</gaussianNoise>
 	       	<ignoreTfPrefix>1</ignoreTfPrefix>

File: urdf/kinect.urdf.xacro (robot description, xacro)
@@ -12,7 +12,7 @@
       <xacro:insert_block name="origin" />
       <parent link="${parent}"/>
-      <child link="${prefix}_rgb_frame" />
+      <child link="${prefix}_rgb_base_link" />
     </joint>
-    <link name="${prefix}_rgb_frame">
+    <link name="${prefix}_rgb_base_link">
       <inertial>
         <mass value="0.001" />
@@ -25,8 +25,8 @@
     <joint name="${prefix}_rgb_optical_joint" type="fixed">
       <origin xyz="0 0 0" rpy="${-M_PI/2} 0 ${-M_PI/2}" />
-      <parent link="${prefix}_rgb_frame" />
-      <child link="${prefix}_rgb_optical_frame" />
+      <parent link="${prefix}_rgb_base_link" />
+      <child link="${prefix}_rgb_optical_link" />
     </joint>
-    <link name="${prefix}_rgb_optical_frame">
+    <link name="${prefix}_rgb_optical_link">
       <inertial>
         <mass value="0.001" />
@@ -39,5 +39,5 @@
   <joint name="${prefix}_joint" type="fixed">
     <origin xyz="-0.031 ${-cam_py} -0.016" rpy="0 0 0"/>
-    <parent link="${prefix}_rgb_frame"/>
+    <parent link="${prefix}_rgb_base_link"/>
     <child link="${prefix}_link"/>
   </joint>
@@ -68,8 +68,8 @@
 	<joint name="${prefix}_depth_joint" type="fixed">
 	  <origin xyz="0 ${2 * -cam_py} 0" rpy="0 0 0" />
-	  <parent link="${prefix}_rgb_frame" />
-	  <child link="${prefix}_depth_frame" />
+	  <parent link="${prefix}_rgb_base_link" />
+	  <child link="${prefix}_depth_link" />
 	</joint>
-	<link name="${prefix}_depth_frame">
+	<link name="${prefix}_depth_link">
     <inertial>
       <mass value="0.001" />
@@ -82,8 +82,8 @@
 	<joint name="${prefix}_depth_optical_joint" type="fixed">
 	  <origin xyz="0 0 0" rpy="${-M_PI/2} 0 ${-M_PI/2}" />
-	  <parent link="${prefix}_depth_frame" />
-	  <child link="${prefix}_depth_optical_frame" />
+	  <parent link="${prefix}_depth_link" />
+	  <child link="${prefix}_depth_optical_link" />
 	</joint>
-	<link name="${prefix}_depth_optical_frame">
+	<link name="${prefix}_depth_optical_link">
     <inertial>
       <mass value="0.001" />
@@ -123,5 +123,5 @@
           <cameraInfoTopicName>rgb/camera_info</cameraInfoTopicName>
           <depthImageCameraInfoTopicName>depth/camera_info</depthImageCameraInfoTopicName>
-          <frameName>${prefix}_depth_optical_frame</frameName>
+          <frameName>${prefix}_depth_optical_link</frameName>
           <baseline>0.1</baseline>
           <distortion_k1>0.0</distortion_k1>

File: urdf/kinectv2.urdf.xacro (robot description, xacro)
@@ -12,7 +12,7 @@
       <xacro:insert_block name="origin" />
       <parent link="${parent}"/>
-      <child link="${prefix}_rgb_frame" />
+      <child link="${prefix}_rgb_base_link" />
     </joint>
-    <link name="${prefix}_rgb_frame">
+    <link name="${prefix}_rgb_base_link">
       <inertial>
         <mass value="0.001" />
@@ -25,8 +25,8 @@
     <joint name="${prefix}_rgb_optical_joint" type="fixed">
       <origin xyz="0 0 0" rpy="${-M_PI/2} 0 ${-M_PI/2}" />
-      <parent link="${prefix}_rgb_frame" />
-      <child link="${prefix}_rgb_optical_frame" />
+      <parent link="${prefix}_rgb_base_link" />
+      <child link="${prefix}_rgb_optical_link" />
     </joint>
-    <link name="${prefix}_rgb_optical_frame">
+    <link name="${prefix}_rgb_optical_link">
       <inertial>
         <mass value="0.001" />
@@ -45,5 +45,5 @@
         <origin xyz="-0.031 ${-cam_py} -0.016" rpy="0 0 0"/>
     </xacro:unless>
-    <parent link="${prefix}_rgb_frame"/>
+    <parent link="${prefix}_rgb_base_link"/>
     <child link="${prefix}_link"/>
   </joint>
@@ -88,8 +88,8 @@
     <joint name="${prefix}_depth_joint" type="fixed">
       <origin xyz="0 ${2 * -cam_py} 0" rpy="0 0 0" />
-      <parent link="${prefix}_rgb_frame" />
-      <child link="${prefix}_depth_frame" />
+      <parent link="${prefix}_rgb_base_link" />
+      <child link="${prefix}_depth_link" />
     </joint>
-    <link name="${prefix}_depth_frame">
+    <link name="${prefix}_depth_link">
     <inertial>
       <mass value="0.001" />
@@ -102,8 +102,8 @@
     <joint name="${prefix}_depth_optical_joint" type="fixed">
       <origin xyz="0 0 0" rpy="${-M_PI/2} 0 ${-M_PI/2}" />
-      <parent link="${prefix}_depth_frame" />
-      <child link="${prefix}_depth_optical_frame" />
+      <parent link="${prefix}_depth_link" />
+      <child link="${prefix}_depth_optical_link" />
     </joint>
-    <link name="${prefix}_depth_optical_frame">
+    <link name="${prefix}_depth_optical_link">
     <inertial>
       <mass value="0.001" />
@@ -143,5 +143,5 @@
           <cameraInfoTopicName>rgb/camera_info</cameraInfoTopicName>
           <depthImageCameraInfoTopicName>depth/camera_info</depthImageCameraInfoTopicName>
-          <frameName>${prefix}_depth_optical_frame</frameName>
+          <frameName>${prefix}_depth_optical_link</frameName>
           <baseline>0.1</baseline>
           <distortion_k1>0.0</distortion_k1>

File: urdf/orbbec_astra.urdf.xacro (robot description, xacro)
@@ -17,7 +17,7 @@
 	  <xacro:insert_block name="origin" />
       <parent link="${parent}"/>
-      <child link="${prefix}_rgb_frame_link" />
+      <child link="${prefix}_rgb_base_link" />
     </joint>
-    <link name="${prefix}_rgb_frame_link">
+    <link name="${prefix}_rgb_base_link">
       <inertial>
         <mass value="0.001" />
@@ -30,5 +30,5 @@
     <joint name="${prefix}_rgb_optical_joint" type="fixed">
       <origin xyz="0.0 0.0 0.0" rpy="${-M_PI/2} 0 ${-M_PI/2}" />
-      <parent link="${prefix}_rgb_frame_link" />
+      <parent link="${prefix}_rgb_base_link" />
       <child link="${prefix}_rgb_optical_frame_link" />
     </joint>
@@ -45,5 +45,5 @@
       <origin xyz="${orbbec_astra_rel_rgb_px} ${orbbec_astra_rel_rgb_py} ${orbbec_astra_rel_rgb_pz}"
               rpy="0.0 0 0"/>
-      <parent link="${prefix}_rgb_frame_link"/>
+      <parent link="${prefix}_rgb_base_link"/>
       <child link="${prefix}_link"/>
     </joint>
@@ -76,5 +76,5 @@
     <joint name="${prefix}_depth_joint" type="fixed">
       <origin xyz="${orbbec_astra_depth_rel_rgb_px} ${orbbec_astra_depth_rel_rgb_py} ${orbbec_astra_depth_rel_rgb_pz}" rpy="0 0 0" />
-      <parent link="${prefix}_rgb_frame_link" />
+      <parent link="${prefix}_rgb_base_link" />
       <child link="${prefix}_depth_frame_link" />
     </joint>
@@ -106,5 +106,5 @@
   </xacro:macro>
    <xacro:macro name="sensor_orbbec_astra_gazebo">
-    <gazebo reference="${prefix}_rgb_frame_link">
+    <gazebo reference="${prefix}_rgb_base_link">
       <sensor type="depth" name="${prefix}_depth_sensor">
         <always_on>true</always_on>

File: urdf/sick_s300.urdf.xacro (robot description, xacro)
@@ -2,10 +2,10 @@
 <robot name="sensor_sick_s300" xmlns:xacro="http://www.ros.org/wiki/xacro">
   <xacro:macro name="sensor_sick_s300" params="prefix parent *origin">
-    <joint name="${prefix}_fix_joint" type="fixed">
+    <joint name="${prefix}_base_joint" type="fixed">
       <xacro:insert_block name="origin" />
       <parent link="${parent}"/>
-      <child link="${prefix}_fix_link"/>
+      <child link="${prefix}_base_link"/>
 	</joint>
-	<link name="${prefix}_fix_link">
+	<link name="${prefix}_base_link">
 		<collision>
 			<origin xyz="0 0 0.076" rpy="0 0 0"/>
@@ -29,5 +29,5 @@
 	</link>
     <joint name="${prefix}_joint" type="fixed">
-      <parent link="${prefix}_fix_link"/>
+      <parent link="${prefix}_base_link"/>
       <child link="${prefix}_link"/>
       <origin xyz="0.0 0 0.116" rpy="0 0 0"/>

File: urdf/sick_s3000.urdf.xacro (robot description, xacro)
@@ -5,7 +5,7 @@
       <xacro:insert_block name="origin" />
       <parent link="${parent}"/>
-      <child link="${prefix}_link"/>
+      <child link="${prefix}_base_link"/>
 	</joint>
-	<link name="${prefix}_link">
+	<link name="${prefix}_base_link">
 		<collision>
 			<origin xyz="-0.093 0 -0.0625" rpy="0 0 0"/>
@@ -30,5 +30,5 @@
   </xacro:macro>
   <xacro:macro name="sensor_sick_s3000_gazebo">
-    <gazebo reference="${prefix}_link">
+    <gazebo reference="${prefix}_base_link">
 			<sensor type="ray" name="${prefix}_sensor">
 				<pose>0 0 0 0 0 0</pose>
@@ -57,5 +57,5 @@
 				<plugin name="${prefix}_controller" filename="libgazebo_ros_laser.so">
 					<topicName>scan</topicName>
-					<frameName>${prefix}_link</frameName>
+					<frameName>${prefix}_base_link</frameName>
 					<ignoreTfPrefix>1</ignoreTfPrefix>
 				</plugin>

File: urdf/ueye_cp_gige.urdf.xacro (robot description, xacro)
@@ -5,7 +5,7 @@
       <insert_block name="origin"/>
       <parent link="${parent}"/>
-      <child link="${prefix}_link"/>
+      <child link="${prefix}_base_link"/>
     </joint>
-    <link name="${prefix}_link"> <!-- TODO: review masses, inertial -->
+    <link name="${prefix}_base_link"> <!-- TODO: review masses, inertial -->
       <inertial>
         <origin xyz="0.0 0.0 0." rpy="0 0 0"/>
@@ -33,8 +33,8 @@
     <joint name="${prefix}_rgb_joint" type="fixed">
       <origin xyz="0 0 0" rpy="0 0 0" />
-      <parent link="${prefix}_link"/>
-      <child link="${prefix}_rgb_frame"/>
+      <parent link="${prefix}_base_link"/>
+      <child link="${prefix}_rgb_frame_link"/>
     </joint>
-    <link name="${prefix}_rgb_frame">
+    <link name="${prefix}_rgb_frame_link">
     <inertial>
       <mass value="0.001" />
@@ -47,8 +47,8 @@
     <joint name="${prefix}_rgb_optical_joint" type="fixed">
       <origin xyz="0 0 0" rpy="0 0 0" />
-      <parent link="${prefix}_rgb_frame"/>
-      <child link="${prefix}_rgb_optical_frame"/>
+      <parent link="${prefix}_rgb_frame_link"/>
+      <child link="${prefix}_rgb_optical_frame_link"/>
     </joint>
-    <link name="${prefix}_rgb_optical_frame">
+    <link name="${prefix}_rgb_optical_frame_link">
     <inertial>
       <mass value="0.001" />
@@ -62,5 +62,5 @@
   </xacro:macro>
   <xacro:macro name="sensor_ueye_cp_gige_gazebo">
-    <gazebo reference="${prefix}_link">
+    <gazebo reference="${prefix}_base_link">
       <sensor type="camera" name="${prefix}_sensor">
         <update_rate>30.0</update_rate>
@@ -88,5 +88,5 @@
           <imageTopicName>image_raw</imageTopicName>
           <cameraInfoTopicName>camera_info</cameraInfoTopicName>
-          <frameName>${prefix}_rgb_frame</frameName>
+          <frameName>${prefix}_rgb_frame_link</frameName>
           <distortionK1>0.0</distortionK1>
           <distortionK2>0.0</distortionK2>
