Commit message: robotnik_sensors: changed wrong name using prefix

File: urdf/axis_m5013.urdf.xacro (robot description, xacro)
@@ -62,5 +62,5 @@
         <hardwareInterface>PositionJointInterface</hardwareInterface>
       </joint>
-      <actuator name="pan_motor">
+      <actuator name="${prefix}pan_motor">
         <hardwareInterface>PositionJointInterface</hardwareInterface>
         <mechanicalReduction>${ptz_mechanical_reduction}</mechanicalReduction>
@@ -82,10 +82,10 @@
       </inertial>
     </link>
-    <transmission name="${name}_tilt_trans">
+    <transmission name="${prefix}_tilt_trans">
       <type>transmission_interface/SimpleTransmission</type>
-      <joint name="${name}_tilt_joint">
+      <joint name="${prefix}_tilt_joint">
         <hardwareInterface>PositionJointInterface</hardwareInterface>
       </joint>
-      <actuator name="tilt_motor">
+      <actuator name="${prefix}tilt_motor">
         <hardwareInterface>PositionJointInterface</hardwareInterface>
         <mechanicalReduction>${ptz_mechanical_reduction}</mechanicalReduction>

Commit message: urdf: updated axis_m5013 inertia based on datasheet and using inertia.urdf.xacro

File: urdf/axis_m5013.urdf.xacro (robot description, xacro)
@@ -16,8 +16,7 @@
     <link name="${prefix}_base_link">
       <inertial>
-        <origin xyz="0 0 0" rpy="0 0 0"/>
-        <mass value="0.1"/>
-        <origin xyz="0 0 0" rpy="0 0 0"/>
-        <inertia ixx="0.1" ixy="0" ixz="0" iyy="0.1" iyz="0" izz="0.1"/>
+        <origin xyz="0.0175 0 0" rpy="0 ${M_PI/2} 0"/>
+        <mass value="0.3"/>
+        <xacro:solid_cuboid_inertia m="0.3" w="0.130" h="0.130" d="0.035" /> <!-- Data from axis M5013 datasheet -->
       </inertial>
       <visual>
@@ -49,7 +48,7 @@
     <link name="${prefix}_pan_link">
       <inertial>
-        <mass value="0.1"/>
+        <mass value="0.01"/>
         <origin xyz="0 0 0" rpy="0 0 0"/>
-        <inertia ixx="0.1" ixy="0" ixz="0" iyy="0.1" iyz="0" izz="0.1"/>
+        <xacro:solid_cuboid_inertia m="0.01" w="0.03" h="0.06" d="0.06" />
       </inertial>
     </link>
@@ -74,7 +73,7 @@
     <link name="${prefix}_tilt_link">
       <inertial>
-        <mass value="0.1"/>
+        <mass value="0.01"/>
         <origin xyz="0 0 0" rpy="0 0 0"/>
-        <inertia ixx="0.1" ixy="0" ixz="0" iyy="0.1" iyz="0" izz="0.1"/>
+        <xacro:solid_cuboid_inertia m="0.01" w="0.06" h="0.06" d="0.03" />
       </inertial>
     </link>
@@ -96,7 +95,7 @@
     <link name="${prefix}_frame_link">
       <inertial>
-        <mass value="0.001"/>
-        <origin xyz="0 0 0"/>
-        <inertia ixx="0.0001" ixy="0.0" ixz="0.0" iyy="0.0001" iyz="0.0" izz="0.0001"/>
+        <mass value="0.01"/>
+        <origin xyz="0 0 0" rpy="0 0 0"/>
+        <xacro:solid_cuboid_inertia m="0.01" w="0.06" h="0.06" d="0.03" />
       </inertial>
     </link>
@@ -109,11 +108,11 @@
     <link name="${prefix}_optical_frame_link">
       <inertial>
-        <mass value="0.001"/>
-        <origin xyz="0 0 0"/>
-        <inertia ixx="0.0001" ixy="0.0" ixz="0.0" iyy="0.0001" iyz="0.0" izz="0.0001"/>
+        <mass value="0.01"/>
+        <origin xyz="0 0 0" rpy="0 0 0"/>
+        <xacro:solid_cuboid_inertia m="0.01" w="0.06" h="0.03" d="0.06" />
       </inertial>
     </link>
     <gazebo reference="${prefix}_base_link">
-      <material>Gazebo/FlatBlack</material>
+      <material>Gazebo/DarkGrey</material>
     </gazebo>
     <!-- Axis sensor for simulation -->

Commit message: Add zoom link and joint to axis cameras

File: urdf/axis_m5013.urdf.xacro (robot description, xacro)
@@ -69,5 +69,5 @@
     <joint name="${prefix}_tilt_joint" type="revolute">
       <axis xyz="0 0 1"/>
-      <origin xyz="0.0 0.0 0.0" rpy="${-PI/2} 0 0"/>
+      <origin xyz="0.0 0.0 0.0" rpy="${PI/2} 0 0"/>
       <parent link="${prefix}_pan_link"/>
       <child link="${prefix}_tilt_link"/>
@@ -90,4 +90,31 @@
       </joint>
       <actuator name="${prefix}tilt_motor">
+        <hardwareInterface>hardware_interface/PositionJointInterface</hardwareInterface>
+        <mechanicalReduction>${ptz_mechanical_reduction}</mechanicalReduction>
+      </actuator>
+    </transmission>
+    <joint name="${prefix}_zoom_joint" type="prismatic">
+      <axis xyz="1 0 0"/>
+      <origin xyz="0.0 0.0 0.0" rpy="${-PI/2} 0 0"/>
+      <parent link="${prefix}_tilt_link"/>
+      <child link="${prefix}_zoom_link"/>
+      <limit effort="${ptz_joint_effort_limit}" velocity="${ptz_joint_velocity_limit}" lower="-1.5708" upper="1.5708"/>
+      <joint_properties damping="${ptz_joint_damping}" friction="{ptz_joint_friction}"/>
+    </joint>
+    <link name="${prefix}_zoom_link">
+      <xacro:if value="${include_inertial}">
+        <inertial>
+          <mass value="0.1"/>
+          <origin xyz="0 0 0" rpy="0 0 0"/>
+          <xacro:solid_cuboid_inertia m="0.1" w="0.11" h="0.11" d="0.1" />
+        </inertial>
+      </xacro:if>
+    </link>
+    <transmission name="${prefix}_zoom_trans">
+      <type>transmission_interface/SimpleTransmission</type>
+      <joint name="${prefix}_zoom_joint">
+        <hardwareInterface>hardware_interface/PositionJointInterface</hardwareInterface>
+      </joint>
+      <actuator name="${prefix}zoom_motor">
         <hardwareInterface>hardware_interface/PositionJointInterface</hardwareInterface>
         <mechanicalReduction>${ptz_mechanical_reduction}</mechanicalReduction>

File: urdf/axis_m5525.urdf.xacro (robot description, xacro)
@@ -69,5 +69,5 @@
     <joint name="${prefix}_tilt_joint" type="revolute">
       <axis xyz="0 0 1"/>
-      <origin xyz="0.0 0.0 0.0" rpy="${-PI/2} 0 0"/>
+      <origin xyz="0.0 0.0 0.0" rpy="${PI/2} 0 0"/>
       <parent link="${prefix}_pan_link"/>
       <child link="${prefix}_tilt_link"/>
@@ -90,4 +90,31 @@
       </joint>
       <actuator name="${prefix}tilt_motor">
+        <hardwareInterface>hardware_interface/PositionJointInterface</hardwareInterface>
+        <mechanicalReduction>${ptz_mechanical_reduction}</mechanicalReduction>
+      </actuator>
+    </transmission>
+    <joint name="${prefix}_zoom_joint" type="prismatic">
+      <axis xyz="1 0 0"/>
+      <origin xyz="0.0 0.0 0.0" rpy="${-PI/2} 0 0"/>
+      <parent link="${prefix}_tilt_link"/>
+      <child link="${prefix}_zoom_link"/>
+      <limit effort="${ptz_joint_effort_limit}" velocity="${ptz_joint_velocity_limit}" lower="-1.5708" upper="1.5708"/>
+      <joint_properties damping="${ptz_joint_damping}" friction="{ptz_joint_friction}"/>
+    </joint>
+    <link name="${prefix}_zoom_link">
+      <xacro:if value="${include_inertial}">
+        <inertial>
+          <mass value="0.1"/>
+          <origin xyz="0 0 0" rpy="0 0 0"/>
+          <xacro:solid_cuboid_inertia m="0.1" w="0.11" h="0.11" d="0.1" />
+        </inertial>
+      </xacro:if>
+    </link>
+    <transmission name="${prefix}_zoom_trans">
+      <type>transmission_interface/SimpleTransmission</type>
+      <joint name="${prefix}_zoom_joint">
+        <hardwareInterface>hardware_interface/PositionJointInterface</hardwareInterface>
+      </joint>
+      <actuator name="${prefix}zoom_motor">
         <hardwareInterface>hardware_interface/PositionJointInterface</hardwareInterface>
         <mechanicalReduction>${ptz_mechanical_reduction}</mechanicalReduction>
