Commit message: Reduce size & quality of most of mesh files

File: urdf/axis_p5676.urdf.xacro (robot description, xacro)
@@ -29,5 +29,5 @@
         </material>
         <geometry>
-          <mesh filename="package://robotnik_sensors/meshes/axis_p5676.stl" scale="1.0 1.0 1.0"/>
+          <mesh filename="package://robotnik_sensors/meshes/axis_p5676.dae" scale="1.0 1.0 1.0"/>
         </geometry>
       </visual>

File: urdf/rs_helios_16p.urdf.xacro (robot description, xacro)
@@ -18,8 +18,8 @@
       </visual>
       <collision>
-        <origin xyz="0 0 0" rpy="0 0 0"/>
-        <geometry>
-          <mesh filename="package://robotnik_sensors/meshes/rs_helios_16p.stl" />
-        </geometry>
+        <origin rpy="0 0 0" xyz="0 0 0.05"/>
+	      <geometry>
+	        <cylinder radius="0.05" length="0.1"/>
+	      </geometry>
       </collision>
       <xacro:if value="${include_inertial}">
