Commit message: Fixes mesh dimensions link 750

File: urdf/link_750_nh.urdf.xacro (robot description, xacro)
@@ -21,16 +21,16 @@
       </inertial>
       <visual>
-        <origin xyz="0 0 0" rpy="0 0 0"/>
+        <origin xyz="-0.07 -0.07 -0.045" rpy="0 0 0"/>
         <material name="grey_color">
           <color rgba="0.1 0.1 0.1 1"/>
         </material>
         <geometry>
-          <mesh filename="package://robotnik_sensors/meshes/link_750_base.stl" scale="1.0 1.0 1.0"/>
+          <mesh filename="package://robotnik_sensors/meshes/link_750_base.stl" scale="0.001 0.001 0.001"/>
         </geometry>
       </visual>
       <collision>
-        <origin xyz="0.0 0.0 0" rpy="0 0 0"/>
+        <origin xyz="-0.07 -0.07 -0.045" rpy="0 0 0"/>
         <geometry>
-          <mesh filename="package://robotnik_sensors/meshes/link_750_base.stl" scale="1.0 1.0 1.0"/>
+          <mesh filename="package://robotnik_sensors/meshes/link_750_base.stl" scale="0.001 0.001 0.001"/>
         </geometry>
       </collision>

Commit message: Updates image frame link for link 750 in sim

File: urdf/link_750_nh.urdf.xacro (robot description, xacro)
@@ -131,5 +131,5 @@
     <!-- Optical frame -->
     <joint name="${prefix}_optical_joint" type="fixed">
-      <origin xyz="0 0 0" rpy="${-M_PI/2} 0 ${-M_PI/2}"/>
+      <origin xyz="0.02 0 0" rpy="0 0 0"/>
       <parent link="${prefix}_frame_link"/>
       <child link="${prefix}_optical_frame_link"/>
@@ -149,5 +149,5 @@
   </xacro:macro>
   <xacro:macro name="sensor_link_750_nh_gazebo">
-    <gazebo reference="${prefix}_frame_link"> <!-- the image will be generated from this (${name}_frame) point of view, with the front being the X axis -->
+    <gazebo reference="${prefix}_optical_frame_link"> <!-- the image will be generated from this (${name}_frame) point of view, with the front being the X axis -->
       <sensor type="camera" name="${prefix}_sensor">
         <update_rate>30.0</update_rate>

Commit message: Modify link_750 urdf for rotatinf in the correct axis

File: urdf/link_750_nh.urdf.xacro (robot description, xacro)
@@ -37,5 +37,5 @@
     </link>
     <joint name="${prefix}_pan_joint" type="revolute">
-      <axis xyz="1 0 0"/>
+      <axis xyz="0 0 -1"/>
       <origin xyz="0.0 0.0 0.0318" rpy="0 0 0"/>
       <!-- check the displacement -->
@@ -78,5 +78,5 @@
     </transmission>
     <joint name="${prefix}_tilt_joint" type="revolute">
-      <axis xyz="0 1 0"/>
+      <axis xyz="0 -1 0"/>
       <origin xyz="0.0 0.0 0.102" rpy="0 0 0"/>
       <parent link="${prefix}_pan_link"/>

Commit message: Updates link750 urdf

File: urdf/link_750_nh.urdf.xacro (robot description, xacro)
@@ -123,12 +123,12 @@
       </actuator>
     </transmission>
-    <joint name="${prefix}_zoom_joint" type="prismatic">
+    <joint name="${prefix}_zoom_color_joint" type="prismatic">
       <axis xyz="0 0 1"/>
       <origin xyz="0.0 0.0 0.0" rpy="0 0 0"/>
       <parent link="${prefix}_optical_frame_link"/>
-      <child link="${prefix}_zoom_link"/>
+      <child link="${prefix}_zoom_color_link"/>
       <limit effort="10000.0" velocity="5" lower="0" upper="10000"/>
     </joint>
-    <link name="${prefix}_zoom_link">
+    <link name="${prefix}_zoom_color_link">
       <xacro:if value="${include_inertial}">
         <inertial>
@@ -139,7 +139,7 @@
       </xacro:if>
     </link>
-    <transmission name="${prefix}_zoom_trans">
+    <transmission name="${prefix}_zoom_color_trans">
       <type>transmission_interface/SimpleTransmission</type>
-      <joint name="${prefix}_zoom_joint">
+      <joint name="${prefix}_zoom_color_joint">
         <hardwareInterface>hardware_interface/PositionJointInterface</hardwareInterface>
       </joint>
@@ -150,5 +150,5 @@
     </transmission>
     <joint name="${prefix}_frame_joint" type="fixed">
-      <origin xyz="0.06 0 0" rpy="${-PI/2} 0 0"/>
+      <origin xyz="0.05 0.025 0" rpy="${-PI/2} 0 0"/>
       <parent link="${prefix}_tilt_link"/>
       <child link="${prefix}_frame_link"/>
@@ -178,4 +178,62 @@
       </xacro:if>
     </link>
+    <gazebo reference="${prefix}_base_link">
+      <material>Gazebo/DarkGrey</material>
+    </gazebo>
+    <joint name="${prefix}_thermal_frame_joint" type="fixed">
+      <origin xyz="0.05 -0.025 0.0" rpy="${-PI/2} 0 0"/>
+      <parent link="${prefix}_tilt_link"/>
+      <child link="${prefix}_thermal_frame_link"/>
+    </joint>
+    <link name="${prefix}_thermal_frame_link">
+      <xacro:if value="${include_inertial}">
+        <inertial>
+          <mass value="0.1"/>
+          <origin xyz="0 0 0"/>
+          <xacro:solid_cuboid_inertia m="0.1" w="0.11" h="0.11" d="0.1" />
+        </inertial>
+      </xacro:if>
+    </link>
+    <!-- Optical frame ${-M_PI/2} -->
+    <joint name="${prefix}_optical_thermal_joint" type="fixed">
+      <origin xyz="0.0 0 0" rpy="${-M_PI/2} 0 ${-M_PI/2}"/>
+      <parent link="${prefix}_thermal_frame_link"/>
+      <child link="${prefix}_optical_thermal_frame_link"/>
+    </joint>
+    <link name="${prefix}_optical_thermal_frame_link">
+      <xacro:if value="${include_inertial}">
+        <inertial>
+          <mass value="0.1"/>
+          <origin xyz="0 0 0"/>
+          <xacro:solid_cuboid_inertia m="0.1" w="0.11" h="0.11" d="0.1" />
+        </inertial>
+      </xacro:if>
+    </link>
+    <joint name="${prefix}_zoom_thermal_joint" type="prismatic">
+      <axis xyz="0 0 1"/>
+      <origin xyz="0.0 0.0 0.0" rpy="0 0 0"/>
+      <parent link="${prefix}_optical_thermal_frame_link"/>
+      <child link="${prefix}_zoom_thermal_link"/>
+      <limit effort="10000.0" velocity="5" lower="0" upper="10000"/>
+    </joint>
+    <link name="${prefix}_zoom_thermal_link">
+      <xacro:if value="${include_inertial}">
+        <inertial>
+          <mass value="0.00001"/>
+          <origin xyz="0 0 0" rpy="0 0 0"/>
+          <xacro:solid_cuboid_inertia m="0.00001" w="0.11" h="0.11" d="0.1" />
+        </inertial>
+      </xacro:if>
+    </link>
+    <transmission name="${prefix}_zoom_thermal_trans">
+      <type>transmission_interface/SimpleTransmission</type>
+      <joint name="${prefix}_zoom_thermal_joint">
+        <hardwareInterface>hardware_interface/PositionJointInterface</hardwareInterface>
+      </joint>
+      <actuator name="${prefix}zoom_thermal_motor">
+        <hardwareInterface>hardware_interface/PositionJointInterface</hardwareInterface>
+        <mechanicalReduction>1</mechanicalReduction>
+      </actuator>
+    </transmission>
     <gazebo reference="${prefix}_base_link">
       <material>Gazebo/DarkGrey</material>
@@ -238,5 +296,5 @@
           <imageTopicName>thermal/image_raw</imageTopicName>
           <cameraInfoTopicName>thermal/camera_info</cameraInfoTopicName>
-          <frameName>${prefix}_frame_link</frameName>
+          <frameName>${prefix}_thermal_frame_link</frameName>
         </plugin>
       </sensor>
