Commit message: Corrects optical center for helios sensor

File: urdf/rs_helios_16p.urdf.xacro (robot description, xacro)
@@ -32,5 +32,5 @@
       <parent link="${prefix}_base_link"/>
       <child link="${prefix}_link" />
-      <origin xyz="0.0 0 0.0405" rpy="0 0 0"/>
+      <origin xyz="0.0 0 0.0635" rpy="0 0 0"/>
     </joint>
     <link name="${prefix}_link"/>

Commit message: rs_helios_16p: Fix black_alu material

File: urdf/rs_helios_16p.urdf.xacro (robot description, xacro)
@@ -15,5 +15,5 @@
           <mesh filename="package://robotnik_sensors/meshes/rs_helios_16p.stl" />
         </geometry>
-        <material name="black_alu"/>
+        <xacro:black_alu_material/>
       </visual>
       <collision>

Commit message: Adds suffix_topic to helios

File: urdf/rs_helios_16p.urdf.xacro (robot description, xacro)
@@ -2,5 +2,5 @@
 <robot name="sensor_rslidar" xmlns:xacro="http://wiki.ros.org/xacro">
   <xacro:property name="M_PI" value="3.1415926535897931" />
-  <xacro:macro name="sensor_rs_helios" params="prefix parent prefix_topic *origin range_min range_max hfov hres vfov vres fps gpu:=^|true include_inertial">
+  <xacro:macro name="sensor_rs_helios" params="prefix parent prefix_topic suffix_topic:='' *origin range_min range_max hfov hres vfov vres fps gpu:=^|true include_inertial">
     <joint name="${prefix}_base_joint" type="fixed">
       <xacro:insert_block name="origin" />
@@ -78,5 +78,5 @@
           </ray>
           <plugin name="${prefix}_controller" filename="${plugin_lib}">
-            <topicName>${prefix_topic}/points</topicName>
+            <topicName>${prefix_topic}/points${suffix_topic}</topicName>
             <frameName>/${prefix}_link</frameName>
             <min_range>${range_min}</min_range>
@@ -87,6 +87,6 @@
     </gazebo>
   </xacro:macro>
-  <xacro:macro name="sensor_rs_helios_16p" params="prefix parent prefix_topic:='lidar_3d' *origin gpu:=false include_inertial:=^|true">
-    <xacro:sensor_rs_helios prefix="${prefix}" parent="${parent}" prefix_topic="${prefix_topic}" range_min="0.2" range_max="150.0" hfov="360.0" hres="0.2" vfov="30.0" vres="2" fps="10.0" gpu="${gpu}" include_inertial="${include_inertial}">
+  <xacro:macro name="sensor_rs_helios_16p" params="prefix parent prefix_topic:='lidar_3d' suffix_topic:='' *origin gpu:=false include_inertial:=^|true">
+    <xacro:sensor_rs_helios prefix="${prefix}" parent="${parent}" prefix_topic="${prefix_topic}" suffix_topic="${suffix_topic}" range_min="0.2" range_max="150.0" hfov="360.0" hres="0.2" vfov="30.0" vres="2" fps="10.0" gpu="${gpu}" include_inertial="${include_inertial}">
       <xacro:insert_block name="origin" />
     </xacro:sensor_rs_helios>
