Commit message: rs_airy: Fix collision origin

File: urdf/rs_airy.urdf.xacro (robot description, xacro)
@@ -18,5 +18,5 @@
       </visual>
       <collision>
-        <origin rpy="0 0 0" xyz="0 0 0.05"/>
+        <origin rpy="0 0 0" xyz="0 0 0.032"/>
 	      <geometry>
 	        <cylinder radius="0.0305" length="0.064"/>

Commit message: rs_airy: Add default prefix_topic

File: urdf/rs_airy.urdf.xacro (robot description, xacro)
@@ -2,5 +2,5 @@
 <robot name="sensor_rsairy" xmlns:xacro="http://wiki.ros.org/xacro">
   <xacro:property name="M_PI" value="3.1415926535897931" />
-  <xacro:macro name="sensor_rs_airy" params="prefix parent *origin prefix_topic suffix_topic:='' range_min:=0.1 range_max:=60.0 hfov:=360 hres:=0.2 vfov:=30.0 vres:=2 fps:=10.0 gpu:=^|true include_inertial:=^|true">
+  <xacro:macro name="sensor_rs_airy" params="prefix parent *origin prefix_topic:='top_3d_laser' suffix_topic:='' range_min:=0.1 range_max:=60.0 hfov:=360 hres:=0.2 vfov:=30.0 vres:=2 fps:=10.0 gpu:=^|true include_inertial:=^|true">
     <joint name="${prefix}_base_joint" type="fixed">
       <xacro:insert_block name="origin" />
