Commit message: Added name space param

File: urdf/gps.urdf.xacro (robot description, xacro)
@@ -1,5 +1,5 @@
 <?xml version="1.0"?>
 <robot name="sensor_gps" xmlns:xacro="http://www.ros.org/wiki/xacro">
-  <xacro:macro name="sensor_gps" params="prefix parent *origin">
+  <xacro:macro name="sensor_gps" params="prefix ns parent *origin">
 	  <!-- ANTENNA GPS -->
 	  <joint name="${prefix}_joint" type="fixed">
@@ -40,6 +40,6 @@
         <updateRate>5</updateRate>
         <bodyName>${prefix}_base_link</bodyName> <!-- must be the link of the gps device, not the base_link or base_footprint -->
-        <frameId>/${prefix}_base_link</frameId>
-        <topicName>fix</topicName>
+        <frameId>${prefix}_base_link</frameId>
+        <topicName>${ns}gps/fix</topicName>
         <!-- Robotnik position at Fuente del Jarro -->
         <referenceLatitude>39.5080331</referenceLatitude>
@@ -47,5 +47,5 @@
         <!-- To set heading in ENU orientation (degrees) -->
         <referenceHeading>90</referenceHeading>
-        <velocityTopicName>fix_velocity</velocityTopicName>
+        <velocityTopicName>${ns}gps/fix_velocity</velocityTopicName>
         <drift>0.0 0.0 0.0</drift>
         <!--<drift>0.0001 0.0001 0.0001</drift>-->

File: urdf/imu.urdf.xacro (robot description, xacro)
@@ -1,5 +1,5 @@
 <?xml version="1.0"?>
 <robot name="sensor_imu" xmlns:xacro="http://www.ros.org/wiki/xacro">
-  <xacro:macro name="sensor_imu" params="prefix parent *origin">
+  <xacro:macro name="sensor_imu" params="prefix ns:='' parent *origin">
 	  <joint name="${prefix}_joint" type="fixed">
 	      <axis xyz="1 0 0"/>
@@ -30,5 +30,5 @@
 	  <gazebo>
 	    <plugin name="${prefix}_controller" filename="libgazebo_ros_imu.so">
-	       <topicName>imu/data</topicName>
+	       <topicName>${ns}imu/data</topicName>
 	       <serviceName>imu/service</serviceName>
 		   <bodyName>${prefix}_link</bodyName>

File: urdf/sick_s3000.urdf.xacro (robot description, xacro)
@@ -1,5 +1,5 @@
 <?xml version="1.0"?>
 <robot name="sensor_sick_s3000" xmlns:xacro="http://www.ros.org/wiki/xacro">
-  <xacro:macro name="sensor_sick_s3000" params="prefix parent prefix_topic:='front_laser' *origin">
+  <xacro:macro name="sensor_sick_s3000" params="prefix parent ns='' prefix_topic:='front_laser' *origin">
     <joint name="${prefix}_joint" type="fixed">
       <xacro:insert_block name="origin" />
@@ -56,5 +56,5 @@
 				</ray>
 				<plugin name="${prefix}_controller" filename="libgazebo_ros_laser.so">
-					<topicName>${prefix_topic}/scan</topicName>
+					<topicName>${ns}${prefix_topic}/scan</topicName>
 					<frameName>/${prefix}_base_link</frameName>
 				</plugin>

Commit message: gps: removed namespace

File: urdf/gps.urdf.xacro (robot description, xacro)
@@ -1,5 +1,5 @@
 <?xml version="1.0"?>
 <robot name="sensor_gps" xmlns:xacro="http://www.ros.org/wiki/xacro">
-  <xacro:macro name="sensor_gps" params="prefix ns parent *origin">
+  <xacro:macro name="sensor_gps" params="prefix parent *origin">
 	  <!-- ANTENNA GPS -->
 	  <joint name="${prefix}_joint" type="fixed">
@@ -41,5 +41,5 @@
         <bodyName>${prefix}_base_link</bodyName> <!-- must be the link of the gps device, not the base_link or base_footprint -->
         <frameId>${prefix}_base_link</frameId>
-        <topicName>${ns}gps/fix</topicName>
+        <topicName>gps/fix</topicName>
         <!-- Robotnik position at Fuente del Jarro -->
         <referenceLatitude>39.5080331</referenceLatitude>
@@ -47,5 +47,5 @@
         <!-- To set heading in ENU orientation (degrees) -->
         <referenceHeading>90</referenceHeading>
-        <velocityTopicName>${ns}gps/fix_velocity</velocityTopicName>
+        <velocityTopicName>gps/fix_velocity</velocityTopicName>
         <drift>0.0 0.0 0.0</drift>
         <!--<drift>0.0001 0.0001 0.0001</drift>-->

Commit message: Added the capability to set the GPS coordinates from launch file

File: urdf/gps.urdf.xacro (robot description, xacro)
@@ -1,5 +1,5 @@
 <?xml version="1.0"?>
 <robot name="sensor_gps" xmlns:xacro="http://wiki.ros.org/xacro">
-  <xacro:macro name="sensor_gps" params="prefix parent *origin">
+  <xacro:macro name="sensor_gps" params="prefix parent *origin gps_latitude:=^|0.0 gps_longitude:=^|0.0">
 	  <!-- ANTENNA GPS -->
 	  <joint name="${prefix}_joint" type="fixed">
@@ -42,7 +42,7 @@
         <frameId>${prefix}_base_link</frameId>
         <topicName>gps/fix</topicName>
-        <!-- Robotnik position at Fuente del Jarro -->
-        <referenceLatitude>39.5080331</referenceLatitude>
-        <referenceLongitude>-0.4619816</referenceLongitude>
+        <!-- GPS coordinates -->
+        <referenceLatitude>${gps_latitude}</referenceLatitude>
+        <referenceLongitude>${gps_longitude}</referenceLongitude>
         <!-- To set heading in ENU orientation (degrees) -->
         <referenceHeading>90</referenceHeading>

File: urdf/gps_with_mast.urdf.xacro (robot description, xacro)
@@ -3,5 +3,5 @@
   <xacro:property name="mast_height" value="0.5" />
   <xacro:property name="mast_radius" value="0.010" />
-  <xacro:macro name="sensor_gps_with_mast" params="prefix parent *origin">
+  <xacro:macro name="sensor_gps_with_mast" params="prefix parent *origin gps_latitude:=^|0.0 gps_longitude:=^|0.0">
 	  <!-- MAST OF THE ANTENNA GPS -->
 	  <joint name="${prefix}_joint" type="fixed">
@@ -77,7 +77,7 @@
         <frameId>${prefix}_link</frameId>   <!-- which frame_id would be on the published message -->
         <topicName>fix</topicName>
-        <!-- Robotnik position at Fuente del Jarro -->
-        <referenceLatitude>39.5080331</referenceLatitude>
-        <referenceLongitude>-0.4619816</referenceLongitude>
+        <!-- GPS coordinates -->
+        <referenceLatitude>${gps_latitude}</referenceLatitude>
+        <referenceLongitude>${gps_longitude}</referenceLongitude>
         <!-- To set heading in ENU orientation (degrees) -->
         <referenceHeading>90</referenceHeading>

Commit message: default coordinates for gps at fuente del jarro

File: urdf/gps.urdf.xacro (robot description, xacro)
@@ -1,5 +1,6 @@
 <?xml version="1.0"?>
 <robot name="sensor_gps" xmlns:xacro="http://wiki.ros.org/xacro">
-  <xacro:macro name="sensor_gps" params="prefix parent *origin gps_latitude:=^|0.0 gps_longitude:=^|0.0">
+  <!-- if no latitude/longitud is specified, then use Fuente del Jarro as default -->
+  <xacro:macro name="sensor_gps" params="prefix parent *origin gps_latitude:=^|39.5080331 gps_longitude:=^|-0.4619816">
 	  <!-- ANTENNA GPS -->
 	  <joint name="${prefix}_joint" type="fixed">

File: urdf/gps_with_mast.urdf.xacro (robot description, xacro)
@@ -3,5 +3,6 @@
   <xacro:property name="mast_height" value="0.5" />
   <xacro:property name="mast_radius" value="0.010" />
-  <xacro:macro name="sensor_gps_with_mast" params="prefix parent *origin gps_latitude:=^|0.0 gps_longitude:=^|0.0">
+  <!-- if no latitude/longitud is specified, then use Fuente del Jarro as default -->
+  <xacro:macro name="sensor_gps_with_mast" params="prefix parent *origin gps_latitude:=^|39.5080331 gps_longitude:=^|-0.4619816">
 	  <!-- MAST OF THE ANTENNA GPS -->
 	  <joint name="${prefix}_joint" type="fixed">

Commit message: added param to change the update_rate

File: urdf/gps.urdf.xacro (robot description, xacro)
@@ -2,5 +2,5 @@
 <robot name="sensor_gps" xmlns:xacro="http://wiki.ros.org/xacro">
   <!-- if no latitude/longitud is specified, then use Fuente del Jarro as default -->
-  <xacro:macro name="sensor_gps" params="prefix parent *origin gps_latitude:=^|39.5080331 gps_longitude:=^|-0.4619816">
+  <xacro:macro name="sensor_gps" params="prefix parent *origin gps_latitude:=^|39.5080331 gps_longitude:=^|-0.4619816 update_rate:=^|5">
 	  <!-- ANTENNA GPS -->
 	  <joint name="${prefix}_joint" type="fixed">
@@ -39,5 +39,5 @@
       <plugin name="${prefix}_controller" filename="libhector_gazebo_ros_gps.so">
         <alwaysOn>1</alwaysOn>
-        <updateRate>5</updateRate>
+        <updateRate>${update_rate}</updateRate>
         <bodyName>${prefix}_base_link</bodyName> <!-- must be the link of the gps device, not the base_link or base_footprint -->
         <frameId>${prefix}_base_link</frameId>

Commit message: Update gps inertia

File: urdf/gps.urdf.xacro (robot description, xacro)
@@ -11,9 +11,9 @@
 	  </joint>
 	  <link name="${prefix}_base_link">
-	    <inertial>
-	      <mass value="0.001"/>
-	      <origin rpy="0 0 0" xyz="0 0 0"/>
-	      <inertia ixx="0.0001" ixy="0" ixz="0" iyy="0.000001" iyz="0" izz="0.0001"/>
-	    </inertial>
+		<inertial>
+			<origin xyz="0.0 0 0.015" rpy="0 0 0" />
+			<mass value="0.2" />
+			<xacro:solid_cuboid_inertia m="0.2" w="0.081" h="0.081" d="0.03" />
+      </inertial>
 	    <visual>
 	      <origin rpy="0 0 0" xyz="0 0 0"/>

Commit message: urdf/gps: link frame fixed

File: urdf/gps.urdf.xacro (robot description, xacro)
@@ -8,7 +8,7 @@
 	    <xacro:insert_block name="origin"/>
 	    <parent link="${parent}"/>
-	    <child link="${prefix}_base_link"/>
+	    <child link="${prefix}_link"/>
 	  </joint>
-	  <link name="${prefix}_base_link">
+	  <link name="${prefix}_link">
 		<inertial>
 			<origin xyz="0.0 0 0.015" rpy="0 0 0" />
@@ -32,5 +32,5 @@
 	    </collision>
 	  </link>
-	  <gazebo reference="${prefix}_base_link">
+	  <gazebo reference="${prefix}_link">
 	    <material>Gazebo/White</material>
 	    <gravity>true</gravity>
@@ -40,6 +40,6 @@
         <alwaysOn>1</alwaysOn>
         <updateRate>${update_rate}</updateRate>
-        <bodyName>${prefix}_base_link</bodyName> <!-- must be the link of the gps device, not the base_link or base_footprint -->
-        <frameId>${prefix}_base_link</frameId>
+        <bodyName>${prefix}_link</bodyName>
+        <frameId>${prefix}_link</frameId>
         <topicName>gps/fix</topicName>
         <!-- GPS coordinates -->
