Commit message: Refactor GPS sensor URDF to remove latitude/longitude parameters and enhance Gazebo integration

File: urdf/gps.urdf.xacro (robot description, xacro)
@@ -1,64 +1,92 @@
 <?xml version="1.0"?>
 <robot name="sensor_gps" xmlns:xacro="http://wiki.ros.org/xacro">
-  <!-- if no latitude/longitud is specified, then use Fuente del Jarro as default -->
-  <xacro:macro name="sensor_gps" params="prefix parent *origin gps_latitude:=^|39.5080331 gps_longitude:=^|-0.4619816 update_rate:=^|5 include_inertial:=^|true">
-	  <!-- ANTENNA GPS -->
-	  <joint name="${prefix}_joint" type="fixed">
-	    <axis xyz="0 1 0"/>
-	    <xacro:insert_block name="origin"/>
-	    <parent link="${parent}"/>
-	    <child link="${prefix}_base_link"/>
-	  </joint>
-	  <link name="${prefix}_base_link">
-		<xacro:if value="${include_inertial}">
-			<inertial>
-				<origin xyz="0.0 0 0.015" rpy="0 0 0" />
-				<mass value="0.2" />
-				<xacro:solid_cuboid_inertia m="0.2" w="0.081" h="0.081" d="0.03" />
-      		</inertial>
-	  	</xacro:if>
-	    <visual>
-	      <origin rpy="0 0 0" xyz="0 0 0"/>
-	      <material name="gps_color">
-           <color rgba="1 1 1 1"/>
+  <!-- Note: gps_latitude/longitude are NOT needed anymore; world defines WGS84 origin -->
+  <xacro:macro name="sensor_gps" params="prefix parent *origin update_rate:=^|5 include_inertial:=^|true frame_id:=^|${prefix}_base_link topic_ns:=^|gps">
+    <!-- ANTENNA GPS -->
+    <joint name="${prefix}_joint" type="fixed">
+      <axis xyz="0 1 0"/>
+      <xacro:insert_block name="origin"/>
+      <parent link="${parent}"/>
+      <child link="${prefix}_base_link"/>
+    </joint>
+    <link name="${prefix}_base_link">
+      <xacro:if value="${include_inertial}">
+        <inertial>
+          <origin xyz="0.0 0 0.015" rpy="0 0 0" />
+          <mass value="0.2" />
+          <xacro:solid_cuboid_inertia m="0.2" w="0.081" h="0.081" d="0.03" />
+        </inertial>
+      </xacro:if>
+      <visual>
+        <origin rpy="0 0 0" xyz="0 0 0"/>
+        <material name="gps_color">
+          <color rgba="1 1 1 1"/>
         </material>
-	      <geometry>
-	        <mesh filename="package://robotnik_sensors/meshes/antenna_3GO16.stl" scale="1.0 1.0 1.0"/>
-	      </geometry>
-	    </visual>
-	    <collision>
-	      <origin rpy="0 0 0" xyz="0 0 0"/>
-	      <geometry>
-	        <mesh filename="package://robotnik_sensors/meshes/antenna_3GO16.stl" scale="1.0 1.0 1.0"/>
-	      </geometry>
-	    </collision>
-	  </link>
-	  <gazebo reference="${prefix}_base_link">
-	    <material>Gazebo/White</material>
-	    <gravity>true</gravity>
-	  </gazebo>
-    <gazebo>
-      <plugin name="${prefix}_controller" filename="libhector_gazebo_ros_gps.so">
-        <alwaysOn>1</alwaysOn>
-        <updateRate>${update_rate}</updateRate>
-        <bodyName>${prefix}_base_link</bodyName> <!-- must be the link of the gps device, not the base_link or base_footprint -->
-        <frameId>${prefix}_base_link</frameId>
-        <topicName>gps/fix</topicName>
-        <!-- GPS coordinates -->
-        <referenceLatitude>${gps_latitude}</referenceLatitude>
-        <referenceLongitude>${gps_longitude}</referenceLongitude>
-        <!-- To set heading in ENU orientation (degrees) -->
-        <referenceHeading>90</referenceHeading>
-        <velocityTopicName>gps/fix_velocity</velocityTopicName>
-        <drift>0.0 0.0 0.0</drift>
-        <!--<drift>0.0001 0.0001 0.0001</drift>-->
-        <!--<drift>0.3 0.3 0.3</drift>-->
-        <gaussianNoise>0.00001 0.00001 0.00001</gaussianNoise>
-        <!--<gaussianNoise>0.00001 0.00001 0.00001</gaussianNoise>-->
-        <velocityDrift>0.00001 0.00001 0.00001</velocityDrift>
-        <!--<velocityGaussianNoise>0.1 0.1 0.1</velocityGaussianNoise>-->
-        <velocityGaussianNoise>0.00001 0.00001 0.00001</velocityGaussianNoise>
-      </plugin>
-	</gazebo>
+        <geometry>
+          <mesh filename="package://robotnik_sensors/meshes/antenna_3GO16.stl" scale="1.0 1.0 1.0"/>
+        </geometry>
+      </visual>
+      <collision>
+        <origin rpy="0 0 0" xyz="0 0 0"/>
+        <geometry>
+          <mesh filename="package://robotnik_sensors/meshes/antenna_3GO16.stl" scale="1.0 1.0 1.0"/>
+        </geometry>
+      </collision>
+    </link>
+    <!-- Gazebo visuals/physics for the link -->
+    <gazebo reference="${prefix}_base_link">
+      <material>Gazebo/White</material>
+      <gravity>true</gravity>
+    </gazebo>
+    <!-- Native Gazebo GPS sensor + ROS bridge -->
+    <gazebo reference="${prefix}_base_link">
+      <sensor name="${prefix}_gps" type="gps">
+        <always_on>true</always_on>
+        <update_rate>${update_rate}</update_rate>
+        <!-- Native GPS noise model; tune to your needs -->
+        <gps>
+          <position_sensing>
+            <horizontal>
+              <noise type="gaussian">
+                <mean>0.0</mean>
+                <stddev>0.05</stddev> <!-- ~0.05 m horiz -->
+              </noise>
+            </horizontal>
+            <vertical>
+              <noise type="gaussian">
+                <mean>0.0</mean>
+                <stddev>0.05</stddev> <!-- ~0.05 m vert -->
+              </noise>
+            </vertical>
+          </position_sensing>
+          <velocity_sensing>
+            <horizontal>
+              <noise type="gaussian">
+                <mean>0.0</mean>
+                <stddev>0.01</stddev>
+              </noise>
+            </horizontal>
+            <vertical>
+              <noise type="gaussian">
+                <mean>0.0</mean>
+                <stddev>0.02</stddev>
+              </noise>
+            </vertical>
+          </velocity_sensing>
+        </gps>
+        <!-- ROS bridge: publishes NavSatFix (+ optional velocity) -->
+        <plugin name="${prefix}_ros_gps" filename="libgazebo_ros_gps.so">
+          <!-- Namespace is optional; leave '/' for absolute topics or set a relative ns -->
+          <ros>
+            <namespace>/</namespace>
+          </ros>
+          <!-- Frame id used in published messages -->
+          <frame_name>${frame_id}</frame_name>
+          <!-- Topics: you can remap at launch if needed -->
+          <topic_name>${topic_ns}/fix</topic_name>
+          <velocity_topic_name>${topic_ns}/fix_velocity</velocity_topic_name>
+        </plugin>
+      </sensor>
+    </gazebo>
   </xacro:macro>
 </robot>

File: urdf/gps_with_mast.urdf.xacro (robot description, xacro)
@@ -3,99 +3,127 @@
   <xacro:property name="mast_height" value="0.5" />
   <xacro:property name="mast_radius" value="0.010" />
-  <!-- if no latitude/longitud is specified, then use Fuente del Jarro as default -->
-  <xacro:macro name="sensor_gps_with_mast" params="prefix parent *origin gps_latitude:=^|39.5080331 gps_longitude:=^|-0.4619816 update_rate:=^|5 include_inertial:=^|true">
-	  <!-- MAST OF THE ANTENNA GPS -->
-	  <joint name="${prefix}_joint" type="fixed">
-	    <axis xyz="0 1 0"/>
-	    <xacro:insert_block name="origin"/>
-	    <parent link="${parent}"/>
-	    <child link="${prefix}_mast_base_link"/>
-	  </joint>
-	  <link name="${prefix}_mast_base_link">
-		<xacro:if value="${include_inertial}">
-			<inertial>
-				<origin xyz="0.0 0 0.0" rpy="0 0 0" />
-				<mass value="1.0" />
-				<xacro:solid_cuboid_inertia m="1.0" w="${mast_radius}" h="${mast_radius}" d="${mast_height}" />
-			</inertial>
-	  	</xacro:if>
-	    <visual>
-	      <origin rpy="0 0 0" xyz="0 0 0"/>
-	      <material name="mast_color">
-            <color rgba="0.1 0.1 0.1 1"/>
-          </material>
-	      <geometry>
-	        <cylinder length="${mast_height}" radius="${mast_radius}" />
-	      </geometry>
-	    </visual>
-	    <collision>
-	      <origin rpy="0 0 0" xyz="0 0 0"/>
-	      <geometry>
-	        <cylinder length="${mast_height}" radius="${mast_radius}" />
-	      </geometry>
-	    </collision>
-	  </link>
-	  <joint name="${prefix}_mast_joint" type="fixed">
-	    <axis xyz="0 1 0"/>
-	    <parent link="${prefix}_mast_base_link"/>
-	    <child link="${prefix}_base_link"/>
-	    <origin xyz="0 0 ${mast_height/2.0}" rpy="0 0 0" />
-	  </joint>
-	  <gazebo reference="${prefix}_mast_base_link">
-	    <material>Gazebo/Black</material>
-	    <gravity>true</gravity>
-	  </gazebo>
-      <!-- ANTENNA GPS -->
-	  <link name="${prefix}_base_link">
-		<xacro:if value="${include_inertial}">
-	    	<inertial>
-				<origin xyz="0.0 0 0.015" rpy="0 0 0" />
-				<mass value="0.2" />
-				<xacro:solid_cuboid_inertia m="0.2" w="0.081" h="0.081" d="0.03" />
-      		</inertial>
-		</xacro:if>
-	    <visual>
-	      <origin rpy="0 0 0" xyz="0 0 0"/>
-	      <material name="gps_color">
-           <color rgba="1 1 1 1"/>
+  <!-- English code, with English comments -->
+  <!-- NOTE: world provides spherical_coordinates (WGS84), so no per-sensor reference lat/lon needed -->
+  <xacro:macro name="sensor_gps_with_mast" params="prefix parent *origin update_rate:=^|5 include_inertial:=^|true frame_id:=^|${prefix}_base_link topic_ns:=^|gps">
+    <!-- Fixed joint from parent to mast base -->
+    <joint name="${prefix}_joint" type="fixed">
+      <axis xyz="0 1 0"/>
+      <xacro:insert_block name="origin"/>
+      <parent link="${parent}"/>
+      <child link="${prefix}_mast_base_link"/>
+    </joint>
+    <!-- Mast base link -->
+    <link name="${prefix}_mast_base_link">
+      <xacro:if value="${include_inertial}">
+        <inertial>
+          <origin xyz="0.0 0 0.0" rpy="0 0 0" />
+          <mass value="1.0" />
+          <xacro:solid_cuboid_inertia m="1.0" w="${mast_radius}" h="${mast_radius}" d="${mast_height}" />
+        </inertial>
+      </xacro:if>
+      <visual>
+        <origin rpy="0 0 0" xyz="0 0 0"/>
+        <material name="mast_color">
+          <color rgba="0.1 0.1 0.1 1"/>
         </material>
-	      <geometry>
-	        <mesh filename="package://robotnik_sensors/meshes/antenna_3GO16.stl" scale="1.0 1.0 1.0"/>
-	      </geometry>
-	    </visual>
-	    <collision>
-	      <origin rpy="0 0 0" xyz="0 0 0"/>
-	      <geometry>
-	        <mesh filename="package://robotnik_sensors/meshes/antenna_3GO16.stl" scale="1.0 1.0 1.0"/>
-	      </geometry>
-	    </collision>
-	  </link>
-	  <gazebo reference="${prefix}_base_link">
-	    <material>Gazebo/White</material>
-	    <gravity>true</gravity>
-	  </gazebo>
-    <gazebo>
-      <plugin name="${prefix}_controller" filename="libhector_gazebo_ros_gps.so">
-        <alwaysOn>1</alwaysOn>
-        <updateRate>${update_rate}</updateRate>
-        <bodyName>${prefix}_base_link</bodyName> <!-- must be the link of the gps device, not the base_link or base_footprint -->
-        <frameId>${prefix}_base_link</frameId>   <!-- which frame_id would be on the published message -->
-        <topicName>gps/fix</topicName>
-        <!-- GPS coordinates -->
-        <referenceLatitude>${gps_latitude}</referenceLatitude>
-        <referenceLongitude>${gps_longitude}</referenceLongitude>
-        <!-- To set heading in ENU orientation (degrees) -->
-        <referenceHeading>90</referenceHeading>
-        <velocityTopicName>gps/fix_velocity</velocityTopicName>
-        <drift>0.0 0.0 0.0</drift>
-        <!--<drift>0.0001 0.0001 0.0001</drift>-->
-        <!--<drift>0.3 0.3 0.3</drift>-->
-        <gaussianNoise>0.00001 0.00001 0.00001</gaussianNoise>
-        <!--<gaussianNoise>0.00001 0.00001 0.00001</gaussianNoise>-->
-        <velocityDrift>0.00001 0.00001 0.00001</velocityDrift>
-        <!--<velocityGaussianNoise>0.1 0.1 0.1</velocityGaussianNoise>-->
-        <velocityGaussianNoise>0.00001 0.00001 0.00001</velocityGaussianNoise>
-      </plugin>
-	</gazebo>
+        <geometry>
+          <cylinder length="${mast_height}" radius="${mast_radius}" />
+        </geometry>
+      </visual>
+      <collision>
+        <origin rpy="0 0 0" xyz="0 0 0"/>
+        <geometry>
+          <cylinder length="${mast_height}" radius="${mast_radius}" />
+        </geometry>
+      </collision>
+    </link>
+    <!-- Joint to antenna link placed at mast top (z = mast_height/2) -->
+    <joint name="${prefix}_mast_joint" type="fixed">
+      <axis xyz="0 1 0"/>
+      <parent link="${prefix}_mast_base_link"/>
+      <child link="${prefix}_base_link"/>
+      <origin xyz="0 0 ${mast_height/2.0}" rpy="0 0 0" />
+    </joint>
+    <!-- Antenna (GPS) link -->
+    <link name="${prefix}_base_link">
+      <xacro:if value="${include_inertial}">
+        <inertial>
+          <origin xyz="0.0 0 0.015" rpy="0 0 0" />
+          <mass value="0.2" />
+          <xacro:solid_cuboid_inertia m="0.2" w="0.081" h="0.081" d="0.03" />
+        </inertial>
+      </xacro:if>
+      <visual>
+        <origin rpy="0 0 0" xyz="0 0 0"/>
+        <material name="gps_color">
+          <color rgba="1 1 1 1"/>
+        </material>
+        <geometry>
+          <mesh filename="package://robotnik_sensors/meshes/antenna_3GO16.stl" scale="1.0 1.0 1.0"/>
+        </geometry>
+      </visual>
+      <collision>
+        <origin rpy="0 0 0" xyz="0 0 0"/>
+        <geometry>
+          <mesh filename="package://robotnik_sensors/meshes/antenna_3GO16.stl" scale="1.0 1.0 1.0"/>
+        </geometry>
+      </collision>
+    </link>
+    <!-- Gazebo visuals/physics -->
+    <gazebo reference="${prefix}_mast_base_link">
+      <material>Gazebo/Black</material>
+      <gravity>true</gravity>
+    </gazebo>
+    <gazebo reference="${prefix}_base_link">
+      <material>Gazebo/White</material>
+      <gravity>true</gravity>
+    </gazebo>
+    <!-- Native Gazebo GPS sensor attached to the antenna link (at mast top) -->
+    <gazebo reference="${prefix}_base_link">
+      <sensor name="${prefix}_gps" type="gps">
+        <always_on>true</always_on>
+        <update_rate>${update_rate}</update_rate>
+        <!-- Noise model: tune as needed -->
+        <gps>
+          <position_sensing>
+            <horizontal>
+              <noise type="gaussian">
+                <mean>0.0</mean>
+                <stddev>0.05</stddev> <!-- ~0.05 m horiz -->
+              </noise>
+            </horizontal>
+            <vertical>
+              <noise type="gaussian">
+                <mean>0.0</mean>
+                <stddev>0.05</stddev> <!-- ~0.05 m vert -->
+              </noise>
+            </vertical>
+          </position_sensing>
+          <velocity_sensing>
+            <horizontal>
+              <noise type="gaussian">
+                <mean>0.0</mean>
+                <stddev>0.01</stddev>
+              </noise>
+            </horizontal>
+            <vertical>
+              <noise type="gaussian">
+                <mean>0.0</mean>
+                <stddev>0.02</stddev>
+              </noise>
+            </vertical>
+          </velocity_sensing>
+        </gps>
+        <!-- ROS bridge: publishes NavSatFix (+ velocity) using world spherical_coordinates -->
+        <plugin name="${prefix}_ros_gps" filename="libgazebo_ros_gps.so">
+          <ros>
+            <namespace>/</namespace> <!-- set to robot ns if needed -->
+          </ros>
+          <frame_name>${frame_id}</frame_name>
+          <topic_name>${topic_ns}/fix</topic_name>
+          <velocity_topic_name>${topic_ns}/fix_velocity</velocity_topic_name>
+        </plugin>
+      </sensor>
+    </gazebo>
   </xacro:macro>
 </robot>
