Commit message: fix typo in imu_joint

File: urdf/sick_multiscan.urdf.xacro (robot description, xacro)
@@ -43,5 +43,5 @@
     <link name="${prefix}_link_6"/> -->
     <!-- Relative position of the IMU to the optical origin (-17 mm, +23.5 mm, -30 mm) -->
-    <joint name="${prefix}imu_joint" type="fixed">
+    <joint name="${prefix}_imu_joint" type="fixed">
       <parent link="${prefix}_link"/>
       <child link="${prefix}_imu_link" />
