Commit message: added kinectv2 urdf (to be improved)

File: urdf/all_sensors.urdf.xacro (robot description, xacro)
@@ -22,3 +22,5 @@
   <!-- Hokuyo 3d -->
   <xacro:include filename="$(find robotnik_sensors)/urdf/hokuyo3d.urdf.xacro" />
+  <!-- KinectV2 -->
+  <xacro:include filename="$(find robotnik_sensors)/urdf/kinectv2.urdf.xacro" />
 </robot>

File: urdf/kinectv2.urdf.xacro (robot description, xacro)
@@ -1,4 +1,4 @@
 <?xml version="1.0"?>
-<robot name="sensor_kinect" xmlns:xacro="http://ros.org/wiki/xacro">
+<robot name="sensor_kinectv2" xmlns:xacro="http://ros.org/wiki/xacro">
   <xacro:property name="M_PI" value="3.1415926535897931" />
 	<xacro:property name="cam_px" value="-0.087" />
@@ -8,5 +8,5 @@
 	<xacro:property name="cam_op" value="0" />
 	<xacro:property name="cam_oy" value="0" />
-  <xacro:macro name="sensor_kinect" params="name parent *origin">
+  <xacro:macro name="sensor_kinectv2" params="name parent *origin">
     <joint name="${name}_rgb_joint" type="fixed">
       <insert_block name="origin" />
@@ -46,5 +46,5 @@
      <origin xyz="0 0 0" rpy="0 0 ${M_PI/2}"/>
       <geometry>
-       <mesh filename="package://robotnik_sensors/meshes/sensors/kinectv2.dae"/>
+       <mesh filename="package://robotnik_sensors/meshes/kinectv2.dae"/>
       </geometry>
     </visual>
@@ -95,7 +95,7 @@
 	</link>
 		<!-- Kinect sensor for simulation -->
-	  <sensor_kinect_gazebo/>
+	  <sensor_kinectv2_gazebo/>
   </xacro:macro>
-  <xacro:macro name="sensor_kinect_gazebo">
+  <xacro:macro name="sensor_kinectv2_gazebo">
     <gazebo reference="${name}_link">
       <sensor type="depth" name="cam">

Commit message: sensors updated to multirobot

File: urdf/all_sensors.urdf.xacro (robot description, xacro)
@@ -32,4 +32,6 @@
   <!-- KinectV2 -->
   <xacro:include filename="$(find robotnik_sensors)/urdf/kinectv2.urdf.xacro" />
+  <!-- Sick Tim 551 -->
+  <xacro:include filename="$(find robotnik_sensors)/urdf/sick_tim551.urdf.xacro" />
   <!-- Sick Tim 571 -->
   <xacro:include filename="$(find robotnik_sensors)/urdf/sick_tim571.urdf.xacro" />
@@ -38,4 +40,6 @@
   <!-- Rplidar -->
   <xacro:include filename="$(find robotnik_sensors)/urdf/rplidar.urdf.xacro" />
+  <!-- Rplidar A2 -->
+  <xacro:include filename="$(find robotnik_sensors)/urdf/rplidar_a2.urdf.xacro" />
   <!-- uEye CP Gige -->
   <xacro:include filename="$(find robotnik_sensors)/urdf/ueye_cp_gige.urdf.xacro" />

File: urdf/hokuyo_urg04lx.urdf.xacro (robot description, xacro)
@@ -34,6 +34,6 @@
   </xacro:macro>
   <xacro:macro name="sensor_hokuyo_urg_gazebo">
-    <gazebo reference="${name}_link">
-			<sensor type="ray" name="${name}_sensor">
+    <gazebo reference="${prefix_frame}${name}_link">
+			<sensor type="ray" name="${prefix_frame}${name}_sensor">
 				<pose>0 0 0 0 0 0</pose>
 				<visualize>false</visualize>
@@ -60,6 +60,7 @@
 				</ray>
 				<plugin name="${name}_controller" filename="libgazebo_ros_laser.so">
-					<topicName>${prefix_topic}${name}/scan</topicName>
+					<topicName>${prefix_topic}scan</topicName>
 					<frameName>${prefix_frame}_${name}_link</frameName>
+					<ignoreTfPrefix>1</ignoreTfPrefix>
 				</plugin>
 			</sensor>

File: urdf/hokuyo_ust10lx.urdf.xacro (robot description, xacro)
@@ -1,12 +1,12 @@
 <?xml version="1.0"?>
 <robot name="sensor_hokuyo_ust10lx" xmlns:xacro="http://www.ros.org/wiki/xacro">
-  <xacro:macro name="sensor_hokuyo_ust10lx" params="prefix_frame prefix_topic parent *origin min_angle:=-2.3562 max_angle:=2.3562">
+  <xacro:macro name="sensor_hokuyo_ust10lx" params="name prefix_frame prefix_topic parent *origin min_angle:=-2.3562 max_angle:=2.3562">
 			<!--arg name="namespace" value="$(arg namespace)"/-->
-    <joint name="${prefix_frame}_joint" type="fixed">
+    <joint name="${name}_joint" type="fixed">
       <xacro:insert_block name="origin" />
       <parent link="${parent}"/>
-      <child link="${prefix_frame}_link"/>
+      <child link="${prefix_frame}${name}_link"/>
     </joint>
-    <link name="${prefix_frame}_link">
+    <link name="${prefix_frame}${name}_link">
       <collision>
         <origin xyz="0 0 -0.05" rpy="0 0 0"/>
@@ -28,9 +28,9 @@
     </link>
     <!-- Hokuyo sensor for simulation -->
-    <sensor_hokuyo_ust_gazebo/>
+    <xacro:sensor_hokuyo_ust_gazebo/>
   </xacro:macro>
   <xacro:macro name="sensor_hokuyo_ust_gazebo">
-    <gazebo reference="${prefix_frame}_link">
-			<sensor type="ray" name="${prefix_frame}_sensor">
+    <gazebo reference="${prefix_frame}${name}_link">
+			<sensor type="ray" name="${prefix_frame}${name}_sensor">
 				<pose>0 0 0 0 0 0</pose>
 				<visualize>false</visualize>
@@ -58,7 +58,7 @@
 					</noise>
 				</ray>
-				<plugin name="${prefix_frame}_controller" filename="libgazebo_ros_laser.so">
-					<topicName>${prefix_topic}hokuyo_base/scan</topicName>
-					<frameName>${prefix_frame}_${name}_link</frameName>
+				<plugin name="${prefix_frame}${name}_controller" filename="libgazebo_ros_laser.so">
+					<topicName>${prefix_topic}scan</topicName>
+					<frameName>${prefix_frame}${name}_link</frameName>
 					<ignoreTfPrefix>1</ignoreTfPrefix>
 				</plugin>

File: urdf/imu.urdf.xacro (robot description, xacro)
@@ -7,7 +7,7 @@
 	      <xacro:insert_block name="origin"/>
 	      <parent link="${parent}"/>
-	      <child link="${prefix_frame}_link"/>
+	      <child link="${prefix_frame}${name}_link"/>
 	  </joint>
-	  <link name="${name}_link">
+	  <link name="${prefix_frame}${name}_link">
 	      <inertial>
 	        <mass value="0.001"/>
@@ -29,8 +29,8 @@
 	  </link>
 	  <gazebo>
-	    <plugin name="${name}_controller" filename="libgazebo_ros_imu.so">
+	    <plugin name="${prefix_frame}${name}_controller" filename="libgazebo_ros_imu.so">
 	       <topicName>${prefix_topic}data</topicName>
 		   <serviceName>${prefix_topic}service</serviceName>
-		   <bodyName>${prefix_frame}_link</bodyName>
+		   <bodyName>${prefix_frame}${name}_link</bodyName>
 	       <gaussianNoise>0.005</gaussianNoise>
 	    </plugin>

File: urdf/orbbec_astra.urdf.xacro (robot description, xacro)
@@ -17,7 +17,7 @@
 	  <xacro:insert_block name="origin" />
       <parent link="${parent}"/>
-      <child link="${name}_rgb_frame" />
+      <child link="${prefix_frame}${name}_rgb_frame_link" />
     </joint>
-    <link name="${name}_rgb_frame">
+    <link name="${prefix_frame}${name}_rgb_frame_link">
       <inertial>
         <mass value="0.001" />
@@ -30,8 +30,8 @@
     <joint name="${name}_rgb_optical_joint" type="fixed">
       <origin xyz="0.0 0.0 0.0" rpy="${-M_PI/2} 0 ${-M_PI/2}" />
-      <parent link="${name}_rgb_frame" />
-      <child link="${name}_rgb_optical_frame" />
+      <parent link="${prefix_frame}${name}_rgb_frame_link" />
+      <child link="${prefix_frame}${name}_rgb_optical_frame_link" />
     </joint>
-    <link name="${name}_rgb_optical_frame">
+    <link name="${prefix_frame}${name}_rgb_optical_frame_link">
       <!--inertial>
         <mass value="0.001" />
@@ -45,8 +45,8 @@
       <origin xyz="${orbbec_astra_rel_rgb_px} ${orbbec_astra_rel_rgb_py} ${orbbec_astra_rel_rgb_pz}"
               rpy="0.0 0 0"/>
-      <parent link="${name}_rgb_frame"/>
-      <child link="${name}_link"/>
+      <parent link="${prefix_frame}${name}_rgb_frame_link"/>
+      <child link="${prefix_frame}${name}_link"/>
     </joint>
-    <link name="${name}_link">
+    <link name="${prefix_frame}${name}_link">
       <visual>
         <origin xyz="0 0 0" rpy="0 0 0"/>
@@ -76,8 +76,8 @@
     <joint name="${name}_depth_joint" type="fixed">
       <origin xyz="${orbbec_astra_depth_rel_rgb_px} ${orbbec_astra_depth_rel_rgb_py} ${orbbec_astra_depth_rel_rgb_pz}" rpy="0 0 0" />
-      <parent link="${name}_rgb_frame" />
-      <child link="${name}_depth_frame" />
+      <parent link="${prefix_frame}${name}_rgb_frame_link" />
+      <child link="${prefix_frame}${name}_depth_frame_link" />
     </joint>
-    <link name="${name}_depth_frame">
+    <link name="${prefix_frame}${name}_depth_frame_link">
       <!--inertial>
         <mass value="0.01" />
@@ -90,8 +90,8 @@
     <joint name="${name}_depth_optical_joint" type="fixed">
       <origin xyz="0 0 0" rpy="${-M_PI/2} 0 ${-M_PI/2}" />
-      <parent link="${name}_depth_frame" />
-      <child link="${name}_depth_optical_frame" />
+      <parent link="${prefix_frame}${name}_depth_frame_link" />
+      <child link="${prefix_frame}${name}_depth_optical_frame_link" />
     </joint>
-    <link name="${name}_depth_optical_frame">
+    <link name="${prefix_frame}${name}_depth_optical_frame_link">
       <!--inertial>
         <mass value="0.001" />
@@ -106,5 +106,5 @@
   </xacro:macro>
    <xacro:macro name="sensor_orbbec_astra_gazebo">
-    <gazebo reference="${name}_link">
+    <gazebo reference="${prefix_frame}${name}_rgb_frame_link">
       <sensor type="depth" name="${name}">
         <always_on>true</always_on>
@@ -131,5 +131,5 @@
           <cameraInfoTopicName>${prefix_topic}rgb/camera_info</cameraInfoTopicName>
           <depthImageCameraInfoTopicName>${prefix_topic}depth/camera_info</depthImageCameraInfoTopicName>
-          <frameName>${prefix_frame}_${name}_depth_optical_frame</frameName>
+          <frameName>${prefix_frame}${name}_depth_optical_frame_link</frameName>
           <baseline>0.1</baseline>
           <distortion_k1>0.0</distortion_k1>
@@ -139,4 +139,5 @@
           <distortion_t2>0.0</distortion_t2>
           <pointCloudCutoff>0.4</pointCloudCutoff>
+          <ignoreTfPrefix>1</ignoreTfPrefix>
         </plugin>
       </sensor>

File: urdf/rplidar.urdf.xacro (robot description, xacro)
@@ -5,7 +5,7 @@
       <xacro:insert_block name="origin" />
       <parent link="${parent}"/>
-      <child link="${name}_laser_base_link"/>
+      <child link="${prefix_frame}${name}_laser_base_link"/>
     </joint>
-    <link name="${name}_laser_base_link">
+    <link name="${prefix_frame}${name}_laser_base_link">
       <collision>
         <origin xyz="0 0 0" rpy="0 0 0"/>
@@ -28,14 +28,14 @@
     <joint name="${name}_laser_joint" type="fixed">
       <origin xyz="0 0 0.0461" rpy="0 0 0"/>
-      <parent link="${name}_laser_base_link"/>
-      <child link="${name}_laser_link"/>
+      <parent link="${prefix_frame}${name}_laser_base_link"/>
+      <child link="${prefix_frame}${name}_laser_link"/>
     </joint>
-    <link name="${name}_laser_link">
+    <link name="${prefix_frame}${name}_laser_link">
     </link>
     <sensor_rplidar_gazebo/>
   </xacro:macro>
   <xacro:macro name="sensor_rplidar_gazebo">
-    <gazebo reference="${name}_laser_link">
-			<sensor type="ray" name="${name}_rplidar_sensor">
+    <gazebo reference="${prefix_frame}${name}_laser_link">
+			<sensor type="ray" name="${prefix_frame}${name}_rplidar_sensor">
 				<pose>0 0 0 0 0 0</pose>
 				<visualize>false</visualize>
@@ -62,6 +62,7 @@
 				</ray>
 				<plugin name="gazebo_ros_rplidar_controller" filename="libgazebo_ros_laser.so">
-					<topicName>${prefix_topic}${name}/scan</topicName>
-					<frameName>${prefix_frame}_${name}_laser_link</frameName>
+					<topicName>${prefix_topic}scan</topicName>
+					<frameName>${prefix_frame}${name}_laser_link</frameName>
+					<ignoreTfPrefix>1</ignoreTfPrefix>
 				</plugin>
 			</sensor>

File: urdf/sick_s3000.urdf.xacro (robot description, xacro)
@@ -56,6 +56,7 @@
 				</ray>
 				<plugin name="${name}_controller" filename="libgazebo_ros_laser.so">
-					<topicName>${prefix_topic}${name}/scan</topicName>
+					<topicName>${prefix_topic}scan</topicName>
 					<frameName>${prefix_frame}_${name}_link</frameName>
+					<ignoreTfPrefix>1</ignoreTfPrefix>
 				</plugin>
 			</sensor>

File: urdf/sick_tim571.urdf.xacro (robot description, xacro)
@@ -36,6 +36,6 @@
   </xacro:macro>
   <xacro:macro name="sensor_sick_tim571_gazebo">
-    <gazebo reference="${name}_link">
-			<sensor type="ray" name="${name}_sensor">
+	<gazebo reference="${prefix_frame}${name}_link">
+			<sensor type="ray" name="${prefix_frame}${name}_sensor">
 				<pose>0 0 0 0 0 0</pose>
 				<visualize>false</visualize>
@@ -61,7 +61,8 @@
 					</noise>
 				</ray>
-				<plugin name="${name}_controller" filename="libgazebo_ros_laser.so">
-					<topicName>${prefix_topic}${name}/scan</topicName>
-					<frameName>${prefix_frame}_${name}_link</frameName>
+				<plugin name="${prefix_frame}${name}_controller" filename="libgazebo_ros_laser.so">
+					<topicName>${prefix_topic}scan</topicName>
+					<frameName>${prefix_frame}${name}_link</frameName>
+					<ignoreTfPrefix>1</ignoreTfPrefix>
 				</plugin>
 			</sensor>

Commit message: added benewake models

File: urdf/all_sensors.urdf.xacro (robot description, xacro)
@@ -66,4 +66,8 @@
   <!-- Benewake CE-30s -->
   <xacro:include filename="$(find robotnik_sensors)/urdf/benewake_ce30s.urdf.xacro" />
+  <!-- Benewake CE-30c -->
+  <xacro:include filename="$(find robotnik_sensors)/urdf/benewake_ce30c.urdf.xacro" />
+  <!-- Benewake CE-30d -->
+  <xacro:include filename="$(find robotnik_sensors)/urdf/benewake_ce30d.urdf.xacro" />
   <!-- Rubedos Viper -->
   <xacro:include filename="$(find robotnik_sensors)/urdf/rubedos_viper.urdf.xacro" />

File: urdf/benewake_ce30s.urdf.xacro (robot description, xacro)
@@ -54,4 +54,102 @@
 	    </inertial>
 	  </link>
+    <sensor_ce30s_gazebo/>
   </xacro:macro>
+ <xacro:macro name="sensor_ce30s_gazebo">
+    <!-- Gazebo requires the velodyne_gazebo_plugins package -->
+    <gazebo reference="${prefix}_link">
+      <sensor type="ray" name="${prefix}_sensor">
+          <pose>0 0 0 0 0 0.0</pose>
+          <visualize>false</visualize>
+          <update_rate>20.0</update_rate>
+          <ray>
+            <scan>
+              <horizontal>
+				<!-- for a high quality simulation -->
+                <samples>320</samples>
+                <!-- Configuration for the ROS ce30s ros driver as provided by Benewake, with sensor front axis being y -->
+                <!-- min_angle>-${132/2.0*M_PI/180.0-M_PI/2.0}</min_angle>
+                <max_angle>${132/2.0*M_PI/180.0+M_PI/2.0}</max_angle -->
+				<!-- Configuration for modified ce30s ros driver x2=y1 y2=-x1 -->
+                <min_angle>-${132/2.0*M_PI/180.0}</min_angle>
+                <max_angle>${132/2.0*M_PI/180.0}</max_angle>
+                <!-- samples>132</samples>
+                <resolution>1</resolution>
+                <min_angle>-1.15192</min_angle>
+                <max_angle>1.15192</max_angle -->
+              </horizontal>
+              <vertical>
+                <!-- samples>24</samples -->
+                <!-- min_angle>-${9.0/2.0*M_PI/180.0}</min_angle>
+                <max_angle> ${9.0/2.0*M_PI/180.0}</max_angle -->
+                <samples>10</samples>
+                <resolution>1</resolution>
+                <min_angle>-0.07854</min_angle>
+                <max_angle>0.07854</max_angle>
+              </vertical>
+            </scan>
+            <range>
+              <min>0.3</min>
+              <max>4.5</max>
+              <resolution>0.01</resolution>
+            </range>
+            <noise>
+              <type>gaussian</type>
+              <mean>0.0</mean>
+              <stddev>0.0</stddev>
+            </noise>
+          </ray>
+          <plugin name="gazebo_ros_laser_controller" filename="libgazebo_ros_block_laser2.so">
+            <topicName>ce30s_output</topicName>
+            <frameName>ce30s</frameName>
+            <min_range>0.3</min_range>
+            <max_range>5.0</max_range>
+            <gaussianNoise>0.008</gaussianNoise>
+          </plugin>
+        </sensor>
+		<!--<sensor type="depth" name="${prefix}_depth_sensor">-->
+		  <!--<update_rate>30.0</update_rate>-->
+		  <!--<camera name="fotonic">-->
+			<!--<horizontal_fov>1.221730476</horizontal_fov>  [> 70 deg <]-->
+			<!--<image>-->
+			  <!--<width>160</width>  [> 160 <]-->
+			  <!--<height>120</height> [> 120 <]-->
+			  <!--<format>L8</format> [> gray <]-->
+			<!--</image>-->
+			<!--<clip>-->
+			  <!--<near>0.05</near>-->
+			  <!--<far>7.0</far>         [> outdoor down to 3m depending on luminosity <]-->
+			<!--</clip>-->
+			<!--<noise>-->
+			  <!--<type>gaussian</type>-->
+			  <!--<mean>0.0</mean>-->
+			  <!--<stddev>0.007</stddev>-->
+			<!--</noise>-->
+		  <!--</camera>-->
+			<!--<plugin name="${prefix}_controller" filename="libgazebo_ros_openni_kinect.so">-->
+					<!--<alwaysOn>true</alwaysOn>-->
+					<!--<updateRate>10.0</updateRate>-->
+					<!--<cameraName>${prefix}</cameraName>-->
+					<!--<imageTopicName>ir/image_raw</imageTopicName>-->
+					<!--<cameraInfoTopicName>ir/camera_info</cameraInfoTopicName>-->
+					<!--<depthImageTopicName>depth/image_raw</depthImageTopicName>-->
+					<!--<depthImageCameraInfoTopicName>depth/camera_info</depthImageCameraInfoTopicName>-->
+					<!--<pointCloudTopicName>points</pointCloudTopicName>-->
+					<!--<frameName>${prefix}_depth_optical_frame_link</frameName>-->
+					<!--<pointCloudCutoff>0.5</pointCloudCutoff>-->
+					<!--<distortionK1>0</distortionK1>-->
+					<!--<distortionK2>0</distortionK2>-->
+					<!--<distortionK3>0</distortionK3>-->
+					<!--<distortionT1>0</distortionT1>-->
+					<!--<distortionT2>0</distortionT2>-->
+					<!--<CxPrime>0</CxPrime>-->
+					<!--<Cx>0</Cx>-->
+					<!--<Cy>0</Cy>-->
+					<!--<focalLength>0</focalLength>-->
+					<!--<hackBaseline>0</hackBaseline>-->
+					<!--<ignoreTfPrefix>1</ignoreTfPrefix>-->
+			  <!--</plugin>      -->
+		<!--</sensor>-->
+    </gazebo>
+    </xacro:macro>
 </robot>

Commit message: unified benewake models

File: urdf/all_sensors.urdf.xacro (robot description, xacro)
@@ -64,10 +64,6 @@
   <!-- Roboteq MGS -->
   <xacro:include filename="$(find robotnik_sensors)/urdf/roboteq_mgs.urdf.xacro" />
-  <!-- Benewake CE-30s -->
-  <xacro:include filename="$(find robotnik_sensors)/urdf/benewake_ce30s.urdf.xacro" />
-  <!-- Benewake CE-30c -->
-  <xacro:include filename="$(find robotnik_sensors)/urdf/benewake_ce30c.urdf.xacro" />
-  <!-- Benewake CE-30d -->
-  <xacro:include filename="$(find robotnik_sensors)/urdf/benewake_ce30d.urdf.xacro" />
+  <!-- Benewake CE-30 (all, includes a, c and d) -->
+  <xacro:include filename="$(find robotnik_sensors)/urdf/benewake_ce30.urdf.xacro" />
   <!-- Rubedos Viper -->
   <xacro:include filename="$(find robotnik_sensors)/urdf/rubedos_viper.urdf.xacro" />

File: urdf/benewake_ce30.urdf.xacro (robot description, xacro)
@@ -1,4 +1,4 @@
 <?xml version="1.0"?>
-<robot name="sensor_benewake_ce30d" xmlns:xacro="http://www.ros.org/wiki/xacro">
+<robot name="sensor_benewake_ce30" xmlns:xacro="http://www.ros.org/wiki/xacro">
   <xacro:property name="M_PI" value="3.1415926535897931" />
   <xacro:property name="ce30d_width" value="0.079"/>
@@ -8,5 +8,5 @@
   <xacro:property name="ce30d_depth_py" value="-0.0115"/>
   <xacro:property name="ce30d_depth_pz" value="0.0"/>
-  <xacro:macro name="sensor_benewake_ce30d" params="prefix parent *origin">
+  <xacro:macro name="sensor_benewake_ce30" params="prefix parent *origin range_min range_max hfov vfov fps">
     <material name="black_alu">
       <color rgba="0.9 0.9 0.9 1"/>
@@ -48,12 +48,12 @@
     <link name="${prefix}_link"/>
   <!-- Ray sensor for simulation, same as Hokuyo3d -->
-  <sensor_benewake_ce30d_gazebo/>
+  <sensor_benewake_ce30_gazebo range_min="${range_min}" range_max="${range_max}" hfov="${hfov}" vfov="${vfov}" fps="${fps}"/>
   </xacro:macro>
-  <xacro:macro name="sensor_benewake_ce30d_gazebo">
+  <xacro:macro name="sensor_benewake_ce30_gazebo" params="range_min range_max hfov vfov fps">
     <gazebo reference="${prefix}_link">
       <sensor type="ray" name="${prefix}_sensor">
           <pose>0 0 0 0 0 0.0</pose>
           <visualize>false</visualize>
-          <update_rate>20.0</update_rate>
+          <update_rate>${fps}</update_rate>
           <ray>
             <scan>
@@ -61,16 +61,16 @@
 				<!-- for a high quality simulation -->
                 <samples>320</samples>
-                <min_angle>-${60/2.0*M_PI/180.0}</min_angle>
-                <max_angle>${60/2.0*M_PI/180.0}</max_angle>
+                <min_angle>-${hfov/2.0*M_PI/180.0}</min_angle>
+                <max_angle>${hfov/2.0*M_PI/180.0}</max_angle>
               </horizontal>
               <vertical>
                 <samples>20</samples>
-                <min_angle>-${10/2.0*M_PI/180.0}</min_angle>
-                <max_angle>${10/2.0*M_PI/180.0}</max_angle>
+                <min_angle>-${vfov/2.0*M_PI/180.0}</min_angle>
+                <max_angle>${vfov/2.0*M_PI/180.0}</max_angle>
               </vertical>
             </scan>
             <range>
               <min>0.4</min>
-              <max>28</max>
+              <max>${range_max}</max>
               <resolution>0.01</resolution>
             </range>
@@ -89,3 +89,18 @@
     </gazebo>
   </xacro:macro>
+  <xacro:macro name="sensor_benewake_ce30a" params="prefix parent *origin">
+    <sensor_benewake_ce30 prefix="${prefix}" parent="${parent}" range_min="0.1" range_max="4.0" hfov="132.0" vfov="9.0" fps="20.0" >
+      <xacro:insert_block name="origin" />
+    </sensor_benewake_ce30>
+  </xacro:macro>
+  <xacro:macro name="sensor_benewake_ce30c" params="prefix parent *origin">
+    <sensor_benewake_ce30 prefix="${prefix}" parent="${parent}" range_min="0.1" range_max="4.0" hfov="132.0" vfov="9.0" fps="20.0" >
+      <xacro:insert_block name="origin" />
+    </sensor_benewake_ce30>
+  </xacro:macro>
+  <xacro:macro name="sensor_benewake_ce30d" params="prefix parent *origin">
+    <sensor_benewake_ce30 prefix="${prefix}" parent="${parent}" range_min="0.4" range_max="28.0" hfov="60.0" vfov="20.0" fps="30.0" >
+      <xacro:insert_block name="origin" />
+    </sensor_benewake_ce30>
+  </xacro:macro>
 </robot>
