Commit message: Updated parameters for rs_bpearl + name changes

File: urdf/all_sensors.urdf.xacro (robot description, xacro)
@@ -77,5 +77,5 @@
   <!-- RoboSense RS-Lidar -->
   <xacro:include filename="$(find robotnik_sensors)/urdf/rslidar.urdf.xacro" />
-    <!-- RoboSense RS-BPearl-Lidar -->
-  <xacro:include filename="$(find robotnik_sensors)/urdf/rs_bpearl_lidar.urdf.xacro" />
+    <!-- RoboSense RS-BPearl -->
+  <xacro:include filename="$(find robotnik_sensors)/urdf/rs_bpearl.urdf.xacro" />
 </robot>

File: urdf/rs_bpearl.urdf.xacro (robot description, xacro)
@@ -1,6 +1,6 @@
 <?xml version="1.0"?>
-<robot name="sensor_rs_bpearl_lidar" xmlns:xacro="http://wiki.ros.org/xacro">
+<robot name="sensor_rs_bpearl" xmlns:xacro="http://wiki.ros.org/xacro">
   <xacro:property name="M_PI" value="3.1415926535897931" />
-  <xacro:macro name="sensor_rs_bpearl_lidar" params="prefix parent prefix_topic *origin range_min range_max hfov samples vfov lasers fps gpu:=^|true">
+  <xacro:macro name="sensor_rs_bpearl" params="prefix parent prefix_topic *origin range_min range_max hfov samples vfov lasers fps gpu:=^|true">
     <material name="black_alu">
       <color rgba="0.9 0.9 0.9 1"/>
@@ -16,5 +16,5 @@
       <origin xyz="0 0 0" rpy="0 0 0"/>
         <geometry>
-          <mesh filename="package://robotnik_sensors/meshes/rs_bpearl_lidar.stl" />
+          <mesh filename="package://robotnik_sensors/meshes/rs_bpearl.stl" />
         </geometry>
         <material name="black_alu"/>
@@ -23,5 +23,5 @@
         <origin xyz="0 0 0" rpy="0 0 0"/>
         <geometry>
-          <mesh filename="package://robotnik_sensors/meshes/rs_bpearl_lidar.stl" />
+          <mesh filename="package://robotnik_sensors/meshes/rs_bpearl.stl" />
         </geometry>
       </collision>
@@ -36,10 +36,10 @@
       <parent link="${prefix}_base_link"/>
       <child link="${prefix}_link" />
-      <origin xyz="0 0 0.06" rpy="0 ${5*M_PI/180.0} 0"/>
+      <origin xyz="0 0 0.06" rpy="0 0 0"/>
     </joint>
     <link name="${prefix}_link"/>
-  <sensor_rs_bpearl_lidar_gazebo range_min="${range_min}" range_max="${range_max}" hfov="${hfov}" samples="${samples}" vfov="${vfov}" lasers="${lasers}" fps="${fps}" gpu="${gpu}"/>
+  <sensor_rs_bpearl_gazebo range_min="${range_min}" range_max="${range_max}" hfov="${hfov}" samples="${samples}" vfov="${vfov}" lasers="${lasers}" fps="${fps}" gpu="${gpu}"/>
   </xacro:macro>
-  <xacro:macro name="sensor_rs_bpearl_lidar_gazebo" params="range_min range_max hfov samples vfov lasers fps gpu">
+  <xacro:macro name="sensor_rs_bpearl_gazebo" params="range_min range_max hfov samples vfov lasers fps gpu">
     <gazebo reference="${prefix}_link">
       <xacro:if value="${gpu}">
@@ -54,5 +54,5 @@
         <sensor type="${ray_type}" name="${prefix}_sensor">
           <pose>0 0 0 0 0 0.0</pose>
-          <visualize>true</visualize>
+          <visualize>false</visualize>
           <update_rate>${fps}</update_rate>
           <ray>
@@ -66,5 +66,5 @@
               <vertical>
                 <samples>${lasers}</samples>
-                <min_angle>-${5*M_PI/180.0}</min_angle>  <!-- bpearl has 90 degrees of vertival field of view-->
+                <min_angle>-${5*M_PI/180.0}</min_angle>  <!-- bpearl has 90 degrees of vertical field of view-->
                 <max_angle> ${(vfov-5)*M_PI/180.0}</max_angle>
               </vertical>
@@ -87,8 +87,3 @@
     </gazebo>
   </xacro:macro>
-  <!--xacro:macro name="sensor_rs_bpearl_lidar" params="prefix parent prefix_topic:='lidar_3d' *origin gpu:=false">
-    <sensor_rs_bpearl_lidar prefix="${prefix}" parent="${parent}" prefix_topic="${prefix_topic}" range_min="0.4" range_max="250.0" hfov="360.0" hres="0.1" vfov="40.0" vres="0.1" fps="20.0" gpu="${gpu}" >
-      <xacro:insert_block name="origin" />
-    </sensor_rs_bpearl_lidar>
-  </xacro:macro-->
 </robot>

Commit message: Update ydlidar
- Add to all_sensors file
- Fix inertia
- Fix ray link position
- Add gazebo plugin

File: urdf/all_sensors.urdf.xacro (robot description, xacro)
@@ -78,5 +78,7 @@
   <!-- RoboSense RS-Lidar -->
   <xacro:include filename="$(find robotnik_sensors)/urdf/rslidar.urdf.xacro" />
-    <!-- RoboSense RS-BPearl -->
+  <!-- RoboSense RS-BPearl -->
   <xacro:include filename="$(find robotnik_sensors)/urdf/rs_bpearl.urdf.xacro" />
+  <!-- Ydlidar -->
+  <xacro:include filename="$(find robotnik_sensors)/urdf/ydlidar_4f.urdf.xacro" />
 </robot>

File: urdf/ydlidar_4f.urdf.xacro (robot description, xacro)
@@ -1,5 +1,5 @@
 <?xml version="1.0"?>
 <robot name="sensor_ydlidar_4f" xmlns:xacro="http://wiki.ros.org/xacro">
-  <xacro:macro name="sensor_ydlidar_4f" params="prefix parent prefix_topic:='front_laser' *origin">
+  <xacro:macro name="sensor_ydlidar_4f" params="prefix parent prefix_topic:='front_laser' *origin min_angle:=-3.14 max_angle:=3.14 gpu:=^true">
     <joint name="${prefix}_base_joint" type="fixed">
       <xacro:insert_block name="origin" />
@@ -9,7 +9,8 @@
     <link name="${prefix}_base_link">
       <inertial>
-        <origin xyz="-0.00029774 0.0066667 0.00013047" rpy="0 0 0" />
-        <mass value="0.15717" />
-        <inertia
+        <origin xyz="-0.0 0.0 0.0205" rpy="0 0 0" />
+        <mass value="0.188" />
+        <xacro:solid_cuboid_inertia m="0.189" w="0.071" h="0.071" d="0.041" />
+        <!--inertia
           ixx="6.7885E-05"
           ixy="-1.3987E-07"
@@ -17,5 +18,5 @@
           iyy="0.00013173"
           iyz="-9.0932E-08"
-          izz="7.1972E-05" />
+          izz="7.1972E-05" /-->
       </inertial>
       <visual>
@@ -38,11 +39,13 @@
       <parent link="${prefix}_base_link"/>
       <child link="${prefix}_link"/>
-      <origin xyz="0.0 0 0.0116" rpy="0 0 0"/>
+      <!--origin xyz="0.0 0 0.0116" rpy="0 0 0"/-->
+      <origin xyz="0.0 0 0.0312" rpy="0 0 0"/>
 	  </joint>
     <link name="${prefix}_link">
       <inertial>
-        <origin xyz="-0.00036659 0.00064155 -0.00027052" rpy="0 0 0" />
-        <mass value="0.25482" />
-        <inertia
+        <origin xyz="-0.0 0.0 -0.0107" rpy="0 0 0" />
+        <mass value="0.001" />
+        <xacro:solid_cuboid_inertia m="0.001" w="0.071" h="0.071" d="0.041" />
+        <!--inertia
           ixx="8.9194E-05"
           ixy="1.8116E-07"
@@ -50,7 +53,49 @@
           iyy="0.00018279"
           iyz="2.423E-07"
-          izz="0.00011103" />
+          izz="0.00011103" /-->
       </inertial>
     </link>
+    <sensor_ydlidar_4f_gazebo />
+  </xacro:macro>
+  <xacro:macro name="sensor_ydlidar_4f_gazebo">
+    <gazebo reference="${prefix}_link">
+      <xacro:if value="${gpu}">
+        <xacro:property name="ray_type" value="gpu_ray" />
+        <xacro:property name="plugin_lib" value="libgazebo_ros_gpu_laser.so" />
+      </xacro:if>
+      <xacro:unless value="${gpu}">
+        <xacro:property name="ray_type" value="ray" />
+        <xacro:property name="plugin_lib" value="libgazebo_ros_laser.so" />
+      </xacro:unless>
+      <sensor type="${ray_type}" name="${prefix}_sensor">
+        <pose>0 0 0 0 0 0</pose>
+        <visualize>false</visualize>
+        <update_rate>12.5</update_rate>
+        <ray>
+          <scan>
+            <horizontal>
+              <samples>1384</samples>
+              <resolution>0.26</resolution>
+              <min_angle>${min_angle}</min_angle>
+              <max_angle>${max_angle}</max_angle>
+            </horizontal>
+          </scan>
+          <range>
+            <min>0.10</min>
+            <max>16.0</max>
+            <resolution>0.03</resolution>
+          </range>
+          <noise>
+            <type>gaussian</type>
+            <mean>0.0</mean>
+            <stddev>0.03</stddev>
+          </noise>
+        </ray>
+        <plugin name="${prefix}_controller" filename="${plugin_lib}">
+          <topicName>${prefix_topic}/scan</topicName>
+          <frameName>/${prefix}_link</frameName><!-- if not global (leading /) sets the current namespace as a prefix (/ns/name_laser_link) -->
+        </plugin>
+      </sensor>
+    </gazebo>
   </xacro:macro>
 </robot>

Commit message: Merge from melodic-devel

File: urdf/all_sensors.urdf.xacro (robot description, xacro)
@@ -10,8 +10,11 @@
   <!-- Axis m5525 -->
   <xacro:include filename="$(find robotnik_sensors)/urdf/axis_m5525.urdf.xacro" />
+  <!-- Axis q8641 -->
+  <xacro:include filename="$(find robotnik_sensors)/urdf/axis_q8641.urdf.xacro" />
   <!-- Fotonic E Series -->
   <xacro:include filename="$(find robotnik_sensors)/urdf/fotonic_e.urdf.xacro" />
   <!-- GPS -->
   <xacro:include filename="$(find robotnik_sensors)/urdf/gps.urdf.xacro" />
+  <xacro:include filename="$(find robotnik_sensors)/urdf/gps_with_mast.urdf.xacro" />
   <!-- Hokuyo urg04lx -->
   <xacro:include filename="$(find robotnik_sensors)/urdf/hokuyo_urg04lx.urdf.xacro" />
@@ -76,4 +79,6 @@
   <!-- Benewake CE-30D -->
   <xacro:include filename="$(find robotnik_sensors)/urdf/benewake_ce30d.urdf.xacro" />
+  <!-- RoboSense RS-Lidar MEMS (includes M100) -->
+  <xacro:include filename="$(find robotnik_sensors)/urdf/rslidar_mems.urdf.xacro" />
   <!-- Rubedos Viper -->
   <xacro:include filename="$(find robotnik_sensors)/urdf/rubedos_viper.urdf.xacro" />
@@ -84,3 +89,5 @@
   <!-- Ydlidar -->
   <xacro:include filename="$(find robotnik_sensors)/urdf/ydlidar_4f.urdf.xacro" />
+  <!-- Ouster 1 -->
+  <xacro:include filename="$(find robotnik_sensors)/urdf/ouster1.urdf.xacro" />
 </robot>

File: urdf/benewake_ce30.urdf.xacro (robot description, xacro)
@@ -97,3 +97,8 @@
     </sensor_benewake_ce30>
   </xacro:macro>
+  <xacro:macro name="sensor_benewake_ce30d" params="prefix parent prefix_topic:='lidar_3d' *origin gpu:=false">
+    <sensor_benewake_ce30 prefix="${prefix}" parent="${parent}" prefix_topic="${prefix_topic}" range_min="0.4" range_max="28.0" hfov="60.0" vfov="4.0" fps="30.0" gpu="${gpu}" >
+      <xacro:insert_block name="origin" />
+    </sensor_benewake_ce30>
+  </xacro:macro>
 </robot>

File: urdf/rs_bpearl.urdf.xacro (robot description, xacro)
@@ -6,10 +6,10 @@
       <color rgba="0.9 0.9 0.9 1"/>
     </material>
-    <joint name="${prefix}bpearl_base_joint" type="fixed">
+    <joint name="${prefix}_base_joint" type="fixed">
       <xacro:insert_block name="origin" />
       <parent link="${parent}"/>
-      <child link="${prefix}bpearl_base_link" />
+      <child link="${prefix}_base_link" />
     </joint>
-    <link name="${prefix}bpearl_base_link">
+    <link name="${prefix}_base_link">
       <visual>
       <!-- origin xyz="0 0 0" rpy="0 0 1.5708"/ -->
@@ -33,10 +33,10 @@
       </inertial>
     </link>
-    <joint name="${prefix}bpearl_joint" type="fixed">
-      <parent link="${prefix}bpearl_base_link"/>
-      <child link="${prefix}bpearl_link" />
+    <joint name="${prefix}_joint" type="fixed">
+      <parent link="${prefix}_base_link"/>
+      <child link="${prefix}_link" />
       <origin xyz="0 0 0.06" rpy="0 0 0"/>
     </joint>
-    <link name="${prefix}bpearl_link"/>
+    <link name="${prefix}_link"/>
   <sensor_rs_bpearl_gazebo range_min="${range_min}" range_max="${range_max}" hfov="${hfov}" samples="${samples}" vfov="${vfov}" lasers="${lasers}" fps="${fps}" gpu="${gpu}"/>
   </xacro:macro>

Commit message: Update with melodic-devel changes

File: urdf/all_sensors.urdf.xacro (robot description, xacro)
@@ -43,4 +43,6 @@
   <!-- Sick microscan3 -->
   <xacro:include filename="$(find robotnik_sensors)/urdf/sick_microscan3.urdf.xacro" />
+  <!-- Sick outdoorscan3 -->
+  <xacro:include filename="$(find robotnik_sensors)/urdf/sick_outdoorscan3.urdf.xacro" />
   <!-- KinectV2 -->
   <xacro:include filename="$(find robotnik_sensors)/urdf/kinectv2.urdf.xacro" />

File: urdf/rs_bpearl.urdf.xacro (robot description, xacro)
@@ -3,7 +3,4 @@
   <xacro:property name="M_PI" value="3.1415926535897931" />
   <xacro:macro name="sensor_rs_bpearl" params="prefix parent prefix_topic *origin range_min range_max hfov samples vfov lasers fps gpu:=^|true">
-    <material name="black_alu">
-      <color rgba="0.9 0.9 0.9 1"/>
-    </material>
     <joint name="${prefix}_base_joint" type="fixed">
       <xacro:insert_block name="origin" />
@@ -18,5 +15,7 @@
           <mesh filename="package://robotnik_sensors/meshes/rs_bpearl.stl" />
         </geometry>
-        <material name="black_alu"/>
+        <material name="blackgray_color">
+          <color rgba="0.25 0.25 0.25 1"/>
+        </material>
       </visual>
       <collision>
@@ -42,5 +41,23 @@
   </xacro:macro>
   <xacro:macro name="sensor_rs_bpearl_gazebo" params="range_min range_max hfov samples vfov lasers fps gpu">
+    <gazebo reference="${prefix}_base_link">
+      <visual>
+        <material>
+          <ambient>0.5 0.5 0.5 1.0</ambient>
+          <diffuse>0.250754 0.250754 0.250754 1.0</diffuse>
+          <specular>0.2508273 0.2508273 0.2508273 1.0</specular>
+          <emissive>0.0 0.0 0.0 0.0</emissive>
+        </material>
+      </visual>
+    </gazebo>
     <gazebo reference="${prefix}_link">
+      <visual>
+        <material>
+          <ambient>1.2 0.2 0.2 1.0</ambient>
+          <diffuse>0.250754 0.250754 0.250754 1.0</diffuse>
+          <specular>0.2508273 0.2508273 0.2508273 1.0</specular>
+          <emissive>0.0 0.0 0.0 0.0</emissive>
+        </material>
+      </visual>
       <xacro:if value="${gpu}">
         <!-- Using GPU needs: https://github.com/RobotnikAutomation/velodyne_simulator -->

File: urdf/rslidar.urdf.xacro (robot description, xacro)
@@ -35,4 +35,5 @@
       <parent link="${prefix}_base_link"/>
       <child link="${prefix}_link" />
+      <origin xyz="0.0 0 0.038" rpy="0 0 0"/>
     </joint>
     <link name="${prefix}_link"/>

File: urdf/zed.urdf.xacro (robot description, xacro)
@@ -1,37 +1,95 @@
 <?xml version="1.0"?>
-<robot name="sensor_zed" xmlns:xacro="http://wiki.ros.org/xacro">
-  <!-- Xacro properties -->
-  <xacro:property name="M_PI" value="3.1415926535897931" />
-  <xacro:macro name="sensor_zed" params="prefix parent prefix_topic:='front_rgbd_camera' *origin">
-    <joint name="${prefix}_rgb_joint" type="fixed">
-	    <xacro:insert_block name="origin" />
+<robot xmlns:xacro="http://wiki.ros.org/xacro">
+  <xacro:macro name="stereo_camera"
+    params="prefix fps baseline hfov width height format near far">
+    <gazebo reference="${prefix}_base_link">
+      <visual>
+        <material>
+          <ambient>0.35 0.35 0.35 1.0</ambient>
+          <diffuse>0.350754 0.350754 0.350754 1.0</diffuse>
+          <specular>0.308273 0.3508273 0.3508273 1.0</specular>
+          <emissive>0.0 0.0 0.0 0.0</emissive>
+        </material>
+      </visual>
+      <sensor type="multicamera" name="stereo_camera">
+        <update_rate>${fps}</update_rate>
+        <camera name="left">
+          <pose>0 0 0 0 0 0 </pose>
+          <horizontal_fov>${hfov}</horizontal_fov>
+          <image>
+            <width>${width}</width>
+            <height>${height}</height>
+            <format>${format}</format>
+          </image>
+          <clip>
+            <near>${near}</near>
+            <far>${far}</far>
+          </clip>
+          <noise>
+            <type>gaussian</type>
+            <mean>0.0</mean>
+            <stddev>0.007</stddev>
+          </noise>
+        </camera>
+        <camera name="right">
+          <pose>${baseline} 0 0 0 0 0</pose>
+          <horizontal_fov>${hfov}</horizontal_fov>
+          <image>
+            <width>${width}</width>
+            <height>${height}</height>
+            <format>${format}</format>
+          </image>
+          <clip>
+            <near>${near}</near>
+            <far>${far}</far>
+          </clip>
+          <noise>
+            <type>gaussian</type>
+            <mean>0.0</mean>
+            <stddev>0.007</stddev>
+          </noise>
+        </camera>
+        <plugin name="stereo_camera_controller" filename="libgazebo_ros_multicamera.so">
+          <alwaysOn>true</alwaysOn>
+          <cameraName>${prefix}</cameraName>
+          <imageTopicName>image_raw</imageTopicName>
+          <cameraInfoTopicName>camera_info</cameraInfoTopicName>
+          <frameName>${prefix}_base_link</frameName>
+          <hackBaseline>${baseline}</hackBaseline>
+          <!-- NOTE: Distortion is currently unused -->
+          <distortionK1>0.0</distortionK1>
+          <distortionK2>0.0</distortionK2>
+          <distortionK3>0.0</distortionK3>
+          <distortionT1>0.0</distortionT1>
+          <distortionT2>0.0</distortionT2>
+          <ignoreTfPrefix>1</ignoreTfPrefix>
+        </plugin>
+      </sensor>
+    </gazebo>
+  </xacro:macro>
+  <xacro:macro name="stereolabs_zed"
+    params="prefix:=zed parent *origin model:=zed format:=R8G8B8 near:=0.05 far:=2500">
+    <xacro:if value="${model == 'zed'}">
+        <xacro:property name="baseline" value="0.12" />
+    </xacro:if>
+    <xacro:if value="${model == 'zedm'}">
+        <xacro:property name="baseline" value="0.06" />
+    </xacro:if>
+    <xacro:if value="${model == 'zed2'}">
+        <xacro:property name="baseline" value="0.12" />
+    </xacro:if>
+    <joint name="${prefix}_base_joint" type="fixed">
+      <xacro:insert_block name="origin" />
       <parent link="${parent}"/>
-      <child link="${prefix}_rgb_base_link" />
+      <child link="${prefix}_base_link" />
     </joint>
-    <link name="${prefix}_rgb_base_link">
-      <inertial>
-        <mass value="0.135" />
-        <origin xyz="0 0 0" />
-        <xacro:solid_cuboid_inertia m="0.135" w="0.033" h="0.175" d="0.03" />
-        <!--inertia ixx="0.0001" ixy="0.0" ixz="0.0"
-          iyy="0.0001" iyz="0.0"
-          izz="0.0001" /-->
-      </inertial>
-    </link>
-    <!-- Camera center -->
-    <joint name="${prefix}_joint" type="fixed">
-      <origin xyz="0.0 0.0 0.0"
-              rpy="0.0 0.0 0.0"/>
-      <parent link="${prefix}_rgb_base_link"/>
-      <child link="${prefix}_link"/>
-    </joint>
-    <link name="${prefix}_link">
-      <visual>
+    <link name="${prefix}_base_link">
+       <visual>
         <origin xyz="0 0 0" rpy="0 0 0"/>
         <geometry>
-          <mesh filename="package://robotnik_sensors/meshes/zed.stl"/>
+          <mesh filename="package://robotnik_sensors/meshes/${model}.stl"/>
         </geometry>
-        <material name="light_grey">
-          <color rgba="0.8 0.8 0.8 0.8"/>
+        <material name="light_zed_grey">
+          <color rgba="0.35 0.35 0.35 1"/>
         </material>
       </visual>
@@ -39,5 +97,5 @@
         <origin xyz="0.0 0.0 0.0" rpy="0 0 0" />
         <geometry>
-          <mesh filename="package://robotnik_sensors/meshes/zed.stl" />
+          <mesh filename="package://robotnik_sensors/meshes/${model}.stl" />
         </geometry>
       </collision>
@@ -46,13 +104,10 @@
         <origin xyz="0 0 0" />
         <xacro:solid_cuboid_inertia m="0.135" w="0.033" h="0.175" d="0.03" />
-        <!--inertia ixx="0.003881243" ixy="0.0" ixz="0.0"
-                  iyy="0.000498940" iyz="0.0"
-                  izz="0.003879257" /-->
       </inertial>
     </link>
-    <!-- Left camera -->
+   <!-- Left camera -->
     <joint name="${prefix}_rgb_left_joint" type="fixed">
       <origin xyz="0.0 0.06 0.0" rpy="0.0 0.0 0.0" />
-      <parent link="${prefix}_link" />
+      <parent link="${prefix}_base_link" />
       <child link="${prefix}_left_rgb_frame" />
     </joint>
@@ -67,5 +122,5 @@
     <joint name="${prefix}_rgb_right_joint" type="fixed">
       <origin xyz="0.0 -0.06 0.0" rpy="0.0 0.0 0.0" />
-      <parent link="${prefix}_link" />
+      <parent link="${prefix}_base_link" />
       <child link="${prefix}_right_rgb_frame" />
     </joint>
@@ -77,5 +132,19 @@
     </joint>
     <link name="${prefix}_right_rgb_optical_frame"/>
-  <!-- TODO: simulation -->
+      <xacro:stereo_camera
+        prefix="${prefix}"
+        hfov="1.2217"
+        baseline="${baseline}"
+        fps="40"
+        width="640"
+        height="480"
+        format="${format}"
+        near="${near}"
+        far="${far}"/>
+  </xacro:macro>
+  <xacro:macro name="sensor_zed" params="prefix:=myzed parent *origin model:=zed" >
+    <stereolabs_zed prefix="${prefix}" parent="${parent}" model="${model}">
+      <xacro:insert_block name="origin" />
+    </stereolabs_zed>
   </xacro:macro>
 </robot>
