Commit message: Add material like a xacro. This solves the problem of having two sensors with the same material name.

File: urdf/all_sensors.urdf.xacro (robot description, xacro)
@@ -3,4 +3,5 @@
   xmlns:xacro="http://wiki.ros.org/xacro">
   <xacro:include filename="$(find robotnik_sensors)/urdf/utils/inertia.urdf.xacro" />
+  <xacro:include filename="$(find robotnik_sensors)/urdf/utils/material.urdf.xacro" />
   <!-- This file unifies all sensors that can be used on simulation, defined as xacro:macros -->
   <!-- Pantilt -->

File: urdf/benewake_ce30.urdf.xacro (robot description, xacro)
@@ -3,7 +3,4 @@
   <xacro:property name="M_PI" value="3.1415926535897931" />
   <xacro:macro name="sensor_benewake_ce30" params="prefix parent prefix_topic *origin range_min range_max hfov vfov fps gpu:=^|true">
-    <material name="black_alu">
-      <color rgba="0.9 0.9 0.9 1"/>
-    </material>
     <joint name="${prefix}_base_joint" type="fixed">
       <xacro:insert_block name="origin" />

File: urdf/benewake_ce30d.urdf.xacro (robot description, xacro)
@@ -3,7 +3,4 @@
   <xacro:property name="M_PI" value="3.1415926535897931" />
   <xacro:macro name="sensor_benewake_ce30d" params="prefix parent prefix_topic:='lidar_3d' *origin range_min:=0.4 range_max:=28.0 hfov:=60.0 vfov:=4.0 fps:=30.0 gpu:=^|true">
-    <material name="black_alu">
-      <color rgba="0.9 0.9 0.9 1"/>
-    </material>
     <joint name="${prefix}_base_joint" type="fixed">
       <xacro:insert_block name="origin" />
@@ -18,5 +15,5 @@
           <mesh filename="package://robotnik_sensors/meshes/benewake_ce30d.stl" />
         </geometry>
-        <material name="black_alu"/>
+	<material name="black_alu"/>
       </visual>
       <collision>

File: urdf/ouster1.urdf.xacro (robot description, xacro)
@@ -3,7 +3,4 @@
   <xacro:property name="M_PI" value="3.1415926535897931" />
   <xacro:macro name="sensor_ouster1" params="prefix parent prefix_topic *origin range_min range_max hfov hsamples vfov vsamples fps gpu:=^|true">
-    <material name="black_alu">
-      <color rgba="0.9 0.9 0.9 1"/>
-    </material>
     <joint name="${prefix}_base_joint" type="fixed">
       <xacro:insert_block name="origin" />

File: urdf/rslidar.urdf.xacro (robot description, xacro)
@@ -3,7 +3,4 @@
   <xacro:property name="M_PI" value="3.1415926535897931" />
   <xacro:macro name="sensor_rslidar" params="prefix parent prefix_topic *origin range_min range_max hfov hres vfov vres fps gpu:=^|true">
-    <material name="black_alu">
-      <color rgba="0.9 0.9 0.9 1"/>
-    </material>
     <joint name="${prefix}_base_joint" type="fixed">
       <xacro:insert_block name="origin" />

File: urdf/rslidar_mems.urdf.xacro (robot description, xacro)
@@ -3,7 +3,4 @@
   <xacro:property name="M_PI" value="3.1415926535897931" />
   <xacro:macro name="sensor_rslidar_mems" params="prefix parent *origin">
-    <material name="black_alu">
-      <color rgba="0.9 0.9 0.9 1"/>
-    </material>
     <joint name="${prefix}_base_joint" type="fixed">
       <xacro:insert_block name="origin" />

Commit message: feat: Add new sensor models and update URDF files for axis_1798le, flir_645r, flir_ptu_5, and rs_airy

File: urdf/all_sensors.urdf.xacro (robot description, xacro)
@@ -149,3 +149,9 @@
   <xacro:include filename="$(find robotnik_sensors)/urdf/sensia_raismart.urdf.xacro" />
   <xacro:include filename="$(find robotnik_sensors)/urdf/sensia_raismart_pt.urdf.xacro" />
+  <!-- axis_1798le -->
+  <xacro:include filename="$(find robotnik_sensors)/urdf/axis_1798le.urdf.xacro" />
+  <!-- flir_645r -->
+  <xacro:include filename="$(find robotnik_sensors)/urdf/flir_645r.urdf.xacro" />
+  <!-- flir_ptu_5 -->
+  <xacro:include filename="$(find robotnik_sensors)/urdf/flir_ptu_5.urdf.xacro" />
 </robot>

File: urdf/rs_airy.urdf.xacro (robot description, xacro)
@@ -39,5 +39,5 @@
   <xacro:sensor_rslidar_gazebo range_min="${range_min}" range_max="${range_max}" hfov="${hfov}" hres="${hres}" vfov="${vfov}" vres="${vres}" fps="${fps}" gpu="${gpu}"/>
   </xacro:macro>
-  <xacro:macro name="sensor_rslidar_gazebo" params="range_min range_max hfov hres vfov vres fps gpu">
+  <xacro:macro name="sensor_rslidar_gazebo" params="range_min range_max hfov hres vfov vres fps gpu prefix_topic:='top_3d_laser' suffix_topic:=''">
     <gazebo reference="${prefix}_link">
       <xacro:if value="${gpu}">
