Commit message: Changed to default gazebo plugin, not used realsense plugin

File: robotnik_sensors/urdf/orbbec_astra.urdf.xacro (robot description, xacro)
@@ -3,5 +3,5 @@
   <xacro:macro name="sensor_orbbec_astra" params="ns prefix parent *origin">
     <joint name="${prefix}_joint" type="fixed">
-    	<xacro:insert_block name="origin" />
+    	<xacro:insert_block name="origin"/>
       <parent link="${parent}"/>
       <child link="${prefix}_link"/>
@@ -15,6 +15,7 @@
       </visual>
       <collision>
+        <origin xyz="-0.02 0 0.015" rpy="0 0 0"/>
         <geometry>
-          <box size="0.1 0.1 0.1"/>
+          <box size="0.042 0.155 0.03"/>
         </geometry>
       </collision>
@@ -30,11 +31,5 @@
       <child link="${prefix}_rgb_frame" />
     </joint>
-    <link name="${prefix}_rgb_frame">
-      <inertial>
-        <mass value="0.297" />
-        <origin xyz="-0.02 -0.0125 0.0" />
-        <xacro:solid_cuboid_inertia m="0.297" w="0.04" h="0.165" d="0.03" />
-      </inertial>
-    </link>
+    <link name="${prefix}_rgb_frame"/>
     <joint name="${prefix}_rgb_optical_joint" type="fixed">
       <origin xyz="0.0 0.0 0.0" rpy="${-M_PI/2} 0 ${-M_PI/2}" />
@@ -42,11 +37,5 @@
       <child link="${prefix}_rgb_optical_frame" />
     </joint>
-    <link name="${prefix}_rgb_optical_frame">
-      <inertial>
-        <mass value="0.001" />
-        <origin xyz="0 0 0" rpy="${M_PI/2} 0 ${M_PI/2}"/>
-        <xacro:solid_cuboid_inertia m="0.001" w="0.04" h="0.165" d="0.03" />
-      </inertial>
-    </link>
+    <link name="${prefix}_rgb_optical_frame"/>
     <joint name="${prefix}_depth_joint" type="fixed">
       <origin xyz="0.0 0.0375 0.0150" rpy="0 0 0" />
@@ -54,11 +43,5 @@
       <child link="${prefix}_depth_frame" />
     </joint>
-    <link name="${prefix}_depth_frame">
-      <inertial>
-        <mass value="0.001" />
-        <origin xyz="0 0 0" />
-        <xacro:solid_cuboid_inertia m="0.001" w="0.04" h="0.165" d="0.03" />
-      </inertial>
-    </link>
+    <link name="${prefix}_depth_frame"/>
     <joint name="${prefix}_depth_optical_joint" type="fixed">
       <origin xyz="0 0 0" rpy="${-M_PI/2} 0 ${-M_PI/2}" />
@@ -66,148 +49,36 @@
       <child link="${prefix}_depth_optical_frame" />
     </joint>
-    <link name="${prefix}_depth_optical_frame">
-      <inertial>
-        <mass value="0.001" />
-        <origin xyz="0 0 0" />
-        <xacro:solid_cuboid_inertia m="0.001" w="0.04" h="0.165" d="0.03" />
-      </inertial>
-    </link>
-  <xacro:sensor_orbbec_astra_gazebo/>
-  <xacro:sensor_orbbec_astra_gazebo/>
-    <xacro:sensor_orbbec_astra_gazebo/>
+    <link name="${prefix}_depth_optical_frame"/>
+    <xacro:sensor_orbbec_astra_gazebo ns="${ns}" prefix="${prefix}"/>
   </xacro:macro>
-  <xacro:macro name="sensor_orbbec_astra_gazebo">
-    <xacro:property name="deg_to_rad" value="0.01745329251994329577" />
+  <xacro:macro name="sensor_orbbec_astra_gazebo" params="ns prefix">
+    <xacro:property name="deg_to_rad" value="0.01745329251994329577"/>
     <gazebo reference="${prefix}_link">
-      <self_collide>0</self_collide>
-      <enable_wind>0</enable_wind>
-      <kinematic>0</kinematic>
-      <gravity>1</gravity>
-      <!--<mu>1</mu>-->
-      <mu2>1</mu2>
-      <fdir1>0 0 0</fdir1>
-      <!--<slip1>0</slip1>
-      <slip2>0</slip2>-->
-      <kp>1e+13</kp>
-      <kd>1</kd>
-      <!--<max_vel>0.01</max_vel>
-      <min_depth>0</min_depth>-->
-      <sensor name="${prefix}color" type="camera">
-        <camera name="${prefix}">
-          <vertical_fov>${49.5*deg_to_rad}</vertical_fov>
-          <horizontal_fov>${60*deg_to_rad}</horizontal_fov>
+      <sensor name="${prefix}" type="depth">
+        <pose>0 0 0 0 0 0</pose>
+        <visualize>false</visualize>
+        <update_rate>30</update_rate>
+        <camera>
+          <horizontal_fov>1,04719755</horizontal_fov>
+          <vertical_fov>0.86393798</vertical_fov>
           <image>
-            <format>RGB_INT8</format>
-            <width>1280</width>
-            <height>960</height>
-          </image>
-          <clip>
-            <near>0.1</near>
-            <far>100</far>
-          </clip>
-          <noise>
-            <type>gaussian</type>
-            <mean>0.0</mean>
-            <stddev>0.004</stddev>
-          </noise>
-        </camera>
-        <always_on>1</always_on>
-        <update_rate>10</update_rate>
-        <visualize>false</visualize>
-      </sensor>
-      <sensor name="${prefix}ired1" type="camera">
-        <camera name="${prefix}">
-          <vertical_fov>${49.5*deg_to_rad}</vertical_fov>
-          <horizontal_fov>${60*deg_to_rad}</horizontal_fov>
-          <image>
-            <format>L_INT8</format>
+            <format>B8G8R8</format>
             <width>640</width>
             <height>480</height>
           </image>
           <clip>
-            <near>0.1</near>
-            <far>100</far>
+            <near>0.05</near>
+            <far>100.0</far>
           </clip>
-          <noise>
-            <type>gaussian</type>
-            <mean>0.0</mean>
-            <stddev>0.004</stddev>
-          </noise>
         </camera>
-        <always_on>1</always_on>
-        <update_rate>10</update_rate>
-        <visualize>false</visualize>
+        <plugin name="${prefix}" filename="libgazebo_ros_camera.so">
+          <ros>
+            <namespace>${ns}</namespace>
+          </ros>
+          <frame_name>${ns}/${prefix}_rgb_optical_frame</frame_name>
+          <min_depth>0.4</min_depth>
+          <max_depth>6.5</max_depth>
+        </plugin>
       </sensor>
-      <sensor name="${prefix}ired2" type="camera">
-        <camera name="${prefix}">
-          <vertical_fov>${49.5*deg_to_rad}</vertical_fov>
-          <horizontal_fov>${60*deg_to_rad}</horizontal_fov>
-          <image>
-            <format>L_INT8</format>
-            <width>640</width>
-            <height>480</height>
-          </image>
-          <clip>
-            <near>0.1</near>
-            <far>100</far>
-          </clip>
-          <noise>
-            <type>gaussian</type>
-            <mean>0.0</mean>
-            <stddev>0.004</stddev>
-          </noise>
-        </camera>
-        <always_on>1</always_on>
-        <update_rate>30</update_rate>
-        <visualize>false</visualize>
-      </sensor>
-      <sensor name="${prefix}depth" type="depth">
-        <camera name="${prefix}">
-          <vertical_fov>${49.5*deg_to_rad}</vertical_fov>
-          <horizontal_fov>${60*deg_to_rad}</horizontal_fov>
-          <image>
-            <format>R8G8B8</format>
-            <width>640</width>
-            <height>480</height>
-          </image>
-          <clip>
-            <near>0.1</near>
-            <far>100</far>
-          </clip>
-          <noise>
-            <type>gaussian</type>
-            <mean>0.0</mean>
-            <stddev>0.004</stddev>
-          </noise>
-        </camera>
-        <always_on>1</always_on>
-        <update_rate>10</update_rate>
-        <visualize>false</visualize>
-      </sensor>
-    </gazebo>
-    <gazebo>
-      <plugin name="${ns}" filename="librealsense_gazebo_plugin.so">
-        <prefix>${prefix}</prefix>
-        <depthUpdateRate>60.0</depthUpdateRate>
-        <colorUpdateRate>60.0</colorUpdateRate>
-        <infraredUpdateRate>60.0</infraredUpdateRate>
-        <depthTopicName>${ns}/${prefix}/depth/image_raw</depthTopicName>
-        <depthCameraInfoTopicName>${ns}/${prefix}/depth/camera_info</depthCameraInfoTopicName>
-        <colorTopicName>${ns}/${prefix}/color/image_raw</colorTopicName>
-        <colorCameraInfoTopicName>${ns}/${prefix}/color/camera_info</colorCameraInfoTopicName>
-        <infrared1TopicName>${ns}/${prefix}/infra1/image_rect_raw</infrared1TopicName>
-        <infrared1CameraInfoTopicName>${ns}/${prefix}/infra1/camera_info</infrared1CameraInfoTopicName>
-        <infrared2TopicName>${ns}/${prefix}/infra2/image_rect_raw</infrared2TopicName>
-        <infrared2CameraInfoTopicName>${ns}/${prefix}/infra2/camera_info</infrared2CameraInfoTopicName>
-        <colorOpticalframeName>${ns}/${prefix}_rgb_optical_frame</colorOpticalframeName>
-        <depthOpticalframeName>${ns}/${prefix}_depth_optical_frame</depthOpticalframeName>
-        <infrared1OpticalframeName>${ns}/${prefix}_left_ir_optical_frame</infrared1OpticalframeName>
-        <infrared2OpticalframeName>${ns}/${prefix}_right_ir_optical_frame</infrared2OpticalframeName>
-        <rangeMinDepth>0.4</rangeMinDepth>
-        <rangeMaxDepth>6.0</rangeMaxDepth>
-        <pointCloud>true</pointCloud>
-        <pointCloudTopicName>${ns}/${prefix}/depth/color/points</pointCloudTopicName>
-        <pointCloudCutoff>0.5</pointCloudCutoff>
-      </plugin>
     </gazebo>
   </xacro:macro>
