Commit message: robotnik_sensors: solves wrong tags when instanciating gazebo plugins

File: robotnik_sensors/urdf/rs_bpearl.urdf.xacro (robot description, xacro)
@@ -38,7 +38,7 @@
     </joint>
     <link name="${prefix}_link"/>
-  <xacro:sensor_rs_bpearl_gazebo range_min="${range_min}" range_max="${range_max}" hfov="${hfov}" samples="${samples}" vfov="${vfov}" lasers="${lasers}" fps="${fps}" gpu="${gpu}"/>
+    <xacro:sensor_rs_bpearl_gazebo prefix="${prefix}" range_min="${range_min}" range_max="${range_max}" hfov="${hfov}" samples="${samples}" vfov="${vfov}" lasers="${lasers}" fps="${fps}" gpu="${gpu}"/>
   </xacro:macro>
-  <xacro:macro name="sensor_rs_bpearl_gazebo" params="range_min range_max hfov samples vfov lasers fps gpu">
+  <xacro:macro name="sensor_rs_bpearl_gazebo" params="prefix range_min range_max hfov samples vfov lasers fps gpu">
     <gazebo reference="${prefix}_base_link">
       <visual>
@@ -75,5 +75,5 @@
             <scan>
               <horizontal>
-				<!-- for a high quality simulation -->
+		<!-- for a high quality simulation -->
                 <samples>${samples}</samples>
                 <min_angle>-${hfov/2*M_PI/180.0}</min_angle>
@@ -97,6 +97,9 @@
           <plugin name="${prefix}_controller" filename="${plugin_lib}">
             <topicName>${prefix_topic}/points</topicName>
-            <frameName>/${prefix}_link</frameName>
-            <gaussianNoise>0.008</gaussianNoise>
+            <gaussian_noise>0.008</gaussian_noise>
+            <organize_cloud>0</organize_cloud>
+            <frame_name>${prefix}_base_link</frame_name>
+            <min_range>${range_min}</min_range>
+            <max_range>${range_max}</max_range>
           </plugin>
         </sensor>

File: robotnik_sensors/urdf/rslidar.urdf.xacro (robot description, xacro)
@@ -79,7 +79,7 @@
           </ray>
           <plugin name="${prefix}_controller" filename="${plugin_lib}">
-            <topicName>${prefix_topic}/points</topicName>
-            <frameName>/${prefix}_link</frameName>
-            <gaussianNoise>0.008</gaussianNoise>
+            <topic_name>${prefix_topic}/points</topic_name>
+            <frame_name>/${prefix}_link</frame_name>
+            <gaussian_noise>0.008</gaussian_noise>
           </plugin>
         </sensor>
