Commit message: feat: Add picoscan120 (#73)

File: robotnik_sensors/urdf/all_sensors.urdf.xacro (robot description, xacro)
@@ -5,6 +5,10 @@
   <!-- This file unifies all sensors that can be used on simulation, defined as xacro:macros -->
   <!-- Declare global argument to set low_performance mode -->
-  <xacro:arg name="low_performance" default="false" />
-  <xacro:property name="low_performance" value="$(arg low_performance)" />
+  <xacro:arg
+    name="low_performance"
+    default="false" />
+  <xacro:property
+    name="low_performance"
+    value="$(arg low_performance)" />
   <xacro:include
     filename="$(find robotnik_sensors)/urdf/utils/inertia.urdf.xacro" />
@@ -41,4 +45,6 @@
   <xacro:include
     filename="$(find robotnik_sensors)/urdf/2d_lidar/sick_tim571.urdf.xacro" />
+  <xacro:include
+    filename="$(find robotnik_sensors)/urdf/2d_lidar/sick_picoscan120.urdf.xacro" />
   <xacro:include
     filename="$(find robotnik_sensors)/urdf/2d_lidar/hokuyo_urg04lx.urdf.xacro" />
