Commit message: Added vectornav

File: robotnik_sensors/urdf/imu/vectornav.urdf.xacro (robot description, xacro)
@@ -1,13 +1,18 @@
 <?xml version="1.0"?>
 <robot name="sensor_vectornav" xmlns:xacro="http://wiki.ros.org/xacro">
-  <xacro:macro name="sensor_vectornav" params="prefix parent *origin topic:='imu/data'">
-    <xacro:include filename="$(find robotnik_sensors)/urdf/utils/inertia.urdf.xacro" />
-    <joint name="${prefix}imu_base_joint" type="fixed">
-      <axis xyz="1 0 0"/>
+  <xacro:macro name="sensor_vectornav"
+               params="frame_prefix
+                       parent
+                       *origin
+                       simulation:=false
+                       node_name:=imu
+                       node_namespace:=${None}
+                       topic_prefix:=~/">
+    <joint name="${frame_prefix}base_joint" type="fixed">
       <xacro:insert_block name="origin"/>
       <parent link="${parent}"/>
-      <child link="${prefix}imu_base_link"/>
+      <child link="${frame_prefix}base_link"/>
     </joint>
-    <link name="${prefix}imu_base_link">
+    <link name="${frame_prefix}base_link">
       <inertial>
         <origin xyz="0.0 0 0.01" rpy="0 0 0" />
@@ -21,5 +26,5 @@
         </material>
         <geometry>
-          <mesh filename="package://robotnik_sensors/meshes/vectornav_vn100.stl"/>
+          <mesh filename="package://robotnik_sensors/meshes/imu/vectornav_vn100.stl"/>
         </geometry>
       </visual>
@@ -31,17 +36,17 @@
       </collision>
     </link>
-    <joint name="${prefix}imu_joint" type="fixed">
+    <joint name="${frame_prefix}joint" type="fixed">
         <axis xyz="1 0 0"/>
         <origin xyz="-0.00745 0.0 0.0088"/>
-        <parent link="${prefix}imu_base_link"/>
-        <child link="${prefix}imu_link"/>
+        <parent link="${frame_prefix}base_link"/>
+        <child link="${frame_prefix}link"/>
     </joint>
-    <link name="${prefix}imu_link" />
-    <gazebo reference="${prefix}imu_base_link">
+    <link name="${frame_prefix}link" />
+    <gazebo reference="${frame_prefix}base_link">
       <material>Gazebo/Red</material>
     </gazebo>
-    <gazebo reference="${prefix}imu_link">
+    <gazebo reference="${frame_prefix}link">
       <gravity>true</gravity>
-      <sensor name="${prefix}imu_sensor" type="imu">
+      <sensor name="${frame_prefix}sensor" type="imu">
         <always_on>true</always_on>
         <update_rate>200</update_rate>
@@ -109,10 +114,11 @@
           </linear_acceleration>
         </imu>
-        <plugin name="${prefix}imu_controller" filename="libgazebo_ros_imu_sensor.so">
+        <plugin name="${node_name}" filename="libgazebo_ros_imu_sensor.so">
+          <ros>
+            <namespace>${node_namespace}</namespace>
+            <remapping>~/out:=${topic_prefix}data</remapping>
+          </ros>
           <initial_orientation_as_reference>false</initial_orientation_as_reference>
-          <frame_name>${prefix}imu_link</frame_name>
-          <ros>
-            <remapping>~/out:=${topic}</remapping>
-          </ros>
+          <frame_name>${node_namespace}/${frame_prefix}link</frame_name>
         </plugin>
       </sensor>
