Commit message: fix: apply prettier format URDF files for lidar and camera

File: robotnik_sensors/urdf/3d_lidar/robosense_helios_16p.urdf.xacro (robot description, xacro)
@@ -80,6 +80,5 @@
       rate="10"
       horizontal_samples="1800"
-      vertical_samples="16">
-    </xacro:lidar_3d_plugin>
+      vertical_samples="16" />
   </xacro:macro>
 </robot>

File: robotnik_sensors/urdf/camera/link_750_nh.urdf.xacro (robot description, xacro)
@@ -114,5 +114,5 @@
           rpy="0 0 0" />
         <material name="grey_color">
-          <color rgba="0.1 0.1 0.1 1"/>
+          <color rgba="0.1 0.1 0.1 1" />
         </material>
         <geometry>
@@ -129,5 +129,5 @@
           <mesh
             filename="package://robotnik_sensors/meshes/camera/link_750_pan.stl"
-            scale="1.0 1.0 1.0"/>
+            scale="1.0 1.0 1.0" />
         </geometry>
       </collision>
@@ -166,7 +166,7 @@
         <origin
           xyz="0 0 0"
-          rpy="${radians(90)} 0 0"/>
+          rpy="${radians(90)} 0 0" />
         <material name="grey_color">
-          <color rgba="0.1 0.1 0.1 1"/>
+          <color rgba="0.1 0.1 0.1 1" />
         </material>
         <geometry>
@@ -187,14 +187,22 @@
       </collision>
     </link>
-    <joint name="${frame_prefix}zoom_color_joint" type="prismatic">
-      <axis xyz="0 0 1"/>
-      <origin xyz="0.0 0.0 0.0" rpy="0 0 0"/>
-      <parent link="${frame_prefix}optical_frame_link"/>
-      <child link="${frame_prefix}zoom_color_link"/>
-      <limit effort="10000.0" velocity="10" lower="0" upper="${ptz_zoom}"/>
+    <joint
+      name="${frame_prefix}zoom_color_joint"
+      type="prismatic">
+      <axis xyz="0 0 1" />
+      <origin
+        xyz="0.0 0.0 0.0"
+        rpy="0 0 0" />
+      <parent link="${frame_prefix}optical_frame_link" />
+      <child link="${frame_prefix}zoom_color_link" />
+      <limit
+        effort="10000.0"
+        velocity="10"
+        lower="0"
+        upper="${ptz_zoom}" />
     </joint>
     <link name="${frame_prefix}zoom_color_link">
       <inertial>
-        <mass value="0.00001"/>
+        <mass value="0.00001" />
         <origin
           xyz="0 0 0"

Commit message: add global arg

File: robotnik_sensors/urdf/3d_lidar/robosense_helios_16p.urdf.xacro (robot description, xacro)
@@ -14,6 +14,5 @@
             node_namespace:=${None}
             topic_prefix:=~/
-            gpu:=false
-            low_performance:=false">
+            gpu:=false">
     <xacro:if value="${node_namespace == None}">
       <xacro:property

File: robotnik_sensors/urdf/all_sensors.urdf.xacro (robot description, xacro)
@@ -4,4 +4,7 @@
   xmlns:xacro="http://wiki.ros.org/xacro">
   <!-- This file unifies all sensors that can be used on simulation, defined as xacro:macros -->
+  <!-- Declare global argument to set low_performance mode -->
+  <xacro:arg name="low_performance" default="false" />
+  <xacro:property name="low_performance" value="$(arg low_performance)" />
   <xacro:include
     filename="$(find robotnik_sensors)/urdf/utils/inertia.urdf.xacro" />

File: robotnik_sensors/urdf/camera/link_750_nh.urdf.xacro (robot description, xacro)
@@ -33,6 +33,5 @@
             node_name:=link_750_nh
             node_namespace:=${None}
-            topic_prefix:=~/
-            low_performance:=false">
+            topic_prefix:=~/">
     <joint
       name="${frame_prefix}base_joint"

File: robotnik_sensors/urdf/depth/intel_realsense_d435.urdf.xacro (robot description, xacro)
@@ -17,6 +17,5 @@
             node_name:=realsense_d435
             node_namespace:=${None}
-            topic_prefix:=~/
-            low_performance:=false">
+            topic_prefix:=~/">
     <!-- node_namespace is used from node_name if not set -->
     <xacro:if value="${node_namespace == None}">

Commit message: feat: add low performance argument (#64)

File: robotnik_sensors/urdf/3d_lidar/robosense_helios_16p.urdf.xacro (robot description, xacro)
@@ -69,16 +69,32 @@
     </joint>
     <link name="${frame_prefix}link" />
-    <xacro:lidar_3d_plugin
-      node_namespace="${node_namespace}"
-      node_name="${node_name}"
-      gazebo_ignition="${gazebo_ignition}"
-      min_range="0.2"
-      max_range="150.0"
-      min_angle="-15.0"
-      max_angle="15.0"
-      frame_link="${frame_prefix}link"
-      rate="10"
-      horizontal_samples="1800"
-      vertical_samples="16" />
+    <xacro:if value="${low_performance}">
+      <xacro:lidar_3d_plugin
+        node_namespace="${node_namespace}"
+        node_name="${node_name}"
+        gazebo_ignition="${gazebo_ignition}"
+        min_range="0.2"
+        max_range="60.0"
+        min_angle="-15.0"
+        max_angle="15.0"
+        frame_link="${frame_prefix}link"
+        rate="5"
+        horizontal_samples="900"
+        vertical_samples="16" />
+    </xacro:if>
+    <xacro:unless value="${low_performance}">
+      <xacro:lidar_3d_plugin
+        node_namespace="${node_namespace}"
+        node_name="${node_name}"
+        gazebo_ignition="${gazebo_ignition}"
+        min_range="0.2"
+        max_range="150.0"
+        min_angle="-15.0"
+        max_angle="15.0"
+        frame_link="${frame_prefix}link"
+        rate="10"
+        horizontal_samples="1800"
+        vertical_samples="16" />
+    </xacro:unless>
   </xacro:macro>
 </robot>

File: robotnik_sensors/urdf/all_sensors.urdf.xacro (robot description, xacro)
@@ -4,4 +4,7 @@
   xmlns:xacro="http://wiki.ros.org/xacro">
   <!-- This file unifies all sensors that can be used on simulation, defined as xacro:macros -->
+  <!-- Declare global argument to set low_performance mode -->
+  <xacro:arg name="low_performance" default="false" />
+  <xacro:property name="low_performance" value="$(arg low_performance)" />
   <xacro:include
     filename="$(find robotnik_sensors)/urdf/utils/inertia.urdf.xacro" />

File: robotnik_sensors/urdf/camera/link_750_nh.urdf.xacro (robot description, xacro)
@@ -264,18 +264,36 @@
     </gazebo>
     <!-- camera sensor for simulation -->
-    <xacro:camera_plugin
-      node_namespace="${node_namespace}"
-      node_name="${node_name}_color"
-      topic_prefix="${topic_prefix}_color"
-      gazebo_ignition="${gazebo_ignition}"
-      optical_frame="${frame_prefix}optical_frame_link"
-      reference_frame="${frame_prefix}frame_link"
-      horizontal_fov="63.7"
-      vertical_fov="32"
-      video_width="1920"
-      video_height="1080"
-      min_depth="0.1"
-      max_depth="100"
-      rate="30" />
+    <xacro:if value="${low_performance}">
+      <xacro:camera_plugin
+        node_namespace="${node_namespace}"
+        node_name="${node_name}_color"
+        topic_prefix="${topic_prefix}_color"
+        gazebo_ignition="${gazebo_ignition}"
+        optical_frame="${frame_prefix}optical_frame_link"
+        reference_frame="${frame_prefix}frame_link"
+        horizontal_fov="63.7"
+        vertical_fov="32"
+        video_width="1280"
+        video_height="720"
+        min_depth="0.1"
+        max_depth="100"
+        rate="5" />
+    </xacro:if>
+    <xacro:unless value="${low_performance}">
+      <xacro:camera_plugin
+        node_namespace="${node_namespace}"
+        node_name="${node_name}_color"
+        topic_prefix="${topic_prefix}_color"
+        gazebo_ignition="${gazebo_ignition}"
+        optical_frame="${frame_prefix}optical_frame_link"
+        reference_frame="${frame_prefix}frame_link"
+        horizontal_fov="63.7"
+        vertical_fov="32"
+        video_width="1920"
+        video_height="1080"
+        min_depth="0.1"
+        max_depth="100"
+        rate="25" />
+    </xacro:unless>
     <ros2_control
       name="${node_name}_control"

File: robotnik_sensors/urdf/depth/intel_realsense_d435.urdf.xacro (robot description, xacro)
@@ -198,18 +198,36 @@
     </joint>
     <link name="${frame_prefix}color_optical_frame" />
-    <xacro:camera_plugin
-      node_namespace="${node_namespace}"
-      node_name="${node_name}_color"
-      topic_prefix="${topic_prefix}_color"
-      gazebo_ignition="${gazebo_ignition}"
-      optical_frame="${frame_prefix}color_optical_frame"
-      reference_frame="${frame_prefix}color_frame"
-      horizontal_fov="69.4"
-      vertical_fov="39"
-      video_width="1920"
-      video_height="1080"
-      min_depth="0.1"
-      max_depth="100"
-      rate="30" />
+    <xacro:if value="${low_performance}">
+      <xacro:camera_plugin
+        node_namespace="${node_namespace}"
+        node_name="${node_name}_color"
+        topic_prefix="${topic_prefix}_color"
+        gazebo_ignition="${gazebo_ignition}"
+        optical_frame="${frame_prefix}color_optical_frame"
+        reference_frame="${frame_prefix}color_frame"
+        horizontal_fov="69.4"
+        vertical_fov="39"
+        video_width="1280"
+        video_height="720"
+        min_depth="0.1"
+        max_depth="100"
+        rate="5" />
+    </xacro:if>
+    <xacro:unless value="${low_performance}">
+      <xacro:camera_plugin
+        node_namespace="${node_namespace}"
+        node_name="${node_name}_color"
+        topic_prefix="${topic_prefix}_color"
+        gazebo_ignition="${gazebo_ignition}"
+        optical_frame="${frame_prefix}color_optical_frame"
+        reference_frame="${frame_prefix}color_frame"
+        horizontal_fov="69.4"
+        vertical_fov="39"
+        video_width="1920"
+        video_height="1080"
+        min_depth="0.1"
+        max_depth="100"
+        rate="30" />
+    </xacro:unless>
   </xacro:macro>
 </robot>
