Commit message: change mesh ublox mast

File: robotnik_sensors/urdf/gps/ublox_with_mast.urdf.xacro (robot description, xacro)
@@ -30,5 +30,5 @@
           </material>
 	      <geometry>
-	        <cylinder length="${mast_height}" radius="${mast_radius}" />
+                <mesh filename="package://robotnik_sensors/meshes/os1_128_support.STL" scale="1.0 1.0 1.0"/>
 	      </geometry>
 	    </visual>
@@ -36,5 +36,5 @@
 	      <origin rpy="0 0 0" xyz="0 0 0"/>
 	      <geometry>
-	        <cylinder length="${mast_height}" radius="${mast_radius}" />
+                <box size="0.05 0.05 0.2"/>
 	      </geometry>
 	    </collision>

Commit message: orient mesh

File: robotnik_sensors/urdf/gps/ublox_with_mast.urdf.xacro (robot description, xacro)
@@ -25,5 +25,5 @@
 		</inertial>
 	    <visual>
-	      <origin rpy="0 0 0" xyz="0 0 0"/>
+	      <origin rpy="0 0 -1.57" xyz="0 0 0"/>
 	      <material name="mast_color">
             <color rgba="0.1 0.1 0.1 1"/>
@@ -43,5 +43,5 @@
 	    <parent link="${frame_prefix}mast_base_link"/>
 	    <child link="${frame_prefix}base_link"/>
-	    <origin xyz="0 0 ${mast_height/2.0}" rpy="0 0 0" />
+	    <origin xyz="0 0 0" rpy="0 0 0" />
 	  </joint>
 	  <gazebo reference="${frame_prefix}mast_base_link">

Commit message: change mesh

File: robotnik_sensors/urdf/gps/ublox_with_mast.urdf.xacro (robot description, xacro)
@@ -25,10 +25,10 @@
 		</inertial>
 	    <visual>
-	      <origin rpy="0 0 -1.57" xyz="0 0 0"/>
+	      <origin rpy="0 0 0" xyz="0 0 0"/>
 	      <material name="mast_color">
             <color rgba="0.1 0.1 0.1 1"/>
           </material>
 	      <geometry>
-                <mesh filename="package://robotnik_sensors/meshes/os1_128_support.STL" scale="1.0 1.0 1.0"/>
+	            <mesh filename="package://robotnik_sensors/meshes/ublox_support.STL" scale="1.0 1.0 1.0"/>
 	      </geometry>
 	    </visual>
@@ -43,5 +43,5 @@
 	    <parent link="${frame_prefix}mast_base_link"/>
 	    <child link="${frame_prefix}base_link"/>
-	    <origin xyz="0 0 0" rpy="0 0 0" />
+	    <origin xyz="0 0 0.257" rpy="0 0 0" />
 	  </joint>
 	  <gazebo reference="${frame_prefix}mast_base_link">

Commit message: fix tests

File: robotnik_sensors/urdf/gps/ublox_with_mast.urdf.xacro (robot description, xacro)
@@ -32,5 +32,5 @@
           </material>
 	      <geometry>
-	            <mesh filename="package://robotnik_sensors/meshes/ublox_support.STL" scale="1.0 1.0 1.0"/>
+                <box size="0.05 0.05 0.2"/>
 	      </geometry>
 	    </visual>

Commit message: Update ublox_with_mast.urdf.xacro

File: robotnik_sensors/urdf/gps/ublox_with_mast.urdf.xacro (robot description, xacro)
@@ -25,20 +25,20 @@
 			<mass value="0.2" />
 			<xacro:solid_cuboid_inertia m="0.2" w="0.081" h="0.081" d="0.03" />
-      </inertial>
-	    <visual>
-	      <origin rpy="0 0 0" xyz="0 0 0"/>
-		  <material name="ublox_gps_color">
-           <color rgba="0.5 0.5 0.5 1"/>
-          </material>
-	      <geometry>
-	        <mesh filename="package://robotnik_sensors/meshes/gps/antenna_ANN_MB.stl" scale="1.0 1.0 1.0"/>
-	      </geometry>
-	    </visual>
-	    <collision>
-	      <origin rpy="0 0 0" xyz="0 0 0.01125"/>
-	        <geometry>
-	          <box size="0.0607 0.083 0.0225"/>
-	        </geometry>
-	    </collision>
+      		</inertial>
+	    	<visual>
+	      		<origin rpy="0 0 0" xyz="0 0 0"/>
+		  	<material name="ublox_gps_color">
+           			<color rgba="0.5 0.5 0.5 1"/>
+          		</material>
+		        <geometry>
+				<mesh filename="package://robotnik_sensors/meshes/gps/antenna_ANN_MB.stl" scale="1.0 1.0 1.0"/>
+		        </geometry>
+	    	</visual>
+	        <collision>
+	          	<origin rpy="0 0 0" xyz="0 0 0.01125"/>
+		        <geometry>
+		     		<box size="0.0607 0.083 0.0225"/>
+		        </geometry>
+	        </collision>
 	  </link>
 	  <joint name="${frame_prefix}mast_joint" type="fixed">
@@ -53,19 +53,19 @@
 			<xacro:solid_cuboid_inertia m="1.0" w="${mast_radius}" h="${mast_radius}" d="${mast_height}" />
 		</inertial>
-	    <visual>
-	      <origin rpy="0 0 0" xyz="0 0 0"/>
-	      <material name="mast_color">
-            <color rgba="0.1 0.1 0.1 1"/>
-          </material>
-	      <geometry>
-	            <mesh filename="package://robotnik_sensors/meshes/gps/mastil_gps.stl" scale="1.0 1.0 1.0"/>
-	      </geometry>
-	    </visual>
-	    <collision>
-	      <origin rpy="0 0 0" xyz="0 0 0"/>
-	      <geometry>
-                <box size="0.05 0.05 0.2"/>
-	      </geometry>
-	    </collision>
+	    	<visual>
+		      <origin rpy="0 0 0" xyz="0 0 0"/>
+		      <material name="mast_color">
+	              	    <color rgba="0.1 0.1 0.1 1"/>
+         	      </material>
+		      <geometry>
+		            <mesh filename="package://robotnik_sensors/meshes/gps/mastil_gps.stl" scale="1.0 1.0 1.0"/>
+		      </geometry>
+	    	</visual>
+	        <collision>
+	            <origin rpy="0 0 0" xyz="0 0 0"/>
+	            <geometry>
+			<box size="0.05 0.05 0.2"/>
+	            </geometry>
+	    	</collision>
 	  </link>
 	  <gazebo reference="${frame_prefix}mast_base_link">
@@ -76,5 +76,5 @@
 	    <material>Gazebo/White</material>
 	    <gravity>true</gravity>
-	  </gazebo>
+	</gazebo>
     <xacro:gps_plugin
       node_namespace="${node_namespace}"
