Commit message: fix gps

File: robotnik_sensors/urdf/gps/ublox.urdf.xacro (robot description, xacro)
@@ -40,12 +40,4 @@
 	    </collision>
 	  </link>
-	  <joint name="${frame_prefix}joint" type="fixed">
-	      <axis xyz="1 0 0"/>
-	      <origin xyz="0.0 0.0 0.01125"/>
-	      <parent link="${frame_prefix}base_link"/>
-	      <child link="${frame_prefix}link"/>
-	  </joint>
-	  <link name="${frame_prefix}link">
-	  </link>
 	<gazebo reference="${frame_prefix}base_link">
 	    <material>Gazebo/White</material>

File: robotnik_sensors/urdf/gps/ublox_with_mast.urdf.xacro (robot description, xacro)
@@ -15,43 +15,7 @@
 						update_rate:=5.0">
 	  <!-- ANTENNA GPS -->
-	  <joint name="${frame_prefix}joint" type="fixed">
+	  <joint name="${frame_prefix}base_joint" type="fixed">
 	    <xacro:insert_block name="origin"/>
 	    <parent link="${parent}"/>
-	    <child link="${frame_prefix}mast_base_link"/>
-	  </joint>
-	  <link name="${frame_prefix}mast_base_link">
-		<inertial>
-			<origin xyz="0.0 0 0.0" rpy="0 0 0" />
-			<mass value="1.0" />
-			<xacro:solid_cuboid_inertia m="1.0" w="${mast_radius}" h="${mast_radius}" d="${mast_height}" />
-		</inertial>
-	    <visual>
-	      <origin rpy="0 0 0" xyz="0 0 0"/>
-	      <material name="mast_color">
-            <color rgba="0.1 0.1 0.1 1"/>
-          </material>
-	      <geometry>
-                <box size="0.05 0.05 0.2"/>
-	      </geometry>
-	    </visual>
-	    <collision>
-	      <origin rpy="0 0 0" xyz="0 0 0"/>
-	      <geometry>
-                <box size="0.05 0.05 0.2"/>
-	      </geometry>
-	    </collision>
-	  </link>
-	  <joint name="${frame_prefix}mast_joint" type="fixed">
-	    <parent link="${frame_prefix}mast_base_link"/>
-	    <child link="${frame_prefix}base_link"/>
-	    <origin xyz="0 0 0.257" rpy="0 0 0" />
-	  </joint>
-	  <gazebo reference="${frame_prefix}mast_base_link">
-	    <material>Gazebo/Black</material>
-	    <gravity>true</gravity>
-	  </gazebo>
-	  <joint name="${frame_prefix}base_joint" type="fixed">
-	    <xacro:insert_block name="origin"/>
-	    <parent link="${frame_prefix}mast_base_link"/>
 	    <child link="${frame_prefix}base_link"/>
 	  </joint>
@@ -78,4 +42,35 @@
 	    </collision>
 	  </link>
+	  <joint name="${frame_prefix}mast_joint" type="fixed">
+	    <parent link="${frame_prefix}base_link"/>
+	    <child link="${frame_prefix}mast_base_link"/>
+	    <origin xyz="0 0 -0.37" rpy="0 0 0" />
+	  </joint>
+	  <link name="${frame_prefix}mast_base_link">
+		<inertial>
+			<origin xyz="0.0 0 0.0" rpy="0 0 0" />
+			<mass value="1.0" />
+			<xacro:solid_cuboid_inertia m="1.0" w="${mast_radius}" h="${mast_radius}" d="${mast_height}" />
+		</inertial>
+	    <visual>
+	      <origin rpy="0 0 0" xyz="0 0 0"/>
+	      <material name="mast_color">
+            <color rgba="0.1 0.1 0.1 1"/>
+          </material>
+	      <geometry>
+	            <mesh filename="package://robotnik_sensors/meshes/gps/mastil_gps.stl" scale="1.0 1.0 1.0"/>
+	      </geometry>
+	    </visual>
+	    <collision>
+	      <origin rpy="0 0 0" xyz="0 0 0"/>
+	      <geometry>
+                <box size="0.05 0.05 0.2"/>
+	      </geometry>
+	    </collision>
+	  </link>
+	  <gazebo reference="${frame_prefix}mast_base_link">
+	    <material>Gazebo/Black</material>
+	    <gravity>true</gravity>
+	  </gazebo>
 	<gazebo reference="${frame_prefix}base_link">
 	    <material>Gazebo/White</material>

Commit message: Update ublox.urdf.xacro

File: robotnik_sensors/urdf/gps/ublox.urdf.xacro (robot description, xacro)
@@ -23,5 +23,5 @@
 			<mass value="0.2" />
 			<xacro:solid_cuboid_inertia m="0.2" w="0.081" h="0.081" d="0.03" />
-      </inertial>
+                </inertial>
 	    <visual>
 	      <origin rpy="0 0 0" xyz="0 0 0"/>
@@ -40,8 +40,16 @@
 	    </collision>
 	  </link>
-	<gazebo reference="${frame_prefix}base_link">
+	  <gazebo reference="${frame_prefix}base_link">
 	    <material>Gazebo/White</material>
 	    <gravity>true</gravity>
 	  </gazebo>
+	  <joint name="${frame_prefix}joint" type="fixed">
+	      <axis xyz="1 0 0"/>
+	      <origin xyz="0.0 0.0 0.01125"/>
+	      <parent link="${frame_prefix}base_link"/>
+	      <child link="${frame_prefix}link"/>
+	  </joint>
+	  <link name="${frame_prefix}link">
+	  </link>
     <xacro:gps_plugin
       node_namespace="${node_namespace}"

Commit message: Update ublox.urdf.xacro

File: robotnik_sensors/urdf/gps/ublox.urdf.xacro (robot description, xacro)
@@ -45,5 +45,4 @@
 	  </gazebo>
 	  <joint name="${frame_prefix}joint" type="fixed">
-	      <axis xyz="1 0 0"/>
 	      <origin xyz="0.0 0.0 0.01125"/>
 	      <parent link="${frame_prefix}base_link"/>
