Commit message: Fix/ros2/fix jazzy sensors (#50)
* fix gps

* fix lidar 3D gazebo

* removed temporary plugins for depth image in gazebo (issues with computation)

* Update intel_realsense_d435.urdf.xacro

remove plugin that are not working #49

* Update ublox_with_mast.urdf.xacro

* Update ublox.urdf.xacro

* Update ublox.urdf.xacro

* Update lidar_3d_plugin.urdf.xacro

* Changed CHANGELOG

File: robotnik_sensors/urdf/depth/intel_realsense_d435.urdf.xacro (robot description, xacro)
@@ -137,55 +137,4 @@
       >
       </xacro:camera_plugin>
-      <xacro:irred_camera_plugin
-        node_namespace="${node_namespace}"
-        node_name="${node_name}_irred1"
-        topic_prefix="${topic_prefix}_irred1"
-        gazebo_classic="${gazebo_classic}"
-        gazebo_ignition="${gazebo_ignition}"
-        optical_frame="${frame_prefix}infra1_optical_frame"
-        reference_frame="${frame_prefix}infra2_frame"
-        horizontal_fov="85.2"
-        vertical_fov="48"
-        video_width="1280"
-        video_height="720"
-        min_depth="0.1"
-        max_depth="100"
-        rate="30"
-      >
-      </xacro:irred_camera_plugin>
-      <xacro:irred_camera_plugin
-        node_namespace="${node_namespace}"
-        node_name="${node_name}_irred2"
-        topic_prefix="${topic_prefix}_irred2"
-        gazebo_classic="${gazebo_classic}"
-        gazebo_ignition="${gazebo_ignition}"
-        optical_frame="${frame_prefix}infra2_optical_frame"
-        reference_frame="${frame_prefix}infra2_frame"
-        horizontal_fov="85.2"
-        vertical_fov="48"
-        video_width="1280"
-        video_height="720"
-        min_depth="0.1"
-        max_depth="100"
-        rate="30"
-      >
-      </xacro:irred_camera_plugin>
-      <xacro:depth_camera_plugin
-        node_namespace="${node_namespace}"
-        node_name="${node_name}_depth"
-        topic_prefix="${topic_prefix}_depth"
-        gazebo_classic="${gazebo_classic}"
-        gazebo_ignition="${gazebo_ignition}"
-        optical_frame="${frame_prefix}depth_optical_frame"
-        reference_frame="${frame_prefix}depth_frame"
-        horizontal_fov="85.2"
-        vertical_fov="48"
-        video_width="1280"
-        video_height="720"
-        min_depth="0.1"
-        max_depth="100"
-        rate="30"
-      >
-      </xacro:depth_camera_plugin>
   </xacro:macro>
 </robot>

File: robotnik_sensors/urdf/gps/ublox.urdf.xacro (robot description, xacro)
@@ -23,5 +23,5 @@
 			<mass value="0.2" />
 			<xacro:solid_cuboid_inertia m="0.2" w="0.081" h="0.081" d="0.03" />
-      </inertial>
+                </inertial>
 	    <visual>
 	      <origin rpy="0 0 0" xyz="0 0 0"/>
@@ -40,6 +40,9 @@
 	    </collision>
 	  </link>
+	  <gazebo reference="${frame_prefix}base_link">
+	    <material>Gazebo/White</material>
+	    <gravity>true</gravity>
+	  </gazebo>
 	  <joint name="${frame_prefix}joint" type="fixed">
-	      <axis xyz="1 0 0"/>
 	      <origin xyz="0.0 0.0 0.01125"/>
 	      <parent link="${frame_prefix}base_link"/>
@@ -48,8 +51,4 @@
 	  <link name="${frame_prefix}link">
 	  </link>
-	<gazebo reference="${frame_prefix}base_link">
-	    <material>Gazebo/White</material>
-	    <gravity>true</gravity>
-	  </gazebo>
     <xacro:gps_plugin
       node_namespace="${node_namespace}"

File: robotnik_sensors/urdf/gps/ublox_with_mast.urdf.xacro (robot description, xacro)
@@ -15,8 +15,35 @@
 						update_rate:=5.0">
 	  <!-- ANTENNA GPS -->
-	  <joint name="${frame_prefix}joint" type="fixed">
+	  <joint name="${frame_prefix}base_joint" type="fixed">
 	    <xacro:insert_block name="origin"/>
 	    <parent link="${parent}"/>
+	    <child link="${frame_prefix}base_link"/>
+	  </joint>
+	  <link name="${frame_prefix}base_link">
+		<inertial>
+			<origin xyz="0.0 0 0.015" rpy="0 0 0" />
+			<mass value="0.2" />
+			<xacro:solid_cuboid_inertia m="0.2" w="0.081" h="0.081" d="0.03" />
+      		</inertial>
+	    	<visual>
+	      		<origin rpy="0 0 0" xyz="0 0 0"/>
+		  	<material name="ublox_gps_color">
+           			<color rgba="0.5 0.5 0.5 1"/>
+          		</material>
+		        <geometry>
+				<mesh filename="package://robotnik_sensors/meshes/gps/antenna_ANN_MB.stl" scale="1.0 1.0 1.0"/>
+		        </geometry>
+	    	</visual>
+	        <collision>
+	          	<origin rpy="0 0 0" xyz="0 0 0.01125"/>
+		        <geometry>
+		     		<box size="0.0607 0.083 0.0225"/>
+		        </geometry>
+	        </collision>
+	  </link>
+	  <joint name="${frame_prefix}mast_joint" type="fixed">
+	    <parent link="${frame_prefix}base_link"/>
 	    <child link="${frame_prefix}mast_base_link"/>
+	    <origin xyz="0 0 -0.37" rpy="0 0 0" />
 	  </joint>
 	  <link name="${frame_prefix}mast_base_link">
@@ -26,60 +53,28 @@
 			<xacro:solid_cuboid_inertia m="1.0" w="${mast_radius}" h="${mast_radius}" d="${mast_height}" />
 		</inertial>
-	    <visual>
-	      <origin rpy="0 0 0" xyz="0 0 0"/>
-	      <material name="mast_color">
-            <color rgba="0.1 0.1 0.1 1"/>
-          </material>
-	      <geometry>
-                <box size="0.05 0.05 0.2"/>
-	      </geometry>
-	    </visual>
-	    <collision>
-	      <origin rpy="0 0 0" xyz="0 0 0"/>
-	      <geometry>
-                <box size="0.05 0.05 0.2"/>
-	      </geometry>
-	    </collision>
+	    	<visual>
+		      <origin rpy="0 0 0" xyz="0 0 0"/>
+		      <material name="mast_color">
+	              	    <color rgba="0.1 0.1 0.1 1"/>
+         	      </material>
+		      <geometry>
+		            <mesh filename="package://robotnik_sensors/meshes/gps/mastil_gps.stl" scale="1.0 1.0 1.0"/>
+		      </geometry>
+	    	</visual>
+	        <collision>
+	            <origin rpy="0 0 0" xyz="0 0 0"/>
+	            <geometry>
+			<box size="0.05 0.05 0.2"/>
+	            </geometry>
+	    	</collision>
 	  </link>
-	  <joint name="${frame_prefix}mast_joint" type="fixed">
-	    <parent link="${frame_prefix}mast_base_link"/>
-	    <child link="${frame_prefix}base_link"/>
-	    <origin xyz="0 0 0.257" rpy="0 0 0" />
-	  </joint>
 	  <gazebo reference="${frame_prefix}mast_base_link">
 	    <material>Gazebo/Black</material>
 	    <gravity>true</gravity>
 	  </gazebo>
-	  <joint name="${frame_prefix}base_joint" type="fixed">
-	    <xacro:insert_block name="origin"/>
-	    <parent link="${frame_prefix}mast_base_link"/>
-	    <child link="${frame_prefix}base_link"/>
-	  </joint>
-	  <link name="${frame_prefix}base_link">
-		<inertial>
-			<origin xyz="0.0 0 0.015" rpy="0 0 0" />
-			<mass value="0.2" />
-			<xacro:solid_cuboid_inertia m="0.2" w="0.081" h="0.081" d="0.03" />
-      </inertial>
-	    <visual>
-	      <origin rpy="0 0 0" xyz="0 0 0"/>
-		  <material name="ublox_gps_color">
-           <color rgba="0.5 0.5 0.5 1"/>
-          </material>
-	      <geometry>
-	        <mesh filename="package://robotnik_sensors/meshes/gps/antenna_ANN_MB.stl" scale="1.0 1.0 1.0"/>
-	      </geometry>
-	    </visual>
-	    <collision>
-	      <origin rpy="0 0 0" xyz="0 0 0.01125"/>
-	        <geometry>
-	          <box size="0.0607 0.083 0.0225"/>
-	        </geometry>
-	    </collision>
-	  </link>
 	<gazebo reference="${frame_prefix}base_link">
 	    <material>Gazebo/White</material>
 	    <gravity>true</gravity>
-	  </gazebo>
+	</gazebo>
     <xacro:gps_plugin
       node_namespace="${node_namespace}"
