Commit message: added readme and improved linter config

File: robotnik_sensors/urdf/2d_lidar/hokuyo_urg04lx.urdf.xacro (robot description, xacro)
@@ -33,5 +33,5 @@
           rpy="0 0 0" />
         <geometry>
-            <mesh
+          <mesh
             filename="package://robotnik_sensors/meshes/hokuyo_urg_04lx.dae" />
         </geometry>
@@ -58,6 +58,5 @@
         rpy="0 0 0" />
     </joint>
-    <link name="${frame_prefix}link">
-    </link>
+    <link name="${frame_prefix}link" />
     <!-- Hokuyo sensor for simulation -->
     <xacro:lidar_2d_plugin
@@ -72,6 +71,5 @@
       rate="10"
       resolution="0.004359297"
-      samples="640">
-    </xacro:lidar_2d_plugin>
+      samples="640" />
   </xacro:macro>
 </robot>

File: robotnik_sensors/urdf/2d_lidar/hokuyo_ust10lx.urdf.xacro (robot description, xacro)
@@ -42,5 +42,5 @@
           rpy="0 0 0" />
         <geometry>
-            <mesh
+          <mesh
             filename="package://robotnik_sensors/meshes/hokuyo_ust_10lx.dae" />
         </geometry>
@@ -67,6 +67,5 @@
       <child link="${frame_prefix}link" />
     </joint>
-    <link name="${frame_prefix}link">
-    </link>
+    <link name="${frame_prefix}link" />
     <!-- Hokuyo sensor for simulation -->
     <xacro:lidar_2d_plugin
@@ -81,6 +80,5 @@
       rate="40"
       resolution="0.004359297"
-      samples="1081">
-    </xacro:lidar_2d_plugin>
+      samples="1081" />
   </xacro:macro>
 </robot>

File: robotnik_sensors/urdf/2d_lidar/hokuyo_ust20lx.urdf.xacro (robot description, xacro)
@@ -68,5 +68,5 @@
         xyz="0.00 0.0 0.0474"
         rpy="0 0 0" />
-	  </joint>
+    </joint>
     <link name="${frame_prefix}link" />
     <!-- Hokuyo sensor for simulation -->
@@ -82,6 +82,5 @@
       rate="40"
       resolution="0.004359297"
-      samples="1081">
-    </xacro:lidar_2d_plugin>
+      samples="1081" />
   </xacro:macro>
 </robot>

File: robotnik_sensors/urdf/2d_lidar/hokuyo_utm30lx.urdf.xacro (robot description, xacro)
@@ -38,5 +38,5 @@
           rpy="0 0 0" />
         <geometry>
-            <mesh
+          <mesh
             filename="package://robotnik_sensors/meshes/hokuyo_utm_30lx.dae" />
         </geometry>
@@ -62,7 +62,6 @@
         xyz="0.00 0 0.055"
         rpy="0 0 0" />
-	  </joint>
-    <link name="${frame_prefix}link">
-    </link>
+    </joint>
+    <link name="${frame_prefix}link" />
     <!-- Hokuyo sensor for simulation -->
     <xacro:lidar_2d_plugin
@@ -77,6 +76,5 @@
       rate="30"
       resolution="0.01"
-      samples="1081">
-    </xacro:lidar_2d_plugin>
+      samples="1081" />
   </xacro:macro>
 </robot>

File: robotnik_sensors/urdf/2d_lidar/sick_microscan3.urdf.xacro (robot description, xacro)
@@ -34,5 +34,5 @@
           rpy="0 0 0" />
         <geometry>
-		  <mesh
+          <mesh
             filename="package://robotnik_sensors/meshes/2d_lidar/sick/microscan3.dae" />
         </geometry>
@@ -43,5 +43,5 @@
           rpy="0 0 0" />
         <geometry>
-		  <mesh
+          <mesh
             filename="package://robotnik_sensors/meshes/2d_lidar/sick/microscan3.dae" />
         </geometry>
@@ -62,5 +62,5 @@
       name="${frame_prefix}joint"
       type="fixed">
-		  <origin
+      <origin
         xyz="0.0 0 0.110"
         rpy="0 0 0" />
@@ -81,6 +81,5 @@
       rate="30"
       resolution="0.00575"
-      samples="700">
-    </xacro:lidar_2d_plugin>
+      samples="700" />
   </xacro:macro>
 </robot>

File: robotnik_sensors/urdf/2d_lidar/sick_nanoscan3.urdf.xacro (robot description, xacro)
@@ -34,5 +34,5 @@
           rpy="0 0 0" />
         <geometry>
-		  <mesh
+          <mesh
             filename="package://robotnik_sensors/meshes/2d_lidar/sick/nanoscan3.stl" />
         </geometry>
@@ -43,5 +43,5 @@
           rpy="0 0 0" />
         <geometry>
-		  <mesh
+          <mesh
             filename="package://robotnik_sensors/meshes/2d_lidar/sick/nanoscan3.stl" />
         </geometry>
@@ -57,5 +57,5 @@
           h="0.1006"
           d="0.08" />
-	  </inertial>
+      </inertial>
     </link>
     <joint
@@ -81,6 +81,5 @@
       rate="12.5"
       resolution="0.00575"
-      samples="1600">
-    </xacro:lidar_2d_plugin>
+      samples="1600" />
   </xacro:macro>
 </robot>

File: robotnik_sensors/urdf/2d_lidar/sick_outdoorscan3.urdf.xacro (robot description, xacro)
@@ -34,5 +34,5 @@
           rpy="0 0 0" />
         <geometry>
-		  <mesh
+          <mesh
             filename="package://robotnik_sensors/meshes/2d_lidar/sick/outdoorscan3.dae" />
         </geometry>
@@ -43,24 +43,24 @@
           rpy="0 0 0" />
         <geometry>
-		  <mesh
+          <mesh
             filename="package://robotnik_sensors/meshes/2d_lidar/sick/outdoorscan3.dae" />
         </geometry>
       </collision>
       <inertial>
-		<mass value="1.15" />
-		<origin
+        <mass value="1.15" />
+        <origin
           xyz="0 0 0.075"
           rpy="0 0 0" />
-		<xacro:solid_cuboid_inertia
+        <xacro:solid_cuboid_inertia
           m="1.15"
           w="0.112"
           h="0.111"
           d="0.15" />
-	  </inertial>
+      </inertial>
     </link>
     <joint
       name="${frame_prefix}joint"
       type="fixed">
-	  <origin
+      <origin
         xyz="0.0 0 0.110"
         rpy="0 0 0" />
@@ -80,6 +80,5 @@
       rate="12.5"
       resolution="0.00575"
-      samples="700">
-    </xacro:lidar_2d_plugin>
+      samples="700" />
   </xacro:macro>
   <xacro:macro name="sensor_sick_outdoorscan3_gazebo">
@@ -94,43 +93,43 @@
         value="ray" />
     </xacro:unless>
-      <gazebo reference="${frame_prefix}link">
-        <sensor
+    <gazebo reference="${frame_prefix}link">
+      <sensor
         type="${ray_type}"
         name="${frame_prefix}sensor">
-          <pose>0.0 0.0 0.0 0.0 0.0 0.0</pose>
-          <visualize>false</visualize>
-		      <update_rate>12.5</update_rate>
-          <ray>
-            <scan>
-              <horizontal>
-                <samples>700</samples>
-                <resolution>1</resolution>
-                <min_angle>${-radians(135)}</min_angle>
-                <max_angle>${radians(135)}</max_angle>
-              </horizontal>
-            </scan>
-            <range>
-              <min>0.05</min>
-			        <max>40.0</max>
-              <resolution>0.00575</resolution>
-            </range>
-            <noise>
-              <type>gaussian</type>
-              <mean>0.0</mean>
-              <stddev>0.01</stddev>
-            </noise>
-          </ray>
-          <plugin
+        <pose>0.0 0.0 0.0 0.0 0.0 0.0</pose>
+        <visualize>false</visualize>
+        <update_rate>12.5</update_rate>
+        <ray>
+          <scan>
+            <horizontal>
+              <samples>700</samples>
+              <resolution>1</resolution>
+              <min_angle>${-radians(135)}</min_angle>
+              <max_angle>${radians(135)}</max_angle>
+            </horizontal>
+          </scan>
+          <range>
+            <min>0.05</min>
+            <max>40.0</max>
+            <resolution>0.00575</resolution>
+          </range>
+          <noise>
+            <type>gaussian</type>
+            <mean>0.0</mean>
+            <stddev>0.01</stddev>
+          </noise>
+        </ray>
+        <plugin
           name="${node_name}"
           filename="libgazebo_ros_ray_sensor.so">
-            <ros>
-              <namespace>${node_namespace}</namespace>
-              <remapping>~/out:=~/scan</remapping>
-            </ros>
-            <output_type>sensor_msgs/LaserScan</output_type>
-            <frame_name>${frame_prefix}link</frame_name>
-          </plugin>
-        </sensor>
-      </gazebo>
+          <ros>
+            <namespace>${node_namespace}</namespace>
+            <remapping>~/out:=~/scan</remapping>
+          </ros>
+          <output_type>sensor_msgs/LaserScan</output_type>
+          <frame_name>${frame_prefix}link</frame_name>
+        </plugin>
+      </sensor>
+    </gazebo>
   </xacro:macro>
 </robot>

File: robotnik_sensors/urdf/2d_lidar/sick_s300.urdf.xacro (robot description, xacro)
@@ -80,6 +80,5 @@
       rate="25.0"
       resolution="0.00575"
-      samples="270">
-    </xacro:lidar_2d_plugin>
+      samples="270" />
   </xacro:macro>
 </robot>

File: robotnik_sensors/urdf/2d_lidar/sick_s3000.urdf.xacro (robot description, xacro)
@@ -34,5 +34,5 @@
           rpy="0 0 0" />
         <geometry>
-		  <mesh
+          <mesh
             filename="package://robotnik_sensors/meshes/2d_lidar/sick/s3000.dae" />
         </geometry>
@@ -43,5 +43,5 @@
           rpy="0 0 0" />
         <geometry>
-		  <mesh
+          <mesh
             filename="package://robotnik_sensors/meshes/2d_lidar/sick/s3000.dae" />
         </geometry>
@@ -57,5 +57,5 @@
           h="0.160"
           d="0.185" />
-	  </inertial>
+      </inertial>
     </link>
     <joint
@@ -80,6 +80,5 @@
       rate="15.0"
       resolution="0.00575"
-      samples="380">
-    </xacro:lidar_2d_plugin>
+      samples="380" />
   </xacro:macro>
 </robot>

File: robotnik_sensors/urdf/2d_lidar/sick_tim551.urdf.xacro (robot description, xacro)
@@ -34,5 +34,5 @@
           rpy="0 0 0" />
         <geometry>
-         <mesh
+          <mesh
             filename="package://robotnik_sensors/meshes/2d_lidar/sick/tim551.dae" />
         </geometry>
@@ -43,5 +43,5 @@
           rpy="0 0 0" />
         <geometry>
-            <mesh
+          <mesh
             filename="package://robotnik_sensors/meshes/2d_lidar/sick/tim551.dae" />
         </geometry>
@@ -80,6 +80,5 @@
       rate="15.0"
       resolution="0.00575"
-      samples="1600">
-    </xacro:lidar_2d_plugin>
+      samples="1600" />
   </xacro:macro>
 </robot>

File: robotnik_sensors/urdf/2d_lidar/sick_tim571.urdf.xacro (robot description, xacro)
@@ -34,5 +34,5 @@
           rpy="0 0 0" />
         <geometry>
-         <mesh
+          <mesh
             filename="package://robotnik_sensors/meshes/2d_lidar/sick/tim571.dae" />
         </geometry>
@@ -43,5 +43,5 @@
           rpy="0 0 0" />
         <geometry>
-            <mesh
+          <mesh
             filename="package://robotnik_sensors/meshes/2d_lidar/sick/tim571.dae" />
         </geometry>
@@ -80,6 +80,5 @@
       rate="15.0"
       resolution="0.00575"
-      samples="810">
-    </xacro:lidar_2d_plugin>
+      samples="810" />
   </xacro:macro>
 </robot>

File: robotnik_sensors/urdf/3d_lidar/livox_mid_360.urdf.xacro (robot description, xacro)
@@ -85,6 +85,5 @@
       rate="10"
       horizontal_samples="1200"
-      vertical_samples="32">
-    </xacro:lidar_3d_plugin>
+      vertical_samples="32" />
   </xacro:macro>
 </robot>

File: robotnik_sensors/urdf/3d_lidar/ouster.urdf.xacro (robot description, xacro)
@@ -83,6 +83,5 @@
       rate="10"
       horizontal_samples="1200"
-      vertical_samples="32">
-    </xacro:lidar_3d_plugin>
+      vertical_samples="32" />
   </xacro:macro>
 </robot>

File: robotnik_sensors/urdf/3d_lidar/robosense_bpearl.urdf.xacro (robot description, xacro)
@@ -80,6 +80,5 @@
       rate="10"
       horizontal_samples="1200"
-      vertical_samples="32">
-    </xacro:lidar_3d_plugin>
+      vertical_samples="32" />
   </xacro:macro>
 </robot>

File: robotnik_sensors/urdf/3d_lidar/robosense_helios_16p.urdf.xacro (robot description, xacro)
@@ -52,5 +52,5 @@
         <mass value="0.840" />
         <origin xyz="0 0 0.04135" />
-		<xacro:solid_cuboid_inertia
+        <xacro:solid_cuboid_inertia
           m="0.840"
           w="0.109"
@@ -80,6 +80,5 @@
       rate="10"
       horizontal_samples="1200"
-      vertical_samples="16">
-    </xacro:lidar_3d_plugin>
+      vertical_samples="16" />
   </xacro:macro>
 </robot>

File: robotnik_sensors/urdf/3d_lidar/sick_multiscan_100.urdf.xacro (robot description, xacro)
@@ -85,6 +85,5 @@
       rate="10"
       horizontal_samples="1200"
-      vertical_samples="16">
-    </xacro:lidar_3d_plugin>
+      vertical_samples="16" />
   </xacro:macro>
 </robot>

File: robotnik_sensors/urdf/3d_lidar/velodyne_vlp16.urdf.xacro (robot description, xacro)
@@ -79,6 +79,5 @@
       rate="10"
       horizontal_samples="1200"
-      vertical_samples="15">
-    </xacro:lidar_3d_plugin>
+      vertical_samples="15" />
   </xacro:macro>
 </robot>

File: robotnik_sensors/urdf/camera/axis_m5013.urdf.xacro (robot description, xacro)
@@ -20,5 +20,6 @@
   <xacro:arg
     name="axis_m5013_controllers_params_file"
-    default="" /> <!-- $(find robotnik_sensors_gazebo)/config/camera/axis_m5013.yaml -->
+    default="" />
+  <!-- $(find robotnik_sensors_gazebo)/config/camera/axis_m5013.yaml -->
   <xacro:macro
     name="sensor_axis_m5013"
@@ -48,5 +49,6 @@
           w="0.130"
           h="0.130"
-          d="0.035" /> <!-- Data from axis M5013 datasheet -->
+          d="0.035" />
+        <!-- Data from axis M5013 datasheet -->
       </inertial>
       <visual>
@@ -200,6 +202,5 @@
       min_depth="0.1"
       max_depth="100"
-      rate="30">
-    </xacro:camera_plugin>
+      rate="30" />
   </xacro:macro>
 </robot>

File: robotnik_sensors/urdf/camera/axis_m5074.urdf.xacro (robot description, xacro)
@@ -20,5 +20,6 @@
   <xacro:arg
     name="axis_m5074_controllers_params_file"
-    default="" /> <!-- $(find robotnik_sensors_gazebo)/config/camera/axis_m5074.yaml-->
+    default="" />
+  <!-- $(find robotnik_sensors_gazebo)/config/camera/axis_m5074.yaml-->
   <xacro:macro
     name="sensor_axis_m5074"
@@ -48,5 +49,6 @@
           w="0.130"
           h="0.130"
-          d="0.035" /> <!-- Data from axis M5013 datasheet -->
+          d="0.035" />
+        <!-- Data from axis M5013 datasheet -->
       </inertial>
       <visual>
@@ -200,6 +202,5 @@
       min_depth="0.1"
       max_depth="100"
-      rate="30">
-    </xacro:camera_plugin>
+      rate="30" />
   </xacro:macro>
 </robot>

File: robotnik_sensors/urdf/camera/axis_m5525.urdf.xacro (robot description, xacro)
@@ -20,5 +20,6 @@
   <xacro:arg
     name="axis_m5525_controllers_params_file"
-    default="" /> <!-- $(find robotnik_sensors_gazebo)/config/camera/axis_m5525.yaml -->
+    default="" />
+  <!-- $(find robotnik_sensors_gazebo)/config/camera/axis_m5525.yaml -->
   <xacro:macro
     name="sensor_axis_m5525"
@@ -196,6 +197,5 @@
       min_depth="0.1"
       max_depth="100"
-      rate="30">
-    </xacro:camera_plugin>
+      rate="30" />
   </xacro:macro>
 </robot>
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