Commit message: Add low_performance parameter to 3D lidar, camera, depth, and partial 2D lidar sensors
Co-authored-by: rafa-martin <23015374+rafa-martin@users.noreply.github.com>

File: robotnik_sensors/urdf/2d_lidar/hokuyo_urg04lx.urdf.xacro (robot description, xacro)
@@ -13,5 +13,6 @@
             node_name:=hokuyo_urg04lx
             node_namespace:=${None}
-            topic_prefix:=~/">
+            topic_prefix:=~/
+            low_performance:=false">
     <!-- node_namespace is used from node_name if not set -->
     <xacro:if value="${node_namespace == None}">
@@ -60,16 +61,32 @@
     <link name="${frame_prefix}link" />
     <!-- Hokuyo sensor for simulation -->
-    <xacro:lidar_2d_plugin
-      node_namespace="${node_namespace}"
-      node_name="${node_name}"
-      gazebo_ignition="${gazebo_ignition}"
-      min_range="0.06"
-      max_range="4.0"
-      min_angle="-2.0943"
-      max_angle="2.0943"
-      frame_link="${frame_prefix}link"
-      rate="10"
-      resolution="0.004359297"
-      samples="640" />
+    <xacro:if value="${low_performance}">
+      <xacro:lidar_2d_plugin
+        node_namespace="${node_namespace}"
+        node_name="${node_name}"
+        gazebo_ignition="${gazebo_ignition}"
+        min_range="0.06"
+        max_range="4.0"
+        min_angle="-2.0943"
+        max_angle="2.0943"
+        frame_link="${frame_prefix}link"
+        rate="5"
+        resolution="0.004359297"
+        samples="640" />
+    </xacro:if>
+    <xacro:unless value="${low_performance}">
+      <xacro:lidar_2d_plugin
+        node_namespace="${node_namespace}"
+        node_name="${node_name}"
+        gazebo_ignition="${gazebo_ignition}"
+        min_range="0.06"
+        max_range="4.0"
+        min_angle="-2.0943"
+        max_angle="2.0943"
+        frame_link="${frame_prefix}link"
+        rate="10"
+        resolution="0.004359297"
+        samples="640" />
+    </xacro:unless>
   </xacro:macro>
 </robot>

File: robotnik_sensors/urdf/3d_lidar/livox_mid_360.urdf.xacro (robot description, xacro)
@@ -14,5 +14,6 @@
             node_namespace:=${None}
             topic_prefix:=~/
-            gpu:=false">
+            gpu:=false
+            low_performance:=false">
     <material name="black_alu">
       <color rgba="0.9 0.9 0.9 1" />
@@ -74,16 +75,32 @@
     </joint>
     <link name="${frame_prefix}link" />
-    <xacro:lidar_3d_plugin
-      node_namespace="${node_namespace}"
-      node_name="${node_name}"
-      gazebo_ignition="${gazebo_ignition}"
-      min_range="0.1"
-      max_range="100.0"
-      min_angle="0.0"
-      max_angle="85"
-      frame_link="${frame_prefix}link"
-      rate="10"
-      horizontal_samples="1200"
-      vertical_samples="32" />
+    <xacro:if value="${low_performance}">
+      <xacro:lidar_3d_plugin
+        node_namespace="${node_namespace}"
+        node_name="${node_name}"
+        gazebo_ignition="${gazebo_ignition}"
+        min_range="0.1"
+        max_range="50.0"
+        min_angle="0.0"
+        max_angle="85"
+        frame_link="${frame_prefix}link"
+        rate="5"
+        horizontal_samples="600"
+        vertical_samples="32" />
+    </xacro:if>
+    <xacro:unless value="${low_performance}">
+      <xacro:lidar_3d_plugin
+        node_namespace="${node_namespace}"
+        node_name="${node_name}"
+        gazebo_ignition="${gazebo_ignition}"
+        min_range="0.1"
+        max_range="100.0"
+        min_angle="0.0"
+        max_angle="85"
+        frame_link="${frame_prefix}link"
+        rate="10"
+        horizontal_samples="1200"
+        vertical_samples="32" />
+    </xacro:unless>
   </xacro:macro>
 </robot>

File: robotnik_sensors/urdf/3d_lidar/ouster.urdf.xacro (robot description, xacro)
@@ -14,5 +14,6 @@
             node_namespace:=${None}
             topic_prefix:=~/
-            gpu:=false">
+            gpu:=false
+            low_performance:=false">
     <material name="black_alu">
       <color rgba="0.9 0.9 0.9 1" />
@@ -72,16 +73,32 @@
     </joint>
     <link name="${frame_prefix}link" />
-    <xacro:lidar_3d_plugin
-      node_namespace="${node_namespace}"
-      node_name="${node_name}"
-      gazebo_ignition="${gazebo_ignition}"
-      min_range="0.1"
-      max_range="50.0"
-      min_angle="0.0"
-      max_angle="85"
-      frame_link="${frame_prefix}link"
-      rate="10"
-      horizontal_samples="1200"
-      vertical_samples="32" />
+    <xacro:if value="${low_performance}">
+      <xacro:lidar_3d_plugin
+        node_namespace="${node_namespace}"
+        node_name="${node_name}"
+        gazebo_ignition="${gazebo_ignition}"
+        min_range="0.1"
+        max_range="25.0"
+        min_angle="0.0"
+        max_angle="85"
+        frame_link="${frame_prefix}link"
+        rate="5"
+        horizontal_samples="600"
+        vertical_samples="32" />
+    </xacro:if>
+    <xacro:unless value="${low_performance}">
+      <xacro:lidar_3d_plugin
+        node_namespace="${node_namespace}"
+        node_name="${node_name}"
+        gazebo_ignition="${gazebo_ignition}"
+        min_range="0.1"
+        max_range="50.0"
+        min_angle="0.0"
+        max_angle="85"
+        frame_link="${frame_prefix}link"
+        rate="10"
+        horizontal_samples="1200"
+        vertical_samples="32" />
+    </xacro:unless>
   </xacro:macro>
 </robot>

File: robotnik_sensors/urdf/3d_lidar/robosense_bpearl.urdf.xacro (robot description, xacro)
@@ -14,5 +14,6 @@
             node_namespace:=${None}
             topic_prefix:=~/
-            gpu:=false">
+            gpu:=false
+            low_performance:=false">
     <xacro:if value="${node_namespace == None}">
       <xacro:property
@@ -69,16 +70,32 @@
     </joint>
     <link name="${frame_prefix}link" />
-    <xacro:lidar_3d_plugin
-      node_namespace="${node_namespace}"
-      node_name="${node_name}"
-      gazebo_ignition="${gazebo_ignition}"
-      min_range="0.1"
-      max_range="100.0"
-      min_angle="0.0"
-      max_angle="85.0"
-      frame_link="${frame_prefix}link"
-      rate="10"
-      horizontal_samples="1200"
-      vertical_samples="32" />
+    <xacro:if value="${low_performance}">
+      <xacro:lidar_3d_plugin
+        node_namespace="${node_namespace}"
+        node_name="${node_name}"
+        gazebo_ignition="${gazebo_ignition}"
+        min_range="0.1"
+        max_range="50.0"
+        min_angle="0.0"
+        max_angle="85.0"
+        frame_link="${frame_prefix}link"
+        rate="5"
+        horizontal_samples="600"
+        vertical_samples="32" />
+    </xacro:if>
+    <xacro:unless value="${low_performance}">
+      <xacro:lidar_3d_plugin
+        node_namespace="${node_namespace}"
+        node_name="${node_name}"
+        gazebo_ignition="${gazebo_ignition}"
+        min_range="0.1"
+        max_range="100.0"
+        min_angle="0.0"
+        max_angle="85.0"
+        frame_link="${frame_prefix}link"
+        rate="10"
+        horizontal_samples="1200"
+        vertical_samples="32" />
+    </xacro:unless>
   </xacro:macro>
 </robot>

File: robotnik_sensors/urdf/3d_lidar/sick_multiscan_100.urdf.xacro (robot description, xacro)
@@ -14,5 +14,6 @@
             node_namespace:=${None}
             topic_prefix:=~/
-            gpu:=false">
+            gpu:=false
+            low_performance:=false">
     <material name="black_alu">
       <color rgba="0.9 0.9 0.9 1" />
@@ -74,16 +75,32 @@
     </joint>
     <link name="${frame_prefix}link" />
-    <xacro:lidar_3d_plugin
-      node_namespace="${node_namespace}"
-      node_name="${node_name}"
-      gazebo_ignition="${gazebo_ignition}"
-      min_range="0.1"
-      max_range="52.0"
-      min_angle="0.0"
-      max_angle="65"
-      frame_link="${frame_prefix}link"
-      rate="10"
-      horizontal_samples="1200"
-      vertical_samples="16" />
+    <xacro:if value="${low_performance}">
+      <xacro:lidar_3d_plugin
+        node_namespace="${node_namespace}"
+        node_name="${node_name}"
+        gazebo_ignition="${gazebo_ignition}"
+        min_range="0.1"
+        max_range="26.0"
+        min_angle="0.0"
+        max_angle="65"
+        frame_link="${frame_prefix}link"
+        rate="5"
+        horizontal_samples="600"
+        vertical_samples="16" />
+    </xacro:if>
+    <xacro:unless value="${low_performance}">
+      <xacro:lidar_3d_plugin
+        node_namespace="${node_namespace}"
+        node_name="${node_name}"
+        gazebo_ignition="${gazebo_ignition}"
+        min_range="0.1"
+        max_range="52.0"
+        min_angle="0.0"
+        max_angle="65"
+        frame_link="${frame_prefix}link"
+        rate="10"
+        horizontal_samples="1200"
+        vertical_samples="16" />
+    </xacro:unless>
   </xacro:macro>
 </robot>

File: robotnik_sensors/urdf/3d_lidar/velodyne_vlp16.urdf.xacro (robot description, xacro)
@@ -14,5 +14,6 @@
             node_namespace:=${None}
             topic_prefix:=~/
-            gpu:=false">
+            gpu:=false
+            low_performance:=false">
     <xacro:if value="${node_namespace == None}">
       <xacro:property
@@ -68,16 +69,32 @@
     </joint>
     <link name="${frame_prefix}link" />
-    <xacro:lidar_3d_plugin
-      node_namespace="${node_namespace}"
-      node_name="${node_name}"
-      gazebo_ignition="${gazebo_ignition}"
-      min_range="0.1"
-      max_range="100.0"
-      min_angle="-15"
-      max_angle="15"
-      frame_link="${frame_prefix}link"
-      rate="10"
-      horizontal_samples="1200"
-      vertical_samples="15" />
+    <xacro:if value="${low_performance}">
+      <xacro:lidar_3d_plugin
+        node_namespace="${node_namespace}"
+        node_name="${node_name}"
+        gazebo_ignition="${gazebo_ignition}"
+        min_range="0.1"
+        max_range="50.0"
+        min_angle="-15"
+        max_angle="15"
+        frame_link="${frame_prefix}link"
+        rate="5"
+        horizontal_samples="600"
+        vertical_samples="15" />
+    </xacro:if>
+    <xacro:unless value="${low_performance}">
+      <xacro:lidar_3d_plugin
+        node_namespace="${node_namespace}"
+        node_name="${node_name}"
+        gazebo_ignition="${gazebo_ignition}"
+        min_range="0.1"
+        max_range="100.0"
+        min_angle="-15"
+        max_angle="15"
+        frame_link="${frame_prefix}link"
+        rate="10"
+        horizontal_samples="1200"
+        vertical_samples="15" />
+    </xacro:unless>
   </xacro:macro>
 </robot>

File: robotnik_sensors/urdf/camera/axis_m5013.urdf.xacro (robot description, xacro)
@@ -30,5 +30,6 @@
             node_name:=axis_m5013
             node_namespace:=${None}
-            topic_prefix:=~/">
+            topic_prefix:=~/
+            low_performance:=false">
     <joint
       name="${frame_prefix}base_joint"
@@ -189,18 +190,36 @@
     </gazebo>
     <!-- Axis sensor for simulation -->
-    <xacro:camera_plugin
-      node_namespace="${node_namespace}"
-      node_name="${node_name}_color"
-      topic_prefix="${topic_prefix}_color"
-      gazebo_ignition="${gazebo_ignition}"
-      optical_frame="${frame_prefix}color_optical_frame"
-      reference_frame="${frame_prefix}color_frame"
-      horizontal_fov="45"
-      vertical_fov="32"
-      video_width="640"
-      video_height="480"
-      min_depth="0.1"
-      max_depth="100"
-      rate="30" />
+    <xacro:if value="${low_performance}">
+      <xacro:camera_plugin
+        node_namespace="${node_namespace}"
+        node_name="${node_name}_color"
+        topic_prefix="${topic_prefix}_color"
+        gazebo_ignition="${gazebo_ignition}"
+        optical_frame="${frame_prefix}color_optical_frame"
+        reference_frame="${frame_prefix}color_frame"
+        horizontal_fov="45"
+        vertical_fov="32"
+        video_width="640"
+        video_height="480"
+        min_depth="0.1"
+        max_depth="100"
+        rate="5" />
+    </xacro:if>
+    <xacro:unless value="${low_performance}">
+      <xacro:camera_plugin
+        node_namespace="${node_namespace}"
+        node_name="${node_name}_color"
+        topic_prefix="${topic_prefix}_color"
+        gazebo_ignition="${gazebo_ignition}"
+        optical_frame="${frame_prefix}color_optical_frame"
+        reference_frame="${frame_prefix}color_frame"
+        horizontal_fov="45"
+        vertical_fov="32"
+        video_width="640"
+        video_height="480"
+        min_depth="0.1"
+        max_depth="100"
+        rate="30" />
+    </xacro:unless>
   </xacro:macro>
 </robot>

File: robotnik_sensors/urdf/camera/axis_m5074.urdf.xacro (robot description, xacro)
@@ -30,5 +30,6 @@
             node_name:=axis_m5074
             node_namespace:=${None}
-            topic_prefix:=~/">
+            topic_prefix:=~/
+            low_performance:=false">
     <joint
       name="${frame_prefix}base_joint"
@@ -189,18 +190,36 @@
     </gazebo>
     <!-- Axis sensor for simulation -->
-    <xacro:camera_plugin
-      node_namespace="${node_namespace}"
-      node_name="${node_name}_color"
-      topic_prefix="${topic_prefix}_color"
-      gazebo_ignition="${gazebo_ignition}"
-      optical_frame="${frame_prefix}color_optical_frame"
-      reference_frame="${frame_prefix}color_frame"
-      horizontal_fov="45"
-      vertical_fov="32"
-      video_width="640"
-      video_height="480"
-      min_depth="0.1"
-      max_depth="100"
-      rate="30" />
+    <xacro:if value="${low_performance}">
+      <xacro:camera_plugin
+        node_namespace="${node_namespace}"
+        node_name="${node_name}_color"
+        topic_prefix="${topic_prefix}_color"
+        gazebo_ignition="${gazebo_ignition}"
+        optical_frame="${frame_prefix}color_optical_frame"
+        reference_frame="${frame_prefix}color_frame"
+        horizontal_fov="45"
+        vertical_fov="32"
+        video_width="640"
+        video_height="480"
+        min_depth="0.1"
+        max_depth="100"
+        rate="5" />
+    </xacro:if>
+    <xacro:unless value="${low_performance}">
+      <xacro:camera_plugin
+        node_namespace="${node_namespace}"
+        node_name="${node_name}_color"
+        topic_prefix="${topic_prefix}_color"
+        gazebo_ignition="${gazebo_ignition}"
+        optical_frame="${frame_prefix}color_optical_frame"
+        reference_frame="${frame_prefix}color_frame"
+        horizontal_fov="45"
+        vertical_fov="32"
+        video_width="640"
+        video_height="480"
+        min_depth="0.1"
+        max_depth="100"
+        rate="30" />
+    </xacro:unless>
   </xacro:macro>
 </robot>

File: robotnik_sensors/urdf/camera/axis_m5525.urdf.xacro (robot description, xacro)
@@ -30,5 +30,6 @@
             node_name:=axis_m5525
             node_namespace:=${None}
-            topic_prefix:=~/">
+            topic_prefix:=~/
+            low_performance:=false">
     <joint
       name="${frame_prefix}base_joint"
@@ -184,18 +185,36 @@
     </gazebo>
     <!-- Axis sensor for simulation -->
-    <xacro:camera_plugin
-      node_namespace="${node_namespace}"
-      node_name="${node_name}_color"
-      topic_prefix="${topic_prefix}_color"
-      gazebo_ignition="${gazebo_ignition}"
-      optical_frame="${frame_prefix}color_optical_frame"
-      reference_frame="${frame_prefix}color_frame"
-      horizontal_fov="45"
-      vertical_fov="32"
-      video_width="640"
-      video_height="480"
-      min_depth="0.1"
-      max_depth="100"
-      rate="30" />
+    <xacro:if value="${low_performance}">
+      <xacro:camera_plugin
+        node_namespace="${node_namespace}"
+        node_name="${node_name}_color"
+        topic_prefix="${topic_prefix}_color"
+        gazebo_ignition="${gazebo_ignition}"
+        optical_frame="${frame_prefix}color_optical_frame"
+        reference_frame="${frame_prefix}color_frame"
+        horizontal_fov="45"
+        vertical_fov="32"
+        video_width="640"
+        video_height="480"
+        min_depth="0.1"
+        max_depth="100"
+        rate="5" />
+    </xacro:if>
+    <xacro:unless value="${low_performance}">
+      <xacro:camera_plugin
+        node_namespace="${node_namespace}"
+        node_name="${node_name}_color"
+        topic_prefix="${topic_prefix}_color"
+        gazebo_ignition="${gazebo_ignition}"
+        optical_frame="${frame_prefix}color_optical_frame"
+        reference_frame="${frame_prefix}color_frame"
+        horizontal_fov="45"
+        vertical_fov="32"
+        video_width="640"
+        video_height="480"
+        min_depth="0.1"
+        max_depth="100"
+        rate="30" />
+    </xacro:unless>
   </xacro:macro>
 </robot>

File: robotnik_sensors/urdf/camera/axis_m5526.urdf.xacro (robot description, xacro)
@@ -30,5 +30,6 @@
             node_name:=axis_m5526
             node_namespace:=${None}
-            topic_prefix:=~/">
+            topic_prefix:=~/
+            low_performance:=false">
     <joint
       name="${frame_prefix}base_joint"
@@ -184,18 +185,36 @@
     </gazebo>
     <!-- Axis sensor for simulation -->
-    <xacro:camera_plugin
-      node_namespace="${node_namespace}"
-      node_name="${node_name}_color"
-      topic_prefix="${topic_prefix}_color"
-      gazebo_ignition="${gazebo_ignition}"
-      optical_frame="${frame_prefix}color_optical_frame"
-      reference_frame="${frame_prefix}color_frame"
-      horizontal_fov="45"
-      vertical_fov="32"
-      video_width="640"
-      video_height="480"
-      min_depth="0.1"
-      max_depth="100"
-      rate="30" />
+    <xacro:if value="${low_performance}">
+      <xacro:camera_plugin
+        node_namespace="${node_namespace}"
+        node_name="${node_name}_color"
+        topic_prefix="${topic_prefix}_color"
+        gazebo_ignition="${gazebo_ignition}"
+        optical_frame="${frame_prefix}color_optical_frame"
+        reference_frame="${frame_prefix}color_frame"
+        horizontal_fov="45"
+        vertical_fov="32"
+        video_width="640"
+        video_height="480"
+        min_depth="0.1"
+        max_depth="100"
+        rate="5" />
+    </xacro:if>
+    <xacro:unless value="${low_performance}">
+      <xacro:camera_plugin
+        node_namespace="${node_namespace}"
+        node_name="${node_name}_color"
+        topic_prefix="${topic_prefix}_color"
+        gazebo_ignition="${gazebo_ignition}"
+        optical_frame="${frame_prefix}color_optical_frame"
+        reference_frame="${frame_prefix}color_frame"
+        horizontal_fov="45"
+        vertical_fov="32"
+        video_width="640"
+        video_height="480"
+        min_depth="0.1"
+        max_depth="100"
+        rate="30" />
+    </xacro:unless>
   </xacro:macro>
 </robot>

File: robotnik_sensors/urdf/depth/azure_kinect.urdf.xacro (robot description, xacro)
@@ -13,5 +13,6 @@
             node_namespace:=${None}
             node_name:=azure_kinect
-            topic_prefix:=~/">
+            topic_prefix:=~/
+            low_performance:=false">
     <xacro:if value="${node_namespace == None}">
       <xacro:property
@@ -120,18 +121,36 @@
     </material>
     <!-- RGBD sensor for simulation, same as Kinect -->
-    <xacro:depth_camera_plugin
-      node_namespace="${node_namespace}"
-      node_name="${node_name}"
-      topic_prefix="${topic_prefix}"
-      gazebo_ignition="${gazebo_ignition}"
-      optical_frame="${frame_prefix}color_optical_frame"
-      reference_frame="${frame_prefix}color_frame"
-      horizontal_fov="60"
-      vertical_fov="45"
-      video_width="640"
-      video_height="480"
-      min_depth="0.05"
-      max_depth="3.5"
-      rate="30" />
+    <xacro:if value="${low_performance}">
+      <xacro:depth_camera_plugin
+        node_namespace="${node_namespace}"
+        node_name="${node_name}"
+        topic_prefix="${topic_prefix}"
+        gazebo_ignition="${gazebo_ignition}"
+        optical_frame="${frame_prefix}color_optical_frame"
+        reference_frame="${frame_prefix}color_frame"
+        horizontal_fov="60"
+        vertical_fov="45"
+        video_width="320"
+        video_height="240"
+        min_depth="0.05"
+        max_depth="3.5"
+        rate="5" />
+    </xacro:if>
+    <xacro:unless value="${low_performance}">
+      <xacro:depth_camera_plugin
+        node_namespace="${node_namespace}"
+        node_name="${node_name}"
+        topic_prefix="${topic_prefix}"
+        gazebo_ignition="${gazebo_ignition}"
+        optical_frame="${frame_prefix}color_optical_frame"
+        reference_frame="${frame_prefix}color_frame"
+        horizontal_fov="60"
+        vertical_fov="45"
+        video_width="640"
+        video_height="480"
+        min_depth="0.05"
+        max_depth="3.5"
+        rate="30" />
+    </xacro:unless>
   </xacro:macro>
 </robot>
