Commit message: Add low_performance parameter to 3D lidar, camera, depth, and partial 2D lidar sensors
Co-authored-by: rafa-martin <23015374+rafa-martin@users.noreply.github.com>

File: robotnik_sensors/urdf/depth/intel_realsense_d435i.urdf.xacro (robot description, xacro)
@@ -19,5 +19,6 @@
             node_name:=realsense_d435i
             node_namespace:=${None}
-            topic_prefix:=~/">
+            topic_prefix:=~/
+            low_performance:=false">
     <!-- node_namespace is used from node_name if not set -->
     <xacro:if value="${node_namespace == None}">
@@ -211,60 +212,120 @@
     </joint>
     <link name="${frame_prefix}imu_frame" />
-    <xacro:camera_plugin
-      node_namespace="${node_namespace}"
-      node_name="${node_name}_color"
-      topic_prefix="${topic_prefix}_color"
-      gazebo_ignition="${gazebo_ignition}"
-      optical_frame="${frame_prefix}color_optical_frame"
-      reference_frame="${frame_prefix}color_frame"
-      horizontal_fov="69.4"
-      vertical_fov="39"
-      video_width="1920"
-      video_height="1080"
-      min_depth="0.1"
-      max_depth="100"
-      rate="30" />
-    <xacro:irred_camera_plugin
-      node_namespace="${node_namespace}"
-      node_name="${node_name}_irred1"
-      topic_prefix="${topic_prefix}_irred1"
-      gazebo_ignition="${gazebo_ignition}"
-      optical_frame="${frame_prefix}infra1_optical_frame"
-      reference_frame="${frame_prefix}infra2_frame"
-      horizontal_fov="85.2"
-      vertical_fov="48"
-      video_width="1280"
-      video_height="720"
-      min_depth="0.1"
-      max_depth="100"
-      rate="30" />
-    <xacro:irred_camera_plugin
-      node_namespace="${node_namespace}"
-      node_name="${node_name}_irred2"
-      topic_prefix="${topic_prefix}_irred2"
-      gazebo_ignition="${gazebo_ignition}"
-      optical_frame="${frame_prefix}infra2_optical_frame"
-      reference_frame="${frame_prefix}infra2_frame"
-      horizontal_fov="85.2"
-      vertical_fov="48"
-      video_width="1280"
-      video_height="720"
-      min_depth="0.1"
-      max_depth="100"
-      rate="30" />
-    <xacro:depth_camera_plugin
-      node_namespace="${node_namespace}"
-      node_name="${node_name}_depth"
-      topic_prefix="${topic_prefix}_depth"
-      gazebo_ignition="${gazebo_ignition}"
-      optical_frame="${frame_prefix}depth_optical_frame"
-      reference_frame="${frame_prefix}depth_frame"
-      horizontal_fov="85.2"
-      vertical_fov="48"
-      video_width="1280"
-      video_height="720"
-      min_depth="0.1"
-      max_depth="100"
-      rate="30" />
+    <xacro:if value="${low_performance}">
+      <xacro:camera_plugin
+        node_namespace="${node_namespace}"
+        node_name="${node_name}_color"
+        topic_prefix="${topic_prefix}_color"
+        gazebo_ignition="${gazebo_ignition}"
+        optical_frame="${frame_prefix}color_optical_frame"
+        reference_frame="${frame_prefix}color_frame"
+        horizontal_fov="69.4"
+        vertical_fov="39"
+        video_width="1280"
+        video_height="720"
+        min_depth="0.1"
+        max_depth="100"
+        rate="5" />
+      <xacro:irred_camera_plugin
+        node_namespace="${node_namespace}"
+        node_name="${node_name}_irred1"
+        topic_prefix="${topic_prefix}_irred1"
+        gazebo_ignition="${gazebo_ignition}"
+        optical_frame="${frame_prefix}infra1_optical_frame"
+        reference_frame="${frame_prefix}infra2_frame"
+        horizontal_fov="85.2"
+        vertical_fov="48"
+        video_width="640"
+        video_height="480"
+        min_depth="0.1"
+        max_depth="100"
+        rate="5" />
+      <xacro:irred_camera_plugin
+        node_namespace="${node_namespace}"
+        node_name="${node_name}_irred2"
+        topic_prefix="${topic_prefix}_irred2"
+        gazebo_ignition="${gazebo_ignition}"
+        optical_frame="${frame_prefix}infra2_optical_frame"
+        reference_frame="${frame_prefix}infra2_frame"
+        horizontal_fov="85.2"
+        vertical_fov="48"
+        video_width="640"
+        video_height="480"
+        min_depth="0.1"
+        max_depth="100"
+        rate="5" />
+      <xacro:depth_camera_plugin
+        node_namespace="${node_namespace}"
+        node_name="${node_name}_depth"
+        topic_prefix="${topic_prefix}_depth"
+        gazebo_ignition="${gazebo_ignition}"
+        optical_frame="${frame_prefix}depth_optical_frame"
+        reference_frame="${frame_prefix}depth_frame"
+        horizontal_fov="85.2"
+        vertical_fov="48"
+        video_width="640"
+        video_height="480"
+        min_depth="0.1"
+        max_depth="100"
+        rate="5" />
+    </xacro:if>
+    <xacro:unless value="${low_performance}">
+      <xacro:camera_plugin
+        node_namespace="${node_namespace}"
+        node_name="${node_name}_color"
+        topic_prefix="${topic_prefix}_color"
+        gazebo_ignition="${gazebo_ignition}"
+        optical_frame="${frame_prefix}color_optical_frame"
+        reference_frame="${frame_prefix}color_frame"
+        horizontal_fov="69.4"
+        vertical_fov="39"
+        video_width="1920"
+        video_height="1080"
+        min_depth="0.1"
+        max_depth="100"
+        rate="30" />
+      <xacro:irred_camera_plugin
+        node_namespace="${node_namespace}"
+        node_name="${node_name}_irred1"
+        topic_prefix="${topic_prefix}_irred1"
+        gazebo_ignition="${gazebo_ignition}"
+        optical_frame="${frame_prefix}infra1_optical_frame"
+        reference_frame="${frame_prefix}infra2_frame"
+        horizontal_fov="85.2"
+        vertical_fov="48"
+        video_width="1280"
+        video_height="720"
+        min_depth="0.1"
+        max_depth="100"
+        rate="30" />
+      <xacro:irred_camera_plugin
+        node_namespace="${node_namespace}"
+        node_name="${node_name}_irred2"
+        topic_prefix="${topic_prefix}_irred2"
+        gazebo_ignition="${gazebo_ignition}"
+        optical_frame="${frame_prefix}infra2_optical_frame"
+        reference_frame="${frame_prefix}infra2_frame"
+        horizontal_fov="85.2"
+        vertical_fov="48"
+        video_width="1280"
+        video_height="720"
+        min_depth="0.1"
+        max_depth="100"
+        rate="30" />
+      <xacro:depth_camera_plugin
+        node_namespace="${node_namespace}"
+        node_name="${node_name}_depth"
+        topic_prefix="${topic_prefix}_depth"
+        gazebo_ignition="${gazebo_ignition}"
+        optical_frame="${frame_prefix}depth_optical_frame"
+        reference_frame="${frame_prefix}depth_frame"
+        horizontal_fov="85.2"
+        vertical_fov="48"
+        video_width="1280"
+        video_height="720"
+        min_depth="0.1"
+        max_depth="100"
+        rate="30" />
+    </xacro:unless>
     <!-- <gazebo>
         <plugin name="${node_name}" filename="librealsense_gazebo_plugin.so">

File: robotnik_sensors/urdf/depth/orbbec_astra.urdf.xacro (robot description, xacro)
@@ -13,5 +13,6 @@
             node_namespace:=${None}
             node_name:=orbbec_astra
-            topic_prefix:=~/">
+            topic_prefix:=~/
+            low_performance:=false">
     <!-- node_namespace is used from node_name if not set -->
     <xacro:if value="${node_namespace == None}">
@@ -95,18 +96,36 @@
     </joint>
     <link name="${frame_prefix}depth_optical_frame" />
-    <xacro:depth_camera_plugin
-      node_namespace="${node_namespace}"
-      node_name="${node_name}"
-      topic_prefix="${topic_prefix}"
-      gazebo_ignition="${gazebo_ignition}"
-      optical_frame="${frame_prefix}depth_optical_frame"
-      reference_frame="${frame_prefix}depth_frame"
-      horizontal_fov="60"
-      vertical_fov="45"
-      video_width="640"
-      video_height="480"
-      min_depth="0.05"
-      max_depth="8.0"
-      rate="30" />
+    <xacro:if value="${low_performance}">
+      <xacro:depth_camera_plugin
+        node_namespace="${node_namespace}"
+        node_name="${node_name}"
+        topic_prefix="${topic_prefix}"
+        gazebo_ignition="${gazebo_ignition}"
+        optical_frame="${frame_prefix}depth_optical_frame"
+        reference_frame="${frame_prefix}depth_frame"
+        horizontal_fov="60"
+        vertical_fov="45"
+        video_width="320"
+        video_height="240"
+        min_depth="0.05"
+        max_depth="8.0"
+        rate="5" />
+    </xacro:if>
+    <xacro:unless value="${low_performance}">
+      <xacro:depth_camera_plugin
+        node_namespace="${node_namespace}"
+        node_name="${node_name}"
+        topic_prefix="${topic_prefix}"
+        gazebo_ignition="${gazebo_ignition}"
+        optical_frame="${frame_prefix}depth_optical_frame"
+        reference_frame="${frame_prefix}depth_frame"
+        horizontal_fov="60"
+        vertical_fov="45"
+        video_width="640"
+        video_height="480"
+        min_depth="0.05"
+        max_depth="8.0"
+        rate="30" />
+    </xacro:unless>
   </xacro:macro>
 </robot>

File: robotnik_sensors/urdf/depth/stereolabs_generic.urdf.xacro (robot description, xacro)
@@ -25,5 +25,6 @@
             video_fps:=30
             min_depth:=0.4
-            max_depth:=6.5">
+            max_depth:=6.5
+            low_performance:=false">
     <!-- node_namespace is used from node_name if not set -->
     <xacro:if value="${node_namespace == None}">
@@ -46,4 +47,16 @@
         name="baseline"
         value="0.12" />
+    </xacro:if>
+    <!-- Override parameters for low performance mode -->
+    <xacro:if value="${low_performance}">
+      <xacro:property
+        name="video_width"
+        value="640" />
+      <xacro:property
+        name="video_height"
+        value="480" />
+      <xacro:property
+        name="video_fps"
+        value="5" />
     </xacro:if>
     <joint
@@ -165,5 +178,5 @@
       min_depth="0.1"
       max_depth="100"
-      rate="30" />
+      rate="${video_fps}" />
     <xacro:camera_plugin
       node_namespace="${node_namespace}"
@@ -179,5 +192,5 @@
       min_depth="0.1"
       max_depth="100"
-      rate="30" />
+      rate="${video_fps}" />
     <xacro:depth_camera_plugin
       node_namespace="${node_namespace}"
@@ -193,5 +206,5 @@
       min_depth="${min_depth}"
       max_depth="${max_depth}"
-      rate="30" />
+      rate="${video_fps}" />
   </xacro:macro>
 </robot>

File: robotnik_sensors/urdf/depth/stereolabs_zed2i.urdf.xacro (robot description, xacro)
@@ -13,5 +13,6 @@
             node_namespace:=stereolabs_zed2i
             node_name:=stereolabs_zed2i
-            topic_prefix:=~/">
+            topic_prefix:=~/
+            low_performance:=false">
     <xacro:sensor_stereolabs_generic
       frame_prefix="${frame_prefix}"
@@ -28,5 +29,6 @@
       video_fps="30"
       min_depth="0.2"
-      max_depth="20.0">
+      max_depth="20.0"
+      low_performance="${low_performance}">
       <xacro:insert_block name="origin" />
     </xacro:sensor_stereolabs_generic>
