Commit message: Fix picoscan120 mesh and standarize urdf

File: robotnik_sensors/urdf/2d_lidar/sick_picoscan120.urdf.xacro (robot description, xacro)
@@ -33,6 +33,6 @@
       <collision>
         <origin
-          xyz="0 0 0.0628"
-          rpy="3.1416 0 0" />
+          xyz="0 0 0"
+          rpy="0 0 0" />
         <geometry>
           <mesh
@@ -42,6 +42,6 @@
       <visual>
         <origin
-          xyz="0 0 0.0628"
-          rpy="3.1416 0 0" />
+          xyz="0 0 0"
+          rpy="0 0 0" />
         <geometry>
           <mesh
@@ -52,6 +52,6 @@
         <mass value="0.25" />
         <origin
-          xyz="0.0 0.0628 0.0"
-          rpy="3.1416 0 0" />
+          xyz="0 0 0"
+          rpy="0 0 0" />
         <xacro:solid_cuboid_inertia
           m="0.25"
@@ -65,10 +65,10 @@
       type="fixed">
       <origin
-        xyz="0 0 0.0628"
+        xyz="0 0 0.062212"
         rpy="0 0 0" />
       <parent link="${frame_prefix}base_link" />
-      <child link="${frame_prefix}link_1" />
+      <child link="${frame_prefix}link" />
     </joint>
-    <link name="${frame_prefix}link_1" />
+    <link name="${frame_prefix}link" />
     <xacro:lidar_2d_plugin
       node_namespace="${node_namespace}"
@@ -79,5 +79,5 @@
       min_angle="${min_angle}"
       max_angle="${max_angle}"
-      frame_link="${frame_prefix}link_1"
+      frame_link="${frame_prefix}link"
       rate="15.0"
       resolution="0.00575"

File: robotnik_sensors/urdf/all_sensors.urdf.xacro (robot description, xacro)
@@ -5,6 +5,10 @@
   <!-- This file unifies all sensors that can be used on simulation, defined as xacro:macros -->
   <!-- Declare global argument to set low_performance mode -->
-  <xacro:arg name="low_performance" default="false" />
-  <xacro:property name="low_performance" value="$(arg low_performance)" />
+  <xacro:arg
+    name="low_performance"
+    default="false" />
+  <xacro:property
+    name="low_performance"
+    value="$(arg low_performance)" />
   <xacro:include
     filename="$(find robotnik_sensors)/urdf/utils/inertia.urdf.xacro" />

Commit message: Add joint_1 and link_1 for 2D lidar in URDF

File: robotnik_sensors/urdf/2d_lidar/sick_picoscan120.urdf.xacro (robot description, xacro)
@@ -71,4 +71,14 @@
     </joint>
     <link name="${frame_prefix}link" />
+    <joint
+      name="${frame_prefix}joint_1"
+      type="fixed">
+      <origin
+        xyz="0 0 0"
+        rpy="0 0 0" />
+      <parent link="${frame_prefix}link" />
+      <child link="${frame_prefix}link_1" />
+    </joint>
+    <link name="${frame_prefix}link_1" />
     <xacro:lidar_2d_plugin
       node_namespace="${node_namespace}"
